File: hardware/65C816.sch (KiCad schematic (older format))
At the start: 12 parts, among them J1 POWER, U1 74AC04, U2 74AC04, U3 74AC04

Commit message: Add data pins buffer and pull downs
Parts:
- added C7: 100nF, symbol Device:C
- added RN1: 1k, Resistor_THT:R_Array_SIP9, symbol Device:R_Network08
- added U4: 74AC245, symbol AKs_Library:74AC245
- U1: symbol AK's_Library:74AC04 -> AKs_Library:74AC04
- U2: value 74AC04 -> W65C816SxP; symbol 65xx:W65C816SxP -> AKs_Library:W65C816SxP
- U3: value 74AC04 -> 74AC573; symbol AK's_Library:74AC573 -> AKs_Library:74AC573
Connections:
- net labels added: D0, D0..7, D1, D2, D3, D4, D5, D6, D7, R~W
- wire segments 63 -> 90

Commit message: Add Bus Enable to the logic for data bus buffer & bank address latch
Parts:
- removed U1: 74AC04, symbol AKs_Library:74AC04
- added U1: 74AC00, symbol 74xx:74HC00
- U2: symbol AKs_Library:W65C816SxP -> AK's_Library:W65C816SxP
- U3: symbol AKs_Library:74AC573 -> AK's_Library:74AC573
- U4: symbol AKs_Library:74AC245 -> AK's_Library:74AC245
Connections:
- net labels added: BE, B_~OE, L_~LE, L_~OE
- net labels removed: ~CLK
- wire segments 90 -> 94
- no-connect marks 5 -> 1
Changed lines of the file:
@@
 	1    0    0    -1
 $EndComp
-Text GLabel 1200 2300 0    50   Input ~ 0
+Text GLabel 1100 2400 0    50   Input ~ 0
 CLK
-Text GLabel 1800 2300 2    50   Output ~ 0
-~CLK
+Text GLabel 1950 2300 2    50   Output ~ 0
+L_~LE
 Entry Wire Line
 	3900 2400 4000 2500
@@
 Text Label 4450 2450 0    50   ~ 0
 DBA5
-Text GLabel 4750 4950 0    50   Input ~ 0
-~CLK
-$Comp
-L power:GND #PWR013
-U 1 1 615F69AE
-P 4750 5050
-F 0 "#PWR013" H 4750 4800 50  0001 C CNN
-F 1 "GND" H 4755 4877 50  0000 C CNN
-F 2 "" H 4750 5050 50  0001 C CNN
-F 3 "" H 4750 5050 50  0001 C CNN
-	1    4750 5050
-	1    0    0    -1
-$EndComp
 $Comp
 L power:GND #PWR015
@@
 	4000 3250 4350 3250
 $Comp
-L AKs_Library:74AC04 U1
-U 1 1 6161E14B
-P 1500 2300
-F 0 "U1" H 1500 2617 50  0000 C CNN
-F 1 "74AC04" H 1500 2526 50  0000 C CNN
-F 2 "" H 1500 2300 50  0001 C CNN
-F 3 "http://www.ti.com/lit/gpn/sn74AC04" H 1500 2300 50  0001 C CNN
-	1    1500 2300
-	1    0    0    -1
-$EndComp
-$Comp
-L AKs_Library:74AC573 U3
+L AK's_Library:74AC573 U3
 U 1 1 61607DB1
 P 5250 4550
@@
 $EndComp
 $Comp
-L AKs_Library:W65C816SxP U2
+L AK's_Library:W65C816SxP U2
 U 1 1 615CDC2D
 P 3150 3600
@@
 F 3 "http://www.westerndesigncenter.com/wdc/documentation/w65c816s.pdf" H 3150 5500 50  0001 C CNN
 	1    3150 3600
-	1    0    0    -1
-$EndComp
-$Comp
-L AKs_Library:74AC04 U1
-U 7 1 61620F57
-P 1400 3350
-F 0 "U1" H 1630 3396 50  0000 L CNN
-F 1 "74AC04" H 1630 3305 50  0000 L CNN
-F 2 "" H 1400 3350 50  0001 C CNN
-F 3 "http://www.ti.com/lit/gpn/sn74AC04" H 1400 3350 50  0001 C CNN
-	7    1400 3350
-	1    0    0    -1
-$EndComp
-$Comp
-L power:VCC #PWR01
-U 1 1 61622B7F
-P 1400 2850
-F 0 "#PWR01" H 1400 2700 50  0001 C CNN
-F 1 "VCC" H 1415 3023 50  0000 C CNN
-F 2 "" H 1400 2850 50  0001 C CNN
-F 3 "" H 1400 2850 50  0001 C CNN
-	1    1400 2850
-	1    0    0    -1
-$EndComp
-$Comp
-L power:GND #PWR02
-U 1 1 61623095
-P 1400 3850
-F 0 "#PWR02" H 1400 3600 50  0001 C CNN
-F 1 "GND" H 1405 3677 50  0000 C CNN
-F 2 "" H 1400 3850 50  0001 C CNN
-F 3 "" H 1400 3850 50  0001 C CNN
-	1    1400 3850
 	1    0    0    -1
 $EndComp
@@
 	5100 1150 5600 1150
 $Comp
-L AKs_Library:74AC04 U1
-U 2 1 616275C1
-P 8000 1300
-F 0 "U1" H 8000 1617 50  0000 C CNN
-F 1 "74AC04" H 8000 1526 50  0000 C CNN
-F 2 "" H 8000 1300 50  0001 C CNN
-F 3 "http://www.ti.com/lit/gpn/sn74AC04" H 8000 1300 50  0001 C CNN
-	2    8000 1300
-	1    0    0    -1
-$EndComp
-$Comp
-L AKs_Library:74AC04 U1
-U 3 1 61628A5E
-P 8000 1850
-F 0 "U1" H 8000 2167 50  0000 C CNN
-F 1 "74AC04" H 8000 2076 50  0000 C CNN
-F 2 "" H 8000 1850 50  0001 C CNN
-F 3 "http://www.ti.com/lit/gpn/sn74AC04" H 8000 1850 50  0001 C CNN
-	3    8000 1850
-	1    0    0    -1
-$EndComp
-$Comp
-L AKs_Library:74AC04 U1
-U 4 1 61629B31
-P 8000 2400
-F 0 "U1" H 8000 2717 50  0000 C CNN
-F 1 "74AC04" H 8000 2626 50  0000 C CNN
-F 2 "" H 8000 2400 50  0001 C CNN
-F 3 "http://www.ti.com/lit/gpn/sn74AC04" H 8000 2400 50  0001 C CNN
-	4    8000 2400
-	1    0    0    -1
-$EndComp
-$Comp
-L AKs_Library:74AC04 U1
-U 5 1 6162A4ED
-P 8800 1300
-F 0 "U1" H 8800 1617 50  0000 C CNN
-F 1 "74AC04" H 8800 1526 50  0000 C CNN
-F 2 "" H 8800 1300 50  0001 C CNN
-F 3 "http://www.ti.com/lit/gpn/sn74AC04" H 8800 1300 50  0001 C CNN
-	5    8800 1300
-	1    0    0    -1
-$EndComp
-$Comp
-L AKs_Library:74AC04 U1
-U 6 1 6162CB28
-P 8800 1850
-F 0 "U1" H 8800 2167 50  0000 C CNN
-F 1 "74AC04" H 8800 2076 50  0000 C CNN
-F 2 "" H 8800 1850 50  0001 C CNN
-F 3 "http://www.ti.com/lit/gpn/sn74AC04" H 8800 1850 50  0001 C CNN
-	6    8800 1850
-	1    0    0    -1
-$EndComp
-Wire Wire Line
-	7700 2400 7700 1850
-Wire Wire Line
-	7700 850  8150 850
-Wire Wire Line
-	8500 850  8500 1300
-Connection ~ 7700 1300
-Wire Wire Line
-	7700 1300 7700 850
-Connection ~ 7700 1850
-Wire Wire Line
-	7700 1850 7700 1300
-Connection ~ 8500 1300
-Wire Wire Line
-	8500 1300 8500 1850
-$Comp
 L power:VCC #PWR016
 U 1 1 61636624
-P 8150 850
-F 0 "#PWR016" H 8150 700 50  0001 C CNN
-F 1 "VCC" H 8165 1023 50  0000 C CNN
-F 2 "" H 8150 850 50  0001 C CNN
-F 3 "" H 8150 850 50  0001 C CNN
-	1    8150 850
-	1    0    0    -1
-$EndComp
-Connection ~ 8150 850
-Wire Wire Line
-	8150 850  8500 850
+P 7700 850
+F 0 "#PWR016" H 7700 700 50  0001 C CNN
+F 1 "VCC" H 7715 1023 50  0000 C CNN
+F 2 "" H 7700 850 50  0001 C CNN
+F 3 "" H 7700 850 50  0001 C CNN
+	1    7700 850
+	1    0    0    -1
+$EndComp
 NoConn ~ 8300 1300
-NoConn ~ 8300 1850
-NoConn ~ 8300 2400
-NoConn ~ 9100 1850
-NoConn ~ 9100 1300
-$Comp
-L AKs_Library:74AC245 U4
+$Comp
+L AK's_Library:74AC245 U4
 U 1 1 61028F62
 P 5250 2450
@@
 Text GLabel 4750 2850 0    50   Input ~ 0
 R~W
-Text GLabel 4750 2950 0    50   Input ~ 0
-~CLK
 Text Label 3750 4500 0    50   ~ 0
 A12
@@
 Entry Wire Line
 	6000 2550 6100 2650
+$Comp
+L 74xx:74HC00 U1
+U 4 1 610F744F
+P 8000 1300
+F 0 "U1" H 8000 1625 50  0000 C CNN
+F 1 "74AC00" H 8000 1534 50  0000 C CNN
+F 2 "" H 8000 1300 50  0001 C CNN
+F 3 "http://www.ti.com/lit/gpn/sn74ac00" H 8000 1300 50  0001 C CNN
+	4    8000 1300
+	1    0    0    -1
+$EndComp
+Connection ~ 7700 1200
+Wire Wire Line
+	7700 1200 7700 850
+$Comp
+L 74xx:74HC00 U1
+U 1 1 610F8470
+P 1500 2300
+F 0 "U1" H 1500 2625 50  0000 C CNN
+F 1 "74AC00" H 1500 2534 50  0000 C CNN
+F 2 "" H 1500 2300 50  0001 C CNN
+F 3 "http://www.ti.com/lit/gpn/sn74ac00" H 1500 2300 50  0001 C CNN
+	1    1500 2300
+	1    0    0    -1
+$EndComp
+$Comp
+L 74xx:74HC00 U1
+U 2 1 610FA375
+P 1500 2850
+F 0 "U1" H 1500 3175 50  0000 C CNN
+F 1 "74AC00" H 1500 3084 50  0000 C CNN
+F 2 "" H 1500 2850 50  0001 C CNN
+F 3 "http://www.ti.com/lit/gpn/sn74ac00" H 1500 2850 50  0001 C CNN
+	2    1500 2850
+	1    0    0    -1
+$EndComp
+$Comp
+L 74xx:74HC00 U1
+U 3 1 610FBE08
+P 1500 3400
+F 0 "U1" H 1500 3725 50  0000 C CNN
+F 1 "74AC00" H 1500 3634 50  0000 C CNN
+F 2 "" H 1500 3400 50  0001 C CNN
+F 3 "http://www.ti.com/lit/gpn/sn74ac00" H 1500 3400 50  0001 C CNN
+	3    1500 3400
+	1    0    0    -1
+$EndComp
+Wire Wire Line
+	1200 2200 1200 2400
+Connection ~ 1200 2400
+Wire Wire Line
+	1200 2400 1200 2750
+Wire Wire Line
+	1200 2400 1100 2400
+Wire Wire Line
+	1200 2950 1200 3300
+Connection ~ 1200 3300
+Wire Wire Line
+	1200 3300 1200 3500
+Wire Wire Line
+	1200 3300 1100 3300
+Text GLabel 1100 3300 0    50   Input ~ 0
+BE
+Text GLabel 1950 2850 2    50   Output ~ 0
+B_~OE
+Text GLabel 1950 3400 2    50   Output ~ 0
+L_~OE
+Wire Wire Line
+	1800 2300 1950 2300
+Wire Wire Line
+	1950 2850 1800 2850
+Wire Wire Line
+	1800 3400 1950 3400
+$Comp
+L 74xx:74HC00 U1
+U 5 1 6111C4EE
+P 1500 4550
+F 0 "U1" H 1730 4596 50  0000 L CNN
+F 1 "74AC00" H 1730 4505 50  0000 L CNN
+F 2 "" H 1500 4550 50  0001 C CNN
+F 3 "http://www.ti.com/lit/gpn/sn74ac00" H 1500 4550 50  0001 C CNN
+	5    1500 4550
+	1    0    0    -1
+$EndComp
+$Comp
+L power:VCC #PWR01
+U 1 1 61122B84
+P 1500 4050
+F 0 "#PWR01" H 1500 3900 50  0001 C CNN
+F 1 "VCC" H 1515 4223 50  0000 C CNN
+F 2 "" H 1500 4050 50  0001 C CNN
+F 3 "" H 1500 4050 50  0001 C CNN
+	1    1500 4050
+	1    0    0    -1
+$EndComp
+$Comp
+L power:GND #PWR02
+U 1 1 61122FFF
+P 1500 5050
+F 0 "#PWR02" H 1500 4800 50  0001 C CNN
+F 1 "GND" H 1505 4877 50  0000 C CNN
+F 2 "" H 1500 5050 50  0001 C CNN
+F 3 "" H 1500 5050 50  0001 C CNN
+	1    1500 5050
+	1    0    0    -1
+$EndComp
+Wire Wire Line
+	7700 1200 7700 1400
+Text GLabel 4750 4950 0    50   Input ~ 0
+L_~LE
+Text GLabel 4750 2950 0    50   Input ~ 0
+B_~OE
+Text GLabel 4750 5050 0    50   Input ~ 0
+L_~OE
+Text GLabel 2550 4000 0    50   Input ~ 0
+BE
+Text GLabel 2550 2700 0    50   Input ~ 0
+CLK
 Wire Bus Line
 	6000 4150 6000 5700

Commit message: Add pull up/down resistors, project symbol library
Parts:
- added RN1, RN2, RN3, RN4, RN6: 10k, Resistor_THT:R_Array_SIP9, symbol Device:R_Network08
- C1: value 220uF -> 220u; symbol Device:CP -> Device:CP_Small
- C2, C3: value 10uF -> 10u; symbol Device:CP -> Device:CP_Small
- C4, C5, C6, C7: value 100nF -> 100n; symbol Device:C -> Device:C_Small
- D1: symbol Device:LED -> Device:LED_Small
- R1: symbol Device:R -> Device:R_Small
- RN5: renamed from RN1; value 1k -> 10k
- U2: symbol AK's_Library:W65C816SxP -> 65C816:W65C816SxP
- U3: renamed from U4; symbol AK's_Library:74AC245 -> 65C816:74AC245
- U4: renamed from U3; symbol AK's_Library:74AC573 -> 74xx:74LS573
Connections:
- wire segments 94 -> 132
- no-connect marks 1 -> 7
Other:
- moved on the sheet: J1, RN5, U1D

Commit message: Update for episode 5
Parts:
- added C8: 10u, symbol Device:CP_Small
- added C9: 100n, symbol Device:C_Small
- added D2: 1N5817, Diode_THT:D_DO-41_SOD81_P10.16mm_Horizontal, symbol Diode:1N5817
- added R2: 1k, symbol Device:R_Small
- added U5: 74AC04, symbol 74xx:74LS04
Connections:
- net labels added: RDY, RDY_IN, ~WAIT
- wire segments 132 -> 151
- no-connect marks 7 -> 10
Other:
- moved on the sheet: U1D, U1E

Commit message: Update for episode 6
Parts:
- removed unit 2 of U1
- removed U5: 74AC04, symbol 74xx:74LS04
- added C10, C11: 100n, symbol Device:C_Small
- added unit 3 of U1
- added U6: 74AC74, symbol 74xx:74LS74
- added U8: 74AC08, symbol 74xx:74LS08
- added U9: 74AC32, symbol 74xx:74LS32
Connections:
- net labels added: CLK*2, ~CLK
- wire segments 151 -> 191
- no-connect marks 10 -> 13
Other:
- moved on the sheet: D2, R2, RN1, RN2, RN3, RN4, RN5, RN6, U1D, U1E, U2, U3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

Commit message: Updates for episode 7
Parts:
- removed U8: 74AC08, symbol 74xx:74LS08
- added C12: 100n, symbol Device:C_Small
- added U5: DS1035-10, symbol 65C816:DS1035-10
- added U8: 74AC11, symbol 74xx:74LS11
- U3: value 74AC245 -> 74ACT245
Connections:
- wire segments 191 -> 199
Other:
- moved on the sheet: C1, C10, C11, C2, C3, C4, C5, C6, C7, C8, C9, D1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

Commit message: Updates for episode 8
Connections:
- net CLK*2 is gone; now on net VCC: U6.3 (C)
- net CLK: no longer U6.5 (Q)
- net VCC: now also U6.2 (D)
- net ~CLK: no longer U6.2 (D), U6.6 (~Q)
- no-connect marks 13 -> 15
Other:
- moved on the sheet: U1A, U5B, U5C, U6A, U8C, U9B, U9C, U9D

Commit message: Updates for episode 9
Connections:
- net B_~OE: now also U9.11; no longer U9.3
- net L_~OE: now also U9.13; no longer U9.2
- net RDY: now also U1.12, U1.13; no longer U1.10, U1.9
- net VCC: now also U9.1, U9.2; no longer U9.12, U9.13
- net ~WAIT: now also U1.8; no longer U1.11
- net at D2.1 (K), U6.9 (Q), U8.1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: now also U1.10; no longer U1.13
- net at U8.6: now also U9.12; no longer U9.1
- new net: U1.11, U1.9
Changed lines of the file:
@@
 $Comp
 L 74xx:74LS32 U9
-U 4 1 6186BC0D
+U 1 1 6186BC0D
 P 900 6300
 F 0 "U9" H 900 6625 50  0000 C CNN
@@
 F 2 "" H 900 6300 50  0001 C CNN
 F 3 "https://www.ti.com/lit/ds/symlink/sn54ac32.pdf" H 900 6300 50  0001 C CNN
-	4    900  6300
+	1    900  6300
 	1    0    0    -1
 $EndComp
@@
 $Comp
 L 74xx:74HC00 U1
-U 3 1 617F2205
+U 4 1 617F2205
 P 2500 2350
 F 0 "U1" H 2500 2675 50  0000 C CNN
@@
 F 2 "" H 2500 2350 50  0001 C CNN
 F 3 "https://www.ti.com/lit/ds/symlink/sn74ac00.pdf" H 2500 2350 50  0001 C CNN
-	3    2500 2350
+	4    2500 2350
 	1    0    0    -1
 $EndComp
@@
 $Comp
 L 74xx:74LS32 U9
-U 1 1 6161DFB3
+U 4 1 6161DFB3
 P 3250 3950
 F 0 "U9" H 3250 4275 50  0000 C CNN
@@
 F 2 "" H 3250 3950 50  0001 C CNN
 F 3 "https://www.ti.com/lit/ds/symlink/sn54ac32.pdf" H 3250 3950 50  0001 C CNN
-	1    3250 3950
+	4    3250 3950
 	1    0    0    -1
 $EndComp
@@
 $Comp
 L 74xx:74HC00 U1
-U 4 1 610F744F
+U 3 1 610F744F
 P 3100 2450
 F 0 "U1" H 3100 2775 50  0000 C CNN
@@
 F 2 "" H 3100 2450 50  0001 C CNN
 F 3 "https://www.ti.com/lit/ds/symlink/sn74ac00.pdf" H 3100 2450 50  0001 C CNN
-	4    3100 2450
+	3    3100 2450
 	1    0    0    -1
 $EndComp
