File: hardware/65C816.sch (KiCad schematic (older format))
At the start: 29 parts, among them J1 POWER, U1 74AC00, U2 W65C816SxP, U3 74ACT245, U4 74AC573, U5 DS1035-10, U6 74AC74, U8 74AC11, U9 74AC32

Commit message: Re-number parts
Parts:
- renumbered C12 to C10, C4 to C3, C5 to C4, C6 to C5, C7 to C6, C9 to C7, C10 to C8, C11 to C9, D2 to D1, D1 to D2, R2 to R1, R1 to R2, U2 to U1, U8 to U2, U6 to U3, U5 to U4, U1 to U5, U9 to U6, U3 to U7, U4 to U8

Commit message: More episode 11 updates
Changed lines of the file:
@@
 Sheet 1 3
 Title "65C816 Homebrew Computer"
-Date "2021-11-25"
-Rev "A.10"
+Date "2021-11-29"
+Rev "A.11"
 Comp ""
 Comment1 ""
@@
 	2750 600  2750 1500
 $Sheet
-S 3050 850  550  450
+S 3250 900  650  450
 U 6188A63E
 F0 "Clock" 50
 F1 "clock.sch" 50
-F2 "CLK" O R 3600 1000 50
-F3 "~CLK" O R 3600 1150 50
+F2 "CLK" O R 3900 1050 50
+F3 "~CLK" O R 3900 1200 50
+F4 "~PWRUP" I L 3250 1050 50
 $EndSheet
 Wire Wire Line
@@
 NoConn ~ 1200 7550
 $Sheet
-S 4150 850  650  450
+S 4450 900  650  450
 U 61B33617
 F0 "Reset" 50
 F1 "reset.sch" 50
-F2 "~RST" O R 4800 1000 50
-F3 "CLK" I L 4150 1000 50
-F4 "~PWRUP" O R 4800 1200 50
-F5 "RST" O R 4800 1100 50
+F2 "~RST" O R 5100 1050 50
+F3 "CLK" I L 4450 1050 50
+F4 "~PWRUP" O R 5100 1250 50
+F5 "RST" O R 5100 1150 50
 $EndSheet
-Text Label 3800 1000 2    50   ~ 0
+Text Label 4100 1050 2    50   ~ 0
 CLK
-Text Label 3800 1150 2    50   ~ 0
+Text Label 4100 1200 2    50   ~ 0
 ~CLK
 Wire Wire Line
-	3600 1150 3800 1150
-Wire Wire Line
-	3600 1000 3800 1000
-Text Label 3950 1000 0    50   ~ 0
+	3900 1200 4100 1200
+Wire Wire Line
+	3900 1050 4100 1050
+Text Label 4250 1050 0    50   ~ 0
 CLK
-Text Label 5000 1000 2    50   ~ 0
+Text Label 5450 1050 2    50   ~ 0
 ~RST
 Wire Wire Line
-	4800 1000 5000 1000
-Wire Wire Line
-	3950 1000 4150 1000
+	5100 1050 5450 1050
+Wire Wire Line
+	4250 1050 4450 1050
 Text Label 1750 2350 0    50   ~ 0
 RDY
@@
 Connection ~ 7350 1000
 Connection ~ 7000 1000
+$Comp
+L 74xx:74LS32 U6
+U 3 1 6186C713
+P 900 5750
+F 0 "U6" H 900 6075 50  0000 C CNN
+F 1 "74AC32" H 900 5984 50  0000 C CNN
+F 2 "" H 900 5750 50  0001 C CNN
+F 3 "https://www.ti.com/lit/ds/symlink/sn54ac32.pdf" H 900 5750 50  0001 C CNN
+	3    900  5750
+	1    0    0    -1
+$EndComp
+$Comp
+L 74xx:74LS32 U6
+U 2 1 6186A7FA
+P 1750 6300
+F 0 "U6" H 1750 6625 50  0000 C CNN
+F 1 "74AC32" H 1750 6534 50  0000 C CNN
+F 2 "" H 1750 6300 50  0001 C CNN
+F 3 "https://www.ti.com/lit/ds/symlink/sn54ac32.pdf" H 1750 6300 50  0001 C CNN
+	2    1750 6300
+	1    0    0    -1
+$EndComp
+$Comp
+L 74xx:74LS32 U6
+U 1 1 6186BC0D
+P 900 6300
+F 0 "U6" H 900 6625 50  0000 C CNN
+F 1 "74AC32" H 900 6534 50  0000 C CNN
+F 2 "" H 900 6300 50  0001 C CNN
+F 3 "https://www.ti.com/lit/ds/symlink/sn54ac32.pdf" H 900 6300 50  0001 C CNN
+	1    900  6300
+	1    0    0    -1
+$EndComp
+$Comp
+L 74xx:74LS32 U6
+U 4 1 6161DFB3
+P 3250 3950
+F 0 "U6" H 3250 4275 50  0000 C CNN
+F 1 "74AC32" H 3250 4184 50  0000 C CNN
+F 2 "" H 3250 3950 50  0001 C CNN
+F 3 "https://www.ti.com/lit/ds/symlink/sn54ac32.pdf" H 3250 3950 50  0001 C CNN
+	4    3250 3950
+	1    0    0    -1
+$EndComp
+$Comp
+L 65C816:W65C816SxP U1
+U 1 1 615CDC2D
+P 6100 4050
+F 0 "U1" H 5750 5450 50  0000 C CNN
+F 1 "W65C816SxP" H 6400 5450 50  0000 C CIB
+F 2 "" H 6100 6050 50  0001 C CNN
+F 3 "https://www.westerndesigncenter.com/wdc/documentation/w65c816s.pdf" H 6100 5950 50  0001 C CNN
+	1    6100 4050
+	1    0    0    -1
+$EndComp
+$Comp
+L 74xx:74LS32 U6
+U 5 1 6186806D
+P 5350 7050
+F 0 "U6" H 5580 7096 50  0000 L CNN
+F 1 "74AC32" H 5580 7005 50  0000 L CNN
+F 2 "" H 5350 7050 50  0001 C CNN
+F 3 "https://www.ti.com/lit/ds/symlink/sn54ac32.pdf" H 5350 7050 50  0001 C CNN
+	5    5350 7050
+	1    0    0    -1
+$EndComp
+Text Label 5450 1250 2    50   ~ 0
+~PWRUP
+Wire Wire Line
+	5450 1250 5100 1250
+Text Label 2900 1050 0    50   ~ 0
+~PWRUP
+Wire Wire Line
+	2900 1050 3250 1050
 Wire Bus Line
 	9600 2100 9600 2950
@@
 Wire Bus Line
 	6950 3850 6950 6100
-$Comp
-L 74xx:74LS32 U6
-U 3 1 6186C713
-P 900 5750
-F 0 "U6" H 900 6075 50  0000 C CNN
-F 1 "74AC32" H 900 5984 50  0000 C CNN
-F 2 "" H 900 5750 50  0001 C CNN
-F 3 "https://www.ti.com/lit/ds/symlink/sn54ac32.pdf" H 900 5750 50  0001 C CNN
-	3    900  5750
-	1    0    0    -1
-$EndComp
-$Comp
-L 74xx:74LS32 U6
-U 2 1 6186A7FA
-P 1750 6300
-F 0 "U6" H 1750 6625 50  0000 C CNN
-F 1 "74AC32" H 1750 6534 50  0000 C CNN
-F 2 "" H 1750 6300 50  0001 C CNN
-F 3 "https://www.ti.com/lit/ds/symlink/sn54ac32.pdf" H 1750 6300 50  0001 C CNN
-	2    1750 6300
-	1    0    0    -1
-$EndComp
-$Comp
-L 74xx:74LS32 U6
-U 1 1 6186BC0D
-P 900 6300
-F 0 "U6" H 900 6625 50  0000 C CNN
-F 1 "74AC32" H 900 6534 50  0000 C CNN
-F 2 "" H 900 6300 50  0001 C CNN
-F 3 "https://www.ti.com/lit/ds/symlink/sn54ac32.pdf" H 900 6300 50  0001 C CNN
-	1    900  6300
-	1    0    0    -1
-$EndComp
-$Comp
-L 74xx:74LS32 U6
-U 4 1 6161DFB3
-P 3250 3950
-F 0 "U6" H 3250 4275 50  0000 C CNN
-F 1 "74AC32" H 3250 4184 50  0000 C CNN
-F 2 "" H 3250 3950 50  0001 C CNN
-F 3 "https://www.ti.com/lit/ds/symlink/sn54ac32.pdf" H 3250 3950 50  0001 C CNN
-	4    3250 3950
-	1    0    0    -1
-$EndComp
-$Comp
-L 65C816:W65C816SxP U1
-U 1 1 615CDC2D
-P 6100 4050
-F 0 "U1" H 5750 5450 50  0000 C CNN
-F 1 "W65C816SxP" H 6400 5450 50  0000 C CIB
-F 2 "" H 6100 6050 50  0001 C CNN
-F 3 "https://www.westerndesigncenter.com/wdc/documentation/w65c816s.pdf" H 6100 5950 50  0001 C CNN
-	1    6100 4050
-	1    0    0    -1
-$EndComp
-$Comp
-L 74xx:74LS32 U6
-U 5 1 6186806D
-P 5350 7050
-F 0 "U6" H 5580 7096 50  0000 L CNN
-F 1 "74AC32" H 5580 7005 50  0000 L CNN
-F 2 "" H 5350 7050 50  0001 C CNN
-F 3 "https://www.ti.com/lit/ds/symlink/sn54ac32.pdf" H 5350 7050 50  0001 C CNN
-	5    5350 7050
-	1    0    0    -1
-$EndComp
 $EndSCHEMATC

Commit message: Updates for Episode 12
Parts:
- R2: value 220 -> 1k
Connections:
- net GND: no longer RN3.1 (common), RN4.1 (common), RN6.1 (common)
- net VCC: now also RN3.1 (common), RN4.1 (common), RN6.1 (common), U1.3 (~ABORT), U1.4 (~IRQ), U1.6 (~NMI)
- net VDA: now reaches U1.39 (VDA)
- net VPA: now reaches U1.7 (VPA)
- net BA0 renamed A16
- net BA1 renamed A17
- net BA2 renamed A18
- net BA3 renamed A19
- net BA4 renamed A20
- net BA5 renamed A21
- net BA6 renamed A22
- net BA7 renamed A23
- net ~WAIT renamed ~WAI
- no-connect marks 15 -> 20
Changed lines of the file:
@@
 $Descr A4 11693 8268
 encoding utf-8
-Sheet 1 3
+Sheet 1 5
 Title "65C816 Homebrew Computer"
-Date "2021-11-29"
-Rev "A.11"
+Date "2021-12-10"
+Rev "A.12"
 Comp ""
 Comment1 ""
@@
 P 2300 950
 F 0 "R2" H 2200 900 50  0000 R CNN
-F 1 "220" H 2200 1000 50  0000 R CNN
+F 1 "1k" H 2200 1000 50  0000 R CNN
 F 2 "" V 2230 950 50  0001 C CNN
 F 3 "~" H 2300 950 50  0001 C CNN
@@
 $EndComp
 Wire Notes Line
-	4000 1750 4000 4750
+	4000 1700 4000 4750
 Wire Notes Line
 	4000 4750 650  4750
 Wire Notes Line
-	650  4750 650  1750
+	650  4750 650  1700
 Wire Notes Line
-	650  1750 4000 1750
+	650  1700 4000 1700
 Wire Notes Line
 	4100 1750 4100 2950
@@
 Wire Wire Line
 	10250 4450 10300 4450
-$Comp
-L power:GND #PWR025
-U 1 1 613FD3EA
-P 10300 4450
-F 0 "#PWR025" H 10300 4200 50  0001 C CNN
-F 1 "GND" H 10305 4277 50  0000 C CNN
-F 2 "" H 10300 4450 50  0001 C CNN
-F 3 "" H 10300 4450 50  0001 C CNN
-	1    10300 4450
-	1    0    0    -1
-$EndComp
 Text Label 9700 4950 0    50   ~ 0
-BA5
+A21
 Text Label 9700 5150 0    50   ~ 0
-BA7
+A23
 Text Label 9700 5050 0    50   ~ 0
-BA6
+A22
 Text Label 9700 4850 0    50   ~ 0
-BA4
+A20
 Text Label 9700 4750 0    50   ~ 0
-BA3
+A19
 Text Label 9700 4650 0    50   ~ 0
-BA2
+A18
 Text Label 9700 4550 0    50   ~ 0
-BA1
+A17
 Text Label 9700 4450 0    50   ~ 0
-BA0
+A16
 Wire Wire Line
 	9700 5150 9850 5150
@@
 Wire Wire Line
 	7700 3750 7650 3750
-$Comp
-L power:GND #PWR019
-U 1 1 6136B158
-P 7700 4550
-F 0 "#PWR019" H 7700 4300 50  0001 C CNN
-F 1 "GND" H 7705 4377 50  0000 C CNN
-F 2 "" H 7700 4550 50  0001 C CNN
-F 3 "" H 7700 4550 50  0001 C CNN
-	1    7700 4550
-	1    0    0    -1
-$EndComp
-$Comp
-L power:GND #PWR018
-U 1 1 61362D9F
-P 7700 3750
-F 0 "#PWR018" H 7700 3500 50  0001 C CNN
-F 1 "GND" H 7705 3577 50  0000 C CNN
-F 2 "" H 7700 3750 50  0001 C CNN
-F 3 "" H 7700 3750 50  0001 C CNN
-	1    7700 3750
-	1    0    0    -1
-$EndComp
 Wire Wire Line
 	7250 3750 7050 3750
@@
 Wire Wire Line
 	7650 2850 7700 2850
-$Comp
-L power:GND #PWR017
-U 1 1 612F2303
-P 7700 2850
-F 0 "#PWR017" H 7700 2600 50  0001 C CNN
-F 1 "GND" H 7705 2677 50  0000 C CNN
-F 2 "" H 7700 2850 50  0001 C CNN
-F 3 "" H 7700 2850 50  0001 C CNN
-	1    7700 2850
-	1    0    0    -1
-$EndComp
 Entry Wire Line
 	9600 2950 9700 3050
@@
 A0
 Text Label 9350 4950 0    50   ~ 0
-BA5
+A21
 Text Label 9350 5150 0    50   ~ 0
-BA7
+A23
 Text Label 9350 5050 0    50   ~ 0
-BA6
+A22
 Text Label 9350 4850 0    50   ~ 0
-BA4
+A20
 Text Label 9350 4750 0    50   ~ 0
-BA3
+A19
 Text Label 9350 4650 0    50   ~ 0
-BA2
+A18
 Text Label 9350 4550 0    50   ~ 0
-BA1
+A17
 Text Label 9350 4450 0    50   ~ 0
-BA0
+A16
 Wire Wire Line
 	9350 5150 9500 5150
@@
 Text Label 4250 1050 0    50   ~ 0
 CLK
-Text Label 5450 1050 2    50   ~ 0
+Text Label 5600 1050 2    50   ~ 0
 ~RST
 Wire Wire Line
-	5100 1050 5450 1050
+	5100 1050 5600 1050
 Wire Wire Line
 	4250 1050 4450 1050
@@
 Text Label 3750 3200 2    50   ~ 0
 L_~LE
-Text Label 3600 2450 2    50   ~ 0
-~WAIT
+Text Label 3750 2450 2    50   ~ 0
+~WAI
 Text Label 3750 3950 2    50   ~ 0
 B_~OE
@@
 Wire Wire Line
 	1750 2350 2000 2350
-Wire Wire Line
-	3600 2450 3400 2450
 Wire Wire Line
 	2900 3200 3750 3200
@@
 	8350 5350 8150 5350
 Text Label 10500 2100 2    50   ~ 0
-D0..7
+D[0..7]
 Text Label 10400 6100 2    50   ~ 0
-A0..A23
+A[0..23]
 $Comp
 L Device:CP_Small C2
@@
 	1    0    0    -1
 $EndComp
-Text Label 5450 1250 2    50   ~ 0
+Text Label 5600 1250 2    50   ~ 0
 ~PWRUP
 Wire Wire Line
-	5450 1250 5100 1250
+	5600 1250 5100 1250
 Text Label 2900 1050 0    50   ~ 0
 ~PWRUP
 Wire Wire Line
 	2900 1050 3250 1050
+NoConn ~ 5500 5250
+NoConn ~ 5500 5150
+NoConn ~ 5500 4950
+NoConn ~ 5500 4850
+NoConn ~ 5250 1150
+$Comp
+L power:PWR_FLAG #FLG0101
+U 1 1 61C5AC05
+P 1300 950
+F 0 "#FLG0101" H 1300 1025 50  0001 C CNN
+F 1 "PWR_FLAG" H 1300 1123 50  0000 C CNN
+F 2 "" H 1300 950 50  0001 C CNN
+F 3 "~" H 1300 950 50  0001 C CNN
+	1    1300 950
+	1    0    0    -1
+$EndComp
+Connection ~ 1300 950
+$Comp
+L power:PWR_FLAG #FLG0102
+U 1 1 61C5B1E2
+P 1300 1150
+F 0 "#FLG0102" H 1300 1225 50  0001 C CNN
+F 1 "PWR_FLAG" H 1300 1323 50  0000 C CNN
+F 2 "" H 1300 1150 50  0001 C CNN
+F 3 "~" H 1300 1150 50  0001 C CNN
+	1    1300 1150
+	-1   0    0    1
+$EndComp
+Connection ~ 1300 1150
+Wire Wire Line
+	5100 1150 5250 1150
+$Sheet
+S 2950 5050 600  1250
+U 61C859BC
+F0 "Debug" 50
+F1 "debug.sch" 50
+F2 "R~W" I L 2950 5200 50
+F3 "VDA" I L 2950 5300 50
+F4 "VPA" I L 2950 5400 50
+F5 "~IRQ" I L 2950 5700 50
+F6 "RDY" I L 2950 5500 50
+F7 "BE" I L 2950 5600 50
+F8 "~NMI" I L 2950 5800 50
+F9 "~WAI" I L 2950 5900 50
+F10 "a[0..23]" I L 2950 6050 50
+F11 "d[0..7]" I L 2950 6150 50
+$EndSheet
+Wire Wire Line
+	2750 5200 2950 5200
+Wire Wire Line
+	2950 5300 2750 5300
+Wire Wire Line
+	2750 5400 2950 5400
+Wire Wire Line
+	2950 5700 2750 5700
+Wire Wire Line
+	2750 5500 2950 5500
+Wire Wire Line
+	2750 5600 2950 5600
+Wire Wire Line
+	2750 5800 2950 5800
+Text Label 2750 5500 0    50   ~ 0
+RDY
+Text Label 2750 5600 0    50   ~ 0
+BE
+Text Label 2750 5800 0    50   ~ 0
+~NMI
+Text Label 2750 5900 0    50   ~ 0
+~WAI
+Text Label 2750 5700 0    50   ~ 0
+~IRQ
+Text Label 2750 5400 0    50   ~ 0
+VPA
+Text Label 2750 5300 0    50   ~ 0
+VDA
+Text Label 2750 5200 0    50   ~ 0
+R~W
+Wire Wire Line
+	2750 5900 2950 5900
+Text Label 2600 6150 0    50   ~ 0
+D[0..7]
+Text Label 2600 6050 0    50   ~ 0
+A[0..23]
+Wire Wire Line
+	3400 2450 3750 2450
+Text Label 5350 4550 0    50   ~ 0
+VPA
+Wire Wire Line
+	5350 4550 5500 4550
+Text Label 5350 4650 0    50   ~ 0
+VDA
+Wire Wire Line
+	5350 4650 5500 4650
+Text Label 5200 3750 0    50   ~ 0
+~NMI
+Text Label 5200 3650 0    50   ~ 0
+~IRQ
+Wire Wire Line
+	5200 3750 5400 3750
+Wire Wire Line
+	5200 3650 5400 3650
+$Comp
+L power:VCC #PWR0101
+U 1 1 6225E717
+P 5400 3500
+F 0 "#PWR0101" H 5400 3350 50  0001 C CNN
+F 1 "VCC" H 5415 3673 50  0000 C CNN
+F 2 "" H 5400 3500 50  0001 C CNN
+F 3 "" H 5400 3500 50  0001 C CNN
+	1    5400 3500
+	1    0    0    -1
+$EndComp
+Wire Wire Line
+	5400 3500 5400 3550
+Connection ~ 5400 3750
+Wire Wire Line
+	5400 3750 5500 3750
+Wire Wire Line
+	5400 3550 5500 3550
+Connection ~ 5400 3550
+Wire Wire Line
+	5400 3550 5400 3650
+Connection ~ 5400 3650
+Wire Wire Line
+	5400 3650 5500 3650
+Wire Wire Line
+	5400 3650 5400 3750
+Wire Bus Line
+	2950 6150 2600 6150
+Wire Bus Line
+	2600 6050 2950 6050
 Wire Bus Line
 	9600 2100 9600 2950
@@
 Wire Bus Line
 	6950 3850 6950 6100
+$Comp
+L power:GND #PWR017
+U 1 1 612F2303
+P 7700 2850
+F 0 "#PWR017" H 7700 2600 50  0001 C CNN
+F 1 "GND" H 7705 2677 50  0000 C CNN
+F 2 "" H 7700 2850 50  0001 C CNN
+F 3 "" H 7700 2850 50  0001 C CNN
+	1    7700 2850
+	1    0    0    -1
+$EndComp
+$Comp
+L power:VCC #PWR018
+U 1 1 61D625DC
+P 7700 3750
+F 0 "#PWR018" H 7700 3600 50  0001 C CNN
+F 1 "VCC" H 7715 3923 50  0000 C CNN
+F 2 "" H 7700 3750 50  0001 C CNN
+F 3 "" H 7700 3750 50  0001 C CNN
+	1    7700 3750
+	1    0    0    -1
+$EndComp
+$Comp
+L power:VCC #PWR019
+U 1 1 61D62AFC
+P 7700 4550
+F 0 "#PWR019" H 7700 4400 50  0001 C CNN
+F 1 "VCC" H 7715 4723 50  0000 C CNN
+F 2 "" H 7700 4550 50  0001 C CNN
+F 3 "" H 7700 4550 50  0001 C CNN
+	1    7700 4550
+	1    0    0    -1
+$EndComp
+$Comp
+L power:VCC #PWR025
+U 1 1 61D63001
+P 10300 4450
+F 0 "#PWR025" H 10300 4300 50  0001 C CNN
+F 1 "VCC" H 10315 4623 50  0000 C CNN
+F 2 "" H 10300 4450 50  0001 C CNN
+F 3 "" H 10300 4450 50  0001 C CNN
+	1    10300 4450
+	1    0    0    -1
+$EndComp
+$Sheet
+S 3900 5050 500  300
+U 61EB86F2
+F0 "Tester" 50
+F1 "tester.sch" 50
+$EndSheet
 $EndSCHEMATC
