File: hardware/clock.sch (KiCad schematic (older format))
At the start: 17 parts, among them SW1 Pulse, U10 74HC14, U11 74HC74, U7 LMC555xN, X1 28.322Mhz

Commit message: Updates for episode 9
Parts:
- added C20, C21: 2.2u, symbol Device:CP_Small
- added C22, C23: 100n, symbol Device:C_Small
- added R10, R8: 10k, symbol Device:R_Small
- added R7, R9: 2.2k, symbol Device:R_Small
- added RN7: 10k, Resistor_THT:R_Array_SIP5, symbol Device:R_Network04
- added SW2: Mode, symbol keyboard:SW_Push
- added SW3: Speed, symbol keyboard:SW_Push
- added SW4: SW_DIP_x04, symbol Switch:SW_DIP_x04
- added U12: 74HC74, symbol 74xx:74LS74
- added U13: 74HC253, symbol 74xx:74LS253
- added U14: 74HC193, symbol 74xx:74LS193
- C13, C14: symbol Device:C_Small -> Device:CP_Small
- X1: value 28.322Mhz -> 20MHz; footprint Oscillator:Oscillator_DIP-8 -> Oscillator:Oscillator_DIP-14; symbol Oscillator:CXO_DIP8 -> Oscillator:CXO_DIP14
Connections:
- net labels added: FAST_~SLOW, MODE, PULSE_~RUN, SPEED
- net labels removed: CLK*2
- wire segments 56 -> 138
- no-connect marks 9 -> 13
Other:
- moved on the sheet: C15, C16, C17, C18, C19, R3, R4, R5, R6, RV1, SW1, U10A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

Commit message: Update for episode 10
Parts:
- added C3: 10u, symbol Device:CP_Small
Connections:
- net GND: now also C3.2
- net VCC: now also C3.1
