File: hardware/clock.sch (KiCad schematic (older format))
At the start: 42 parts, among them SW1 Pulse, SW2 Mode, SW3 Speed, SW4 SW_DIP_x04, SW6 SW_DIP_SPDT_x02, U10 74HC112, U11 74HC74, U12 LMC555xN, U13 74HC112, U14 74HC74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

Commit message: Updates for Episode 12
Parts:
- removed RN7, RN8: 10k, Resistor_THT:R_Array_SIP5, symbol Device:R_Network04
- added D5: Clock, symbol Device:LED_Small
- added R13: 1k, symbol Device:R_Small
- added R14, R15, R16, R17, R18, R19, R20, R21: 10k, symbol Device:R_Small
Connections:
- net FAST_ON_RST: now also R14.1
- net GND: now also R13.1, R18.1, R19.1, R20.1, R21.1
- net PULSE_ON_RST: now also R16.1
- net RUN_ON_RST: now also R17.1
- net SLOW_ON_RST: now also R15.1
- net VCC: now also R14.2, R15.2, R16.2, R17.2; no longer U9.11
- net ~CLK: now also U9.11
- net at SW4.6, U15.1 (B): now also R20.2
- net at SW4.7, U15.10 (C): now also R19.2
- net at SW4.5, U15.15 (A): now also R21.2
- net at SW4.8, U15.9 (D): now also R18.2
- net at U9.10: now also D5.2 (A)
- new net: D5.1 (K), R13.2
- no-connect marks 15 -> 14
Other:
- note added: "LED"
- moved on the sheet: U10B, U10C, U11C, U13C, U14C, U9D, U9E, U9F, U9G, X1
