File: hardware/tester.sch (KiCad schematic (older format))
At the start: 4 parts

Commit message: Annotate tester
Parts:
- gave numbers to parts that had none: 4
Changed lines of the file:
@@
 $EndDescr
 $Comp
-L Device:R_Network08 RN?
+L Device:R_Network08 RN8
 U 1 1 61EBC620
 P 5150 2200
-F 0 "RN?" V 5675 2200 50  0000 C CNN
+F 0 "RN8" V 5675 2200 50  0000 C CNN
 F 1 "1.5k" V 5584 2200 50  0000 C CNN
 F 2 "Resistor_THT:R_Array_SIP9" V 5625 2200 50  0001 C CNN
@@
 $EndComp
 $Comp
-L 65C816:LED-Array-8 BAR?
+L 65C816:LED-Array-8 BAR6
 U 1 1 61EBB5B6
 P 4650 2250
-F 0 "BAR?" H 4650 2835 50  0000 C CNN
+F 0 "BAR6" H 4650 2835 50  0000 C CNN
 F 1 "Red" H 4650 2744 50  0000 C CNN
 F 2 "" H 4680 1675 50  0001 C CNN
@@
 $EndComp
 $Comp
-L Switch:SW_DIP_x08 SW?
+L Switch:SW_DIP_x08 SW7
 U 1 1 61EC1F32
 P 3250 2300
-F 0 "SW?" H 3250 2967 50  0000 C CNN
+F 0 "SW7" H 3250 2967 50  0000 C CNN
 F 1 "SW_DIP_x08" H 3250 2876 50  0000 C CNN
 F 2 "" H 3250 2300 50  0001 C CNN
@@
 	4850 2600 4950 2600
 $Comp
-L power:GND #PWR?
+L power:GND #PWR0109
 U 1 1 61ED15BD
 P 5400 2650
-F 0 "#PWR?" H 5400 2400 50  0001 C CNN
+F 0 "#PWR0109" H 5400 2400 50  0001 C CNN
 F 1 "GND" H 5405 2477 50  0000 C CNN
 F 2 "" H 5400 2650 50  0001 C CNN
@@
 	5400 2600 5350 2600
 $Comp
-L power:VCC #PWR?
+L power:VCC #PWR0110
 U 1 1 61ED1E14
 P 2850 1850
-F 0 "#PWR?" H 2850 1700 50  0001 C CNN
+F 0 "#PWR0110" H 2850 1700 50  0001 C CNN
 F 1 "VCC" H 2865 2023 50  0000 C CNN
 F 2 "" H 2850 1850 50  0001 C CNN
@@
 	2850 1900 2850 2000
 $Comp
-L Device:R_Network08 RN?
+L Device:R_Network08 RN7
 U 1 1 61ED3E98
 P 3900 2950
-F 0 "RN?" H 3420 2904 50  0000 R CNN
+F 0 "RN7" H 3420 2904 50  0000 R CNN
 F 1 "10k" H 3420 2995 50  0000 R CNN
 F 2 "Resistor_THT:R_Array_SIP9" V 4375 2950 50  0001 C CNN
@@
 	4300 1900 3550 1900
 $Comp
-L power:GND #PWR?
+L power:GND #PWR0111
 U 1 1 61EDFF00
 P 4300 3200
-F 0 "#PWR?" H 4300 2950 50  0001 C CNN
+F 0 "#PWR0111" H 4300 2950 50  0001 C CNN
 F 1 "GND" H 4305 3027 50  0000 C CNN
 F 2 "" H 4300 3200 50  0001 C CNN
