File: hardware/65C816.kicad_sch (KiCad schematic)
At the start: 29 parts, among them J1 POWER, U1 W65C816SxP, U2 74AC11, U3 74AC74, U4 DS1035-10, U5 74AC00, U6 74AC32, U7 74ACT245, U8 74AC573

Commit message: Updates for Episode 13
Connections:
- net E: now reaches U1.35 (E)
- no-connect marks 20 -> 19
Other:
- sheet Debug ports: added E; removed none
Changed lines of the file:
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@@
   (title_block
     (title "65C816 Homebrew Computer")
-    (date "2021-12-10")
-    (rev "A.12")
+    (date "2022-01-09")
+    (rev "A.13")
     (comment 2 "https://github.com/adrienkohlbecker/65C816")
     (comment 3 "Licensed under CERN-OHL-W v2")
@@
   (no_connect (at 139.7 123.19))
   (no_connect (at 30.48 160.02))
-  (no_connect (at 139.7 130.81))
   (no_connect (at 44.45 83.82))
   (no_connect (at 52.07 160.02))
@@
     (stroke (width 0) (type default) (color 0 0 0 0))
   )
-  (wire (pts (xy 69.85 147.32) (xy 74.93 147.32))
+  (wire (pts (xy 69.85 144.78) (xy 74.93 144.78))
     (stroke (width 0) (type default) (color 0 0 0 0))
   )
@@
     (stroke (width 0) (type default) (color 0 0 0 0))
   )
-  (wire (pts (xy 74.93 144.78) (xy 69.85 144.78))
+  (wire (pts (xy 74.93 142.24) (xy 69.85 142.24))
     (stroke (width 0) (type default) (color 0 0 0 0))
   )
@@
     (stroke (width 0) (type default) (color 0 0 0 0))
   )
-  (wire (pts (xy 69.85 137.16) (xy 74.93 137.16))
+  (wire (pts (xy 69.85 134.62) (xy 74.93 134.62))
     (stroke (width 0) (type default) (color 0 0 0 0))
   )
@@
     (stroke (width 0) (type default) (color 0 0 0 0))
   )
-  (wire (pts (xy 69.85 132.08) (xy 74.93 132.08))
+  (wire (pts (xy 69.85 129.54) (xy 74.93 129.54))
     (stroke (width 0) (type default) (color 0 0 0 0))
   )
@@
     (stroke (width 0) (type default) (color 0 0 0 0))
   )
+  (wire (pts (xy 69.85 149.86) (xy 74.93 149.86))
+    (stroke (width 0) (type default) (color 0 0 0 0))
+  )
   (polyline (pts (xy 104.14 74.93) (xy 127 74.93))
     (stroke (width 0) (type default) (color 0 0 0 0))
@@
     (stroke (width 0) (type default) (color 0 0 0 0))
   )
-  (wire (pts (xy 69.85 139.7) (xy 74.93 139.7))
+  (wire (pts (xy 69.85 137.16) (xy 74.93 137.16))
     (stroke (width 0) (type default) (color 0 0 0 0))
   )
@@
     (stroke (width 0) (type default) (color 0 0 0 0))
   )
-  (wire (pts (xy 74.93 134.62) (xy 69.85 134.62))
+  (wire (pts (xy 74.93 132.08) (xy 69.85 132.08))
     (stroke (width 0) (type default) (color 0 0 0 0))
   )
@@
     (stroke (width 0) (type default) (color 0 0 0 0))
   )
-  (wire (pts (xy 69.85 149.86) (xy 74.93 149.86))
+  (wire (pts (xy 69.85 147.32) (xy 74.93 147.32))
     (stroke (width 0) (type default) (color 0 0 0 0))
   )
@@
     (stroke (width 0) (type default) (color 0 0 0 0))
   )
+  (wire (pts (xy 137.16 130.81) (xy 139.7 130.81))
+    (stroke (width 0) (type default) (color 0 0 0 0))
+  )
   (wire (pts (xy 15.24 162.56) (xy 15.24 171.45))
     (stroke (width 0) (type default) (color 0 0 0 0))
@@
     (stroke (width 0) (type default) (color 0 0 0 0))
   )
-  (wire (pts (xy 69.85 142.24) (xy 74.93 142.24))
+  (wire (pts (xy 69.85 139.7) (xy 74.93 139.7))
     (stroke (width 0) (type default) (color 0 0 0 0))
   )
@@
     (effects (font (size 1.27 1.27)) (justify left bottom))
   )
-  (label "R~{W}" (at 69.85 132.08 0)
+  (label "R~{W}" (at 69.85 129.54 0)
     (effects (font (size 1.27 1.27)) (justify left bottom))
   )
@@
     (effects (font (size 1.27 1.27)) (justify left bottom))
   )
-  (label "BE" (at 69.85 142.24 0)
+  (label "BE" (at 69.85 139.7 0)
     (effects (font (size 1.27 1.27)) (justify left bottom))
   )
@@
     (effects (font (size 1.27 1.27)) (justify right bottom))
   )
-  (label "VDA" (at 69.85 134.62 0)
+  (label "VDA" (at 69.85 132.08 0)
     (effects (font (size 1.27 1.27)) (justify left bottom))
   )
@@
     (effects (font (size 1.27 1.27)) (justify left bottom))
   )
-  (label "RDY" (at 69.85 139.7 0)
+  (label "RDY" (at 69.85 137.16 0)
     (effects (font (size 1.27 1.27)) (justify left bottom))
   )
@@
     (effects (font (size 1.27 1.27)) (justify left bottom))
   )
-  (label "VPA" (at 69.85 137.16 0)
+  (label "VPA" (at 69.85 134.62 0)
     (effects (font (size 1.27 1.27)) (justify left bottom))
   )
@@
     (effects (font (size 1.27 1.27)) (justify left bottom))
   )
-  (label "~{IRQ}" (at 69.85 144.78 0)
+  (label "~{IRQ}" (at 69.85 142.24 0)
     (effects (font (size 1.27 1.27)) (justify left bottom))
   )
@@
     (effects (font (size 1.27 1.27)) (justify left bottom))
   )
+  (label "E" (at 137.16 130.81 0)
+    (effects (font (size 1.27 1.27)) (justify left bottom))
+  )
   (label "DBA1" (at 204.47 115.57 0)
     (effects (font (size 1.27 1.27)) (justify left bottom))
@@
     (effects (font (size 1.27 1.27)) (justify left bottom))
   )
-  (label "~{WAI}" (at 69.85 149.86 0)
+  (label "~{WAI}" (at 69.85 147.32 0)
     (effects (font (size 1.27 1.27)) (justify left bottom))
   )
@@
     (effects (font (size 1.27 1.27)) (justify left bottom))
   )
+  (label "E" (at 69.85 149.86 0)
+    (effects (font (size 1.27 1.27)) (justify left bottom))
+  )
   (label "A5" (at 179.07 107.95 0)
     (effects (font (size 1.27 1.27)) (justify left bottom))
@@
     (effects (font (size 1.27 1.27)) (justify left bottom))
   )
-  (label "~{NMI}" (at 69.85 147.32 0)
+  (label "~{NMI}" (at 69.85 144.78 0)
     (effects (font (size 1.27 1.27)) (justify left bottom))
   )
@@
     )
   )
-  (sheet (at 74.93 128.27) (size 15.24 31.75) (fields_autoplaced)
+  (sheet (at 74.93 125.73) (size 15.24 34.29) (fields_autoplaced)
     (stroke (width 0) (type solid) (color 0 0 0 0))
     (fill (color 0 0 0 0.0000))
-    (property "Sheet name" "Debug" (id 0) (at 74.93 127.5584 0)
+    (property "Sheet name" "Debug" (id 0) (at 74.93 125.0184 0)
       (effects (font (size 1.27 1.27)) (justify left bottom))
     )
@@
       (effects (font (size 1.27 1.27)) (justify left top))
     )
-    (pin "R~{W}" input (at 74.93 132.08 180)
+    (pin "R~{W}" input (at 74.93 129.54 180)
       (effects (font (size 1.27 1.27)) (justify left))
     )
-    (pin "VDA" input (at 74.93 134.62 180)
+    (pin "VDA" input (at 74.93 132.08 180)
       (effects (font (size 1.27 1.27)) (justify left))
     )
-    (pin "VPA" input (at 74.93 137.16 180)
+    (pin "VPA" input (at 74.93 134.62 180)
       (effects (font (size 1.27 1.27)) (justify left))
     )
-    (pin "~{IRQ}" input (at 74.93 144.78 180)
+    (pin "~{IRQ}" input (at 74.93 142.24 180)
       (effects (font (size 1.27 1.27)) (justify left))
     )
-    (pin "RDY" input (at 74.93 139.7 180)
+    (pin "RDY" input (at 74.93 137.16 180)
       (effects (font (size 1.27 1.27)) (justify left))
     )
-    (pin "BE" input (at 74.93 142.24 180)
+    (pin "BE" input (at 74.93 139.7 180)
       (effects (font (size 1.27 1.27)) (justify left))
     )
-    (pin "~{NMI}" input (at 74.93 147.32 180)
+    (pin "~{NMI}" input (at 74.93 144.78 180)
       (effects (font (size 1.27 1.27)) (justify left))
     )
-    (pin "~{WAI}" input (at 74.93 149.86 180)
+    (pin "~{WAI}" input (at 74.93 147.32 180)
       (effects (font (size 1.27 1.27)) (justify left))
     )
@@
       (effects (font (size 1.27 1.27)) (justify left))
     )
+    (pin "E" input (at 74.93 149.86 180)
+      (effects (font (size 1.27 1.27)) (justify left))
+    )
   )
   (sheet (at 99.06 128.27) (size 12.7 7.62) (fields_autoplaced)
@@
       (reference "#PWR0111") (unit 1) (value "GND") (footprint "")
     )
+    (path "/00000000-0000-0000-0000-000061c859bc/dd61f84d-33a7-40f6-8248-c59e0bd85f7e"
+      (reference "#PWR0112") (unit 1) (value "GND") (footprint "")
+    )
     (path "/00000000-0000-0000-0000-000061c859bc/00000000-0000-0000-0000-000061d2a5dc"
       (reference "BAR1") (unit 1) (value "Blue") (footprint "")
@@
       (reference "D5") (unit 1) (value "Clock") (footprint "")
     )
+    (path "/00000000-0000-0000-0000-000061c859bc/82bb7156-1a6e-4d66-a09d-1fa84847ab75"
+      (reference "D6") (unit 1) (value "EMU") (footprint "")
+    )
     (path "/00000000-0000-0000-0000-0000615d1014"
       (reference "J1") (unit 1) (value "POWER") (footprint "")
@@
       (reference "R21") (unit 1) (value "10k") (footprint "")
     )
+    (path "/00000000-0000-0000-0000-000061c859bc/868e4046-f070-4126-9940-0cf2cdeca915"
+      (reference "R22") (unit 1) (value "1k") (footprint "")
+    )
     (path "/00000000-0000-0000-0000-00006129b21e"

Commit message: Updates for Episode 14
Parts:
- removed C10, C4, C5, C6, C7, C8, C9: 100n, symbol Device:C_Small
- removed D1: 1N5817, Diode_THT:D_DO-41_SOD81_P10.16mm_Horizontal, symbol Diode:1N5817
- removed R1: 1k, symbol Device:R_Small
- removed RN2, RN3, RN4, RN5, RN6: 10k, Resistor_THT:R_Array_SIP9, symbol Device:R_Network08
- removed U2: 74AC11, symbol 74xx:74LS11
- removed U3: 74AC74, symbol 74xx:74LS74
- removed U4: DS1035-10, symbol 65C816:DS1035-10
- removed U5: 74AC00, symbol 74xx:74HC00
- removed U6: 74AC32, symbol 74xx:74LS32
- removed U7: 74ACT245, symbol 65C816:74AC245
- removed U8: 74AC573, symbol 74xx:74LS573
- C1, C2: symbol Device:CP_Small -> Device:C_Polarized_Small
Connections:
- net VCC: no longer U1.3 (~{ABORT}), U1.4 (~{IRQ}), U1.6 (~{NMI})
- net ~{IRQ}: now reaches RN1.5 (R4)
- net ~{IRQ}: now also U1.4 (~{IRQ})
- net ~{NMI}: now reaches RN1.6 (R5)
- net ~{NMI}: now also U1.6 (~{NMI})
- net ~{ABORT}: now reaches RN1.7 (R6)
- net ~{ABORT}: now also U1.3 (~{ABORT})
- no-connect marks 19 -> 6
Other:
- added sheet Address decoding (address_decoding.kicad_sch)
- added sheet Glue Logic (glue_logic.kicad_sch)
- added sheet Memory (memory.kicad_sch)
- sheet Debug ports: added A[0..23], D[0..7]; removed a[0..23], d[0..7]
- moved on the sheet: C2, C3, RN1, U1

Commit message: Start episode 15
Other:
- sheet Address decoding ports: added ~{RAM_CS}; removed none
- sheet Glue Logic ports: added A[16..23], ~{RD}, ~{WR}; removed A[0..23], W~{R}
- sheet Memory ports: added ~{RAM_CS}, ~{RD}, ~{WR}; removed W~{R}
Changed lines of the file:
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@@
   (title_block
     (title "65C816 Homebrew Computer")
-    (date "2022-01-14")
-    (rev "A.14")
+    (date "2022-01-23")
+    (rev "A.15")
     (comment 2 "https://github.com/adrienkohlbecker/65C816")
     (comment 3 "Licensed under CERN-OHL-W v2")
@@
     (stroke (width 0) (type default) (color 0 0 0 0))
   )
+  (wire (pts (xy 180.34 66.04) (xy 185.42 66.04))
+    (stroke (width 0) (type default) (color 0 0 0 0))
+  )
   (bus (pts (xy 106.68 119.38) (xy 106.68 121.92))
     (stroke (width 0) (type default) (color 0 0 0 0))
@@
     (stroke (width 0) (type default) (color 0 0 0 0))
   )
+  (wire (pts (xy 214.63 68.58) (xy 226.06 68.58))
+    (stroke (width 0) (type default) (color 0 0 0 0))
+  )
   (bus (pts (xy 106.68 111.76) (xy 106.68 114.3))
     (stroke (width 0) (type default) (color 0 0 0 0))
@@
     (stroke (width 0) (type default) (color 0 0 0 0))
   )
+  (wire (pts (xy 214.63 58.42) (xy 226.06 58.42))
+    (stroke (width 0) (type default) (color 0 0 0 0))
+  )
   (wire (pts (xy 36.83 85.09) (xy 44.45 85.09))
     (stroke (width 0) (type default) (color 0 0 0 0))
@@
   )
   (bus (pts (xy 106.68 73.66) (xy 106.68 76.2))
+    (stroke (width 0) (type default) (color 0 0 0 0))
+  )
+  (wire (pts (xy 246.38 96.52) (xy 256.54 96.52))
     (stroke (width 0) (type default) (color 0 0 0 0))
   )
@@
     (effects (font (size 1.27 1.27)) (justify left bottom))
   )
+  (label "~{WR}" (at 214.63 68.58 0)
+    (effects (font (size 1.27 1.27)) (justify left bottom))
+  )
   (label "BE" (at 153.67 104.14 0)
     (effects (font (size 1.27 1.27)) (justify left bottom))
+  )
+  (label "~{RAM_CS}" (at 256.54 96.52 180)
+    (effects (font (size 1.27 1.27)) (justify right bottom))
   )
   (label "VPA" (at 66.04 114.3 0)
@@
     (effects (font (size 1.27 1.27)) (justify left bottom))
   )
-  (label "A[0..23]" (at 190.5 74.93 180)
+  (label "A[16..23]" (at 190.5 74.93 180)
     (effects (font (size 1.27 1.27)) (justify right bottom))
   )
@@
     (effects (font (size 1.27 1.27)) (justify right bottom))
   )
-  (label "W~{R}" (at 214.63 66.04 0)
-    (effects (font (size 1.27 1.27)) (justify left bottom))
+  (label "~{RD}" (at 214.63 66.04 0)
+    (effects (font (size 1.27 1.27)) (justify left bottom))
+  )
+  (label "~{WR}" (at 185.42 66.04 180)
+    (effects (font (size 1.27 1.27)) (justify right bottom))
   )
   (label "RDY" (at 153.67 101.6 0)
@@
     (effects (font (size 1.27 1.27)) (justify left bottom))
   )
-  (label "W~{R}" (at 185.42 63.5 180)
+  (label "~{RD}" (at 185.42 63.5 180)
     (effects (font (size 1.27 1.27)) (justify right bottom))
+  )
+  (label "~{RAM_CS}" (at 214.63 58.42 0)
+    (effects (font (size 1.27 1.27)) (justify left bottom))
   )
   (label "DBA3" (at 100.33 78.74 0)
@@
       (effects (font (size 1.27 1.27)) (justify left))
     )
-    (pin "W~{R}" input (at 226.06 66.04 180)
+    (pin "~{RD}" input (at 226.06 66.04 180)
+      (effects (font (size 1.27 1.27)) (justify left))
+    )
+    (pin "~{WR}" input (at 226.06 68.58 180)
+      (effects (font (size 1.27 1.27)) (justify left))
+    )
+    (pin "~{RAM_CS}" input (at 226.06 58.42 180)
       (effects (font (size 1.27 1.27)) (justify left))
     )
@@
       (effects (font (size 1.27 1.27)) (justify right))
     )
-    (pin "A[0..23]" output (at 180.34 74.93 0)
+    (pin "~{RD}" output (at 180.34 63.5 0)
       (effects (font (size 1.27 1.27)) (justify right))
     )
-    (pin "W~{R}" output (at 180.34 63.5 0)
+    (pin "~{WR}" output (at 180.34 66.04 0)
+      (effects (font (size 1.27 1.27)) (justify right))
+    )
+    (pin "A[16..23]" output (at 180.34 74.93 0)
       (effects (font (size 1.27 1.27)) (justify right))
     )
@@
     )
     (pin "~{ROM_CS}" output (at 246.38 93.98 0)
+      (effects (font (size 1.27 1.27)) (justify right))
+    )
+    (pin "~{RAM_CS}" output (at 246.38 96.52 0)
       (effects (font (size 1.27 1.27)) (justify right))
     )
@@
       (reference "#PWR0120") (unit 1) (value "GND") (footprint "")
     )
+    (path "/51a25d9b-b48c-46f9-8897-a7e56a5418ca/1e40ff28-0621-4424-82fd-81f8001b22e6"
+      (reference "#PWR0121") (unit 1) (value "VCC") (footprint "")
+    )
+    (path "/51a25d9b-b48c-46f9-8897-a7e56a5418ca/abb2d525-947e-4d5f-8493-12d9b8f91794"
+      (reference "#PWR0122") (unit 1) (value "GND") (footprint "")
+    )
     (path "/00000000-0000-0000-0000-000061c859bc/00000000-0000-0000-0000-000061d2a5dc"
       (reference "BAR1") (unit 1) (value "Blue") (footprint "")
@@
       (reference "C42") (unit 1) (value "10u") (footprint "")
     )
+    (path "/51a25d9b-b48c-46f9-8897-a7e56a5418ca/cc0e7822-95c2-433c-9a29-9af1a7951302"
+      (reference "C43") (unit 1) (value "100n") (footprint "")
+    )
     (path "/95d65710-49c8-4cb8-9de3-935bd85d56b1/f818d74a-5ffc-4388-be9e-aa337070bc87"
       (reference "D1") (unit 1) (value "1N5817") (footprint "Diode_THT:D_DO-41_SOD81_P10.16mm_Horizontal")
@@
       (reference "U27") (unit 2) (value "74HC10") (footprint "")
     )
-    (path "/95d65710-49c8-4cb8-9de3-935bd85d56b1/8dd2bee0-48bf-4a9f-8928-92398172eb68"
+    (path "/f3e13532-3999-4d1f-800f-4b9a7b3c3e9d/a4ba7831-9238-43e0-8c5c-16ce57651bfc"
       (reference "U27") (unit 3) (value "74HC10") (footprint "")
     )
@@
       (reference "U27") (unit 4) (value "74HC10") (footprint "")
     )
+    (path "/51a25d9b-b48c-46f9-8897-a7e56a5418ca/885ebe43-b6ad-42fe-bc71-d7c9ebc3d292"
+      (reference "U28") (unit 1) (value "KM62256CLP") (footprint "Package_DIP:DIP-28_W15.24mm")
+    )
     (path "/00000000-0000-0000-0000-00006188a63e/00000000-0000-0000-0000-00006194c461"

Commit message: Update for Episode 15
Connections:
- net ~{ROM_WE}: now reaches RN1.8 (R7)
- no-connect marks 6 -> 5
Other:
- sheet Memory ports: added ~{ROM_WE}; removed none

Commit message: Update for Episode 16
Connections:
- no-connect marks 5 -> 14
Other:
- sheet Address decoding ports: added {ADDRESS}, ~{EXTRAM_CS}, ~{IO0}, ~{IO1}, ~{IO2}, ~{IO3}, ~{IO4}, ~{IO5}, ~{IO6}, ~{IO7}; removed A[0..23]
- sheet Debug ports: added RDY_IN, {ADDRESS}, ~{RST}; removed A[0..23], RDY
- sheet Glue Logic ports: added {ADDRESS}; removed A[0..15], A[16..23]
- sheet Memory ports: added {ADDRESS}; removed A[0..23]
