File: hardware/65C816.kicad_sch (KiCad schematic)
At the start: 8 parts, among them J1 POWER, U1 W65C816SxP

Commit message: Updates for episode 17
Other:
- added sheet Monitor (monitor.kicad_sch)
- sheet Clock ports: added MONCLK; removed ~{PWRUP}
- sheet Reset ports: added none; removed ~{PWRUP}

Commit message: Update for episode 18
Other:
- sheet Debug ports: added SYNC, VA; removed VDA, VPA
- sheet Glue Logic ports: added SYNC, VA, VDA, VPA; removed none
- sheet Monitor ports: added SYNC, VA; removed none

Commit message: Update for episode 19
Connections:
- no-connect marks 14 -> 15
Other:
- sheet Glue Logic ports: added CLK_IN; removed none

Commit message: More episode 19 updates
Parts:
- removed RN1: 10k, Resistor_THT:R_Array_SIP9, symbol Device:R_Network08
- added R12, R34, R35, R36, R37: 10k, symbol Device:R_Small
Connections:
- net BE: now also R37.2
- net R~{W}: now also R36.2
- net VCC: now also R12.1, R34.1, R35.1, R36.1, R37.1
- net ~{ABORT}: now also R12.2
- net ~{IRQ}: now also R34.2
- net ~{NMI}: now also R35.2
- no-connect marks 15 -> 14

Commit message: Update for episode 20
Connections:
- no-connect marks 14 -> 13
Other:
- sheet Memory ports: added ~{EXTRAM_CS}; removed none
Changed lines of the file:
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@@
   (title_block
     (title "65C816 Homebrew Computer")
-    (date "2022-03-01")
-    (rev "A.19")
+    (date "2022-03-25")
+    (rev "A.20")
     (comment 2 "https://github.com/adrienkohlbecker/65C816")
     (comment 3 "Licensed under CERN-OHL-W v2")
-    (comment 4 "Copyright © 2021 Adrien Kohlbecker")
+    (comment 4 "Copyright © 2022 Adrien Kohlbecker")
   )
   (bus_alias "ADDRESS" (members "A[0..15]" "~{A[16..23]}"))
@@
   (no_connect (at 69.85 132.08))
   (no_connect (at 69.85 121.92))
-  (no_connect (at 182.88 41.91))
   (no_connect (at 248.92 66.04))
   (no_connect (at 248.92 68.58))
@@
   (no_connect (at 248.92 81.28))
   (no_connect (at 248.92 83.82))
-  (no_connect (at 248.92 62.23))
   (no_connect (at 248.92 73.66))
+  (no_connect (at 182.88 38.1))
   (bus_entry (at 104.14 111.76) (size 2.54 2.54)
     (stroke (width 0) (type default) (color 0 0 0 0))
@@
     (stroke (width 0) (type default) (color 0 0 0 0))
   )
-  (bus (pts (xy 144.78 128.27) (xy 158.75 128.27))
+  (bus (pts (xy 144.78 133.35) (xy 158.75 133.35))
     (stroke (width 0) (type default) (color 0 0 0 0))
   )
@@
     (stroke (width 0) (type default) (color 0 0 0 0))
   )
-  (wire (pts (xy 147.32 116.84) (xy 158.75 116.84))
+  (wire (pts (xy 147.32 120.65) (xy 158.75 120.65))
     (stroke (width 0) (type default) (color 0 0 0 0))
   )
@@
     (stroke (width 0) (type default) (color 0 0 0 0))
   )
-  (wire (pts (xy 246.38 57.15) (xy 256.54 57.15))
+  (wire (pts (xy 246.38 57.15) (xy 259.08 57.15))
     (stroke (width 0) (type default) (color 0 0 0 0))
   )
@@
     (stroke (width 0) (type default) (color 0 0 0 0))
   )
-  (wire (pts (xy 180.34 41.91) (xy 182.88 41.91))
-    (stroke (width 0) (type default) (color 0 0 0 0))
-  )
   (wire (pts (xy 217.17 102.87) (xy 226.06 102.87))
     (stroke (width 0) (type default) (color 0 0 0 0))
@@
     (stroke (width 0) (type default) (color 0 0 0 0))
   )
-  (wire (pts (xy 147.32 119.38) (xy 158.75 119.38))
+  (wire (pts (xy 147.32 123.19) (xy 158.75 123.19))
     (stroke (width 0) (type default) (color 0 0 0 0))
   )
@@
     (stroke (width 0) (type default) (color 0 0 0 0))
   )
+  (wire (pts (xy 180.34 41.91) (xy 189.23 41.91))
+    (stroke (width 0) (type default) (color 0 0 0 0))
+  )
   (wire (pts (xy 83.82 29.21) (xy 92.71 29.21))
     (stroke (width 0) (type default) (color 0 0 0 0))
   )
-  (bus (pts (xy 144.78 130.81) (xy 158.75 130.81))
+  (bus (pts (xy 144.78 135.89) (xy 158.75 135.89))
     (stroke (width 0) (type default) (color 0 0 0 0))
   )
@@
     (stroke (width 0) (type default) (color 0 0 0 0))
   )
-  (wire (pts (xy 147.32 124.46) (xy 158.75 124.46))
+  (wire (pts (xy 147.32 128.27) (xy 158.75 128.27))
     (stroke (width 0) (type default) (color 0 0 0 0))
   )
@@
     (stroke (width 0) (type default) (color 0 0 0 0))
   )
-  (wire (pts (xy 246.38 62.23) (xy 248.92 62.23))
+  (wire (pts (xy 246.38 62.23) (xy 259.08 62.23))
     (stroke (width 0) (type default) (color 0 0 0 0))
   )
@@
     (stroke (width 0) (type default) (color 0 0 0 0))
   )
+  (wire (pts (xy 147.32 114.3) (xy 158.75 114.3))
+    (stroke (width 0) (type default) (color 0 0 0 0))
+  )
   (bus (pts (xy 106.68 129.54) (xy 106.68 132.08))
     (stroke (width 0) (type default) (color 0 0 0 0))
   )
-  (wire (pts (xy 180.34 38.1) (xy 189.23 38.1))
+  (wire (pts (xy 180.34 38.1) (xy 182.88 38.1))
     (stroke (width 0) (type default) (color 0 0 0 0))
   )
@@
     (stroke (width 0) (type default) (color 0 0 0 0))
   )
-  (wire (pts (xy 246.38 59.69) (xy 256.54 59.69))
+  (wire (pts (xy 246.38 59.69) (xy 259.08 59.69))
     (stroke (width 0) (type default) (color 0 0 0 0))
   )
@@
     (effects (font (size 1.27 1.27)) (justify right bottom))
   )
-  (label "~{ROM_WE}" (at 147.32 124.46 0)
-    (effects (font (size 1.27 1.27)) (justify left bottom))
+  (label "~{ROM_WE}" (at 147.32 128.27 0)
+    (effects (font (size 1.27 1.27)) (justify left bottom))
+  )
+  (label "~{EXTRAM_CS}" (at 259.08 62.23 180)
+    (effects (font (size 1.27 1.27)) (justify right bottom))
   )
   (label "{ADDRESS}" (at 213.36 151.13 0)
@@
     (effects (font (size 1.27 1.27)) (justify left bottom))
   )
-  (label "{ADDRESS}" (at 144.78 128.27 0)
+  (label "{ADDRESS}" (at 144.78 133.35 0)
     (effects (font (size 1.27 1.27)) (justify left bottom))
   )
@@
     (effects (font (size 1.27 1.27)) (justify left bottom))
   )
-  (label "~{WR}" (at 147.32 119.38 0)
+  (label "~{WR}" (at 147.32 123.19 0)
     (effects (font (size 1.27 1.27)) (justify left bottom))
   )
@@
     (effects (font (size 1.27 1.27)) (justify right bottom))
   )
-  (label "~{RAM_CS}" (at 256.54 59.69 180)
+  (label "~{RAM_CS}" (at 259.08 59.69 180)
     (effects (font (size 1.27 1.27)) (justify right bottom))
   )
@@
     (effects (font (size 1.27 1.27)) (justify left bottom))
   )
-  (label "CLK_IN" (at 189.23 38.1 180)
+  (label "CLK_IN" (at 189.23 41.91 180)
     (effects (font (size 1.27 1.27)) (justify right bottom))
   )
-  (label "~{RD}" (at 147.32 116.84 0)
+  (label "~{RD}" (at 147.32 120.65 0)
     (effects (font (size 1.27 1.27)) (justify left bottom))
   )
@@
     (effects (font (size 1.27 1.27)) (justify left bottom))
   )
-  (label "D[0..7]" (at 144.78 130.81 0)
+  (label "D[0..7]" (at 144.78 135.89 0)
     (effects (font (size 1.27 1.27)) (justify left bottom))
   )
@@
   )
   (label "E" (at 67.31 129.54 0)
+    (effects (font (size 1.27 1.27)) (justify left bottom))
+  )
+  (label "~{EXTRAM_CS}" (at 147.32 114.3 0)
     (effects (font (size 1.27 1.27)) (justify left bottom))
   )
@@
     (effects (font (size 1.27 1.27)) (justify left bottom))
   )
-  (label "~{ROM_CS}" (at 256.54 57.15 180)
+  (label "~{ROM_CS}" (at 259.08 57.15 180)
     (effects (font (size 1.27 1.27)) (justify right bottom))
   )
@@
     )
   )
-  (sheet (at 158.75 142.24) (size 21.59 7.62) (fields_autoplaced)
+  (sheet (at 158.75 146.05) (size 21.59 7.62) (fields_autoplaced)
     (stroke (width 0) (type solid) (color 0 0 0 0))
     (fill (color 0 0 0 0.0000))
-    (property "Sheet name" "Tester" (id 0) (at 158.75 141.5284 0)
+    (property "Sheet name" "Tester" (id 0) (at 158.75 145.3384 0)
       (effects (font (size 1.27 1.27)) (justify left bottom))
     )
-    (property "Sheet file" "tester.kicad_sch" (id 1) (at 158.75 150.4446 0)
+    (property "Sheet file" "tester.kicad_sch" (id 1) (at 158.75 154.2546 0)
       (effects (font (size 1.27 1.27)) (justify left top))
     )
   )
-  (sheet (at 158.75 105.41) (size 21.59 29.21) (fields_autoplaced)
+  (sheet (at 158.75 105.41) (size 21.59 33.02) (fields_autoplaced)
     (stroke (width 0.1524) (type solid) (color 0 0 0 0))
     (fill (color 0 0 0 0.0000))
@@
       (effects (font (size 1.27 1.27)) (justify left bottom))
     )
-    (property "Sheet file" "memory.kicad_sch" (id 1) (at 158.75 135.2046 0)
+    (property "Sheet file" "memory.kicad_sch" (id 1) (at 158.75 139.0146 0)
       (effects (font (size 1.27 1.27)) (justify left top))
     )
-    (pin "D[0..7]" bidirectional (at 158.75 130.81 180)
+    (pin "D[0..7]" bidirectional (at 158.75 135.89 180)
       (effects (font (size 1.27 1.27)) (justify left))
     )
@@
       (effects (font (size 1.27 1.27)) (justify left))
     )
-    (pin "~{RD}" input (at 158.75 116.84 180)
-      (effects (font (size 1.27 1.27)) (justify left))
-    )
-    (pin "~{WR}" input (at 158.75 119.38 180)
+    (pin "~{RD}" input (at 158.75 120.65 180)
+      (effects (font (size 1.27 1.27)) (justify left))
+    )
+    (pin "~{WR}" input (at 158.75 123.19 180)
       (effects (font (size 1.27 1.27)) (justify left))
     )
@@
       (effects (font (size 1.27 1.27)) (justify left))
     )
-    (pin "~{ROM_WE}" input (at 158.75 124.46 180)
-      (effects (font (size 1.27 1.27)) (justify left))
-    )
-    (pin "{ADDRESS}" input (at 158.75 128.27 180)
+    (pin "~{ROM_WE}" input (at 158.75 128.27 180)
+      (effects (font (size 1.27 1.27)) (justify left))
+    )
+    (pin "{ADDRESS}" input (at 158.75 133.35 180)
+      (effects (font (size 1.27 1.27)) (justify left))
+    )
+    (pin "~{EXTRAM_CS}" input (at 158.75 114.3 180)
       (effects (font (size 1.27 1.27)) (justify left))
     )
@@
       (reference "#PWR0125") (unit 1) (value "VCC") (footprint "")
     )
+    (path "/51a25d9b-b48c-46f9-8897-a7e56a5418ca/e3be4575-4fff-4b16-a449-f39d1ab96f37"
+      (reference "#PWR0126") (unit 1) (value "VCC") (footprint "")
+    )
+    (path "/51a25d9b-b48c-46f9-8897-a7e56a5418ca/108b7719-421b-4157-9322-dfe93655268d"
+      (reference "#PWR0127") (unit 1) (value "GND") (footprint "")
+    )
     (path "/00000000-0000-0000-0000-000061c859bc/a7e376c9-fb69-4975-b411-b7a56874b31b"
       (reference "BAR1") (unit 1) (value "LED-Array-10-BGYR") (footprint "")
@@
       (reference "C50") (unit 1) (value "100n") (footprint "")
     )
+    (path "/51a25d9b-b48c-46f9-8897-a7e56a5418ca/14dd1e19-10dc-465a-8511-75979ee549a5"
+      (reference "C51") (unit 1) (value "100n") (footprint "")
+    )
     (path "/95d65710-49c8-4cb8-9de3-935bd85d56b1/f818d74a-5ffc-4388-be9e-aa337070bc87"
       (reference "D1") (unit 1) (value "1N5817") (footprint "Diode_THT:D_DO-41_SOD81_P10.16mm_Horizontal")
@@
       (reference "U34") (unit 4) (value "74AC10") (footprint "")
     )
+    (path "/51a25d9b-b48c-46f9-8897-a7e56a5418ca/62968bc7-38ef-4ca3-9397-f1d2c6dbc7e2"
+      (reference "U35") (unit 1) (value "AS6C4008-55PCN") (footprint "Package_DIP:DIP-32_W15.24mm")
+    )
     (path "/95d65710-49c8-4cb8-9de3-935bd85d56b1/b67fb8b6-c5be-4798-b081-82d2174f0e9d"

Commit message: Update for episode 21
Parts:
- removed R34: 10k, symbol Device:R_Small
Connections:
- no-connect marks 13 -> 12
Other:
- added sheet GPIO (gpio.kicad_sch)
