File: hardware/65C816.kicad_sch (KiCad schematic)
At the start: 11 parts, among them J1 POWER, U1 W65C816SxP

Commit message: Renumber
Parts:
- renumbered D2 to D1, R2 to R1, R12 to R2, R35 to R3, R36 to R4, R37 to R5

Commit message: Updates for episode 22
Other:
- added sheet Peripherals (peripherals.kicad_sch)
- sheet GPIO ports: added {PORTA}, {PORTB}; removed none
Changed lines of the file:
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@@
   (title_block
     (title "65C816 Homebrew Computer")
-    (date "2022-04-15")
-    (rev "A.21")
+    (date "2022-05-06")
+    (rev "A.22")
     (comment 2 "https://github.com/adrienkohlbecker/65C816")
     (comment 3 "Licensed under CERN-OHL-W v2")
@@
     (stroke (width 0) (type default) (color 0 0 0 0))
   )
+  (bus (pts (xy 271.78 36.83) (xy 283.21 36.83))
+    (stroke (width 0) (type default) (color 0 0 0 0))
+  )
   (wire (pts (xy 191.77 116.84) (xy 200.66 116.84))
     (stroke (width 0) (type default) (color 0 0 0 0))
@@
     (stroke (width 0) (type default) (color 0 0 0 0))
   )
+  (bus (pts (xy 252.73 68.58) (xy 241.3 68.58))
+    (stroke (width 0) (type default) (color 0 0 0 0))
+  )
   (wire (pts (xy 105.41 114.3) (xy 100.33 114.3))
     (stroke (width 0) (type default) (color 0 0 0 0))
@@
     (stroke (width 0) (type default) (color 0 0 0 0))
   )
+  (bus (pts (xy 252.73 66.04) (xy 241.3 66.04))
+    (stroke (width 0) (type default) (color 0 0 0 0))
+  )
   (bus (pts (xy 187.96 147.32) (xy 200.66 147.32))
     (stroke (width 0) (type default) (color 0 0 0 0))
@@
   )
   (wire (pts (xy 105.41 86.36) (xy 100.33 86.36))
+    (stroke (width 0) (type default) (color 0 0 0 0))
+  )
+  (bus (pts (xy 271.78 34.29) (xy 283.21 34.29))
     (stroke (width 0) (type default) (color 0 0 0 0))
   )
@@
     (effects (font (size 1.27 1.27)) (justify left bottom))
   )
+  (label "{PORTA}" (at 241.3 66.04 0)
+    (effects (font (size 1.27 1.27)) (justify left bottom))
+  )
   (label "A12" (at 100.33 124.46 0)
     (effects (font (size 1.27 1.27)) (justify left bottom))
@@
   (label "A14" (at 100.33 129.54 0)
     (effects (font (size 1.27 1.27)) (justify left bottom))
+  )
+  (label "{PORTB}" (at 283.21 36.83 180)
+    (effects (font (size 1.27 1.27)) (justify right bottom))
   )
   (label "DBA1" (at 100.33 73.66 0)
@@
     (effects (font (size 1.27 1.27)) (justify left bottom))
   )
+  (label "{PORTB}" (at 241.3 68.58 0)
+    (effects (font (size 1.27 1.27)) (justify left bottom))
+  )
   (label "CLK" (at 173.99 52.07 180)
     (effects (font (size 1.27 1.27)) (justify right bottom))
@@
   )
   (label "MONCLK" (at 233.68 137.16 180)
+    (effects (font (size 1.27 1.27)) (justify right bottom))
+  )
+  (label "{PORTA}" (at 283.21 34.29 180)
     (effects (font (size 1.27 1.27)) (justify right bottom))
   )
@@
     )
   )
+  (sheet (at 252.73 62.23) (size 19.05 19.05) (fields_autoplaced)
+    (stroke (width 0.1524) (type solid) (color 0 0 0 0))
+    (fill (color 0 0 0 0.0000))
+    (property "Sheet name" "Peripherals" (id 0) (at 252.73 61.5184 0)
+      (effects (font (size 1.27 1.27)) (justify left bottom))
+    )
+    (property "Sheet file" "peripherals.kicad_sch" (id 1) (at 252.73 81.8646 0)
+      (effects (font (size 1.27 1.27)) (justify left top))
+    )
+    (pin "{PORTA}" input (at 252.73 66.04 180)
+      (effects (font (size 1.27 1.27)) (justify left))
+    )
+    (pin "{PORTB}" input (at 252.73 68.58 180)
+      (effects (font (size 1.27 1.27)) (justify left))
+    )
+  )
   (sheet (at 200.66 133.35) (size 20.32 21.59) (fields_autoplaced)
     (stroke (width 0.1524) (type solid) (color 0 0 0 0))
@@
     (pin "VA" input (at 252.73 41.91 180)
       (effects (font (size 1.27 1.27)) (justify left))
+    )
+    (pin "{PORTA}" output (at 271.78 34.29 0)
+      (effects (font (size 1.27 1.27)) (justify right))
+    )
+    (pin "{PORTB}" output (at 271.78 36.83 0)
+      (effects (font (size 1.27 1.27)) (justify right))
     )
   )
@@
     (path "/ad436a76-34c0-4a92-97a3-841d53d56384" (page "9"))
     (path "/d540f930-f1b1-4dbe-a658-53337bc671f7" (page "10"))
+    (path "/9ed7b6bb-7ed2-4702-841f-e7214dc31a3a" (page "11"))
   )
   (symbol_instances
@@
       (reference "#PWR0137") (unit 1) (value "GND") (footprint "")
     )
+    (path "/9ed7b6bb-7ed2-4702-841f-e7214dc31a3a/fa8592f1-e58e-47b1-a136-fdf66694e39e"
+      (reference "#PWR0138") (unit 1) (value "VCC") (footprint "")
+    )
+    (path "/9ed7b6bb-7ed2-4702-841f-e7214dc31a3a/b812a04f-f15d-493c-bc9e-d753041a9d51"
+      (reference "#PWR0139") (unit 1) (value "GND") (footprint "")
+    )
+    (path "/9ed7b6bb-7ed2-4702-841f-e7214dc31a3a/fc71f5a8-1262-4967-95b8-b80e4caa500f"
+      (reference "#PWR0140") (unit 1) (value "VCC") (footprint "")
+    )
+    (path "/9ed7b6bb-7ed2-4702-841f-e7214dc31a3a/7e73d4d5-1427-4f74-a06a-74444b81f42d"
+      (reference "#PWR0141") (unit 1) (value "GND") (footprint "")
+    )
+    (path "/9ed7b6bb-7ed2-4702-841f-e7214dc31a3a/89ff1752-d989-4c90-bc1d-2da58196c565"
+      (reference "#PWR0142") (unit 1) (value "VCC") (footprint "")
+    )
+    (path "/9ed7b6bb-7ed2-4702-841f-e7214dc31a3a/cc4091e5-fde6-42b8-8820-46ea102df2d7"
+      (reference "#PWR0143") (unit 1) (value "GND") (footprint "")
+    )
     (path "/00000000-0000-0000-0000-000061c859bc/a7e376c9-fb69-4975-b411-b7a56874b31b"
       (reference "BAR1") (unit 1) (value "LED-Array-10-BGYR") (footprint "")
@@
       (reference "D3") (unit 1) (value "1N5817") (footprint "Diode_THT:D_DO-41_SOD81_P10.16mm_Horizontal")
     )
+    (path "/9ed7b6bb-7ed2-4702-841f-e7214dc31a3a/26a36c45-d460-4bae-835a-3016e3b778c6"
+      (reference "DS1") (unit 1) (value "HD44780") (footprint "Display:WC1602A")
+    )
     (path "/00000000-0000-0000-0000-0000615d1014"
       (reference "J1") (unit 1) (value "POWER") (footprint "")
@@
       (reference "RV1") (unit 1) (value "500k") (footprint "")
     )
+    (path "/9ed7b6bb-7ed2-4702-841f-e7214dc31a3a/00c27e7c-9cd0-41be-a04c-086ba8f8eabf"
+      (reference "RV2") (unit 1) (value "10k") (footprint "")
+    )
     (path "/00000000-0000-0000-0000-00006188a63e/00000000-0000-0000-0000-000061988e45"

Commit message: Update for episode 23
Other:
- sheet Clock ports: added ~{CLK_EN}; removed MONCLK
- sheet Monitor ports: added CLK_IN, ~{CLK_EN}; removed MONCLK
Changed lines of the file:
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@@
   (title_block
     (title "65C816 Homebrew Computer")
-    (date "2022-05-06")
-    (rev "A.22")
+    (date "2022-05-23")
+    (rev "A.23")
     (comment 2 "https://github.com/adrienkohlbecker/65C816")
     (comment 3 "Licensed under CERN-OHL-W v2")
@@
     (stroke (width 0) (type default) (color 0 0 0 0))
   )
+  (wire (pts (xy 220.98 139.7) (xy 233.68 139.7))
+    (stroke (width 0) (type default) (color 0 0 0 0))
+  )
   (wire (pts (xy 233.68 137.16) (xy 220.98 137.16))
     (stroke (width 0) (type default) (color 0 0 0 0))
@@
     (effects (font (size 1.27 1.27)) (justify left bottom))
   )
-  (label "MONCLK" (at 137.16 34.29 0)
+  (label "~{CLK_EN}" (at 137.16 34.29 0)
     (effects (font (size 1.27 1.27)) (justify left bottom))
   )
@@
     (effects (font (size 1.27 1.27)) (justify left bottom))
   )
-  (label "MONCLK" (at 233.68 137.16 180)
+  (label "~{CLK_EN}" (at 233.68 137.16 180)
+    (effects (font (size 1.27 1.27)) (justify right bottom))
+  )
+  (label "CLK_IN" (at 233.68 139.7 180)
     (effects (font (size 1.27 1.27)) (justify right bottom))
   )
@@
       (effects (font (size 1.27 1.27)) (justify right))
     )
-    (pin "MONCLK" input (at 146.05 34.29 180)
+    (pin "~{CLK_EN}" input (at 146.05 34.29 180)
       (effects (font (size 1.27 1.27)) (justify left))
     )
@@
       (effects (font (size 1.27 1.27)) (justify left))
     )
-    (pin "MONCLK" output (at 220.98 137.16 0)
-      (effects (font (size 1.27 1.27)) (justify right))
-    )
     (pin "SYNC" input (at 200.66 139.7 180)
       (effects (font (size 1.27 1.27)) (justify left))
@@
     (pin "VA" input (at 200.66 142.24 180)
       (effects (font (size 1.27 1.27)) (justify left))
+    )
+    (pin "~{CLK_EN}" output (at 220.98 137.16 0)
+      (effects (font (size 1.27 1.27)) (justify right))
+    )
+    (pin "CLK_IN" bidirectional (at 220.98 139.7 0)
+      (effects (font (size 1.27 1.27)) (justify right))
     )
   )
@@
       (reference "#PWR045") (unit 1) (value "VCC") (footprint "")
     )
-    (path "/00000000-0000-0000-0000-00006188a63e/00000000-0000-0000-0000-000061b55d16"
-      (reference "#PWR046") (unit 1) (value "GND") (footprint "")
+    (path "/00000000-0000-0000-0000-00006188a63e/9046a009-49d0-4967-8780-b19596d2a1b8"
+      (reference "#PWR046") (unit 1) (value "VCC") (footprint "")
     )
     (path "/00000000-0000-0000-0000-00006188a63e/00000000-0000-0000-0000-000061dd67d5"
@@
       (reference "#PWR0143") (unit 1) (value "GND") (footprint "")
     )
+    (path "/00000000-0000-0000-0000-00006188a63e/f10c80e2-e06f-4ff6-97b2-e81734468134"
+      (reference "#PWR0144") (unit 1) (value "GND") (footprint "")
+    )
+    (path "/00000000-0000-0000-0000-00006188a63e/9e40651a-3e1a-4d4e-91b1-8737c6133ef4"
+      (reference "#PWR0145") (unit 1) (value "VCC") (footprint "")
+    )
+    (path "/00000000-0000-0000-0000-00006188a63e/9938f9b2-7d2d-4f02-8ba8-5fa739df5360"
+      (reference "#PWR0146") (unit 1) (value "GND") (footprint "")
+    )
+    (path "/00000000-0000-0000-0000-00006188a63e/f8d2dab6-7ac4-4960-82d1-7ca695ce2fe1"
+      (reference "#PWR0147") (unit 1) (value "GND") (footprint "")
+    )
     (path "/00000000-0000-0000-0000-000061c859bc/a7e376c9-fb69-4975-b411-b7a56874b31b"
       (reference "BAR1") (unit 1) (value "LED-Array-10-BGYR") (footprint "")
@@
       (reference "R16") (unit 1) (value "10k") (footprint "")
     )
-    (path "/00000000-0000-0000-0000-00006188a63e/00000000-0000-0000-0000-000061dc18a8"
+    (path "/00000000-0000-0000-0000-00006188a63e/13fdffb1-a6c7-4690-8695-8477c4aadf42"
       (reference "R17") (unit 1) (value "10k") (footprint "")
     )
@@
       (reference "R23") (unit 1) (value "1k") (footprint "")
     )
-    (path "/00000000-0000-0000-0000-00006188a63e/26c30e6d-c469-4313-a981-55e1711112b8"
-      (reference "R24") (unit 1) (value "100") (footprint "")
-    )
-    (path "/00000000-0000-0000-0000-00006188a63e/b9ccdb07-26ea-4761-ad36-c6c26d163692"
-      (reference "R25") (unit 1) (value "100") (footprint "")
-    )
     (path "/95d65710-49c8-4cb8-9de3-935bd85d56b1/01ddd3b1-919f-4050-9eb5-fe57903e202e"
       (reference "R26") (unit 1) (value "10k") (footprint "")
@@
       (reference "SW4") (unit 1) (value "SW_DIP_SPDT_x02") (footprint "")
     )
-    (path "/00000000-0000-0000-0000-00006188a63e/00000000-0000-0000-0000-00006190529c"
-      (reference "SW5") (unit 1) (value "SW_DIP_x04") (footprint "")
-    )
-    (path "/00000000-0000-0000-0000-00006188a63e/28f8a272-ad05-49f0-b9f0-48cb70ea1d36"
-      (reference "SW6") (unit 1) (value "SW_DIP_SPDT_x01") (footprint "")
+    (path "/00000000-0000-0000-0000-00006188a63e/4ffd8958-74b4-48f4-8dba-37c5d6b7a503"
+      (reference "SW5") (unit 1) (value "SW_DIP_x03") (footprint "")
     )
     (path "/00000000-0000-0000-0000-000061b33617/00000000-0000-0000-0000-000061969d97"
@@
     )
     (path "/00000000-0000-0000-0000-00006188a63e/00000000-0000-0000-0000-000061bdff75"
-      (reference "U5") (unit 1) (value "74HC112") (footprint "")
+      (reference "U5") (unit 1) (value "74AC112") (footprint "")
     )
     (path "/00000000-0000-0000-0000-00006188a63e/00000000-0000-0000-0000-000061be0d5f"
-      (reference "U5") (unit 2) (value "74HC112") (footprint "")
+      (reference "U5") (unit 2) (value "74AC112") (footprint "")
     )
     (path "/00000000-0000-0000-0000-00006188a63e/00000000-0000-0000-0000-000061be1ff1"
-      (reference "U5") (unit 3) (value "74HC112") (footprint "")
+      (reference "U5") (unit 3) (value "74AC112") (footprint "")
     )
     (path "/00000000-0000-0000-0000-00006188a63e/00000000-0000-0000-0000-0000619b42fc"
@@
     )
     (path "/00000000-0000-0000-0000-00006188a63e/00000000-0000-0000-0000-000061c9d37c"
-      (reference "U7") (unit 1) (value "74HC112") (footprint "")
+      (reference "U7") (unit 1) (value "74AC112") (footprint "")
     )
     (path "/00000000-0000-0000-0000-00006188a63e/00000000-0000-0000-0000-000061cf4e59"
-      (reference "U7") (unit 2) (value "74HC112") (footprint "")
+      (reference "U7") (unit 2) (value "74AC112") (footprint "")
     )
     (path "/00000000-0000-0000-0000-00006188a63e/00000000-0000-0000-0000-000061cf632e"
-      (reference "U7") (unit 3) (value "74HC112") (footprint "")
+      (reference "U7") (unit 3) (value "74AC112") (footprint "")
     )
     (path "/00000000-0000-0000-0000-00006188a63e/00000000-0000-0000-0000-00006196ecf1"
       (reference "U8") (unit 1) (value "LMC555xN") (footprint "Package_DIP:DIP-8_W7.62mm")
     )
-    (path "/00000000-0000-0000-0000-00006188a63e/00000000-0000-0000-0000-000061b2bf9d"
-      (reference "U9") (unit 1) (value "74AC151") (footprint "")
+    (path "/00000000-0000-0000-0000-00006188a63e/7b872fee-c441-4c2d-8a8a-8b6e94dc680b"
+      (reference "U9") (unit 1) (value "74HC283") (footprint "")
     )
     (path "/00000000-0000-0000-0000-00006188a63e/00000000-0000-0000-0000-000061dd67c2"
-      (reference "U10") (unit 1) (value "74HC151") (footprint "")
+      (reference "U10") (unit 1) (value "74AC151") (footprint "")
     )
     (path "/00000000-0000-0000-0000-000061b33617/00000000-0000-0000-0000-000061967767"
@@
       (reference "U39") (unit 1) (value "74HC541") (footprint "")
     )
+    (path "/00000000-0000-0000-0000-00006188a63e/12b113e3-01f5-4d85-95a7-8902ccd8f69c"
+      (reference "U40") (unit 1) (value "74HC251") (footprint "")
+    )
     (path "/00000000-0000-0000-0000-00006188a63e/00000000-0000-0000-0000-00006194c461"

Commit message: Snapshot ep 24 work
Parts:
- removed C1: 220u, symbol Device:C_Polarized_Small
- removed C2: 10u, symbol Device:C_Polarized_Small
- removed C3: 100n, symbol Device:C_Small
- removed D1: POWER, symbol Device:LED_Small
- removed J1: POWER, symbol Connector_Generic:Conn_01x02
- removed R1: 1k, symbol Device:R_Small
- removed R2, R3, R4, R5: 10k, symbol Device:R_Small
- removed U1: W65C816SxP, symbol 65C816:W65C816SxP
Connections:
- no-connect marks 12 -> 11
Other:
- sheet Clock renamed Debug Clock
- removed sheet Glue Logic
- removed sheet Reset
- added sheet CPU Breakout (breakout.kicad_sch)
- sheet Address decoding ports: added A[0..23], ~{BANK0}; removed {ADDRESS}
- sheet Debug ports: added A[0..23]; removed {ADDRESS}
- sheet Debug Clock: file clock.kicad_sch -> debug_clock.kicad_sch
- sheet Debug Clock ports: added ~{CLK_EN_IN}, ~{CLK_EN_OUT}; removed ~{CLK_EN}
- sheet GPIO ports: added A[0..23]; removed {ADDRESS}
- sheet Memory ports: added A[0..23]; removed {ADDRESS}
- sheet Monitor ports: added A[0..23], ~{CLK_EN_OUT}; removed {ADDRESS}, ~{CLK_EN}

Commit message: Snapshot ep 24 work
Changed lines of the file:
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@@
     (effects (font (size 1.27 1.27)) (justify left bottom))
+  )
+  (symbol (lib_id "power:VCC") (at 181.61 102.87 90) (unit 1)
+    (in_bom yes) (on_board yes) (fields_autoplaced)
+    (property "Reference" "#PWR0165" (id 0) (at 185.42 102.87 0)
+      (effects (font (size 1.27 1.27)) hide)
+    )
+    (property "Value" "VCC" (id 1) (at 177.8 102.8699 90)
+      (effects (font (size 1.27 1.27)) (justify left))
+    )
+    (property "Footprint" "" (id 2) (at 181.61 102.87 0)
+      (effects (font (size 1.27 1.27)) hide)
+    )
+    (property "Datasheet" "" (id 3) (at 181.61 102.87 0)
+      (effects (font (size 1.27 1.27)) hide)
+    )
+    (pin "1")
   )
   (sheet (at 127 38.1) (size 21.59 15.24) (fields_autoplaced)
@@
       (reference "#PWR0164") (unit 1) (value "VCC") (footprint "")
     )
+    (path "/36f87b18-2ccc-47b1-8c83-cb4010940ee3"
+      (reference "#PWR0165") (unit 1) (value "VCC") (footprint "")
+    )
     (path "/00000000-0000-0000-0000-000061c859bc/a7e376c9-fb69-4975-b411-b7a56874b31b"

Commit message: More updates
Other:
- sheet CPU Breakout ports: added CLK_SRC; removed CLK_IN
- sheet Monitor ports: added CLK_SRC; removed CLK_IN
Changed lines of the file:
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@@
+    (stroke (width 0) (type default) (color 0 0 0 0))
+  )
+  (wire (pts (xy 172.72 102.87) (xy 181.61 102.87))
     (stroke (width 0) (type default) (color 0 0 0 0))
   )
@@
     (effects (font (size 1.27 1.27)) (justify left bottom))
   )
+  (label "E" (at 172.72 102.87 0)
+    (effects (font (size 1.27 1.27)) (justify left bottom))
+  )
   (label "~{ROM_CS}" (at 115.57 66.04 0)
     (effects (font (size 1.27 1.27)) (justify left bottom))
@@
     (effects (font (size 1.27 1.27)) (justify left bottom))
   )
-  (label "CLK_IN" (at 33.02 46.99 0)
+  (label "CLK_SRC" (at 33.02 46.99 0)
     (effects (font (size 1.27 1.27)) (justify left bottom))
   )
@@
     (effects (font (size 1.27 1.27)) (justify right bottom))
   )
-  (label "CLK_IN" (at 162.56 45.72 180)
+  (label "CLK_SRC" (at 162.56 45.72 180)
     (effects (font (size 1.27 1.27)) (justify right bottom))
   )
@@
     (effects (font (size 1.27 1.27)) (justify right bottom))
   )
-  (label "CLK_IN" (at 273.05 102.87 180)
+  (label "CLK_SRC" (at 273.05 102.87 180)
     (effects (font (size 1.27 1.27)) (justify right bottom))
   )
@@
   (label "~{RST}" (at 229.87 40.64 0)
     (effects (font (size 1.27 1.27)) (justify left bottom))
-  )
-  (symbol (lib_id "power:VCC") (at 181.61 102.87 90) (unit 1)
-    (in_bom yes) (on_board yes) (fields_autoplaced)
-    (property "Reference" "#PWR0165" (id 0) (at 185.42 102.87 0)
-      (effects (font (size 1.27 1.27)) hide)
-    )
-    (property "Value" "VCC" (id 1) (at 177.8 102.8699 90)
-      (effects (font (size 1.27 1.27)) (justify left))
-    )
-    (property "Footprint" "" (id 2) (at 181.61 102.87 0)
-      (effects (font (size 1.27 1.27)) hide)
-    )
-    (property "Datasheet" "" (id 3) (at 181.61 102.87 0)
-      (effects (font (size 1.27 1.27)) hide)
-    )
-    (pin "1")
   )
   (sheet (at 127 38.1) (size 21.59 15.24) (fields_autoplaced)
@@
       (effects (font (size 1.27 1.27)) (justify left))
     )
-    (pin "CLK_IN" bidirectional (at 256.54 102.87 0)
+    (pin "CLK_SRC" bidirectional (at 256.54 102.87 0)
       (effects (font (size 1.27 1.27)) (justify right))
     )
@@
       (effects (font (size 1.27 1.27)) (justify left))
     )
-    (pin "CLK_IN" bidirectional (at 46.99 46.99 180)
+    (pin "CLK_SRC" bidirectional (at 46.99 46.99 180)
       (effects (font (size 1.27 1.27)) (justify left))
     )
@@
       (reference "#FLG02") (unit 1) (value "PWR_FLAG") (footprint "")
     )
-    (path "/e5d0483c-6550-44c4-8b9e-8a347a49d5da/a5f491c8-cefa-4711-b3cf-794f723d3875"
-      (reference "#FLG0101") (unit 1) (value "PWR_FLAG") (footprint "")
-    )
-    (path "/e5d0483c-6550-44c4-8b9e-8a347a49d5da/518e5e07-2cf6-402c-a775-d1d24dd787ac"
+    (path "/e5d0483c-6550-44c4-8b9e-8a347a49d5da/62ebe6b3-dd4c-4c55-8d8a-21b9853b1e20"
       (reference "#PWR01") (unit 1) (value "VCC") (footprint "")
     )
@@
       (reference "#PWR0149") (unit 1) (value "GND") (footprint "")
     )
-    (path "/e5d0483c-6550-44c4-8b9e-8a347a49d5da/c19cf0f9-51a5-4b41-9abb-cbc7f35d86e6"
-      (reference "#PWR0150") (unit 1) (value "+5V") (footprint "")
+    (path "/e5d0483c-6550-44c4-8b9e-8a347a49d5da/24076432-06f0-41ae-9974-1a0c8570ee38"
+      (reference "#PWR0150") (unit 1) (value "VCC") (footprint "")
     )
     (path "/e5d0483c-6550-44c4-8b9e-8a347a49d5da/ac283e0f-56bc-4f02-8be9-0348725be0da/71f7c452-3171-4926-b8bf-53972928edbe"
@@
       (reference "#PWR0155") (unit 1) (value "GND") (footprint "")
     )
-    (path "/e5d0483c-6550-44c4-8b9e-8a347a49d5da/c6c85d1d-a22c-4e86-8ce2-daf52ef5ef35"
-      (reference "#PWR0156") (unit 1) (value "+5V") (footprint "")
-    )
-    (path "/e5d0483c-6550-44c4-8b9e-8a347a49d5da/b6844e6a-a82e-4046-aa12-ade336000618"
-      (reference "#PWR0157") (unit 1) (value "+5V") (footprint "")
+    (path "/e5d0483c-6550-44c4-8b9e-8a347a49d5da/2e46f42f-271c-4f1b-945a-fdd447ae38b7"
+      (reference "#PWR0156") (unit 1) (value "VCC") (footprint "")
     )
     (path "/e5d0483c-6550-44c4-8b9e-8a347a49d5da/4b8b470a-01e6-4542-b92a-d84e6f5eca5a"
@@
       (reference "#PWR0164") (unit 1) (value "VCC") (footprint "")
     )
-    (path "/36f87b18-2ccc-47b1-8c83-cb4010940ee3"
-      (reference "#PWR0165") (unit 1) (value "VCC") (footprint "")
+    (path "/e5d0483c-6550-44c4-8b9e-8a347a49d5da/ac283e0f-56bc-4f02-8be9-0348725be0da/1dfb63c7-0e87-4219-93d1-84841b66bb3e"
+      (reference "#PWR0165") (unit 1) (value "GND") (footprint "")
     )
     (path "/00000000-0000-0000-0000-000061c859bc/a7e376c9-fb69-4975-b411-b7a56874b31b"
@@
       (reference "DS1") (unit 1) (value "HD44780") (footprint "Display:WC1602A")
     )
-    (path "/e5d0483c-6550-44c4-8b9e-8a347a49d5da/dbce72ae-5929-4fd8-9d9f-d702fc31f3a5"
-      (reference "F1") (unit 1) (value "Fuse") (footprint "")
-    )
     (path "/e5d0483c-6550-44c4-8b9e-8a347a49d5da/3dad0243-5776-40ec-a406-c461334b4acf"
       (reference "J1") (unit 1) (value "Jack-DC") (footprint "")
@@
       (reference "J2") (unit 1) (value "Tester") (footprint "")
     )
+    (path "/e5d0483c-6550-44c4-8b9e-8a347a49d5da/ac283e0f-56bc-4f02-8be9-0348725be0da/45cc211d-8a75-4d24-a61e-55f7bfca8b8c"
+      (reference "J3") (unit 1) (value "Conn_01x02") (footprint "")
+    )
     (path "/e5d0483c-6550-44c4-8b9e-8a347a49d5da/53bee63e-299d-4029-8191-42375cde4417/3f8ec66d-a42d-4dd5-87bd-ba197deaf9fd"
       (reference "J4") (unit 1) (value "Conn_01x10") (footprint "")
     )
-    (path "/e5d0483c-6550-44c4-8b9e-8a347a49d5da/c2b7db24-ef06-4919-8c04-f22d4ca61f8b"
-      (reference "J5") (unit 1) (value "Conn_01x13") (footprint "")
+    (path "/e5d0483c-6550-44c4-8b9e-8a347a49d5da/751a9dd4-4e8e-43b2-87d2-ec9010be4550"
+      (reference "J5") (unit 1) (value "Conn_01x12") (footprint "")
     )
     (path "/e5d0483c-6550-44c4-8b9e-8a347a49d5da/3f06e0d1-d27c-4d18-90e3-1016a0097024"

Commit message: Updates for episode 25
Other:
- sheet CPU Breakout ports: added CLK_IN, ~{CLK_EN}; removed CLK_SRC, ~{CLK_EN_IN}
- sheet Debug Clock ports: added ~{CLK_EN}; removed ~{CLK_EN_IN}, ~{CLK_EN_OUT}
- sheet Monitor ports: added CLK_IN, ~{CLK_EN}; removed CLK_SRC, ~{CLK_EN_OUT}
