File: hardware/clock.kicad_sch (KiCad schematic)
At the start: 50 parts, among them SW1 Pulse, SW2 Mode, SW3 Speed, SW4 SW_DIP_x04, SW6 SW_DIP_SPDT_x02, U10 74HC112, U11 74HC74, U12 LMC555xN, U13 74HC112, U14 74HC74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

Commit message: Updates for Episode 14
Parts:
- C11, C12, C13, C14, C16: symbol Device:CP_Small -> Device:C_Polarized_Small
- RV1: symbol Device:R_POT -> Device:R_Potentiometer
- SW1, SW2, SW3: symbol keyboard:SW_Push -> Switch:SW_Push
- U12: symbol AK's_Library:LMC555xN -> 65C816:LMC555xN
Changed lines of the file:
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@@
   (title_block
     (title "Clock Module")
-    (date "2022-01-09")
-    (rev "A.13")
+    (date "2022-01-14")
+    (rev "A.14")
     (comment 2 "https://github.com/adrienkohlbecker/65C816")
     (comment 3 "Licensed under CERN-OHL-W v2")
@@
     (pin "1")
   )
-  (symbol (lib_id "keyboard:SW_Push") (at 21.59 102.87 90) (unit 1)
+  (symbol (lib_id "Switch:SW_Push") (at 21.59 102.87 90) (unit 1)
     (in_bom yes) (on_board yes)
     (property "Reference" "SW2" (id 0) (at 22.8092 101.7016 90)
@@
       (effects (font (size 1.27 1.27)) hide)
     )
-    (property "Datasheet" "" (id 3) (at 16.51 102.87 0)
+    (property "Datasheet" "~" (id 3) (at 16.51 102.87 0)
       (effects (font (size 1.27 1.27)) hide)
     )
@@
     (pin "6")
   )
-  (symbol (lib_id "Device:CP_Small") (at 34.29 109.22 0) (unit 1)
+  (symbol (lib_id "Device:C_Polarized_Small") (at 34.29 109.22 0) (unit 1)
     (in_bom yes) (on_board yes)
     (property "Reference" "C12" (id 0) (at 36.6268 108.0516 0)
@@
     (pin "1")
   )
-  (symbol (lib_id "keyboard:SW_Push") (at 21.59 142.24 90) (unit 1)
+  (symbol (lib_id "Switch:SW_Push") (at 21.59 142.24 90) (unit 1)
     (in_bom yes) (on_board yes)
     (property "Reference" "SW3" (id 0) (at 22.8092 141.0716 90)
@@
       (effects (font (size 1.27 1.27)) hide)
     )
-    (property "Datasheet" "" (id 3) (at 16.51 142.24 0)
+    (property "Datasheet" "~" (id 3) (at 16.51 142.24 0)
       (effects (font (size 1.27 1.27)) hide)
     )
@@
     (pin "4")
   )
-  (symbol (lib_id "Device:CP_Small") (at 34.29 148.59 0) (unit 1)
+  (symbol (lib_id "Device:C_Polarized_Small") (at 34.29 148.59 0) (unit 1)
     (in_bom yes) (on_board yes)
     (property "Reference" "C13" (id 0) (at 36.6268 147.4216 0)
@@
     (pin "1")
   )
-  (symbol (lib_id "AK's_Library:LMC555xN") (at 224.79 52.07 0) (unit 1)
+  (symbol (lib_id "65C816:LMC555xN") (at 224.79 52.07 0) (unit 1)
     (in_bom yes) (on_board yes)
     (property "Reference" "U12" (id 0) (at 218.44 43.18 0))
@@
     (pin "2")
   )
-  (symbol (lib_id "Device:R_POT") (at 200.66 57.15 0) (mirror x) (unit 1)
+  (symbol (lib_id "Device:R_Potentiometer") (at 200.66 57.15 0) (mirror x) (unit 1)
     (in_bom yes) (on_board yes)
     (property "Reference" "RV1" (id 0) (at 198.9074 55.9816 0)
@@
     (pin "1")
   )
-  (symbol (lib_id "Device:CP_Small") (at 212.09 62.23 0) (unit 1)
+  (symbol (lib_id "Device:C_Polarized_Small") (at 212.09 62.23 0) (unit 1)
     (in_bom yes) (on_board yes)
     (property "Reference" "C14" (id 0) (at 214.4268 61.0616 0)
@@
     (pin "2")
   )
-  (symbol (lib_id "Device:CP_Small") (at 34.29 68.58 0) (unit 1)
+  (symbol (lib_id "Device:C_Polarized_Small") (at 34.29 68.58 0) (unit 1)
     (in_bom yes) (on_board yes)
     (property "Reference" "C11" (id 0) (at 36.6268 67.4116 0)
@@
     (pin "2")
   )
-  (symbol (lib_id "keyboard:SW_Push") (at 21.59 62.23 90) (unit 1)
+  (symbol (lib_id "Switch:SW_Push") (at 21.59 62.23 90) (unit 1)
     (in_bom yes) (on_board yes)
     (property "Reference" "SW1" (id 0) (at 22.8092 61.0616 90)
@@
       (effects (font (size 1.27 1.27)) hide)
     )
-    (property "Datasheet" "" (id 3) (at 16.51 62.23 0)
+    (property "Datasheet" "~" (id 3) (at 16.51 62.23 0)
       (effects (font (size 1.27 1.27)) hide)
     )
@@
     (pin "1")
   )
-  (symbol (lib_id "Device:CP_Small") (at 20.32 223.52 0) (unit 1)
+  (symbol (lib_id "Device:C_Polarized_Small") (at 20.32 223.52 0) (unit 1)
     (in_bom yes) (on_board yes)
     (property "Reference" "C16" (id 0) (at 23.3172 222.3516 0)
@@
       (effects (font (size 1.27 1.27)) (justify left))
     )
-    (property "Footprint" "" (id 2) (at 21.2852 227.33 0)
-      (effects (font (size 1.27 1.27)) hide)
-    )
+    (property "Footprint" "" (id 2) (at 20.32 223.52 0)
+      (effects (font (size 1.27 1.27)) hide)
+    )

Commit message: Updates for episode 17
Parts:
- added C48: 22u, symbol Device:C_Polarized_Small
- added R11, R32: 100, symbol Device:R_Small
- added R33: 10k, symbol Device:R_Small
- added SW8: SW_DIP_SPDT_x01, symbol 65C816:SW_DIP_SPDT_x01
- U16: value 74HC151 -> 74AC151
Connections:
- net ~{PWRUP} is gone; now on an unnamed net: SW6.1, SW6.2, SW6.3, SW6.4
- net CLK: now also R11.2; no longer U16.5 (Z)
- net GND: now also C48.2
- net SLOW: now also SW8.3, SW8.4; no longer U14.5 (Q)
- net VCC: now also R33.2; no longer U9.13, U9.9
- net ~{CLK}: now also R32.2; no longer U16.6 (~{Z})
- net at U9.8: now also U9.13
- new net: C48.1, R33.1, U9.9
- new net: SW8.2, U14.5 (Q)
- new net: R11.1, U16.5 (Z)
- new net: R32.1, U16.6 (~{Z})
- new net MONCLK: SW8.1
- no-connect marks 14 -> 12
Other:
- moved on the sheet: D5, R13, R14, R15, R16, R17, SW6, U10B, U16, U9D, U9E, U9F
