File: hardware/clock.kicad_sch (KiCad schematic)
At the start: 55 parts, among them SW1 Pulse, SW2 Mode, SW3 Speed, SW4 SW_DIP_x04, SW6 SW_DIP_SPDT_x02, SW8 SW_DIP_SPDT_x01, U10 74HC112, U11 74HC74, U12 LMC555xN, U13 74HC112, U14 74HC74, U15 74HC193, U16 74AC151, U17 74HC151, U9 74HC14, X1 20MHz

Commit message: Updates for episode 20
Connections:
- net FAST: now also U17.14 (I5), U17.15 (I4); no longer U17.1 (I3), U17.2 (I2)
- net FAST_~{SLOW}: now also U16.11 (S0), U17.11 (S0), U17.9 (S2)
- net GND: no longer U17.9 (S2)
- net SLOW: now also U17.1 (I3), U17.2 (I2); no longer U17.14 (I5), U17.15 (I4)
- net VCC: no longer U16.11 (S0), U17.11 (S0)
Changed lines of the file:
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@@
   (junction (at 81.28 226.06) (diameter 0) (color 0 0 0 0)
   )
+  (junction (at 297.18 134.62) (diameter 0) (color 0 0 0 0)
+  )
   (junction (at 293.37 46.99) (diameter 0) (color 0 0 0 0)
   )
@@
   (junction (at 76.2 41.91) (diameter 0) (color 0 0 0 0)
   )
+  (junction (at 297.18 121.92) (diameter 0) (color 0 0 0 0)
+  )
   (junction (at 97.79 41.91) (diameter 0) (color 0 0 0 0)
   )
+  (junction (at 297.18 114.3) (diameter 0) (color 0 0 0 0)
+  )
   (junction (at 76.2 36.83) (diameter 0) (color 0 0 0 0)
   )
@@
   (junction (at 236.22 198.12) (diameter 0) (color 0 0 0 0)
   )
-  (junction (at 298.45 142.24) (diameter 0) (color 0 0 0 0)
-  )
   (junction (at 34.29 142.24) (diameter 0) (color 0 0 0 0)
   )
   (junction (at 102.87 36.83) (diameter 0) (color 0 0 0 0)
   )
+  (junction (at 297.18 111.76) (diameter 0) (color 0 0 0 0)
+  )
   (junction (at 142.24 54.61) (diameter 0) (color 0 0 0 0)
   )
@@
   (junction (at 91.44 220.98) (diameter 0) (color 0 0 0 0)
   )
+  (junction (at 294.64 59.69) (diameter 0) (color 0 0 0 0)
+  )
   (junction (at 58.42 190.5) (diameter 0) (color 0 0 0 0)
   )
@@
   )
   (junction (at 50.8 226.06) (diameter 0) (color 0 0 0 0)
-  )
-  (junction (at 297.18 114.3) (diameter 0) (color 0 0 0 0)
   )
   (junction (at 220.98 134.62) (diameter 0) (color 0 0 0 0)
@@
     (stroke (width 0) (type default) (color 0 0 0 0))
   )
+  (wire (pts (xy 297.18 121.92) (xy 297.18 124.46))
+    (stroke (width 0) (type default) (color 0 0 0 0))
+  )
   (wire (pts (xy 114.3 54.61) (xy 113.03 54.61))
     (stroke (width 0) (type default) (color 0 0 0 0))
@@
     (stroke (width 0) (type default) (color 0 0 0 0))
   )
+  (wire (pts (xy 299.72 137.16) (xy 297.18 137.16))
+    (stroke (width 0) (type default) (color 0 0 0 0))
+  )
   (wire (pts (xy 41.91 26.67) (xy 48.26 26.67))
     (stroke (width 0) (type default) (color 0 0 0 0))
@@
     (stroke (width 0) (type default) (color 0 0 0 0))
   )
+  (wire (pts (xy 281.94 59.69) (xy 294.64 59.69))
+    (stroke (width 0) (type default) (color 0 0 0 0))
+  )
   (wire (pts (xy 97.79 41.91) (xy 114.3 41.91))
     (stroke (width 0) (type default) (color 0 0 0 0))
@@
     (stroke (width 0) (type default) (color 0 0 0 0))
   )
-  (wire (pts (xy 290.83 114.3) (xy 297.18 114.3))
-    (stroke (width 0) (type default) (color 0 0 0 0))
-  )
   (wire (pts (xy 220.98 134.62) (xy 250.19 134.62))
     (stroke (width 0) (type default) (color 0 0 0 0))
@@
     (stroke (width 0) (type default) (color 0 0 0 0))
   )
-  (wire (pts (xy 290.83 124.46) (xy 297.18 124.46))
-    (stroke (width 0) (type default) (color 0 0 0 0))
-  )
   (wire (pts (xy 78.74 41.91) (xy 76.2 41.91))
     (stroke (width 0) (type default) (color 0 0 0 0))
   )
+  (wire (pts (xy 297.18 111.76) (xy 297.18 114.3))
+    (stroke (width 0) (type default) (color 0 0 0 0))
+  )
   (wire (pts (xy 34.29 102.87) (xy 34.29 106.68))
     (stroke (width 0) (type default) (color 0 0 0 0))
@@
     (stroke (width 0) (type default) (color 0 0 0 0))
   )
-  (wire (pts (xy 295.91 59.69) (xy 284.48 59.69))
+  (wire (pts (xy 295.91 59.69) (xy 294.64 59.69))
     (stroke (width 0) (type default) (color 0 0 0 0))
   )
@@
     (stroke (width 0) (type default) (color 0 0 0 0))
   )
-  (wire (pts (xy 284.48 62.23) (xy 295.91 62.23))
+  (wire (pts (xy 281.94 62.23) (xy 295.91 62.23))
     (stroke (width 0) (type default) (color 0 0 0 0))
   )
@@
     (stroke (width 0) (type default) (color 0 0 0 0))
   )
+  (wire (pts (xy 294.64 57.15) (xy 294.64 59.69))
+    (stroke (width 0) (type default) (color 0 0 0 0))
+  )
   (wire (pts (xy 170.18 180.34) (xy 170.18 182.88))
     (stroke (width 0) (type default) (color 0 0 0 0))
@@
     (stroke (width 0) (type default) (color 0 0 0 0))
   )
-  (wire (pts (xy 295.91 57.15) (xy 293.37 57.15))
+  (wire (pts (xy 295.91 57.15) (xy 294.64 57.15))
     (stroke (width 0) (type default) (color 0 0 0 0))
   )
@@
     (stroke (width 0) (type default) (color 0 0 0 0))
   )
+  (wire (pts (xy 297.18 137.16) (xy 297.18 134.62))
+    (stroke (width 0) (type default) (color 0 0 0 0))
+  )
   (wire (pts (xy 257.81 123.19) (xy 271.78 123.19))
     (stroke (width 0) (type default) (color 0 0 0 0))
@@
     (stroke (width 0) (type default) (color 0 0 0 0))
   )
-  (wire (pts (xy 299.72 137.16) (xy 298.45 137.16))
-    (stroke (width 0) (type default) (color 0 0 0 0))
-  )
   (wire (pts (xy 34.29 142.24) (xy 34.29 146.05))
     (stroke (width 0) (type default) (color 0 0 0 0))
@@
     (stroke (width 0) (type default) (color 0 0 0 0))
   )
+  (wire (pts (xy 297.18 134.62) (xy 297.18 132.08))
+    (stroke (width 0) (type default) (color 0 0 0 0))
+  )
   (wire (pts (xy 171.45 177.8) (xy 170.18 177.8))
     (stroke (width 0) (type default) (color 0 0 0 0))
@@
     (stroke (width 0) (type default) (color 0 0 0 0))
   )
-  (wire (pts (xy 298.45 137.16) (xy 298.45 142.24))
-    (stroke (width 0) (type default) (color 0 0 0 0))
-  )
   (wire (pts (xy 254 60.96) (xy 250.19 60.96))
     (stroke (width 0) (type default) (color 0 0 0 0))
@@
     (stroke (width 0) (type default) (color 0 0 0 0))
   )
-  (wire (pts (xy 299.72 134.62) (xy 288.29 134.62))
+  (wire (pts (xy 299.72 134.62) (xy 297.18 134.62))
     (stroke (width 0) (type default) (color 0 0 0 0))
   )
@@
   )
   (wire (pts (xy 236.22 172.72) (xy 254 172.72))
+    (stroke (width 0) (type default) (color 0 0 0 0))
+  )
+  (wire (pts (xy 297.18 134.62) (xy 283.21 134.62))
     (stroke (width 0) (type default) (color 0 0 0 0))
   )
@@
     (effects (font (size 1.27 1.27)) (justify right bottom))
   )
-  (label "PULSE_~{RUN}" (at 284.48 62.23 0)
+  (label "PULSE_~{RUN}" (at 281.94 62.23 0)
     (effects (font (size 1.27 1.27)) (justify left bottom))
   )
@@
     (effects (font (size 1.27 1.27)) (justify left bottom))
   )
-  (label "FAST" (at 290.83 114.3 0)
-    (effects (font (size 1.27 1.27)) (justify left bottom))
-  )
   (label "FAST_ON_RST" (at 77.47 116.84 0)
     (effects (font (size 1.27 1.27)) (justify left bottom))
@@
     (effects (font (size 1.27 1.27)) (justify left bottom))
   )
-  (label "FAST" (at 290.83 124.46 0)
+  (label "FAST" (at 290.83 119.38 0)
     (effects (font (size 1.27 1.27)) (justify left bottom))
   )
@@
     (effects (font (size 1.27 1.27)) (justify right bottom))
   )
-  (label "FAST_~{SLOW}" (at 288.29 134.62 0)
+  (label "FAST_~{SLOW}" (at 283.21 134.62 0)
     (effects (font (size 1.27 1.27)) (justify left bottom))
   )
@@
     (effects (font (size 1.27 1.27)) (justify left bottom))
   )
-  (label "SLOW" (at 290.83 119.38 0)
-    (effects (font (size 1.27 1.27)) (justify left bottom))
-  )
-  (label "FAST_~{SLOW}" (at 284.48 59.69 0)
+  (label "FAST_~{SLOW}" (at 281.94 59.69 0)
     (effects (font (size 1.27 1.27)) (justify left bottom))
   )
@@
     (pin "1")
   )
-  (symbol (lib_id "power:VCC") (at 293.37 57.15 0) (unit 1)
-    (in_bom yes) (on_board yes)
-    (property "Reference" "#PWR068" (id 0) (at 293.37 60.96 0)
-      (effects (font (size 1.27 1.27)) hide)
-    )
-    (property "Value" "VCC" (id 1) (at 290.83 54.61 0))
-    (property "Footprint" "" (id 2) (at 293.37 57.15 0)
-      (effects (font (size 1.27 1.27)) hide)
-    )
-    (property "Datasheet" "" (id 3) (at 293.37 57.15 0)
-      (effects (font (size 1.27 1.27)) hide)
-    )
-    (pin "1")
-  )
   (symbol (lib_id "power:VCC") (at 152.4 63.5 0) (unit 1)
     (in_bom yes) (on_board yes)
@@
       (effects (font (size 1.27 1.27)) hide)
     )
-    (pin "1")
-  )
-  (symbol (lib_id "power:VCC") (at 297.18 132.08 0) (unit 1)
-    (in_bom yes) (on_board yes)
-    (property "Reference" "#PWR069" (id 0) (at 297.18 135.89 0)
-      (effects (font (size 1.27 1.27)) hide)
-    )
-    (property "Value" "VCC" (id 1) (at 294.64 129.54 0))
-    (property "Footprint" "" (id 2) (at 297.18 132.08 0)
-      (effects (font (size 1.27 1.27)) hide)
-    )
-    (property "Datasheet" "" (id 3) (at 297.18 132.08 0)
-      (effects (font (size 1.27 1.27)) hide)
-    )

Commit message: Update for episode 21
Other:
- note added: "0000 10Mhz 0001 5Mhz 0010 3.33Mhz 0011 2.5Mhz 0100 2Mhz 0101 1.67Mhz 0110 1.43Mhz 0111 1.25Mhz 1000 1.11Mhz 1001 1Mhz 1010 0.90Mhz 1011 0.83Mhz 1100 0.76Mhz 1101 0.71Mhz 1110 0.66Mhz 1111 0.62Mhz"
- note added: "Divider setting:"
- moved on the sheet: R18, R19, R20, R21, SW4, U14B, U15, X1

Commit message: Renumber
Parts:
- renumbered C18 to C10, C19 to C11, C20 to C12, C21 to C13, C22 to C14, C23 to C15, C24 to C16, C29 to C17, C30 to C18, C14 to C19, C15 to C20, C16 to C4, C48 to C5, C17 to C6, C11 to C7, C12 to C8, C13 to C9, D5 to D2, R6 to R10, R7 to R11, R8 to R12, R14 to R13, R15 to R14, R16 to R15, R17 to R16, R18 to R17, R19 to R18, R20 to R19, R21 to R20, R13 to R21, R9 to R22, R10 to R23, R11 to R24, R32 to R25, R33 to R6, R3 to R7, R4 to R8, R5 to R9, SW6 to SW4, SW4 to SW5, SW8 to SW6, U17 to U10, U9 to U2, U11 to U3, U15 to U4, U13 to U5, U14 to U6, U10 to U7, U12 to U8, U16 to U9

Commit message: Update for episode 23
Parts:
- removed R24, R25: 100, symbol Device:R_Small
- removed SW5: SW_DIP_x04, symbol Switch:SW_DIP_x04
- removed SW6: SW_DIP_SPDT_x01, symbol 65C816:SW_DIP_SPDT_x01
- removed U9: 74AC151, symbol 74xx:74LS151
- added SW5: SW_DIP_x03, symbol Switch:SW_DIP_x03
- added U40: 74HC251, symbol 74xx:74LS251
- added U9: 74HC283, symbol 74xx:74LS283
- U10: value 74HC151 -> 74AC151
- U5, U7: value 74HC112 -> 74AC112
Connections:
- net CLK: now also U40.5 (Y)
- net FAST: now also U40.1 (I3), U40.2 (I2)
- net FAST_~{SLOW}: now also U40.10 (S1), U40.11 (S0)
- net GND: now also U40.8 (GND), U9.11 (B4), U9.12 (A4), U9.15 (B3), U9.2 (B2), U9.6 (B1), U9.8 (GND)
- net PULSE: now also U40.12 (I7), U40.13 (I6), U40.14 (I5), U40.15 (I4)
- net PULSE_~{RUN}: now also U40.9 (S2)
- net SLOW: now also U6.5 (Q), U40.3 (I1), U40.4 (I0)
- net VCC: now also SW5.1, SW5.2, SW5.3, U40.16 (VCC), U9.16 (VCC), U9.7 (C0)
- net ~{CLK}: now also U40.6 (~{Y})
- net at U4.1 (B): now also U9.1 (S2); no longer R19.2
- net at U4.10 (C): now also U9.13 (S3); no longer R18.2
- net at U4.15 (A): now also U9.4 (S1); no longer R20.2
- net at U4.9 (D): now also U9.10 (S4); no longer R17.2
- new net: R18.2, SW5.6, U9.14 (A3)
- new net: R19.2, SW5.5, U9.3 (A2)
- new net: R20.2, SW5.4, U9.5 (A1)
- new net ~{CLK_EN}: R17.2, U40.7 (~{OE})
- no-connect marks 12 -> 13
Other:
- note added: "000 5Mhz 001 3.33Mhz 010 2.5Mhz 011 2Mhz 100 1.67Mhz 101 1.43Mhz 110 1.25Mhz 111 1.11Mhz"
- note added: "=> overall, maximum frequency of the fast clock is 6.87MHz"
- note added: "Fast clock falling edge => 12.3 ns (74AC151) => RUN => 9.4 ns (74AC112) => PULSE_RUN selection bit => 51 ns (74HC251) => CLK We want the whole chain to happen before the fast clock has a rising edge => minimum half period of the fast clock 12.3+9.4+51ns = 72.7ns => maximum frequency of the fast clock 1000/72.7/2 = 6.87MHz"
- note added: "Fast clock falling edge => 9.4 ns (74AC112) => FAST_SLOW selection bit => 51 ns (74HC251) => CLK We want the whole chain to happen before the fast clock has a rising edge => minimum half period of the fast clock 9.4+51ns = 60.4ns => maximum frequency of the fast clock 1000/60.4/2 = 8.27MHz"
- note removed: "0000 10Mhz 0001 5Mhz 0010 3.33Mhz 0011 2.5Mhz 0100 2Mhz 0101 1.67Mhz 0110 1.43Mhz 0111 1.25Mhz 1000 1.11Mhz 1001 1Mhz 1010 0.90Mhz 1011 0.83Mhz 1100 0.76Mhz 1101 0.71Mhz 1110 0.66Mhz 1111 0.62Mhz"
- moved on the sheet: R18, R19, R20, U4, U6B, X1
