File: hardware/tester.kicad_sch (KiCad schematic)
At the start: 5 parts, among them J2 Tester, SW7 SW_DIP_x08

Commit message: Renumber
Parts:
- renumbered RN7 to RN10, RN8 to RN11, SW7 to SW8
Changed lines of the file:
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@@
   (symbol (lib_id "Device:R_Network08") (at 143.51 58.42 270) (mirror x) (unit 1)
     (in_bom yes) (on_board yes)
-    (property "Reference" "RN8" (id 0) (at 143.51 45.085 90))
+    (property "Reference" "RN11" (id 0) (at 143.51 45.085 90))
     (property "Value" "1.5k" (id 1) (at 143.51 47.3964 90))
     (property "Footprint" "Resistor_THT:R_Array_SIP9" (id 2) (at 143.51 46.355 90)
@@
   (symbol (lib_id "Switch:SW_DIP_x08") (at 68.58 60.96 0) (unit 1)
     (in_bom yes) (on_board yes)
-    (property "Reference" "SW7" (id 0) (at 68.58 44.0182 0))
+    (property "Reference" "SW8" (id 0) (at 68.58 44.0182 0))
     (property "Value" "SW_DIP_x08" (id 1) (at 68.58 46.3296 0))
     (property "Footprint" "" (id 2) (at 68.58 60.96 0)
@@
   (symbol (lib_id "power:GND") (at 149.86 69.85 0) (unit 1)
     (in_bom yes) (on_board yes)
-    (property "Reference" "#PWR0109" (id 0) (at 149.86 76.2 0)
+    (property "Reference" "#PWR0123" (id 0) (at 149.86 76.2 0)
       (effects (font (size 1.27 1.27)) hide)
     )
@@
   (symbol (lib_id "power:VCC") (at 58.42 49.53 0) (unit 1)
     (in_bom yes) (on_board yes)
-    (property "Reference" "#PWR0110" (id 0) (at 58.42 53.34 0)
+    (property "Reference" "#PWR0121" (id 0) (at 58.42 53.34 0)
       (effects (font (size 1.27 1.27)) hide)
     )
@@
   (symbol (lib_id "Device:R_Network08") (at 85.09 77.47 180) (unit 1)
     (in_bom yes) (on_board yes)
-    (property "Reference" "RN7" (id 0) (at 97.282 76.3016 0)
+    (property "Reference" "RN10" (id 0) (at 97.282 76.3016 0)
       (effects (font (size 1.27 1.27)) (justify right))
     )
@@
   (symbol (lib_id "power:GND") (at 95.25 83.82 0) (unit 1)
     (in_bom yes) (on_board yes)
-    (property "Reference" "#PWR0111" (id 0) (at 95.25 90.17 0)
+    (property "Reference" "#PWR0122" (id 0) (at 95.25 90.17 0)
       (effects (font (size 1.27 1.27)) hide)
     )

Commit message: Snapshot ep 24 work
Parts:
- RN10: value 10k -> 3.3k
Changed lines of the file:
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@@
   (title_block
     (title "Tester Module")
-    (date "2022-05-23")
-    (rev "A.23")
+    (date "2022-07-04")
+    (rev "A.24")
     (comment 2 "https://github.com/adrienkohlbecker/65C816")
     (comment 3 "Licensed under CERN-OHL-W v2")
@@
       (effects (font (size 1.27 1.27)) (justify right))
     )
-    (property "Value" "10k" (id 1) (at 97.282 78.613 0)
+    (property "Value" "3.3k" (id 1) (at 97.282 78.613 0)
       (effects (font (size 1.27 1.27)) (justify right))
     )

Commit message: Update main project
Parts:
- renumbered BAR6 to BAR8, J2 to J1, RN10 to RN7, RN11 to RN8, SW8 to SW6
Changed lines of the file:
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@@
   (symbol (lib_id "65C816:LED-Array-8") (at 130.81 59.69 0) (unit 1)
     (in_bom yes) (on_board yes)
-    (property "Reference" "BAR6" (id 0) (at 130.81 44.831 0))
+    (property "Reference" "BAR8" (id 0) (at 130.81 44.831 0))
     (property "Value" "Red" (id 1) (at 130.81 47.1424 0))
     (property "Footprint" "" (id 2) (at 131.572 74.295 0)
@@
   (symbol (lib_id "Device:R_Network08") (at 143.51 58.42 270) (mirror x) (unit 1)
     (in_bom yes) (on_board yes)
-    (property "Reference" "RN11" (id 0) (at 143.51 45.085 90))
+    (property "Reference" "RN8" (id 0) (at 143.51 45.085 90))
     (property "Value" "1.5k" (id 1) (at 143.51 47.3964 90))
     (property "Footprint" "Resistor_THT:R_Array_SIP9" (id 2) (at 143.51 46.355 90)
@@
   (symbol (lib_id "Switch:SW_DIP_x08") (at 68.58 60.96 0) (unit 1)
     (in_bom yes) (on_board yes)
-    (property "Reference" "SW8" (id 0) (at 68.58 44.0182 0))
+    (property "Reference" "SW6" (id 0) (at 68.58 44.0182 0))
     (property "Value" "SW_DIP_x08" (id 1) (at 68.58 46.3296 0))
     (property "Footprint" "" (id 2) (at 68.58 60.96 0)
@@
   (symbol (lib_id "power:GND") (at 149.86 69.85 0) (unit 1)
     (in_bom yes) (on_board yes)
-    (property "Reference" "#PWR0123" (id 0) (at 149.86 76.2 0)
+    (property "Reference" "#PWR0114" (id 0) (at 149.86 76.2 0)
       (effects (font (size 1.27 1.27)) hide)
     )
@@
   (symbol (lib_id "power:VCC") (at 58.42 49.53 0) (unit 1)
     (in_bom yes) (on_board yes)
-    (property "Reference" "#PWR0121" (id 0) (at 58.42 53.34 0)
+    (property "Reference" "#PWR0112" (id 0) (at 58.42 53.34 0)
       (effects (font (size 1.27 1.27)) hide)
     )
@@
   (symbol (lib_id "Device:R_Network08") (at 85.09 77.47 180) (unit 1)
     (in_bom yes) (on_board yes)
-    (property "Reference" "RN10" (id 0) (at 97.282 76.3016 0)
+    (property "Reference" "RN7" (id 0) (at 97.282 76.3016 0)
       (effects (font (size 1.27 1.27)) (justify right))
     )
@@
   (symbol (lib_id "power:GND") (at 95.25 83.82 0) (unit 1)
     (in_bom yes) (on_board yes)
-    (property "Reference" "#PWR0122" (id 0) (at 95.25 90.17 0)
+    (property "Reference" "#PWR0113" (id 0) (at 95.25 90.17 0)
       (effects (font (size 1.27 1.27)) hide)
     )
@@
   (symbol (lib_id "Connector_Generic:Conn_01x08") (at 109.22 41.91 90) (unit 1)
     (in_bom yes) (on_board yes) (fields_autoplaced)
-    (property "Reference" "J2" (id 0) (at 110.49 35.56 90))
+    (property "Reference" "J1" (id 0) (at 110.49 35.56 90))
     (property "Value" "Tester" (id 1) (at 110.49 38.1 90))
     (property "Footprint" "" (id 2) (at 109.22 41.91 0)
