File: hardware/tester.kicad_sch (KiCad schematic)
At the start: 5 parts, among them J1 Tester, SW6 SW_DIP_x08

Commit message: Rename
Parts:
- BAR8: symbol 65C816:LED-Array-8 -> BB816:LED-Array-8
Changed lines of the file:
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@@
   (title_block
     (title "Tester Module")
-    (date "2023-05-14")
+    (date "2023-05-23")
     (rev "A.32")
-    (comment 2 "https://github.com/adrienkohlbecker/65C816")
+    (comment 2 "https://github.com/adrienkohlbecker/BB816")
     (comment 3 "Licensed under CERN-OHL-W v2")
-    (comment 4 "Copyright © 2022 Adrien Kohlbecker")
+    (comment 4 "Copyright © 2022-2023 Adrien Kohlbecker")
   )
   (junction (at 82.55 63.5) (diameter 0) (color 0 0 0 0)
@@
     (stroke (width 0) (type default) (color 0 0 0 0))
   )
-  (symbol (lib_id "65C816:LED-Array-8") (at 130.81 59.69 0) (unit 1)
+  (symbol (lib_id "BB816:LED-Array-8") (at 130.81 59.69 0) (unit 1)
     (in_bom yes) (on_board yes)
     (property "Reference" "BAR8" (id 0) (at 130.81 44.831 0))
