File: hardware/glue_logic.kicad_sch (KiCad schematic)
At the start: 23 parts, among them U2 74AC11, U27 74HC10, U3 74AC74, U4 DS1035-10, U5 74HC00, U6 74AHC32, U7 74ACT245, U8 74AC573

Commit message: Fix gate
Parts:
- U5: value 74HC00 -> 74AHC00
Changed lines of the file:
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@@
     (in_bom yes) (on_board yes)
     (property "Reference" "U5" (id 0) (at 66.04 94.615 0))
-    (property "Value" "74HC00" (id 1) (at 66.04 96.9264 0))
+    (property "Value" "74AHC00" (id 1) (at 66.04 96.9264 0))
     (property "Footprint" "" (id 2) (at 66.04 102.87 0)
       (effects (font (size 1.27 1.27)) hide)
     )
-    (property "Datasheet" "https://www.ti.com/lit/ds/symlink/sn74ac00.pdf" (id 3) (at 66.04 102.87 0)
+    (property "Datasheet" "https://www.ti.com/lit/ds/symlink/sn74ahc00.pdf" (id 3) (at 66.04 102.87 0)
       (effects (font (size 1.27 1.27)) hide)
     )
@@
     (in_bom yes) (on_board yes)
     (property "Reference" "U5" (id 0) (at 49.53 132.715 0))
-    (property "Value" "74HC00" (id 1) (at 49.53 135.0264 0))
+    (property "Value" "74AHC00" (id 1) (at 49.53 135.0264 0))
     (property "Footprint" "" (id 2) (at 49.53 140.97 0)
       (effects (font (size 1.27 1.27)) hide)
     )
-    (property "Datasheet" "https://www.ti.com/lit/ds/symlink/sn74ac00.pdf" (id 3) (at 49.53 140.97 0)
+    (property "Datasheet" "https://www.ti.com/lit/ds/symlink/sn74ahc00.pdf" (id 3) (at 49.53 140.97 0)
       (effects (font (size 1.27 1.27)) hide)
     )
@@
       (effects (font (size 1.27 1.27)) (justify left))
     )
-    (property "Value" "74HC00" (id 1) (at 126.492 176.403 0)
+    (property "Value" "74AHC00" (id 1) (at 126.492 176.403 0)
       (effects (font (size 1.27 1.27)) (justify left))
     )
@@
       (effects (font (size 1.27 1.27)) hide)
     )
-    (property "Datasheet" "https://www.ti.com/lit/ds/symlink/sn74ac00.pdf" (id 3) (at 120.65 175.26 0)
+    (property "Datasheet" "https://www.ti.com/lit/ds/symlink/sn74ahc00.pdf" (id 3) (at 120.65 175.26 0)
       (effects (font (size 1.27 1.27)) hide)
     )
@@
     (in_bom yes) (on_board yes)
     (property "Reference" "U5" (id 0) (at 106.68 94.615 0))
-    (property "Value" "74HC00" (id 1) (at 106.68 96.9264 0))
+    (property "Value" "74AHC00" (id 1) (at 106.68 96.9264 0))
     (property "Footprint" "" (id 2) (at 106.68 102.87 0)
       (effects (font (size 1.27 1.27)) hide)
     )
-    (property "Datasheet" "https://www.ti.com/lit/ds/symlink/sn74ac00.pdf" (id 3) (at 106.68 102.87 0)
+    (property "Datasheet" "https://www.ti.com/lit/ds/symlink/sn74ahc00.pdf" (id 3) (at 106.68 102.87 0)
       (effects (font (size 1.27 1.27)) hide)
     )
@@
     (in_bom yes) (on_board yes)
     (property "Reference" "U5" (id 0) (at 50.8 92.075 0))
-    (property "Value" "74HC00" (id 1) (at 50.8 94.3864 0))
+    (property "Value" "74AHC00" (id 1) (at 50.8 94.3864 0))
     (property "Footprint" "" (id 2) (at 50.8 100.33 0)
       (effects (font (size 1.27 1.27)) hide)
     )
-    (property "Datasheet" "https://www.ti.com/lit/ds/symlink/sn74ac00.pdf" (id 3) (at 50.8 100.33 0)
-      (effects (font (size 1.27 1.27)) hide)
-    )
+    (property "Datasheet" "https://www.ti.com/lit/ds/symlink/sn74ahc00.pdf" (id 3) (at 50.8 100.33 0)
+      (effects (font (size 1.27 1.27)) hide)
+    )

Commit message: Start episode 15
Parts:
- removed U27: 74HC10, symbol 74xx:74LS10
Connections:
- net R~{W}: now also U5.2, U6.1
- net VCC: no longer U5.2, U6.1, U6.2
- net ~{CLK}: now also U6.2
- net ~{WR}: now reaches U6.3
- net ~{RD}: now reaches U5.3
- no-connect marks 10 -> 8
Other:
- note added: "pull-down on buffer is useful if the clock gets paused, since the data bus is only driven for half the cycle pull-up/down on address bus and cpu data bus is useful only if you plan to tie BE low with nothing else driving the bus"
- moved on the sheet: U5A, U6A, U6C

Commit message: Update for Episode 15
Other:
- note added: "pull-down on buffer data bus is useful if you stop the clock, since the data bus is only driven for half the cycle pull-up/down on address bus and cpu data bus is useful only if you plan to tie BE low with nothing else driving the bus"
- note removed: "pull-down on buffer is useful if the clock gets paused, since the data bus is only driven for half the cycle pull-up/down on address bus and cpu data bus is useful only if you plan to tie BE low with nothing else driving the bus"
Changed lines of the file:
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@@
     (stroke (width 0) (type default) (color 0 0 0 0))
   )
-  (text "pull-down on buffer is useful if the clock gets paused, since the data bus is only driven for half the cycle\npull-up/down on address bus and cpu data bus is useful only if you plan to tie BE low with nothing else driving the bus"
+  (text "pull-down on buffer data bus is useful if you stop the clock, since the data bus is only driven for half the cycle\npull-up/down on address bus and cpu data bus is useful only if you plan to tie BE low with nothing else driving the bus"
     (at 161.29 151.13 0)
     (effects (font (size 1.27 1.27)) (justify left bottom))

Commit message: Update for Episode 16
Parts:
- removed U8: 74AC573, symbol 74xx:74LS573
- added U8: 74AC563, symbol 65C816:74AC563
- U3: value 74AC74 -> 74AHC74
Connections:
- net DBA0: now also U8.2 (D0)
- net DBA1: now also U8.3 (D1)
- net DBA2: now also U8.4 (D2)
- net DBA3: now also U8.5 (D3)
- net DBA4: now also U8.6 (D4)
- net DBA5: now also U8.7 (D5)
- net DBA6: now also U8.8 (D6)
- net DBA7: now also U8.9 (D7)
- net GND: now also RN6.1 (common), U8.10 (GND)
- net L_~{LE}: now also U8.11 (LE)
- net L_~{OE}: now also U8.1 (OE)
- net VCC: now also U8.20 (VCC); no longer RN6.1 (common)
- net A16 renamed ~{A16}
- net ~{A16}: now also U8.19 (~{Q0})
- net A17 renamed ~{A17}
- net ~{A17}: now also U8.18 (~{Q1})
- net A18 renamed ~{A18}
- net ~{A18}: now also U8.17 (~{Q2})
- net A19 renamed ~{A19}
- net ~{A19}: now also U8.16 (~{Q3})
- net A20 renamed ~{A20}
- net ~{A20}: now also U8.15 (~{Q4})
- net A21 renamed ~{A21}
- net ~{A21}: now also U8.14 (~{Q5})
- net A22 renamed ~{A22}
- net ~{A22}: now also U8.13 (~{Q6})
- net A23 renamed ~{A23}
- net ~{A23}: now also U8.12 (~{Q7})

Commit message: Update for episode 18
Parts:
- added C49, C50: 100n, symbol Device:C_Small
- added U34: 74AC10, symbol 74xx:74LS10
- added U35: 74AHC367, symbol 74xx:74LS367
Connections:
- net GND: now also C49.2, C50.2, U34.7 (GND), U35.8 (GND)
- net L_~{OE}: now also U35.15 (OEb)
- net RDY_REG: now also U34.9
- net R~{W}: now also U5.1, U34.2; no longer U6.1
- net VCC: now also U6.1, U6.2, C49.1, C50.1, U34.14 (VCC), U35.1 (OEa), U35.10 (I4), U35.16 (VCC), U35.2 (I1), U35.4 (I2), U35.6 (I3); no longer U2.10, U2.11, U2.9, U5.1, U6.10, U6.9
- net ~{CLK}: now also U34.10; no longer U6.2
- net ~{RD}: now also U35.11 (O5b); no longer U5.3
- net ~{WR}: now also U35.13 (O6b); no longer U6.3
- net SYNC: now reaches U2.8
- net ~{CLK+}: now reaches U2.13, U2.5, U4.7
- net ~{CLK+}: now also U34.11
- net VA: now reaches U6.8
- net VA: now also U34.1, U34.3
- new net: U34.13, U34.5, U34.8
- new net: U34.4, U5.3
- new net: U34.12, U35.12 (I5)
- new net: U34.6, U35.14 (I6)
- new net VDA: U2.9, U6.9
- new net VPA: U2.10, U2.11, U6.10
- no-connect marks 8 -> 11
Other:
- note added: "pull-down on buffer data bus is useful if you stop the clock, since the data bus is only driven for half the cycle pull-up/down on address bus and cpu data bus are useful only if you plan to tie BE low with nothing else driving the bus"
- note removed: "pull-down on buffer data bus is useful if you stop the clock, since the data bus is only driven for half the cycle pull-up/down on address bus and cpu data bus is useful only if you plan to tie BE low with nothing else driving the bus"
- moved on the sheet: C10, C4, C42, C5, C6, C7, C8, C9, D1, R1, U2A, U2B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

Commit message: Update for episode 19
Parts:
- removed U2: 74AC11, symbol 74xx:74LS11
- removed U35: 74AHC367, symbol 74xx:74LS367
- added U2: 74AHC125, symbol 74xx:74LS125
- added U36: 74AHC02, symbol 74xx:74LS02
Connections:
- net BE: now also U5.10, U5.12, U5.13; no longer U5.4, U5.5
- net B_~{OE}: now also U5.8; no longer U6.11
- net CLK: now also U4.3, U4.6, U36.11, U36.12, U36.3
- net GND: now also U2.7 (GND), U36.7 (GND)
- net L_~{LE}: now also U36.1
- net L_~{OE}: now also U5.11, U2.1, U2.4; no longer U5.6, U6.13
- net RDY: now also U6.1; no longer U5.12, U5.13
- net RDY_REG: no longer U34.9, U5.10
- net R~{W}: now also U34.10, U34.11, U34.13, U34.9; no longer U34.2, U5.1, U5.2
- net SYNC: now also U5.6
- net VA: now also U34.2; no longer U34.1
- net VCC: now also U2.10, U2.12, U2.13, U2.14 (VCC), U2.9, U36.14 (VCC), U36.5, U36.6, U36.8, U36.9; no longer U4.2, U4.3, U6.1, U6.2, U6.4, U6.5
- net VDA: now also U5.1
- net VPA: now also U5.2
- net ~{CLK}: now also U36.13; no longer U34.10, U4.1
- net ~{RD}: now also U2.3
- net ~{WAI}: now also U6.3; no longer U5.8
- net ~{WR}: now also U2.6
- net at U34.4: now also U34.8; no longer U5.3
- net at U5.9: now also U34.1, U6.11, U36.2; no longer U5.11
- net ~{RDY_REG}: now reaches U6.12
- net ~{RDY_REG}: now also U3.8 (~{Q}), U6.2, U6.4
- net at U6.6: now also U34.5
- net at U34.12: now also U2.2
- net at U34.6: now also U2.5
- net CLK+: now reaches U4.5
- net CLK+: now also U6.13
- net ~{CLK+} renamed CLK-
- net CLK-: now also U4.2; no longer U34.11
- new net: U5.3, U5.4, U5.5
- new net CLK_IN: U4.1, U6.5
- no-connect marks 11 -> 6
Other:
- moved on the sheet: D1, R1, U34A, U34B, U34C, U34D, U3A, U3C, U5A, U5B, U5C, U5D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

Commit message: More episode 19 updates
Parts:
- added R38, R39, R40: 10k, symbol Device:R_Small
Connections:
- net BE: now also U34.10, U34.11; no longer U5.10
- net B_~{OE}: now also U34.8; no longer U5.8
- net RDY_IN: now also R38.2
- net R~{W}: now also U5.10, U5.9; no longer U34.10, U34.11, U34.9
- net VCC: now also R38.1, R39.1, R40.1
- net ~{RD}: now also R39.2
- net ~{WR}: now also R40.2
- net at U34.4: now also U5.8; no longer U34.8
- net at U34.1, U36.2, U6.11: now also U34.9; no longer U5.9
Other:
- moved on the sheet: U34C, U5C
