File: hardware/glue_logic.kicad_sch (KiCad schematic)
At the start: 29 parts, among them U2 74AHC125, U3 74AHC74, U34 74AC10, U36 74AHC02, U4 DS1035-10, U5 74AHC00, U6 74AHC32, U7 74ACT245, U8 74AC563

Commit message: More updates for Episode 19
Connections:
- net BE: now also U36.5, U36.6; no longer U5.12, U5.13
- net CLK: now also U36.2, U6.10; no longer U36.11
- net L_~{LE}: now also U36.13; no longer U36.1
- net L_~{OE}: now also U36.4; no longer U5.11
- net RDY: now also U5.12, U5.13; no longer U6.1
- net RDY_REG: now also U5.10
- net R~{W}: now also U36.8, U36.9; no longer U5.10, U5.9
- net VA: now also U6.3; no longer U6.8
- net VCC: no longer U36.5, U36.6, U36.8, U36.9
- net VDA: now also U6.1; no longer U6.9
- net VPA: now also U6.2; no longer U6.10
- net ~{CLK}: now also U36.1; no longer U36.13
- net ~{RDY_REG}: no longer U6.2
- net ~{WAI}: now also U5.8; no longer U6.3
- net at U34.9, U6.11: now also U36.11, U6.9; no longer U34.1, U36.2
- net at U34.4: now also U36.10; no longer U5.8
- new net: U5.11, U5.9
- new net: U34.1, U6.8
- no-connect marks 6 -> 4
Other:
- moved on the sheet: RN2, RN3, RN4, RN5, RN6, U2E, U36A, U36B, U36C, U36D, U3A, U5C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

Commit message: Update for episode 21
Parts:
- added R34: 10k, symbol Device:R_Small
Connections:
- net GND: now also R34.2
- net L_~{OE}: now also U2.13
- net VA: now also U2.11, R34.1; no longer U34.2, U34.3, U6.3
- net VCC: no longer U2.12, U2.13
- new net: U2.12, U34.2, U34.3, U6.3
- no-connect marks 4 -> 3
Other:
- moved on the sheet: U2C, U2D, U5A, U5B, U6A

Commit message: Renumber
Parts:
- renumbered C42 to C25, C4 to C26, C5 to C27, C6 to C28, C7 to C29, C8 to C30, C9 to C31, C10 to C32, C49 to C33, C50 to C34, D1 to D3, R38 to R26, R1 to R27, R39 to R28, R40 to R29, R34 to R30, RN2 to RN1, RN3 to RN2, RN4 to RN3, RN5 to RN4, RN6 to RN5, U3 to U13, U2 to U14, U4 to U15, U5 to U16, U36 to U17, U6 to U18, U34 to U19, U7 to U20, U8 to U21

Commit message: Update for episode 23
Connections:
- net BUFFER_CLK: now reaches U17.11, U18.11, U18.9, U19.9
- net at U17.10: now also U19.3; no longer U19.4
- net WRITE_CLK: now reaches U18.6, U19.5
- net READ_CLK: now reaches U18.8, U19.1
- net at U14.12, U18.3, U19.2: now also U19.4; no longer U19.3
- net L_~{LE} renamed ~{READ_CLK}
- net L_~{OE} renamed ~{BE}
Other:
- note added: "BUFFER_CLK +10ns"
- note added: "BUS MANAGEMENT"
- note added: "CLK"
- note added: "CLOCK PHASES"
- note added: "I/O CONTROL"
- note added: "MISC"
- note added: "READY PIN"
- note added: "READ_CLK +10ns (falling-edge only)"
- note added: "SHEET I/O"
- note added: "WRITE_CLK -20ns"
- moved on the sheet: C25, C26, C27, C28, C29, C30, C31, C32, C33, C34, D3, R26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

Commit message: Snapshot ep 24 work
Parts:
- removed C25: 10u, symbol Device:C_Polarized_Small
- removed unit 3 of U14
- removed U21: 74AC563, symbol 65C816:74AC563
- added C21, C25: 100n, symbol Device:C_Small
- added J4: Conn_01x10, symbol Connector_Generic:Conn_01x10
- added R24: 100k, symbol Device:R_Small
- added R43, R44, R45: 0R, symbol Device:R_Small
- added U12, U22: 74AHC32, symbol 74xx:74LS32
- added U21: 74AHC573, symbol 74xx:74LS573
- R26: value 10k -> 3.3k
- R28, R29, R30, RN1, RN2, RN3, RN4, RN5: value 10k -> 100k
- U20: value 74ACT245 -> 74AHCT245
Connections:
- net BUFFER_CLK: now also J4.3 (Pin_3)
- net B_~{OE}: now also J4.8 (Pin_8)
- net CLK: now also R44.2; no longer U15.3, U15.6
- net CLK+: now also J4.2 (Pin_2), R45.2; no longer U15.5
- net CLK-: now also J4.1 (Pin_1), R43.2; no longer U15.2, U15.7
- net CLK_IN: now also R24.1
- net DBA0: now also U21.2 (D0)
- net DBA1: now also U21.3 (D1)
- net DBA2: now also U21.4 (D2)
- net DBA3: now also U21.5 (D3)
- net DBA4: now also U21.6 (D4)
- net DBA5: now also U21.7 (D5)
- net DBA6: now also U21.8 (D6)
- net DBA7: now also U21.9 (D7)
- net GND: now also C21.2, C25.2, J4.10 (Pin_10), R24.2, U12.7 (GND), U21.10 (GND), U22.7 (GND)
- net RDY_REG: now also J4.7 (Pin_7)
- net READ_CLK: now also J4.5 (Pin_5)
- net VCC: now also C21.1, C25.1, U12.14 (VCC), U21.20 (VCC), U22.12, U22.13, U22.14 (VCC)
- net WRITE_CLK: now also J4.6 (Pin_6)
- net ~{BE}: now also J4.9 (Pin_9), U21.1 (OE)
- net ~{READ_CLK}: now also J4.4 (Pin_4), U21.11 (Load)
- net RDY renamed RDY⎒
- net ~{A16} renamed A16
- net A16: now also U12.1, U21.19 (Q0)
- net ~{A17} renamed A17
- net A17: now also U12.2, U21.18 (Q1)
- net ~{A18} renamed A18
- net A18: now also U12.4, U21.17 (Q2)
- net ~{A19} renamed A19
- net A19: now also U12.5, U21.16 (Q3)
- net ~{A20} renamed A20
- net A20: now also U12.9, U21.15 (Q4)
- net ~{A21} renamed A21
- net A21: now also U12.10, U21.14 (Q5)
- net ~{A22} renamed A22
- net A22: now also U12.12, U21.13 (Q6)
- net ~{A23} renamed A23
- net A23: now also U12.13, U21.12 (Q7)
- new net: R43.1, U15.2, U15.7
- new net: U12.3, U22.1
- new net: U12.6, U22.2
- new net: U22.3, U22.9
- new net: R44.1, U15.3, U15.6
- new net: R45.1, U15.5
- new net: U12.8, U22.4
- new net: U12.11, U22.5
- new net: U22.10, U22.6
- new net ~{BANK0}: U22.8
Other:
- note added: "BANK ZERO"
- note added: "DEBUG CONNECTOR"
- moved on the sheet: C26, C27, C28, C29, C30, C31, C32, C33, C34, U13A, U13C, U14E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

Commit message: More updates
Connections:
- net CLK_IN renamed CLK_SRC
Changed lines of the file:
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@@
     (stroke (width 0) (type default) (color 0 0 0 0))
   )
-  (wire (pts (xy 43.18 44.45) (xy 50.8 44.45))
+  (wire (pts (xy 43.18 44.45) (xy 53.34 44.45))
     (stroke (width 0) (type default) (color 0 0 0 0))
   )
@@
     (stroke (width 0) (type default) (color 0 0 0 0))
   )
-  (wire (pts (xy 31.75 29.21) (xy 40.64 29.21))
+  (wire (pts (xy 30.48 29.21) (xy 40.64 29.21))
     (stroke (width 0) (type default) (color 0 0 0 0))
   )
@@
     (stroke (width 0) (type default) (color 0 0 0 0))
   )
-  (wire (pts (xy 31.75 36.83) (xy 40.64 36.83))
+  (wire (pts (xy 30.48 36.83) (xy 40.64 36.83))
     (stroke (width 0) (type default) (color 0 0 0 0))
   )
@@
     (stroke (width 0) (type default) (color 0 0 0 0))
   )
-  (wire (pts (xy 43.18 40.64) (xy 50.8 40.64))
+  (wire (pts (xy 43.18 40.64) (xy 53.34 40.64))
     (stroke (width 0) (type default) (color 0 0 0 0))
   )
@@
     (stroke (width 0) (type default) (color 0 0 0 0))
   )
-  (wire (pts (xy 50.8 29.21) (xy 43.18 29.21))
+  (wire (pts (xy 53.34 29.21) (xy 43.18 29.21))
     (stroke (width 0) (type default) (color 0 0 0 0))
   )
@@
     (stroke (width 0) (type default) (color 0 0 0 0))
   )
-  (wire (pts (xy 31.75 44.45) (xy 40.64 44.45))
+  (wire (pts (xy 30.48 44.45) (xy 40.64 44.45))
     (stroke (width 0) (type default) (color 0 0 0 0))
   )
@@
     (stroke (width 0) (type default) (color 0 0 0 0))
   )
-  (wire (pts (xy 40.64 40.64) (xy 31.75 40.64))
+  (wire (pts (xy 40.64 40.64) (xy 30.48 40.64))
     (stroke (width 0) (type default) (color 0 0 0 0))
   )
@@
     (stroke (width 0) (type default) (color 0 0 0 0))
   )
-  (wire (pts (xy 43.18 52.07) (xy 50.8 52.07))
+  (wire (pts (xy 43.18 52.07) (xy 53.34 52.07))
     (stroke (width 0) (type default) (color 0 0 0 0))
   )
@@
     (stroke (width 0) (type default) (color 0 0 0 0))
   )
-  (wire (pts (xy 31.75 25.4) (xy 40.64 25.4))
+  (wire (pts (xy 30.48 25.4) (xy 40.64 25.4))
     (stroke (width 0) (type default) (color 0 0 0 0))
   )
@@
     (stroke (width 0) (type default) (color 0 0 0 0))
   )
-  (wire (pts (xy 96.52 220.98) (xy 105.41 220.98))
+  (wire (pts (xy 96.52 220.98) (xy 106.68 220.98))
     (stroke (width 0) (type default) (color 0 0 0 0))
   )
@@
     (stroke (width 0) (type default) (color 0 0 0 0))
   )
-  (wire (pts (xy 43.18 55.88) (xy 50.8 55.88))
+  (wire (pts (xy 43.18 55.88) (xy 53.34 55.88))
     (stroke (width 0) (type default) (color 0 0 0 0))
   )
@@
     (stroke (width 0) (type default) (color 0 0 0 0))
   )
-  (wire (pts (xy 40.64 33.02) (xy 31.75 33.02))
+  (wire (pts (xy 40.64 33.02) (xy 30.48 33.02))
     (stroke (width 0) (type default) (color 0 0 0 0))
   )
@@
     (stroke (width 0) (type default) (color 0 0 0 0))
   )
-  (wire (pts (xy 161.29 25.4) (xy 169.545 25.4))
+  (wire (pts (xy 160.02 25.4) (xy 169.545 25.4))
     (stroke (width 0) (type default) (color 0 0 0 0))
   )
@@
     (stroke (width 0) (type default) (color 0 0 0 0))
   )
-  (wire (pts (xy 50.8 25.4) (xy 43.18 25.4))
+  (wire (pts (xy 53.34 25.4) (xy 43.18 25.4))
     (stroke (width 0) (type default) (color 0 0 0 0))
   )
@@
     (stroke (width 0) (type solid) (color 0 0 0 0))
   )
-  (wire (pts (xy 43.18 36.83) (xy 50.8 36.83))
+  (wire (pts (xy 43.18 36.83) (xy 53.34 36.83))
     (stroke (width 0) (type default) (color 0 0 0 0))
   )
@@
     (stroke (width 0) (type default) (color 0 0 0 0))
   )
-  (wire (pts (xy 43.18 33.02) (xy 50.8 33.02))
+  (wire (pts (xy 43.18 33.02) (xy 53.34 33.02))
     (stroke (width 0) (type default) (color 0 0 0 0))
   )
@@
     (stroke (width 0) (type default) (color 0 0 0 0))
   )
-  (wire (pts (xy 43.18 48.26) (xy 50.8 48.26))
+  (wire (pts (xy 43.18 48.26) (xy 53.34 48.26))
     (stroke (width 0) (type default) (color 0 0 0 0))
   )
@@
     (effects (font (size 1.27 1.27)) (justify left bottom))
   )
-  (label "VA" (at 105.41 220.98 180)
+  (label "VA" (at 106.68 220.98 180)
     (effects (font (size 1.27 1.27)) (justify right bottom))
   )
@@
     (effects (font (size 1.27 1.27)) (justify left bottom))
   )
-  (label "CLK_IN" (at 162.56 101.6 0)
+  (label "CLK_SRC" (at 162.56 101.6 0)
     (effects (font (size 1.27 1.27)) (justify left bottom))
   )
@@
     (effects (font (size 1.27 1.27)) (justify left bottom))
   )
-  (label "CLK_IN" (at 40.64 25.4 180)
+  (label "CLK_SRC" (at 40.64 25.4 180)
     (effects (font (size 1.27 1.27)) (justify right bottom))
   )
@@
     (effects (font (size 1.27 1.27)) (justify left bottom))
   )
-  (label "CLK_IN" (at 161.29 25.4 0)
+  (label "CLK_SRC" (at 160.02 25.4 0)
     (effects (font (size 1.27 1.27)) (justify left bottom))
   )
@@
     (effects (font (size 1.27 1.27)) (justify left bottom))
   )
-  (hierarchical_label "~{WAI}" (shape output) (at 50.8 33.02 0)
+  (hierarchical_label "~{WAI}" (shape output) (at 53.34 33.02 0)
     (effects (font (size 1.27 1.27)) (justify left))
   )
-  (hierarchical_label "~{BANK0}" (shape output) (at 50.8 55.88 0)
+  (hierarchical_label "~{BANK0}" (shape output) (at 53.34 55.88 0)
     (effects (font (size 1.27 1.27)) (justify left))
   )
-  (hierarchical_label "R~{W}" (shape input) (at 31.75 36.83 180)
+  (hierarchical_label "R~{W}" (shape input) (at 30.48 36.83 180)
     (effects (font (size 1.27 1.27)) (justify right))
   )
-  (hierarchical_label "VPA" (shape input) (at 31.75 44.45 180)
+  (hierarchical_label "VPA" (shape input) (at 30.48 44.45 180)
     (effects (font (size 1.27 1.27)) (justify right))
   )
-  (hierarchical_label "~{RD}" (shape output) (at 50.8 40.64 0)
+  (hierarchical_label "~{RD}" (shape output) (at 53.34 40.64 0)
     (effects (font (size 1.27 1.27)) (justify left))
   )
-  (hierarchical_label "SYNC" (shape output) (at 50.8 52.07 0)
+  (hierarchical_label "SYNC" (shape output) (at 53.34 52.07 0)
     (effects (font (size 1.27 1.27)) (justify left))
   )
-  (hierarchical_label "~{CLK}" (shape output) (at 50.8 29.21 0)
+  (hierarchical_label "~{CLK}" (shape output) (at 53.34 29.21 0)
     (effects (font (size 1.27 1.27)) (justify left))
   )
-  (hierarchical_label "VA" (shape output) (at 50.8 48.26 0)
+  (hierarchical_label "VA" (shape output) (at 53.34 48.26 0)
     (effects (font (size 1.27 1.27)) (justify left))
   )
-  (hierarchical_label "VDA" (shape input) (at 31.75 40.64 180)
+  (hierarchical_label "VDA" (shape input) (at 30.48 40.64 180)
     (effects (font (size 1.27 1.27)) (justify right))
   )
-  (hierarchical_label "RDY_IN" (shape input) (at 31.75 29.21 180)
+  (hierarchical_label "RDY_IN" (shape input) (at 30.48 29.21 180)
     (effects (font (size 1.27 1.27)) (justify right))
   )
-  (hierarchical_label "~{WR}" (shape output) (at 50.8 44.45 0)
+  (hierarchical_label "~{WR}" (shape output) (at 53.34 44.45 0)
     (effects (font (size 1.27 1.27)) (justify left))
   )
@@
     (effects (font (size 1.27 1.27)) (justify left))
   )
-  (hierarchical_label "CLK" (shape output) (at 50.8 25.4 0)
+  (hierarchical_label "CLK" (shape output) (at 53.34 25.4 0)
     (effects (font (size 1.27 1.27)) (justify left))
   )
@@
     (effects (font (size 1.27 1.27)) (justify right))
   )
-  (hierarchical_label "CLK_IN" (shape input) (at 31.75 25.4 180)
+  (hierarchical_label "CLK_SRC" (shape input) (at 30.48 25.4 180)
     (effects (font (size 1.27 1.27)) (justify right))
   )
-  (hierarchical_label "RDY⎒" (shape bidirectional) (at 50.8 36.83 0)
+  (hierarchical_label "RDY⎒" (shape bidirectional) (at 53.34 36.83 0)
     (effects (font (size 1.27 1.27)) (justify left))
   )
-  (hierarchical_label "BE" (shape input) (at 31.75 33.02 180)
+  (hierarchical_label "BE" (shape input) (at 30.48 33.02 180)
     (effects (font (size 1.27 1.27)) (justify right))
   )
