File: hardware/glue_logic.kicad_sch (KiCad schematic)
At the start: 38 parts, among them J4 Conn_01x10, U12 74AHC32, U13 74AHC74, U14 74AHC125, U15 DS1035-10, U16 74AHC00, U17 74AHC02, U18 74AHC32, U19 74AC10, U20 74AHCT245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

Commit message: Updates for episode 25
Parts:
- added C40: 100n, symbol Device:C_Small
- added R46: 0R, symbol Device:R_Small
- added U43: 74AC112, symbol 74xx:74LS112
Connections:
- net CLK: now also U13.3 (C), U43.13 (C)
- net GND: now also C40.2, U43.8 (GND); no longer RN5.1 (common)
- net RDY_REG: no longer U16.10
- net RDY⎒: now also U22.12; no longer U16.12, U16.13
- net VCC: now also RN5.1 (common), U16.10, U16.9, C40.1, U43.1 (C), U43.10 (~{S}), U43.14 (~{R}), U43.15 (~{R}), U43.16 (VCC), U43.2 (K), U43.3 (J), U43.4 (~{S}); no longer U13.2 (D), U13.3 (C), U22.12, U22.13
- net ~{RDY_REG}: now also U22.13
- net ~{WAI}: now also U22.11; no longer U16.8
- net X: now reaches U13.5 (Q)
- net at U16.11: now also U43.12 (K); no longer U16.9
- new net: R46.1, U43.9 (Q)
- new net M: R46.2
- new net MX: U13.2 (D), U16.12, U16.13, U43.11 (J)
- no-connect marks 3 -> 5
Other:
- note added: "M/X demux"
- moved on the sheet: C21, C25, C26, C27, C28, C29, C30, C31, C32, C33, C34, U13A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
