File: hardware/debug.kicad_sch (KiCad schematic)
At the start: 23 parts, among them U20 74HC04, U21 74HC245, U22 74HC245, U23 74HC245, U24 74HC245, U25 74HC245

Commit message: Updates for Episode 13
Parts:
- added D6: EMU, symbol Device:LED_Small
- added R22: 1k, symbol Device:R_Small
Connections:
- net GND: now also D6.1 (K)
- new net: D6.2 (A), R22.2
- new net E: R22.1
Changed lines of the file:
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@@
   (title_block
     (title "Debug module")
-    (date "2021-12-10")
-    (rev "A.12")
+    (date "2022-01-09")
+    (rev "A.13")
     (comment 2 "https://github.com/adrienkohlbecker/65C816")
     (comment 3 "Licensed under CERN-OHL-W v2")
@@
     (stroke (width 0) (type default) (color 0 0 0 0))
   )
+  (wire (pts (xy 92.71 92.71) (xy 92.71 91.44))
+    (stroke (width 0) (type default) (color 0 0 0 0))
+  )
   (wire (pts (xy 36.83 46.99) (xy 48.26 46.99))
     (stroke (width 0) (type default) (color 0 0 0 0))
@@
     (stroke (width 0) (type default) (color 0 0 0 0))
   )
-  (bus (pts (xy 36.83 66.04) (xy 48.26 66.04))
+  (bus (pts (xy 36.83 69.85) (xy 48.26 69.85))
     (stroke (width 0) (type default) (color 0 0 0 0))
   )
@@
     (stroke (width 0) (type default) (color 0 0 0 0))
   )
+  (wire (pts (xy 36.83 62.23) (xy 48.26 62.23))
+    (stroke (width 0) (type default) (color 0 0 0 0))
+  )
   (bus (pts (xy 115.57 140.97) (xy 115.57 143.51))
     (stroke (width 0) (type default) (color 0 0 0 0))
@@
     (stroke (width 0) (type default) (color 0 0 0 0))
   )
+  (wire (pts (xy 82.55 91.44) (xy 85.09 91.44))
+    (stroke (width 0) (type default) (color 0 0 0 0))
+  )
   (wire (pts (xy 118.11 35.56) (xy 125.73 35.56))
     (stroke (width 0) (type default) (color 0 0 0 0))
@@
     (stroke (width 0) (type default) (color 0 0 0 0))
   )
+  (wire (pts (xy 92.71 91.44) (xy 90.17 91.44))
+    (stroke (width 0) (type default) (color 0 0 0 0))
+  )
   (bus (pts (xy 115.57 96.52) (xy 115.57 99.06))
     (stroke (width 0) (type default) (color 0 0 0 0))
@@
     (stroke (width 0) (type default) (color 0 0 0 0))
   )
-  (bus (pts (xy 48.26 62.23) (xy 36.83 62.23))
+  (bus (pts (xy 48.26 66.04) (xy 36.83 66.04))
     (stroke (width 0) (type default) (color 0 0 0 0))
   )
@@
     (stroke (width 0) (type default) (color 0 0 0 0))
   )
+  (wire (pts (xy 73.66 91.44) (xy 77.47 91.44))
+    (stroke (width 0) (type default) (color 0 0 0 0))
+  )
   (wire (pts (xy 153.67 99.06) (xy 151.13 99.06))
     (stroke (width 0) (type default) (color 0 0 0 0))
@@
     (effects (font (size 1.27 1.27)) (justify left bottom))
   )
-  (label "d[0..7]" (at 48.26 66.04 180)
+  (label "d[0..7]" (at 48.26 69.85 180)
     (effects (font (size 1.27 1.27)) (justify right bottom))
   )
@@
     (effects (font (size 1.27 1.27)) (justify left bottom))
   )
-  (label "a[0..23]" (at 48.26 62.23 180)
+  (label "a[0..23]" (at 48.26 66.04 180)
     (effects (font (size 1.27 1.27)) (justify right bottom))
   )
@@
     (effects (font (size 1.27 1.27)) (justify left bottom))
   )
+  (label "E" (at 48.26 62.23 180)
+    (effects (font (size 1.27 1.27)) (justify right bottom))
+  )
   (label "~{NMI}" (at 31.75 157.48 0)
     (effects (font (size 1.27 1.27)) (justify left bottom))
@@
     (effects (font (size 1.27 1.27)) (justify right bottom))
   )
+  (label "E" (at 73.66 91.44 0)
+    (effects (font (size 1.27 1.27)) (justify left bottom))
+  )
   (label "VPA" (at 48.26 39.37 180)
     (effects (font (size 1.27 1.27)) (justify right bottom))
@@
     (effects (font (size 1.27 1.27)) (justify right))
   )
-  (hierarchical_label "a[0..23]" (shape input) (at 36.83 62.23 180)
+  (hierarchical_label "a[0..23]" (shape input) (at 36.83 66.04 180)
     (effects (font (size 1.27 1.27)) (justify right))
   )
@@
     (effects (font (size 1.27 1.27)) (justify right))
   )
+  (hierarchical_label "E" (shape input) (at 36.83 62.23 180)
+    (effects (font (size 1.27 1.27)) (justify right))
+  )
   (hierarchical_label "R~{W}" (shape input) (at 36.83 31.75 180)
     (effects (font (size 1.27 1.27)) (justify right))
@@
     (effects (font (size 1.27 1.27)) (justify right))
   )
-  (hierarchical_label "d[0..7]" (shape input) (at 36.83 66.04 180)
+  (hierarchical_label "d[0..7]" (shape input) (at 36.83 69.85 180)
     (effects (font (size 1.27 1.27)) (justify right))
   )
@@
       (effects (font (size 1.27 1.27)) hide)
     )
+    (pin "1")
+  )
+  (symbol (lib_id "Device:LED_Small") (at 87.63 91.44 180) (unit 1)
+    (in_bom yes) (on_board yes)
+    (property "Reference" "D6" (id 0) (at 87.63 86.36 0))
+    (property "Value" "EMU" (id 1) (at 87.63 88.9 0))
+    (property "Footprint" "" (id 2) (at 87.63 91.44 90)
+      (effects (font (size 1.27 1.27)) hide)
+    )
+    (property "Datasheet" "~" (id 3) (at 87.63 91.44 90)
+      (effects (font (size 1.27 1.27)) hide)
+    )
+    (pin "1")
+    (pin "2")
+  )
+  (symbol (lib_id "Device:R_Small") (at 80.01 91.44 90) (unit 1)
+    (in_bom yes) (on_board yes)
+    (property "Reference" "R22" (id 0) (at 80.01 86.36 90))
+    (property "Value" "1k" (id 1) (at 80.01 88.9 90))
+    (property "Footprint" "" (id 2) (at 80.01 91.44 0)
+      (effects (font (size 1.27 1.27)) hide)
+    )
+    (property "Datasheet" "~" (id 3) (at 80.01 91.44 0)
+      (effects (font (size 1.27 1.27)) hide)
+    )
+    (pin "1")
+    (pin "2")
+  )
+  (symbol (lib_id "power:GND") (at 92.71 92.71 0) (unit 1)
+    (in_bom yes) (on_board yes)
+    (property "Reference" "#PWR0112" (id 0) (at 92.71 99.06 0)
+      (effects (font (size 1.27 1.27)) hide)
+    )
+    (property "Value" "GND" (id 1) (at 92.837 97.1042 0))
+    (property "Footprint" "" (id 2) (at 92.71 92.71 0)
+      (effects (font (size 1.27 1.27)) hide)
+    )
+    (property "Datasheet" "" (id 3) (at 92.71 92.71 0)
+      (effects (font (size 1.27 1.27)) hide)
+    )

Commit message: Updates for Episode 14
Parts:
- removed U21, U22, U23, U24, U25: 74HC245, symbol 74xx:74LS245
- added U21, U22, U23, U24, U25: 74HC541, symbol 74xx:74LS541
- C31: symbol Device:CP_Small -> Device:C_Polarized_Small
Connections:
- net BE: now also U21.7 (A5)
- net GND: now also U21.1 (G1), U21.10 (GND), U21.19 (G2), U22.1 (G1), U22.10 (GND), U22.19 (G2), U23.1 (G1), U23.10 (GND), U23.19 (G2), U24.1 (G1), U24.10 (GND), U24.19 (G2), U25.1 (G1), U25.10 (GND), U25.19 (G2)
- net RDY: now also U21.6 (A4)
- net R~{W}: now also U21.2 (A0)
- net VCC: now also U21.20 (VCC), U22.20 (VCC), U23.20 (VCC), U24.20 (VCC), U25.20 (VCC)
- net ~{IRQ}: now also U21.5 (A3)
- net ~{NMI}: now also U21.8 (A6)
- net ~{VDA}: now also U21.3 (A1)
- net ~{VPA}: now also U21.4 (A2)
- net ~{WAI}: now also U21.9 (A7)
- net at BAR2.1 (A): now also U22.18 (Y0)
- net at BAR2.2 (A): now also U22.17 (Y1)
- net at BAR2.3 (A): now also U22.16 (Y2)
- net at BAR2.4 (A): now also U22.15 (Y3)
- net at BAR2.5 (A): now also U22.14 (Y4)
- net at BAR2.6 (A): now also U22.13 (Y5)
- net at BAR2.7 (A): now also U22.12 (Y6)
- net at BAR2.8 (A): now also U22.11 (Y7)
- net at BAR3.1 (A): now also U23.18 (Y0)
- net at BAR3.2 (A): now also U23.17 (Y1)
- net at BAR3.3 (A): now also U23.16 (Y2)
- net at BAR3.4 (A): now also U23.15 (Y3)
- net at BAR3.5 (A): now also U23.14 (Y4)
- net at BAR3.6 (A): now also U23.13 (Y5)
- net at BAR3.7 (A): now also U23.12 (Y6)
- net at BAR3.8 (A): now also U23.11 (Y7)
- net at BAR4.1 (A): now also U24.18 (Y0)
- net at BAR4.2 (A): now also U24.17 (Y1)
- net at BAR4.3 (A): now also U24.16 (Y2)
- net at BAR4.4 (A): now also U24.15 (Y3)
- net at BAR4.5 (A): now also U24.14 (Y4)
- net at BAR4.6 (A): now also U24.13 (Y5)
- net at BAR4.7 (A): now also U24.12 (Y6)
- net at BAR4.8 (A): now also U24.11 (Y7)
- net at BAR5.8 (A): now also U25.11 (Y7)
- net at BAR5.7 (A): now also U25.12 (Y6)
- net at BAR5.6 (A): now also U25.13 (Y5)
- net at BAR5.5 (A): now also U25.14 (Y4)
- net at BAR5.4 (A): now also U25.15 (Y3)
- net at BAR5.3 (A): now also U25.16 (Y2)
- net at BAR5.2 (A): now also U25.17 (Y1)
- net at BAR5.1 (A): now also U25.18 (Y0)
- net at BAR1.10 (K): now also U21.12 (Y6)
- net at BAR1.11 (K): now also U21.13 (Y5)
- net at BAR1.12 (K): now also U21.14 (Y4)
- net at BAR1.13 (K): now also U21.15 (Y3)
- net at BAR1.14 (K): now also U21.16 (Y2)
- net at BAR1.15 (K): now also U21.17 (Y1)
- net at BAR1.16 (K): now also U21.18 (Y0)
- net at BAR1.9 (K): now also U21.11 (Y7)
- new net A0: U24.9 (A7)
- new net A1: U24.8 (A6)
- new net A10: U23.7 (A5)
- new net A11: U23.6 (A4)
- new net A12: U23.5 (A3)
- new net A13: U23.4 (A2)
- new net A14: U23.3 (A1)
- new net A15: U23.2 (A0)
- new net A16: U22.9 (A7)
- new net A17: U22.8 (A6)
- new net A18: U22.7 (A5)
- new net A19: U22.6 (A4)
- new net A2: U24.7 (A5)
- new net A20: U22.5 (A3)
- new net A21: U22.4 (A2)
- new net A22: U22.3 (A1)
- new net A23: U22.2 (A0)
- new net A3: U24.6 (A4)
- new net A4: U24.5 (A3)
- new net A5: U24.4 (A2)
- new net A6: U24.3 (A1)
- new net A7: U24.2 (A0)
- new net A8: U23.9 (A7)
- new net A9: U23.8 (A6)
- new net D0: U25.9 (A7)
- new net D1: U25.8 (A6)
- new net D2: U25.7 (A5)
- new net D3: U25.6 (A4)
- new net D4: U25.5 (A3)
- new net D5: U25.4 (A2)
- new net D6: U25.3 (A1)
- new net D7: U25.2 (A0)
Other:
- title: Debug module -> Debug Module

Commit message: Update for Episode 16
Parts:
- removed BAR1: Blue, symbol 65C816:LED-Array-8
- removed D6: EMU, symbol Device:LED_Small
- removed RN9: 1.5k, Resistor_THT:R_Array_SIP9, symbol Device:R_Network08
- removed U21, U22: 74HC541, symbol 74xx:74LS541
- added BAR1: LED-Array-10-BGYR, symbol 65C816:LED-Array-10-BGYR
- added R23, R24, R25, R26: 4.7k, symbol Device:R_Small
- added R27, R28, R29: 1k, symbol Device:R_Small
- added R30, R31: 2k, symbol Device:R_Small
- added U21, U22: 74HC540, symbol 74xx:74LS540
- R22: value 1k -> 1.5k
Connections:
- net BE: now also U21.7 (A5)
- net E: now also U20.5; no longer R22.1
- net GND: now also R22.2, R23.2, R24.2, R25.2, R26.2, R27.2, R28.2, R29.2, R30.2, R31.2, U21.1 (G1), U21.10 (GND), U21.19 (G2), U22.1 (G1), U22.10 (GND), U22.19 (G2)
- net R~{W}: now also U21.2 (A0)
- net VCC: now also U21.20 (VCC), U22.20 (VCC); no longer U20.11, U20.5, U20.9
- net ~{IRQ}: now also U21.5 (A3)
- net ~{NMI}: now also U21.8 (A6)
- net ~{VDA}: now also U21.3 (A1)
- net ~{VPA}: now also U21.4 (A2)
- net ~{WAI}: now also U21.9 (A7)
- net at BAR2.1 (A): now also U22.18 (Y0)
- net at BAR2.2 (A): now also U22.17 (Y1)
- net at BAR2.3 (A): now also U22.16 (Y2)
- net at BAR2.4 (A): now also U22.15 (Y3)
- net at BAR2.5 (A): now also U22.14 (Y4)
- net at BAR2.6 (A): now also U22.13 (Y5)
- net at BAR2.7 (A): now also U22.12 (Y6)
- net at BAR2.8 (A): now also U22.11 (Y7)
- net at U20.6: now also U20.9
- net RST: now reaches U20.10
- net RST: now also BAR1.10 (A)
- net E_BUF: now reaches U20.8
- net E_BUF: now also BAR1.2 (A)
- new net: BAR1.12 (K), R30.1
- new net: BAR1.13 (K), R29.1
- new net: BAR1.11 (K), R31.1
- new net: BAR1.9 (A), U21.11 (Y7)
- new net: BAR1.8 (A), U21.12 (Y6)
- new net: BAR1.7 (A), U21.13 (Y5)
- new net: BAR1.6 (A), U21.14 (Y4)
- new net: BAR1.5 (A), U21.15 (Y3)
- new net: BAR1.4 (A), U21.16 (Y2)
- new net: BAR1.3 (A), U21.17 (Y1)
- new net: BAR1.1 (A), U21.18 (Y0)
- new net: BAR1.20 (K), R22.1
- new net: BAR1.18 (K), R24.1
- new net: BAR1.15 (K), R27.1
- new net: BAR1.19 (K), R23.1
- new net: BAR1.14 (K), R28.1
- new net: BAR1.16 (K), R26.1
- new net: BAR1.17 (K), R25.1
- new net RDY_IN: U21.6 (A4)
- new net ~{A16}: U22.9 (A7)
- new net ~{A17}: U22.8 (A6)
- new net ~{A18}: U22.7 (A5)
- new net ~{A19}: U22.6 (A4)
- new net ~{A20}: U22.5 (A3)
- new net ~{A21}: U22.4 (A2)
- new net ~{A22}: U22.3 (A1)
- new net ~{A23}: U22.2 (A0)
- new net ~{RST}: U20.11
- no-connect marks 4 -> 1
Other:
- moved on the sheet: U20F

Commit message: Update for episode 18
Connections:
- net RST renamed RST_BUF
- net VDA renamed SYNC
- net VPA renamed VA
- net ~{VDA} renamed ~{SYNC}
- net ~{VPA} renamed ~{VA}
Changed lines of the file:
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@@
   (title_block
     (title "Debug Module")
-    (date "2022-02-09")
-    (rev "A.17")
+    (date "2022-02-21")
+    (rev "A.18")
     (comment 2 "https://github.com/adrienkohlbecker/65C816")
     (comment 3 "Licensed under CERN-OHL-W v2")
@@
     (stroke (width 0) (type default) (color 0 0 0 0))
   )
-  (wire (pts (xy 83.82 115.57) (xy 88.9 115.57))
+  (wire (pts (xy 83.82 115.57) (xy 92.71 115.57))
     (stroke (width 0) (type default) (color 0 0 0 0))
   )
@@
     (effects (font (size 1.27 1.27)) (justify right bottom))
   )
-  (label "RST" (at 67.31 162.56 0)
+  (label "RST_BUF" (at 67.31 162.56 0)
     (effects (font (size 1.27 1.27)) (justify left bottom))
   )
@@
     (effects (font (size 1.27 1.27)) (justify right bottom))
   )
-  (label "VDA" (at 26.67 102.87 0)
+  (label "SYNC" (at 26.67 102.87 0)
     (effects (font (size 1.27 1.27)) (justify left bottom))
   )
@@
     (effects (font (size 1.27 1.27)) (justify right bottom))
   )
-  (label "~{VPA}" (at 29.21 147.32 0)
+  (label "~{VA}" (at 29.21 147.32 0)
     (effects (font (size 1.27 1.27)) (justify left bottom))
   )
@@
     (effects (font (size 1.27 1.27)) (justify left bottom))
   )
-  (label "~{VPA}" (at 52.07 115.57 180)
+  (label "~{VA}" (at 52.07 115.57 180)
     (effects (font (size 1.27 1.27)) (justify right bottom))
   )
@@
     (effects (font (size 1.27 1.27)) (justify right bottom))
   )
-  (label "VPA" (at 48.26 39.37 180)
-    (effects (font (size 1.27 1.27)) (justify right bottom))
-  )
-  (label "~{VDA}" (at 29.21 144.78 0)
+  (label "VA" (at 48.26 39.37 180)
+    (effects (font (size 1.27 1.27)) (justify right bottom))
+  )
+  (label "~{SYNC}" (at 29.21 144.78 0)
     (effects (font (size 1.27 1.27)) (justify left bottom))
   )
@@
     (effects (font (size 1.27 1.27)) (justify left bottom))
   )
-  (label "~{VDA}" (at 52.07 102.87 180)
+  (label "~{SYNC}" (at 52.07 102.87 180)
     (effects (font (size 1.27 1.27)) (justify right bottom))
   )
@@
     (effects (font (size 1.27 1.27)) (justify right bottom))
   )
-  (label "VPA" (at 26.67 115.57 0)
+  (label "VA" (at 26.67 115.57 0)
     (effects (font (size 1.27 1.27)) (justify left bottom))
   )
@@
     (effects (font (size 1.27 1.27)) (justify right bottom))
   )
-  (label "VDA" (at 48.26 35.56 180)
+  (label "SYNC" (at 48.26 35.56 180)
     (effects (font (size 1.27 1.27)) (justify right bottom))
   )
@@
     (effects (font (size 1.27 1.27)) (justify right bottom))
   )
-  (label "RST" (at 88.9 115.57 180)
+  (label "RST_BUF" (at 92.71 115.57 180)
     (effects (font (size 1.27 1.27)) (justify right bottom))
   )
@@
     (effects (font (size 1.27 1.27)) (justify right))
   )
-  (hierarchical_label "VDA" (shape input) (at 36.83 35.56 180)
+  (hierarchical_label "SYNC" (shape input) (at 36.83 35.56 180)
     (effects (font (size 1.27 1.27)) (justify right))
   )
@@
     (effects (font (size 1.27 1.27)) (justify right))
   )
-  (hierarchical_label "VPA" (shape input) (at 36.83 39.37 180)
+  (hierarchical_label "VA" (shape input) (at 36.83 39.37 180)
     (effects (font (size 1.27 1.27)) (justify right))
   )
