File: hardware/debug.kicad_sch (KiCad schematic)
At the start: 32 parts, among them U20 74HC04, U21 74HC540, U22 74HC540, U23 74HC541, U24 74HC541, U25 74HC541

Commit message: Renumber
Parts:
- renumbered C31 to C45, C32 to C46, C33 to C47, C34 to C48, C35 to C49, C36 to C50, C37 to C51, R22 to R32, R23 to R33, R24 to R34, R25 to R35, R26 to R36, R27 to R37, R28 to R38, R29 to R39, R30 to R40, R31 to R41, RN10 to RN6, RN11 to RN7, RN12 to RN8, RN13 to RN9, U20 to U30, U21 to U31, U22 to U32, U23 to U33, U24 to U34, U25 to U35

Commit message: More episode 21 update
Parts:
- R32: value 1.5k -> 3.3k
- R33, R34, R35, R36: value 4.7k -> 6.8k
- R40, R41: value 2k -> 1.5k
Changed lines of the file:
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@@
     (in_bom yes) (on_board yes)
     (property "Reference" "R40" (id 0) (at 102.87 160.02 90))
-    (property "Value" "2k" (id 1) (at 99.06 160.02 90))
+    (property "Value" "1.5k" (id 1) (at 99.06 160.02 90))
     (property "Footprint" "" (id 2) (at 92.71 160.02 0)
       (effects (font (size 1.27 1.27)) hide)
@@
     (in_bom yes) (on_board yes)
     (property "Reference" "R41" (id 0) (at 102.87 162.56 90))
-    (property "Value" "2k" (id 1) (at 99.06 162.56 90))
+    (property "Value" "1.5k" (id 1) (at 99.06 162.56 90))
     (property "Footprint" "" (id 2) (at 92.71 162.56 0)
       (effects (font (size 1.27 1.27)) hide)
@@
     (in_bom yes) (on_board yes)
     (property "Reference" "R32" (id 0) (at 102.87 139.7 90))
-    (property "Value" "1.5k" (id 1) (at 99.06 139.7 90))
+    (property "Value" "3.3k" (id 1) (at 99.06 139.7 90))
     (property "Footprint" "" (id 2) (at 92.71 139.7 0)
       (effects (font (size 1.27 1.27)) hide)
@@
     (in_bom yes) (on_board yes)
     (property "Reference" "R34" (id 0) (at 102.87 144.78 90))
-    (property "Value" "4.7k" (id 1) (at 99.06 144.78 90))
+    (property "Value" "6.8k" (id 1) (at 99.06 144.78 90))
     (property "Footprint" "" (id 2) (at 92.71 144.78 0)
       (effects (font (size 1.27 1.27)) hide)
@@
     (in_bom yes) (on_board yes)
     (property "Reference" "R33" (id 0) (at 102.87 142.24 90))
-    (property "Value" "4.7k" (id 1) (at 99.06 142.24 90))
+    (property "Value" "6.8k" (id 1) (at 99.06 142.24 90))
     (property "Footprint" "" (id 2) (at 92.71 142.24 0)
       (effects (font (size 1.27 1.27)) hide)
@@
     (in_bom yes) (on_board yes)
     (property "Reference" "R36" (id 0) (at 102.87 149.86 90))
-    (property "Value" "4.7k" (id 1) (at 99.06 149.86 90))
+    (property "Value" "6.8k" (id 1) (at 99.06 149.86 90))
     (property "Footprint" "" (id 2) (at 92.71 149.86 0)
       (effects (font (size 1.27 1.27)) hide)
@@
     (in_bom yes) (on_board yes)
     (property "Reference" "R35" (id 0) (at 102.87 147.32 90))
-    (property "Value" "4.7k" (id 1) (at 99.06 147.32 90))
+    (property "Value" "6.8k" (id 1) (at 99.06 147.32 90))
     (property "Footprint" "" (id 2) (at 92.71 147.32 0)
       (effects (font (size 1.27 1.27)) hide)

Commit message: Snapshot ep 24 work
Parts:
- removed U32: 74HC540, symbol 74xx:74LS540
- added U32: 74HC541, symbol 74xx:74LS541
Connections:
- net GND: now also U32.1 (G1), U32.10 (GND), U32.19 (G2)
- net VCC: now also U32.20 (VCC)
- net at BAR2.1 (A): now also U32.18 (Y0)
- net at BAR2.2 (A): now also U32.17 (Y1)
- net at BAR2.3 (A): now also U32.16 (Y2)
- net at BAR2.4 (A): now also U32.15 (Y3)
- net at BAR2.5 (A): now also U32.14 (Y4)
- net at BAR2.6 (A): now also U32.13 (Y5)
- net at BAR2.7 (A): now also U32.12 (Y6)
- net at BAR2.8 (A): now also U32.11 (Y7)
- new net A16: U32.9 (A7)
- new net A17: U32.8 (A6)
- new net A18: U32.7 (A5)
- new net A19: U32.6 (A4)
- new net A20: U32.5 (A3)
- new net A21: U32.4 (A2)
- new net A22: U32.3 (A1)
- new net A23: U32.2 (A0)
