File: hardware/debug.kicad_sch (KiCad schematic)
At the start: 32 parts, among them U30 74HC04, U31 74HC540, U32 74HC541, U33 74HC541, U34 74HC541, U35 74HC541

Commit message: Update main project
Parts:
- renumbered C45 to C27, C46 to C28, C47 to C29, C48 to C30, C49 to C31, C50 to C32, C51 to C33, R32 to R20, R33 to R21, R34 to R22, R35 to R23, R36 to R24, R37 to R25, R38 to R26, R39 to R27, R40 to R28, R41 to R29, RN6 to RN1, RN7 to RN2, RN8 to RN3, RN9 to RN4, U30 to U19, U31 to U20, U32 to U21, U33 to U22, U34 to U23, U35 to U24

Commit message: Update schematic
Parts:
- added BAR9: LED-Array-8-GYR, symbol 65C816:LED-Array-8-GYR
- added C43: 100n, symbol Device:C_Small
- added R40: 1.5k, symbol Device:R_Small
- added R41, R42: 1k, symbol Device:R_Small
- added R43, R44, R45, R46, R47: 6.8k, symbol Device:R_Small
- added U32: 74HC541, symbol 74xx:74LS541
Connections:
- net BE: now also U20.8 (A6); no longer U20.7 (A5)
- net E: now also U19.9; no longer U19.5
- net GND: now also C43.2, U32.1 (G1), U32.10 (GND), U32.19 (G2)
- net RDY_IN: now also U20.7 (A5); no longer U20.6 (A4)
- net SYNC: now also U32.6 (A4); no longer U19.1
- net VA: now also U32.7 (A5); no longer U19.3
- net VCC: now also U19.1, U19.3, U19.5, C43.1, R40.2, R41.2, R42.2, R43.2, R44.2, R45.2, R46.2, R47.2, U32.20 (VCC); no longer U19.13
- net ~{NMI}: now also U20.6 (A4); no longer U20.8 (A6)
- net CLK_EN_BUF: now reaches U19.12
- net CLK_EN_BUF: now also U32.3 (A1)
- net at U19.6: no longer U19.9
- net at U20.16 (Y2): now also BAR9.14 (K); no longer BAR1.4 (A)
- net at U20.17 (Y1): now also BAR9.13 (K); no longer BAR1.3 (A)
- net at U20.18 (Y0): now also BAR1.2 (A); no longer BAR1.1 (A)
- net E_BUF renamed ~{E_BUF}
- net ~{E_BUF}: now also BAR9.12 (K); no longer BAR1.2 (A)
- net ~{SYNC}: no longer names the net of U19.2
- net ~{SYNC}: no longer U20.3 (A1)
- net ~{VA}: no longer names the net of U19.4
- net ~{VA}: no longer U20.4 (A2)
- new net: BAR9.1 (A), R47.1
- new net: BAR9.10 (K), U32.17 (Y1)
- new net: BAR9.11 (K), U32.16 (Y2)
- new net: BAR9.15 (K), U32.12 (Y6)
- new net: BAR9.16 (K), U32.11 (Y7)
- new net: BAR9.2 (A), R46.1
- new net: BAR9.3 (A), R45.1
- new net: BAR9.4 (A), R44.1
- new net: BAR9.5 (A), R43.1
- new net: BAR9.6 (A), R42.1
- new net: BAR9.7 (A), R41.1
- new net: BAR9.8 (A), R40.1
- new net: BAR9.9 (K), U32.18 (Y0)
- new net: BAR1.1 (A), U32.15 (Y3)
- new net: BAR1.3 (A), U32.14 (Y4)
- new net: BAR1.4 (A), U32.13 (Y5)
- new net CLK: U32.5 (A3)
- new net M: U20.3 (A1)
- new net X: U20.4 (A2)
- new net ~{ABORT}: U32.2 (A0)
- new net ~{CLK_EN}: U19.13
- new net ~{ML}: U32.9 (A7)
- new net ~{ROM_WE}: U32.4 (A2)
- new net ~{VP}: U32.8 (A6)
- no-connect marks 1 -> 3
Other:
- moved on the sheet: BAR1, BAR2, BAR3, BAR4, C27, C28, C29, C30, C31, C32, C33, R20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

Commit message: Update for Episode 32
Parts:
- removed unit 1 of U19
- removed unit 2 of U19
- removed unit 3 of U19
Connections:
- net M: now also U32.6 (A4); no longer U20.3 (A1)
- net SYNC: now also U32.3 (A1); no longer U32.6 (A4)
- net VA: now also U19.13; no longer U32.7 (A5)
- net X: now also U32.7 (A5); no longer U20.4 (A2)
- net ~{CLK_EN}: now also U20.3 (A1); no longer U19.13
- net at U20.16 (Y2): now also BAR1.4 (A); no longer BAR9.14 (K)
- net at U20.17 (Y1): now also BAR9.10 (K); no longer BAR9.13 (K)
- net at U32.17 (Y1): now also BAR1.3 (A); no longer BAR9.10 (K)
- net at U32.14 (Y4): now also BAR9.13 (K); no longer BAR1.3 (A)
- net at U32.13 (Y5): now also BAR9.14 (K); no longer BAR1.4 (A)
- net CLK_EN_BUF renamed ~{VA_BUF}
- net ~{VA_BUF}: now also U20.4 (A2); no longer U32.3 (A1)
- no-connect marks 3 -> 0

Commit message: Rename
Parts:
- BAR1: symbol 65C816:LED-Array-10-BGYR -> BB816:LED-Array-10-BGYR
- BAR2, BAR3, BAR4, BAR5: symbol 65C816:LED-Array-8 -> BB816:LED-Array-8
- BAR9: symbol 65C816:LED-Array-8-GYR -> BB816:LED-Array-8-GYR
Changed lines of the file:
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@@
   (title_block
     (title "Debug Module")
-    (date "2023-05-14")
+    (date "2023-05-23")
     (rev "A.32")
-    (comment 2 "https://github.com/adrienkohlbecker/65C816")
+    (comment 2 "https://github.com/adrienkohlbecker/BB816")
     (comment 3 "Licensed under CERN-OHL-W v2")
-    (comment 4 "Copyright © 2022 Adrien Kohlbecker")
+    (comment 4 "Copyright © 2022-2023 Adrien Kohlbecker")
   )
   (junction (at 255.27 96.52) (diameter 0) (color 0 0 0 0)
@@
     (pin "2")
   )
-  (symbol (lib_id "65C816:LED-Array-8") (at 165.1 39.37 0) (unit 1)
+  (symbol (lib_id "BB816:LED-Array-8") (at 165.1 39.37 0) (unit 1)
     (in_bom yes) (on_board yes)
     (property "Reference" "BAR2" (id 0) (at 165.1 24.511 0))
@@
     (pin "1")
   )
-  (symbol (lib_id "65C816:LED-Array-8") (at 165.1 92.71 0) (unit 1)
+  (symbol (lib_id "BB816:LED-Array-8") (at 165.1 92.71 0) (unit 1)
     (in_bom yes) (on_board yes)
     (property "Reference" "BAR3" (id 0) (at 165.1 77.851 0))
@@
     (pin "1")
   )
-  (symbol (lib_id "65C816:LED-Array-8") (at 165.1 144.78 0) (unit 1)
+  (symbol (lib_id "BB816:LED-Array-8") (at 165.1 144.78 0) (unit 1)
     (in_bom yes) (on_board yes)
     (property "Reference" "BAR4" (id 0) (at 165.1 129.921 0))
@@
     (pin "9")
   )
-  (symbol (lib_id "65C816:LED-Array-8") (at 250.19 40.64 0) (unit 1)
+  (symbol (lib_id "BB816:LED-Array-8") (at 250.19 40.64 0) (unit 1)
     (in_bom yes) (on_board yes)
     (property "Reference" "BAR5" (id 0) (at 250.19 25.781 0))
@@
     (pin "9")
   )
-  (symbol (lib_id "65C816:LED-Array-8-GYR") (at 85.09 170.18 180) (unit 1)
+  (symbol (lib_id "BB816:LED-Array-8-GYR") (at 85.09 170.18 180) (unit 1)
     (in_bom yes) (on_board yes) (fields_autoplaced)
     (property "Reference" "BAR9" (id 0) (at 84.455 151.13 0))
@@
     (pin "2")
   )
-  (symbol (lib_id "65C816:LED-Array-10-BGYR") (at 85.09 113.03 0) (unit 1)
+  (symbol (lib_id "BB816:LED-Array-10-BGYR") (at 85.09 113.03 0) (unit 1)
     (in_bom yes) (on_board yes) (fields_autoplaced)
     (property "Reference" "BAR1" (id 0) (at 85.725 96.52 0))
