File: hardware/memory.kicad_sch (KiCad schematic)
At the start: 4 parts, among them U26 28C256

Commit message: Start episode 15
Parts:
- added C43: 100n, symbol Device:C_Small
- added U28: KM62256CLP, Package_DIP:DIP-28_W15.24mm, symbol Memory_RAM:KM62256CLP
Connections:
- net A0: now also U28.10 (A0)
- net A1: now also U28.9 (A1)
- net A10: now also U28.21 (A10)
- net A11: now also U28.23 (A11)
- net A12: now also U28.2 (A12)
- net A13: now also U28.26 (A13)
- net A14: now also U28.1 (A14)
- net A2: now also U28.8 (A2)
- net A3: now also U28.7 (A3)
- net A4: now also U28.6 (A4)
- net A5: now also U28.5 (A5)
- net A6: now also U28.4 (A6)
- net A7: now also U28.3 (A7)
- net A8: now also U28.25 (A8)
- net A9: now also U28.24 (A9)
- net D0: now also U28.11 (Q0)
- net D1: now also U28.12 (Q1)
- net D2: now also U28.13 (Q2)
- net D3: now also U28.15 (Q3)
- net D4: now also U28.16 (Q4)
- net D5: now also U28.17 (Q5)
- net D6: now also U28.18 (Q6)
- net D7: now also U28.19 (Q7)
- net GND: now also C43.2, U28.14 (GND)
- net VCC: now also C43.1, U28.28 (VCC)
- net W~{R} renamed ~{RD}
- net ~{RD}: now also U28.22 (~{OE})
- new net ~{RAM_CS}: U28.20 (~{CS})
- new net ~{WR}: U28.27 (~{WE})
Other:
- moved on the sheet: C38, C39, R23, U26

Commit message: Update for Episode 15
Parts:
- removed R23: 10k, symbol Device:R_Small
- U26: value 28C256 -> AT28C256-15PC
- U28: value KM62256CLP -> LY62256PL-55LL
Connections:
- net ~{ROM_WE}: now reaches U26.27 (~{WE})
Changed lines of the file:
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@@
-    (stroke (width 0) (type default) (color 0 0 0 0))
-  )
-  (wire (pts (xy 88.9 102.87) (xy 88.9 101.6))
     (stroke (width 0) (type default) (color 0 0 0 0))
   )
@@
     (stroke (width 0) (type default) (color 0 0 0 0))
   )
-  (wire (pts (xy 88.9 95.25) (xy 88.9 96.52))
-    (stroke (width 0) (type default) (color 0 0 0 0))
-  )
   (bus (pts (xy 175.26 87.63) (xy 175.26 90.17))
     (stroke (width 0) (type default) (color 0 0 0 0))
@@
     (stroke (width 0) (type default) (color 0 0 0 0))
   )
+  (wire (pts (xy 96.52 102.87) (xy 105.41 102.87))
+    (stroke (width 0) (type default) (color 0 0 0 0))
+  )
   (wire (pts (xy 100.33 95.25) (xy 105.41 95.25))
     (stroke (width 0) (type default) (color 0 0 0 0))
@@
     (stroke (width 0) (type default) (color 0 0 0 0))
   )
-  (bus (pts (xy 30.48 39.37) (xy 44.45 39.37))
+  (wire (pts (xy 30.48 35.56) (xy 44.45 35.56))
+    (stroke (width 0) (type default) (color 0 0 0 0))
+  )
+  (bus (pts (xy 30.48 44.45) (xy 44.45 44.45))
     (stroke (width 0) (type default) (color 0 0 0 0))
   )
@@
     (stroke (width 0) (type default) (color 0 0 0 0))
   )
-  (bus (pts (xy 30.48 35.56) (xy 44.45 35.56))
+  (bus (pts (xy 30.48 40.64) (xy 44.45 40.64))
     (stroke (width 0) (type default) (color 0 0 0 0))
   )
@@
     (stroke (width 0) (type default) (color 0 0 0 0))
   )
-  (wire (pts (xy 105.41 102.87) (xy 88.9 102.87))
-    (stroke (width 0) (type default) (color 0 0 0 0))
-  )
   (wire (pts (xy 125.73 74.93) (xy 130.81 74.93))
     (stroke (width 0) (type default) (color 0 0 0 0))
@@
     (effects (font (size 1.27 1.27)) (justify left bottom))
   )
-  (label "D[0..7]" (at 44.45 39.37 180)
+  (label "D[0..7]" (at 44.45 44.45 180)
     (effects (font (size 1.27 1.27)) (justify right bottom))
   )
@@
     (effects (font (size 1.27 1.27)) (justify left bottom))
   )
-  (label "A[0..23]" (at 44.45 35.56 180)
+  (label "A[0..23]" (at 44.45 40.64 180)
     (effects (font (size 1.27 1.27)) (justify right bottom))
   )
@@
     (effects (font (size 1.27 1.27)) (justify left bottom))
   )
+  (label "~{ROM_WE}" (at 44.45 35.56 180)
+    (effects (font (size 1.27 1.27)) (justify right bottom))
+  )
   (label "~{RD}" (at 96.52 105.41 0)
     (effects (font (size 1.27 1.27)) (justify left bottom))
@@
   )
   (label "A2" (at 177.8 67.31 0)
+    (effects (font (size 1.27 1.27)) (justify left bottom))
+  )
+  (label "~{ROM_WE}" (at 96.52 102.87 0)
     (effects (font (size 1.27 1.27)) (justify left bottom))
   )
@@
     (effects (font (size 1.27 1.27)) (justify right))
   )
+  (hierarchical_label "~{ROM_WE}" (shape input) (at 30.48 35.56 180)
+    (effects (font (size 1.27 1.27)) (justify right))
+  )
   (hierarchical_label "~{ROM_CS}" (shape input) (at 30.48 27.94 180)
     (effects (font (size 1.27 1.27)) (justify right))
   )
-  (hierarchical_label "A[0..23]" (shape input) (at 30.48 35.56 180)
+  (hierarchical_label "A[0..23]" (shape input) (at 30.48 40.64 180)
     (effects (font (size 1.27 1.27)) (justify right))
   )
@@
     (effects (font (size 1.27 1.27)) (justify right))
   )
-  (hierarchical_label "D[0..7]" (shape bidirectional) (at 30.48 39.37 180)
+  (hierarchical_label "D[0..7]" (shape bidirectional) (at 30.48 44.45 180)
     (effects (font (size 1.27 1.27)) (justify right))
   )
@@
     (pin "1")
   )
-  (symbol (lib_id "Device:R_Small") (at 88.9 99.06 0) (unit 1)
-    (in_bom yes) (on_board yes) (fields_autoplaced)
-    (property "Reference" "R23" (id 0) (at 91.44 97.7899 0)
-      (effects (font (size 1.27 1.27)) (justify left))
-    )
-    (property "Value" "10k" (id 1) (at 91.44 100.3299 0)
-      (effects (font (size 1.27 1.27)) (justify left))
-    )
-    (property "Footprint" "" (id 2) (at 88.9 99.06 0)
-      (effects (font (size 1.27 1.27)) hide)
-    )
-    (property "Datasheet" "~" (id 3) (at 88.9 99.06 0)
-      (effects (font (size 1.27 1.27)) hide)
-    )
-    (pin "1")
-    (pin "2")
-  )
   (symbol (lib_id "power:VCC") (at 115.57 57.15 0) (unit 1)
     (in_bom yes) (on_board yes) (fields_autoplaced)
@@
   )
   (symbol (lib_id "Memory_RAM:KM62256CLP") (at 195.58 80.01 0) (unit 1)
-    (in_bom yes) (on_board yes) (fields_autoplaced)
-    (property "Reference" "U28" (id 0) (at 197.5994 54.61 0)
+    (in_bom yes) (on_board yes)
+    (property "Reference" "U28" (id 0) (at 185.42 58.42 0)
       (effects (font (size 1.27 1.27)) (justify left))
     )
-    (property "Value" "KM62256CLP" (id 1) (at 197.5994 57.15 0)
+    (property "Value" "LY62256PL-55LL" (id 1) (at 196.85 58.42 0)
       (effects (font (size 1.27 1.27)) (justify left))
     )
@@
       (effects (font (size 1.27 1.27)) hide)
     )
-    (property "Datasheet" "https://www.futurlec.com/Datasheet/Memory/62256.pdf" (id 3) (at 195.58 82.55 0)
+    (property "Datasheet" "http://www.farnell.com/datasheets/1674430.pdf" (id 3) (at 195.58 82.55 0)
       (effects (font (size 1.27 1.27)) hide)
     )
@@
     (pin "9")
   )
-  (symbol (lib_id "power:VCC") (at 88.9 95.25 0) (unit 1)
-    (in_bom yes) (on_board yes) (fields_autoplaced)
-    (property "Reference" "#PWR099" (id 0) (at 88.9 99.06 0)
-      (effects (font (size 1.27 1.27)) hide)
-    )
-    (property "Value" "VCC" (id 1) (at 88.9 90.17 0))
-    (property "Footprint" "" (id 2) (at 88.9 95.25 0)
-      (effects (font (size 1.27 1.27)) hide)
-    )
-    (property "Datasheet" "" (id 3) (at 88.9 95.25 0)
-      (effects (font (size 1.27 1.27)) hide)
-    )
-    (pin "1")
-  )
   (symbol (lib_id "Device:C_Small") (at 266.7 26.67 0) (unit 1)
     (in_bom yes) (on_board yes) (fields_autoplaced)
@@
   )
   (symbol (lib_id "Memory_EEPROM:28C256") (at 115.57 85.09 0) (unit 1)
-    (in_bom yes) (on_board yes) (fields_autoplaced)
-    (property "Reference" "U26" (id 0) (at 117.5894 54.61 0)
+    (in_bom yes) (on_board yes)
+    (property "Reference" "U26" (id 0) (at 107.95 58.42 0)
       (effects (font (size 1.27 1.27)) (justify left))
     )
-    (property "Value" "28C256" (id 1) (at 117.5894 57.15 0)
+    (property "Value" "AT28C256-15PC" (id 1) (at 116.84 58.42 0)
       (effects (font (size 1.27 1.27)) (justify left))
     )

Commit message: Update for Episode 16
Changed lines of the file:
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@@
   (title_block
     (title "Memory Module")
-    (date "2022-01-23")
-    (rev "A.15")
+    (date "2022-01-30")
+    (rev "A.16")
     (comment 2 "https://github.com/adrienkohlbecker/65C816")
     (comment 3 "Licensed under CERN-OHL-W v2")
@@
     (effects (font (size 1.27 1.27)) (justify left bottom))
   )
-  (label "A[0..23]" (at 44.45 40.64 180)
+  (label "{ADDRESS}" (at 44.45 40.64 180)
     (effects (font (size 1.27 1.27)) (justify right bottom))
   )
@@
     (effects (font (size 1.27 1.27)) (justify left bottom))
   )
-  (label "A[0..23]" (at 162.56 57.15 0)
+  (label "{ADDRESS}" (at 162.56 57.15 0)
     (effects (font (size 1.27 1.27)) (justify left bottom))
   )
@@
     (effects (font (size 1.27 1.27)) (justify right bottom))
   )
-  (label "A[0..23]" (at 85.09 57.15 0)
+  (label "{ADDRESS}" (at 85.09 57.15 0)
     (effects (font (size 1.27 1.27)) (justify left bottom))
   )
@@
     (effects (font (size 1.27 1.27)) (justify right))
   )
-  (hierarchical_label "A[0..23]" (shape input) (at 30.48 40.64 180)
+  (hierarchical_label "{ADDRESS}" (shape input) (at 30.48 40.64 180)
     (effects (font (size 1.27 1.27)) (justify right))
   )

Commit message: More episode 19 updates
Parts:
- added R41: 10k, symbol Device:R_Small
Connections:
- net VCC: now also R41.1
- net ~{ROM_WE}: now also R41.2
Changed lines of the file:
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@@
     (comment 4 "Copyright © 2021 Adrien Kohlbecker")
   )
+  (junction (at 93.98 102.87) (diameter 0) (color 0 0 0 0)
+  )
   (junction (at 257.81 29.21) (diameter 0) (color 0 0 0 0)
   )
@@
     (stroke (width 0) (type default) (color 0 0 0 0))
   )
-  (wire (pts (xy 96.52 107.95) (xy 105.41 107.95))
+  (wire (pts (xy 83.82 107.95) (xy 105.41 107.95))
     (stroke (width 0) (type default) (color 0 0 0 0))
   )
@@
     (stroke (width 0) (type default) (color 0 0 0 0))
   )
-  (wire (pts (xy 96.52 102.87) (xy 105.41 102.87))
+  (wire (pts (xy 83.82 102.87) (xy 93.98 102.87))
     (stroke (width 0) (type default) (color 0 0 0 0))
   )
@@
     (stroke (width 0) (type default) (color 0 0 0 0))
   )
+  (wire (pts (xy 93.98 101.6) (xy 93.98 102.87))
+    (stroke (width 0) (type default) (color 0 0 0 0))
+  )
   (wire (pts (xy 177.8 90.17) (xy 182.88 90.17))
     (stroke (width 0) (type default) (color 0 0 0 0))
@@
     (stroke (width 0) (type default) (color 0 0 0 0))
   )
+  (wire (pts (xy 93.98 102.87) (xy 105.41 102.87))
+    (stroke (width 0) (type default) (color 0 0 0 0))
+  )
   (bus (pts (xy 175.26 59.69) (xy 175.26 62.23))
     (stroke (width 0) (type default) (color 0 0 0 0))
@@
     (stroke (width 0) (type default) (color 0 0 0 0))
   )
-  (wire (pts (xy 96.52 105.41) (xy 105.41 105.41))
+  (wire (pts (xy 83.82 105.41) (xy 105.41 105.41))
+    (stroke (width 0) (type default) (color 0 0 0 0))
+  )
+  (wire (pts (xy 93.98 95.25) (xy 93.98 96.52))
     (stroke (width 0) (type default) (color 0 0 0 0))
   )
@@
     (effects (font (size 1.27 1.27)) (justify left bottom))
   )
-  (label "~{ROM_CS}" (at 96.52 107.95 0)
+  (label "~{ROM_CS}" (at 83.82 107.95 0)
     (effects (font (size 1.27 1.27)) (justify left bottom))
   )
@@
     (effects (font (size 1.27 1.27)) (justify right bottom))
   )
-  (label "~{RD}" (at 96.52 105.41 0)
+  (label "~{RD}" (at 83.82 105.41 0)
     (effects (font (size 1.27 1.27)) (justify left bottom))
   )
@@
     (effects (font (size 1.27 1.27)) (justify left bottom))
   )
-  (label "~{ROM_WE}" (at 96.52 102.87 0)
+  (label "~{ROM_WE}" (at 83.82 102.87 0)
     (effects (font (size 1.27 1.27)) (justify left bottom))
   )
@@
     )
     (pin "1")
+  )
+  (symbol (lib_id "Device:R_Small") (at 93.98 99.06 0) (unit 1)
+    (in_bom yes) (on_board yes)
+    (property "Reference" "R41" (id 0) (at 95.25 97.79 0)
+      (effects (font (size 1.27 1.27)) (justify left))
+    )
+    (property "Value" "10k" (id 1) (at 95.25 100.33 0)
+      (effects (font (size 1.27 1.27)) (justify left))
+    )
+    (property "Footprint" "" (id 2) (at 93.98 99.06 0)
+      (effects (font (size 1.27 1.27)) hide)
+    )
+    (property "Datasheet" "~" (id 3) (at 93.98 99.06 0)
+      (effects (font (size 1.27 1.27)) hide)
+    )
+    (pin "1")
+    (pin "2")
   )
   (symbol (lib_id "power:VCC") (at 115.57 57.15 0) (unit 1)
@@
     (pin "9")
   )
+  (symbol (lib_id "power:VCC") (at 93.98 95.25 0) (unit 1)
+    (in_bom yes) (on_board yes) (fields_autoplaced)
+    (property "Reference" "#PWR0125" (id 0) (at 93.98 99.06 0)
+      (effects (font (size 1.27 1.27)) hide)
+    )
+    (property "Value" "VCC" (id 1) (at 93.98 90.17 0))
+    (property "Footprint" "" (id 2) (at 93.98 95.25 0)
+      (effects (font (size 1.27 1.27)) hide)
+    )
+    (property "Datasheet" "" (id 3) (at 93.98 95.25 0)
+      (effects (font (size 1.27 1.27)) hide)
+    )
+    (pin "1")
+  )
   (symbol (lib_id "power:GND") (at 195.58 102.87 0) (unit 1)

Commit message: Update for episode 20
Parts:
- added C51: 100n, symbol Device:C_Small
- added U35: AS6C4008-55PCN, Package_DIP:DIP-32_W15.24mm, symbol Memory_RAM:AS6C4008-55PCN
Connections:
- net A0: now also U35.12 (A0)
- net A1: now also U35.11 (A1)
- net A10: now also U35.23 (A10)
- net A11: now also U35.25 (A11)
- net A12: now also U35.4 (A12)
- net A13: now also U35.28 (A13)
- net A14: now also U35.3 (A14)
- net A2: now also U35.10 (A2)
- net A3: now also U35.9 (A3)
- net A4: now also U35.8 (A4)
- net A5: now also U35.7 (A5)
- net A6: now also U35.6 (A6)
- net A7: now also U35.5 (A7)
- net A8: now also U35.27 (A8)
- net A9: now also U35.26 (A9)
- net D0: now also U35.13 (DQ0)
- net D1: now also U35.14 (DQ1)
- net D2: now also U35.15 (DQ2)
- net D3: now also U35.17 (DQ3)
- net D4: now also U35.18 (DQ4)
- net D5: now also U35.19 (DQ5)
- net D6: now also U35.20 (DQ6)
- net D7: now also U35.21 (DQ7)
- net GND: now also C51.2, U35.16 (VSS)
- net VCC: now also C51.1, U35.32 (VCC)
- net ~{RD}: now also U35.24 (OE#)
- net ~{WR}: now also U35.29 (WE#)
- new net A15: U35.31 (A15)
- new net ~{A16}: U35.2 (A16)
- new net ~{A17}: U35.30 (A17)
- new net ~{A18}: U35.1 (A18)
- new net ~{EXTRAM_CS}: U35.22 (CE#)
Other:
- moved on the sheet: C38, C39, C43, R41, U26, U28
