File: hardware/memory.kicad_sch (KiCad schematic)
At the start: 8 parts, among them U26 AT28C256-15PC, U28 LY62256PL-55LL, U35 AS6C4008-55PCN

Commit message: Renumber
Parts:
- renumbered C38 to C41, C39 to C42, C51 to C44, R41 to R31, U26 to U27, U35 to U29
Changed lines of the file:
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@@
   (symbol (lib_id "power:GND") (at 218.44 123.19 0) (unit 1)
     (in_bom yes) (on_board yes) (fields_autoplaced)
-    (property "Reference" "#PWR0127" (id 0) (at 218.44 129.54 0)
+    (property "Reference" "#PWR093" (id 0) (at 218.44 129.54 0)
       (effects (font (size 1.27 1.27)) hide)
     )
@@
   (symbol (lib_id "Device:C_Small") (at 270.51 26.67 0) (unit 1)
     (in_bom yes) (on_board yes) (fields_autoplaced)
-    (property "Reference" "C51" (id 0) (at 273.05 25.4062 0)
+    (property "Reference" "C44" (id 0) (at 273.05 25.4062 0)
       (effects (font (size 1.27 1.27)) (justify left))
     )
@@
   (symbol (lib_id "Device:R_Small") (at 40.64 109.22 0) (unit 1)
     (in_bom yes) (on_board yes)
-    (property "Reference" "R41" (id 0) (at 41.91 107.95 0)
+    (property "Reference" "R31" (id 0) (at 41.91 107.95 0)
       (effects (font (size 1.27 1.27)) (justify left))
     )
@@
   (symbol (lib_id "Memory_RAM:AS6C4008-55PCN") (at 218.44 95.25 0) (unit 1)
     (in_bom yes) (on_board yes)
-    (property "Reference" "U35" (id 0) (at 208.28 68.58 0)
+    (property "Reference" "U29" (id 0) (at 208.28 68.58 0)
       (effects (font (size 1.27 1.27)) (justify left))
     )
@@
   (symbol (lib_id "power:VCC") (at 62.23 67.31 0) (unit 1)
     (in_bom yes) (on_board yes) (fields_autoplaced)
-    (property "Reference" "#PWR038" (id 0) (at 62.23 71.12 0)
+    (property "Reference" "#PWR088" (id 0) (at 62.23 71.12 0)
       (effects (font (size 1.27 1.27)) hide)
     )
@@
   (symbol (lib_id "Device:C_Small") (at 252.73 26.67 0) (unit 1)
     (in_bom yes) (on_board yes) (fields_autoplaced)
-    (property "Reference" "C39" (id 0) (at 255.27 25.4062 0)
+    (property "Reference" "C42" (id 0) (at 255.27 25.4062 0)
       (effects (font (size 1.27 1.27)) (justify left))
     )
@@
   (symbol (lib_id "Memory_EEPROM:28C256") (at 62.23 95.25 0) (unit 1)
     (in_bom yes) (on_board yes)
-    (property "Reference" "U26" (id 0) (at 54.61 68.58 0)
+    (property "Reference" "U27" (id 0) (at 54.61 68.58 0)
       (effects (font (size 1.27 1.27)) (justify left))
     )
@@
   (symbol (lib_id "power:VCC") (at 40.64 105.41 0) (unit 1)
     (in_bom yes) (on_board yes) (fields_autoplaced)
-    (property "Reference" "#PWR0125" (id 0) (at 40.64 109.22 0)
+    (property "Reference" "#PWR087" (id 0) (at 40.64 109.22 0)
       (effects (font (size 1.27 1.27)) hide)
     )
@@
   (symbol (lib_id "power:GND") (at 139.7 113.03 0) (unit 1)
     (in_bom yes) (on_board yes) (fields_autoplaced)
-    (property "Reference" "#PWR0122" (id 0) (at 139.7 119.38 0)
+    (property "Reference" "#PWR091" (id 0) (at 139.7 119.38 0)
       (effects (font (size 1.27 1.27)) hide)
     )
@@
   (symbol (lib_id "power:VCC") (at 243.84 22.86 0) (unit 1)
     (in_bom yes) (on_board yes) (fields_autoplaced)
-    (property "Reference" "#PWR066" (id 0) (at 243.84 26.67 0)
+    (property "Reference" "#PWR094" (id 0) (at 243.84 26.67 0)
       (effects (font (size 1.27 1.27)) hide)
     )
@@
   (symbol (lib_id "power:VCC") (at 218.44 67.31 0) (unit 1)
     (in_bom yes) (on_board yes) (fields_autoplaced)
-    (property "Reference" "#PWR0126" (id 0) (at 218.44 71.12 0)
+    (property "Reference" "#PWR092" (id 0) (at 218.44 71.12 0)
       (effects (font (size 1.27 1.27)) hide)
     )
@@
   (symbol (lib_id "power:VCC") (at 139.7 67.31 0) (unit 1)
     (in_bom yes) (on_board yes) (fields_autoplaced)
-    (property "Reference" "#PWR0121" (id 0) (at 139.7 71.12 0)
+    (property "Reference" "#PWR090" (id 0) (at 139.7 71.12 0)
       (effects (font (size 1.27 1.27)) hide)
     )
@@
   (symbol (lib_id "power:GND") (at 243.84 30.48 0) (unit 1)
     (in_bom yes) (on_board yes) (fields_autoplaced)
-    (property "Reference" "#PWR085" (id 0) (at 243.84 36.83 0)
+    (property "Reference" "#PWR095" (id 0) (at 243.84 36.83 0)
       (effects (font (size 1.27 1.27)) hide)
     )
@@
   (symbol (lib_id "power:GND") (at 62.23 123.19 0) (unit 1)
     (in_bom yes) (on_board yes) (fields_autoplaced)
-    (property "Reference" "#PWR062" (id 0) (at 62.23 129.54 0)
+    (property "Reference" "#PWR089" (id 0) (at 62.23 129.54 0)
       (effects (font (size 1.27 1.27)) hide)
     )
@@
   (symbol (lib_id "Device:C_Polarized_Small") (at 243.84 26.67 0) (unit 1)
     (in_bom yes) (on_board yes)
-    (property "Reference" "C38" (id 0) (at 246.38 25.4 0)
-      (effects (font (size 1.27 1.27)) (justify left))
-    )
+    (property "Reference" "C41" (id 0) (at 246.38 25.4 0)
+      (effects (font (size 1.27 1.27)) (justify left))
+    )

Commit message: Snapshot ep 24 work
Parts:
- R31: value 10k -> 3.3k
Connections:
- net ~{A16} renamed A16
- net ~{A17} renamed A17
- net ~{A18} renamed A18
Changed lines of the file:
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@@
   (title_block
     (title "Memory Module")
-    (date "2022-05-23")
-    (rev "A.23")
+    (date "2022-07-04")
+    (rev "A.24")
     (comment 2 "https://github.com/adrienkohlbecker/65C816")
     (comment 3 "Licensed under CERN-OHL-W v2")
@@
     (effects (font (size 1.27 1.27)) (justify left bottom))
   )
+  (label "A18" (at 200.66 118.11 0)
+    (effects (font (size 1.27 1.27)) (justify left bottom))
+  )
   (label "~{WR}" (at 44.45 24.13 180)
     (effects (font (size 1.27 1.27)) (justify right bottom))
@@
     (effects (font (size 1.27 1.27)) (justify left bottom))
   )
-  (label "~{A16}" (at 200.66 113.03 0)
-    (effects (font (size 1.27 1.27)) (justify left bottom))
-  )
   (label "D6" (at 154.94 87.63 0)
     (effects (font (size 1.27 1.27)) (justify left bottom))
@@
     (effects (font (size 1.27 1.27)) (justify left bottom))
   )
-  (label "{ADDRESS}" (at 44.45 44.45 180)
+  (label "A[0..23]" (at 44.45 44.45 180)
     (effects (font (size 1.27 1.27)) (justify right bottom))
   )
@@
     (effects (font (size 1.27 1.27)) (justify left bottom))
   )
-  (label "{ADDRESS}" (at 106.68 67.31 0)
+  (label "A[0..23]" (at 106.68 67.31 0)
     (effects (font (size 1.27 1.27)) (justify left bottom))
   )
@@
     (effects (font (size 1.27 1.27)) (justify left bottom))
   )
-  (label "{ADDRESS}" (at 31.75 67.31 0)
+  (label "A[0..23]" (at 31.75 67.31 0)
     (effects (font (size 1.27 1.27)) (justify left bottom))
   )
@@
     (effects (font (size 1.27 1.27)) (justify left bottom))
   )
+  (label "A17" (at 200.66 115.57 0)
+    (effects (font (size 1.27 1.27)) (justify left bottom))
+  )
   (label "D2" (at 234.95 77.47 0)
     (effects (font (size 1.27 1.27)) (justify left bottom))
@@
     (effects (font (size 1.27 1.27)) (justify left bottom))
   )
+  (label "A16" (at 200.66 113.03 0)
+    (effects (font (size 1.27 1.27)) (justify left bottom))
+  )
   (label "A5" (at 200.66 85.09 0)
     (effects (font (size 1.27 1.27)) (justify left bottom))
   )
-  (label "{ADDRESS}" (at 185.42 67.31 0)
+  (label "A[0..23]" (at 185.42 67.31 0)
     (effects (font (size 1.27 1.27)) (justify left bottom))
   )
@@
     (effects (font (size 1.27 1.27)) (justify left bottom))
   )
-  (label "~{A18}" (at 200.66 118.11 0)
-    (effects (font (size 1.27 1.27)) (justify left bottom))
-  )
   (label "A2" (at 121.92 77.47 0)
     (effects (font (size 1.27 1.27)) (justify left bottom))
@@
   )
   (label "A13" (at 46.99 105.41 0)
-    (effects (font (size 1.27 1.27)) (justify left bottom))
-  )
-  (label "~{A17}" (at 200.66 115.57 0)
     (effects (font (size 1.27 1.27)) (justify left bottom))
   )
@@
     (effects (font (size 1.27 1.27)) (justify right))
   )
-  (hierarchical_label "{ADDRESS}" (shape input) (at 30.48 44.45 180)
+  (hierarchical_label "A[0..23]" (shape input) (at 30.48 44.45 180)
     (effects (font (size 1.27 1.27)) (justify right))
   )
@@
       (effects (font (size 1.27 1.27)) (justify left))
     )
-    (property "Value" "10k" (id 1) (at 41.91 110.49 0)
+    (property "Value" "3.3k" (id 1) (at 41.91 110.49 0)
       (effects (font (size 1.27 1.27)) (justify left))
     )

Commit message: Update main project
Parts:
- renumbered C41 to C6, C42 to C7, C43 to C8, C44 to C9, R31 to R1, U27 to U6, U28 to U7, U29 to U8
Changed lines of the file:
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@@
   (symbol (lib_id "power:GND") (at 218.44 123.19 0) (unit 1)
     (in_bom yes) (on_board yes) (fields_autoplaced)
-    (property "Reference" "#PWR093" (id 0) (at 218.44 129.54 0)
+    (property "Reference" "#PWR018" (id 0) (at 218.44 129.54 0)
       (effects (font (size 1.27 1.27)) hide)
     )
@@
   (symbol (lib_id "Device:C_Small") (at 270.51 26.67 0) (unit 1)
     (in_bom yes) (on_board yes) (fields_autoplaced)
-    (property "Reference" "C44" (id 0) (at 273.05 25.4062 0)
+    (property "Reference" "C9" (id 0) (at 273.05 25.4062 0)
       (effects (font (size 1.27 1.27)) (justify left))
     )
@@
   (symbol (lib_id "Device:R_Small") (at 40.64 109.22 0) (unit 1)
     (in_bom yes) (on_board yes)
-    (property "Reference" "R31" (id 0) (at 41.91 107.95 0)
+    (property "Reference" "R1" (id 0) (at 41.91 107.95 0)
       (effects (font (size 1.27 1.27)) (justify left))
     )
@@
   (symbol (lib_id "Memory_RAM:AS6C4008-55PCN") (at 218.44 95.25 0) (unit 1)
     (in_bom yes) (on_board yes)
-    (property "Reference" "U29" (id 0) (at 208.28 68.58 0)
+    (property "Reference" "U8" (id 0) (at 208.28 68.58 0)
       (effects (font (size 1.27 1.27)) (justify left))
     )
@@
   (symbol (lib_id "power:VCC") (at 62.23 67.31 0) (unit 1)
     (in_bom yes) (on_board yes) (fields_autoplaced)
-    (property "Reference" "#PWR088" (id 0) (at 62.23 71.12 0)
+    (property "Reference" "#PWR013" (id 0) (at 62.23 71.12 0)
       (effects (font (size 1.27 1.27)) hide)
     )
@@
   (symbol (lib_id "Memory_RAM:KM62256CLP") (at 139.7 90.17 0) (unit 1)
     (in_bom yes) (on_board yes)
-    (property "Reference" "U28" (id 0) (at 129.54 68.58 0)
+    (property "Reference" "U7" (id 0) (at 129.54 68.58 0)
       (effects (font (size 1.27 1.27)) (justify left))
     )
@@
   (symbol (lib_id "Device:C_Small") (at 252.73 26.67 0) (unit 1)
     (in_bom yes) (on_board yes) (fields_autoplaced)
-    (property "Reference" "C42" (id 0) (at 255.27 25.4062 0)
+    (property "Reference" "C7" (id 0) (at 255.27 25.4062 0)
       (effects (font (size 1.27 1.27)) (justify left))
     )
@@
   (symbol (lib_id "Memory_EEPROM:28C256") (at 62.23 95.25 0) (unit 1)
     (in_bom yes) (on_board yes)
-    (property "Reference" "U27" (id 0) (at 54.61 68.58 0)
+    (property "Reference" "U6" (id 0) (at 54.61 68.58 0)
       (effects (font (size 1.27 1.27)) (justify left))
     )
@@
   (symbol (lib_id "power:VCC") (at 40.64 105.41 0) (unit 1)
     (in_bom yes) (on_board yes) (fields_autoplaced)
-    (property "Reference" "#PWR087" (id 0) (at 40.64 109.22 0)
+    (property "Reference" "#PWR012" (id 0) (at 40.64 109.22 0)
       (effects (font (size 1.27 1.27)) hide)
     )
@@
   (symbol (lib_id "power:GND") (at 139.7 113.03 0) (unit 1)
     (in_bom yes) (on_board yes) (fields_autoplaced)
-    (property "Reference" "#PWR091" (id 0) (at 139.7 119.38 0)
+    (property "Reference" "#PWR016" (id 0) (at 139.7 119.38 0)
       (effects (font (size 1.27 1.27)) hide)
     )
@@
   (symbol (lib_id "power:VCC") (at 243.84 22.86 0) (unit 1)
     (in_bom yes) (on_board yes) (fields_autoplaced)
-    (property "Reference" "#PWR094" (id 0) (at 243.84 26.67 0)
+    (property "Reference" "#PWR019" (id 0) (at 243.84 26.67 0)
       (effects (font (size 1.27 1.27)) hide)
     )
@@
   (symbol (lib_id "Device:C_Small") (at 261.62 26.67 0) (unit 1)
     (in_bom yes) (on_board yes) (fields_autoplaced)
-    (property "Reference" "C43" (id 0) (at 264.16 25.4062 0)
+    (property "Reference" "C8" (id 0) (at 264.16 25.4062 0)
       (effects (font (size 1.27 1.27)) (justify left))
     )
@@
   (symbol (lib_id "power:VCC") (at 218.44 67.31 0) (unit 1)
     (in_bom yes) (on_board yes) (fields_autoplaced)
-    (property "Reference" "#PWR092" (id 0) (at 218.44 71.12 0)
+    (property "Reference" "#PWR017" (id 0) (at 218.44 71.12 0)
       (effects (font (size 1.27 1.27)) hide)
     )
@@
   (symbol (lib_id "power:VCC") (at 139.7 67.31 0) (unit 1)
     (in_bom yes) (on_board yes) (fields_autoplaced)
-    (property "Reference" "#PWR090" (id 0) (at 139.7 71.12 0)
+    (property "Reference" "#PWR015" (id 0) (at 139.7 71.12 0)
       (effects (font (size 1.27 1.27)) hide)
     )
@@
   (symbol (lib_id "power:GND") (at 243.84 30.48 0) (unit 1)
     (in_bom yes) (on_board yes) (fields_autoplaced)
-    (property "Reference" "#PWR095" (id 0) (at 243.84 36.83 0)
+    (property "Reference" "#PWR020" (id 0) (at 243.84 36.83 0)
       (effects (font (size 1.27 1.27)) hide)
     )
@@
   (symbol (lib_id "power:GND") (at 62.23 123.19 0) (unit 1)
     (in_bom yes) (on_board yes) (fields_autoplaced)
-    (property "Reference" "#PWR089" (id 0) (at 62.23 129.54 0)
+    (property "Reference" "#PWR014" (id 0) (at 62.23 129.54 0)
       (effects (font (size 1.27 1.27)) hide)
     )
@@
   (symbol (lib_id "Device:C_Polarized_Small") (at 243.84 26.67 0) (unit 1)
     (in_bom yes) (on_board yes)
-    (property "Reference" "C41" (id 0) (at 246.38 25.4 0)
-      (effects (font (size 1.27 1.27)) (justify left))
-    )
+    (property "Reference" "C6" (id 0) (at 246.38 25.4 0)
+      (effects (font (size 1.27 1.27)) (justify left))
+    )
