File: hardware/reset.kicad_sch (KiCad schematic)
At the start: 11 parts, among them SW5 Reset, U18 MAX705, U19 74HC175

Commit message: Updates for Episode 14
Parts:
- C25: symbol Device:CP_Small -> Device:C_Polarized_Small
- SW5: symbol keyboard:SW_Push -> Switch:SW_Push
Changed lines of the file:
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@@
   (title_block
     (title "Reset Module")
-    (date "2022-01-09")
-    (rev "A.13")
+    (date "2022-01-14")
+    (rev "A.14")
     (comment 2 "https://github.com/adrienkohlbecker/65C816")
     (comment 3 "Licensed under CERN-OHL-W v2")
@@
     (pin "1")
   )
-  (symbol (lib_id "keyboard:SW_Push") (at 52.07 72.39 90) (unit 1)
+  (symbol (lib_id "Switch:SW_Push") (at 52.07 72.39 90) (unit 1)
     (in_bom yes) (on_board yes)
     (property "Reference" "SW5" (id 0) (at 53.2892 71.2216 90)
@@
       (effects (font (size 1.27 1.27)) hide)
     )
-    (property "Datasheet" "" (id 3) (at 46.99 72.39 0)
+    (property "Datasheet" "~" (id 3) (at 46.99 72.39 0)
       (effects (font (size 1.27 1.27)) hide)
     )
@@
     (pin "1")
   )
-  (symbol (lib_id "Device:CP_Small") (at 24.13 124.46 0) (unit 1)
+  (symbol (lib_id "Device:C_Polarized_Small") (at 24.13 124.46 0) (unit 1)
     (in_bom yes) (on_board yes)
     (property "Reference" "C25" (id 0) (at 27.1272 123.2916 0)
@@
       (effects (font (size 1.27 1.27)) (justify left))
     )
-    (property "Footprint" "" (id 2) (at 25.0952 128.27 0)
-      (effects (font (size 1.27 1.27)) hide)
-    )
+    (property "Footprint" "" (id 2) (at 24.13 124.46 0)
+      (effects (font (size 1.27 1.27)) hide)
+    )

Commit message: Update for Episode 16
Parts:
- removed D3: Reset, symbol Device:LED_Small
- removed R11: 1k, symbol Device:R_Small
Connections:
- net VCC: now also U19.13 (D3)
- net at U19.12 (D2), U19.7 (Q1): no longer U19.13 (D3)
- no-connect marks 6 -> 7
Changed lines of the file:
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@@
   (title_block
     (title "Reset Module")
-    (date "2022-01-23")
-    (rev "A.15")
+    (date "2022-01-30")
+    (rev "A.16")
     (comment 2 "https://github.com/adrienkohlbecker/65C816")
     (comment 3 "Licensed under CERN-OHL-W v2")
@@
   )
   (junction (at 24.13 127) (diameter 0) (color 0 0 0 0)
-  )
-  (junction (at 137.16 67.31) (diameter 0) (color 0 0 0 0)
   )
   (junction (at 52.07 66.04) (diameter 0) (color 0 0 0 0)
@@
   (no_connect (at 66.04 71.12))
   (no_connect (at 86.36 71.12))
+  (no_connect (at 166.37 74.93))
   (no_connect (at 166.37 64.77))
   (wire (pts (xy 138.43 43.18) (xy 138.43 62.23))
@@
     (stroke (width 0) (type default) (color 0 0 0 0))
   )
-  (wire (pts (xy 177.8 74.93) (xy 177.8 76.2))
+  (wire (pts (xy 139.7 72.39) (xy 140.97 72.39))
     (stroke (width 0) (type default) (color 0 0 0 0))
   )
@@
     (stroke (width 0) (type default) (color 0 0 0 0))
   )
-  (wire (pts (xy 177.8 82.55) (xy 177.8 81.28))
-    (stroke (width 0) (type default) (color 0 0 0 0))
-  )
   (wire (pts (xy 52.07 81.28) (xy 52.07 78.74))
     (stroke (width 0) (type default) (color 0 0 0 0))
@@
     (stroke (width 0) (type default) (color 0 0 0 0))
   )
-  (wire (pts (xy 137.16 72.39) (xy 137.16 67.31))
-    (stroke (width 0) (type default) (color 0 0 0 0))
-  )
-  (wire (pts (xy 175.26 74.93) (xy 177.8 74.93))
-    (stroke (width 0) (type default) (color 0 0 0 0))
-  )
   (wire (pts (xy 33.02 127) (xy 24.13 127))
     (stroke (width 0) (type default) (color 0 0 0 0))
   )
   (wire (pts (xy 166.37 67.31) (xy 173.99 67.31))
-    (stroke (width 0) (type default) (color 0 0 0 0))
-  )
-  (wire (pts (xy 170.18 74.93) (xy 166.37 74.93))
-    (stroke (width 0) (type default) (color 0 0 0 0))
-  )
-  (wire (pts (xy 140.97 72.39) (xy 137.16 72.39))
     (stroke (width 0) (type default) (color 0 0 0 0))
   )
@@
     )
     (property "Datasheet" "" (id 3) (at 24.13 127 0)
-      (effects (font (size 1.27 1.27)) hide)
-    )
-    (pin "1")
-  )
-  (symbol (lib_id "Device:LED_Small") (at 172.72 74.93 180) (unit 1)
-    (in_bom yes) (on_board yes)
-    (property "Reference" "D3" (id 0) (at 172.72 78.74 0))
-    (property "Value" "Reset" (id 1) (at 172.72 81.28 0))
-    (property "Footprint" "" (id 2) (at 172.72 74.93 90)
-      (effects (font (size 1.27 1.27)) hide)
-    )
-    (property "Datasheet" "~" (id 3) (at 172.72 74.93 90)
-      (effects (font (size 1.27 1.27)) hide)
-    )
-    (pin "1")
-    (pin "2")
-  )
-  (symbol (lib_id "Device:R_Small") (at 177.8 78.74 180) (unit 1)
-    (in_bom yes) (on_board yes)
-    (property "Reference" "R11" (id 0) (at 179.2986 77.5716 0)
-      (effects (font (size 1.27 1.27)) (justify right))
-    )
-    (property "Value" "1k" (id 1) (at 179.2986 79.883 0)
-      (effects (font (size 1.27 1.27)) (justify right))
-    )
-    (property "Footprint" "" (id 2) (at 177.8 78.74 0)
-      (effects (font (size 1.27 1.27)) hide)
-    )
-    (property "Datasheet" "~" (id 3) (at 177.8 78.74 0)
-      (effects (font (size 1.27 1.27)) hide)
-    )
-    (pin "1")
-    (pin "2")
-  )
-  (symbol (lib_id "power:GND") (at 177.8 82.55 0) (unit 1)
-    (in_bom yes) (on_board yes)
-    (property "Reference" "#PWR084" (id 0) (at 177.8 88.9 0)
-      (effects (font (size 1.27 1.27)) hide)
-    )
-    (property "Value" "GND" (id 1) (at 177.927 86.9442 0))
-    (property "Footprint" "" (id 2) (at 177.8 82.55 0)
-      (effects (font (size 1.27 1.27)) hide)
-    )
-    (property "Datasheet" "" (id 3) (at 177.8 82.55 0)
       (effects (font (size 1.27 1.27)) hide)
     )
@@
       (effects (font (size 1.27 1.27)) hide)
     )
+    (pin "1")
+  )
+  (symbol (lib_id "power:VCC") (at 139.7 72.39 0) (unit 1)
+    (in_bom yes) (on_board yes)
+    (property "Reference" "#PWR0112" (id 0) (at 139.7 76.2 0)
+      (effects (font (size 1.27 1.27)) hide)
+    )
+    (property "Value" "VCC" (id 1) (at 137.16 69.85 0))
+    (property "Footprint" "" (id 2) (at 139.7 72.39 0)
+      (effects (font (size 1.27 1.27)) hide)
+    )
+    (property "Datasheet" "" (id 3) (at 139.7 72.39 0)
+      (effects (font (size 1.27 1.27)) hide)
+    )

Commit message: Updates for episode 17
Parts:
- removed D4: PWRUP, symbol Device:LED_Small
- removed R12: 1k, symbol Device:R_Small
Connections:
- net ~{PWRUP}: no longer names the net of U18.7 (~{RESET}), U19.1 (~{Mr}), U19.4 (D0)
Other:
- moved on the sheet: C27, SW5, U18, U19
