File: hardware/reset.kicad_sch (KiCad schematic)
At the start: 7 parts, among them SW5 Reset, U18 MAX705, U19 74HC175

Commit message: Updates for episode 20
Connections:
- net VCC: no longer U19.13 (D3)
- net at U19.12 (D2), U19.7 (Q1): now also U19.13 (D3)
Changed lines of the file:
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@@
   (junction (at 24.13 121.92) (diameter 0) (color 0 0 0 0)
+  )
+  (junction (at 111.76 67.31) (diameter 0) (color 0 0 0 0)
   )
   (junction (at 33.02 121.92) (diameter 0) (color 0 0 0 0)
@@
     (stroke (width 0) (type default) (color 0 0 0 0))
   )
-  (wire (pts (xy 114.3 72.39) (xy 115.57 72.39))
+  (wire (pts (xy 111.76 72.39) (xy 115.57 72.39))
     (stroke (width 0) (type default) (color 0 0 0 0))
   )
@@
   )
   (wire (pts (xy 110.49 77.47) (xy 115.57 77.47))
+    (stroke (width 0) (type default) (color 0 0 0 0))
+  )
+  (wire (pts (xy 111.76 72.39) (xy 111.76 67.31))
     (stroke (width 0) (type default) (color 0 0 0 0))
   )
@@
     (pin "2")
   )
-  (symbol (lib_id "power:VCC") (at 114.3 72.39 0) (unit 1)
-    (in_bom yes) (on_board yes)
-    (property "Reference" "#PWR0112" (id 0) (at 114.3 76.2 0)
-      (effects (font (size 1.27 1.27)) hide)
-    )
-    (property "Value" "VCC" (id 1) (at 111.76 69.85 0))
-    (property "Footprint" "" (id 2) (at 114.3 72.39 0)
-      (effects (font (size 1.27 1.27)) hide)
-    )
-    (property "Datasheet" "" (id 3) (at 114.3 72.39 0)
-      (effects (font (size 1.27 1.27)) hide)
-    )
-    (pin "1")
-  )
 )

Commit message: Renumber
Parts:
- renumbered C25 to C21, C26 to C22, C28 to C23, C27 to C24, SW5 to SW7, U18 to U11, U19 to U12
Changed lines of the file:
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@@
   (symbol (lib_id "65C816:MAX705") (at 81.28 59.69 0) (unit 1)
     (in_bom yes) (on_board yes)
-    (property "Reference" "U18" (id 0) (at 74.93 49.53 0))
+    (property "Reference" "U11" (id 0) (at 74.93 49.53 0))
     (property "Value" "MAX705" (id 1) (at 87.63 49.53 0))
     (property "Footprint" "" (id 2) (at 78.74 49.53 0)
@@
   (symbol (lib_id "power:VCC") (at 81.28 48.26 0) (unit 1)
     (in_bom yes) (on_board yes)
-    (property "Reference" "#PWR080" (id 0) (at 81.28 52.07 0)
+    (property "Reference" "#PWR056" (id 0) (at 81.28 52.07 0)
       (effects (font (size 1.27 1.27)) hide)
     )
@@
   (symbol (lib_id "power:GND") (at 81.28 71.12 0) (unit 1)
     (in_bom yes) (on_board yes)
-    (property "Reference" "#PWR081" (id 0) (at 81.28 77.47 0)
+    (property "Reference" "#PWR057" (id 0) (at 81.28 77.47 0)
       (effects (font (size 1.27 1.27)) hide)
     )
@@
   (symbol (lib_id "Switch:SW_Push") (at 57.15 63.5 90) (unit 1)
     (in_bom yes) (on_board yes)
-    (property "Reference" "SW5" (id 0) (at 58.3692 62.3316 90)
+    (property "Reference" "SW7" (id 0) (at 58.3692 62.3316 90)
       (effects (font (size 1.27 1.27)) (justify right))
     )
@@
   (symbol (lib_id "power:GND") (at 57.15 72.39 0) (unit 1)
     (in_bom yes) (on_board yes)
-    (property "Reference" "#PWR078" (id 0) (at 57.15 78.74 0)
+    (property "Reference" "#PWR054" (id 0) (at 57.15 78.74 0)
       (effects (font (size 1.27 1.27)) hide)
     )
@@
   (symbol (lib_id "Device:C_Small") (at 33.02 124.46 0) (unit 1)
     (in_bom yes) (on_board yes)
-    (property "Reference" "C26" (id 0) (at 35.3568 123.2916 0)
+    (property "Reference" "C22" (id 0) (at 35.3568 123.2916 0)
       (effects (font (size 1.27 1.27)) (justify left))
     )
@@
   (symbol (lib_id "Device:C_Small") (at 45.72 124.46 0) (unit 1)
     (in_bom yes) (on_board yes)
-    (property "Reference" "C28" (id 0) (at 48.0568 123.2916 0)
+    (property "Reference" "C23" (id 0) (at 48.0568 123.2916 0)
       (effects (font (size 1.27 1.27)) (justify left))
     )
@@
   (symbol (lib_id "power:VCC") (at 24.13 121.92 0) (unit 1)
     (in_bom yes) (on_board yes)
-    (property "Reference" "#PWR076" (id 0) (at 24.13 125.73 0)
+    (property "Reference" "#PWR052" (id 0) (at 24.13 125.73 0)
       (effects (font (size 1.27 1.27)) hide)
     )
@@
   (symbol (lib_id "power:GND") (at 24.13 127 0) (unit 1)
     (in_bom yes) (on_board yes)
-    (property "Reference" "#PWR077" (id 0) (at 24.13 133.35 0)
+    (property "Reference" "#PWR053" (id 0) (at 24.13 133.35 0)
       (effects (font (size 1.27 1.27)) hide)
     )
@@
   (symbol (lib_id "Device:C_Small") (at 46.99 63.5 0) (unit 1)
     (in_bom yes) (on_board yes)
-    (property "Reference" "C27" (id 0) (at 49.3268 62.3316 0)
+    (property "Reference" "C24" (id 0) (at 49.3268 62.3316 0)
       (effects (font (size 1.27 1.27)) (justify left))
     )
@@
   (symbol (lib_id "74xx:74LS175") (at 128.27 67.31 0) (unit 1)
     (in_bom yes) (on_board yes)
-    (property "Reference" "U19" (id 0) (at 121.92 53.34 0))
+    (property "Reference" "U12" (id 0) (at 121.92 53.34 0))
     (property "Value" "74HC175" (id 1) (at 134.62 53.34 0))
     (property "Footprint" "" (id 2) (at 128.27 67.31 0)
@@
   (symbol (lib_id "power:VCC") (at 128.27 49.53 0) (unit 1)
     (in_bom yes) (on_board yes)
-    (property "Reference" "#PWR082" (id 0) (at 128.27 53.34 0)
+    (property "Reference" "#PWR058" (id 0) (at 128.27 53.34 0)
       (effects (font (size 1.27 1.27)) hide)
     )
@@
   (symbol (lib_id "power:GND") (at 128.27 87.63 0) (unit 1)
     (in_bom yes) (on_board yes)
-    (property "Reference" "#PWR083" (id 0) (at 128.27 93.98 0)
+    (property "Reference" "#PWR059" (id 0) (at 128.27 93.98 0)
       (effects (font (size 1.27 1.27)) hide)
     )
@@
   (symbol (lib_id "power:GND") (at 68.58 62.23 0) (unit 1)
     (in_bom yes) (on_board yes)
-    (property "Reference" "#PWR079" (id 0) (at 68.58 68.58 0)
+    (property "Reference" "#PWR055" (id 0) (at 68.58 68.58 0)
       (effects (font (size 1.27 1.27)) hide)
     )
@@
   (symbol (lib_id "Device:C_Polarized_Small") (at 24.13 124.46 0) (unit 1)
     (in_bom yes) (on_board yes)
-    (property "Reference" "C25" (id 0) (at 27.1272 123.2916 0)
-      (effects (font (size 1.27 1.27)) (justify left))
-    )
+    (property "Reference" "C21" (id 0) (at 27.1272 123.2916 0)
+      (effects (font (size 1.27 1.27)) (justify left))
+    )
