File: hardware/address_decoding.kicad_sch (KiCad schematic)
At the start: 4 parts, among them U27 74HC10, U28 74HC10

Commit message: More updates for episode 14
Parts:
- renumbered U28 to U27
Changed lines of the file:
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@@
   (symbol (lib_id "74xx:74LS10") (at 102.87 161.29 0) (unit 4)
     (in_bom yes) (on_board yes)
-    (property "Reference" "U28" (id 0) (at 99.06 152.4 0))
+    (property "Reference" "U27" (id 0) (at 99.06 152.4 0))
     (property "Value" "74HC10" (id 1) (at 107.95 152.4 0))
     (property "Footprint" "" (id 2) (at 102.87 161.29 0)

Commit message: Start episode 15
Parts:
- added unit 3 of U27
Connections:
- net VCC: now also U27.10, U27.11, U27.9
- net A15 renamed ~{RAM_CS}
- no-connect marks 1 -> 2
Changed lines of the file:
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@@
   (title_block
     (title "Address Decoding Module")
-    (date "2022-01-14")
-    (rev "A.14")
+    (date "2022-01-23")
+    (rev "A.15")
     (comment 2 "https://github.com/adrienkohlbecker/65C816")
     (comment 3 "Licensed under CERN-OHL-W v2")
@@
   (junction (at 129.54 91.44) (diameter 0) (color 0 0 0 0)
   )
+  (junction (at 39.37 157.48) (diameter 0) (color 0 0 0 0)
+  )
   (junction (at 39.37 154.94) (diameter 0) (color 0 0 0 0)
   )
+  (junction (at 39.37 170.18) (diameter 0) (color 0 0 0 0)
+  )
+  (junction (at 39.37 167.64) (diameter 0) (color 0 0 0 0)
+  )
   (junction (at 256.54 24.13) (diameter 0) (color 0 0 0 0)
   )
   (junction (at 256.54 29.21) (diameter 0) (color 0 0 0 0)
   )
+  (no_connect (at 57.15 170.18))
   (no_connect (at 57.15 154.94))
+  (bus_entry (at 125.73 107.95) (size 2.54 2.54)
+    (stroke (width 0) (type default) (color 0 0 0 0))
+  )
   (bus_entry (at 125.73 93.98) (size 2.54 2.54)
     (stroke (width 0) (type default) (color 0 0 0 0))
   )
+  (wire (pts (xy 41.91 167.64) (xy 39.37 167.64))
+    (stroke (width 0) (type default) (color 0 0 0 0))
+  )
+  (wire (pts (xy 41.91 170.18) (xy 39.37 170.18))
+    (stroke (width 0) (type default) (color 0 0 0 0))
+  )
+  (wire (pts (xy 39.37 167.64) (xy 39.37 157.48))
+    (stroke (width 0) (type default) (color 0 0 0 0))
+  )
   (wire (pts (xy 39.37 154.94) (xy 39.37 157.48))
     (stroke (width 0) (type default) (color 0 0 0 0))
@@
     (stroke (width 0) (type default) (color 0 0 0 0))
   )
+  (bus (pts (xy 125.73 93.98) (xy 125.73 107.95))
+    (stroke (width 0) (type default) (color 0 0 0 0))
+  )
+  (wire (pts (xy 39.37 170.18) (xy 39.37 167.64))
+    (stroke (width 0) (type default) (color 0 0 0 0))
+  )
   (wire (pts (xy 256.54 24.13) (xy 267.97 24.13))
     (stroke (width 0) (type default) (color 0 0 0 0))
@@
     (stroke (width 0) (type default) (color 0 0 0 0))
   )
+  (wire (pts (xy 128.27 110.49) (xy 158.75 110.49))
+    (stroke (width 0) (type default) (color 0 0 0 0))
+  )
   (wire (pts (xy 129.54 91.44) (xy 129.54 93.98))
     (stroke (width 0) (type default) (color 0 0 0 0))
   )
+  (wire (pts (xy 39.37 172.72) (xy 39.37 170.18))
+    (stroke (width 0) (type default) (color 0 0 0 0))
+  )
   (bus (pts (xy 125.73 81.28) (xy 125.73 93.98))
     (stroke (width 0) (type default) (color 0 0 0 0))
@@
     (stroke (width 0) (type default) (color 0 0 0 0))
   )
+  (wire (pts (xy 63.5 40.64) (xy 73.66 40.64))
+    (stroke (width 0) (type default) (color 0 0 0 0))
+  )
   (wire (pts (xy 129.54 93.98) (xy 132.08 93.98))
+    (stroke (width 0) (type default) (color 0 0 0 0))
+  )
+  (wire (pts (xy 41.91 172.72) (xy 39.37 172.72))
     (stroke (width 0) (type default) (color 0 0 0 0))
   )
@@
     (effects (font (size 1.27 1.27)) (justify right bottom))
   )
+  (label "~{RAM_CS}" (at 158.75 110.49 180)
+    (effects (font (size 1.27 1.27)) (justify right bottom))
+  )
   (label "A[0..23]" (at 109.22 81.28 0)
     (effects (font (size 1.27 1.27)) (justify left bottom))
@@
   )
   (label "~{ROM_CS}" (at 63.5 38.1 0)
+    (effects (font (size 1.27 1.27)) (justify left bottom))
+  )
+  (label "A15" (at 128.27 110.49 0)
     (effects (font (size 1.27 1.27)) (justify left bottom))
   )
@@
     (effects (font (size 1.27 1.27)) (justify right bottom))
   )
+  (label "~{RAM_CS}" (at 63.5 40.64 0)
+    (effects (font (size 1.27 1.27)) (justify left bottom))
+  )
   (hierarchical_label "A[0..23]" (shape input) (at 44.45 38.1 180)
     (effects (font (size 1.27 1.27)) (justify right))
   )
   (hierarchical_label "~{ROM_CS}" (shape output) (at 73.66 38.1 0)
+    (effects (font (size 1.27 1.27)) (justify left))
+  )
+  (hierarchical_label "~{RAM_CS}" (shape output) (at 73.66 40.64 0)
     (effects (font (size 1.27 1.27)) (justify left))
   )
@@
     (pin "1")
   )
+  (symbol (lib_id "74xx:74LS10") (at 49.53 170.18 0) (unit 3)
+    (in_bom yes) (on_board yes) (fields_autoplaced)
+    (property "Reference" "U27" (id 0) (at 49.53 161.29 0))
+    (property "Value" "74HC10" (id 1) (at 49.53 163.83 0))
+    (property "Footprint" "" (id 2) (at 49.53 170.18 0)
+      (effects (font (size 1.27 1.27)) hide)
+    )
+    (property "Datasheet" "https://www.ti.com/lit/ds/symlink/sn74hc10.pdf" (id 3) (at 49.53 170.18 0)
+      (effects (font (size 1.27 1.27)) hide)
+    )
+    (pin "10")
+    (pin "11")
+    (pin "8")
+    (pin "9")
+  )
   (symbol (lib_id "power:GND") (at 256.54 30.48 0) (unit 1)

Commit message: Update for Episode 16
Parts:
- removed U27: 74HC10, symbol 74xx:74LS10
- added C44, C45, C46, C47: 100n, symbol Device:C_Small
- added U27, U29: 74HC30, symbol 74xx:74LS30
- added U30: 74AHC00, symbol 74xx:74LS00
- added U31: 74AHC32, symbol 74xx:74LS32
- added U32: 74AHC138, symbol 74xx:74LS138
Connections:
- net GND: now also C44.2, C45.2, C46.2, C47.2, U27.7 (GND), U29.7 (GND), U30.7 (GND), U31.7 (GND), U32.8 (GND)
- net VCC: now also C44.1, C45.1, C46.1, C47.1, U27.14 (VCC), U29.14 (VCC), U30.14 (VCC), U31.14 (VCC), U32.16 (VCC)
- net ~{RAM_CS}: now also U31.11
- net ~{ROM_CS}: now also U31.8
- new net: U27.8, U31.12, U31.9, U32.5 (E2)
- new net: U30.11, U31.13
- new net: U30.13, U30.8, U31.10, U32.6 (E3)
- new net: U30.3, U31.1
- new net: U30.6, U31.2
- new net: U29.8, U30.12, U32.4 (E1)
- new net: U31.3, U31.5
- new net A10: U29.5
- new net A11: U29.4
- new net A12: U29.3
- new net A13: U29.2
- new net A14: U29.1
- new net A15: U30.10, U30.9
- new net A4: U32.1 (A0)
- new net A5: U32.2 (A1)
- new net A6: U32.3 (A2)
- new net A7: U29.12
- new net A8: U29.11
- new net A9: U29.6
- new net ~{A16}: U27.12
- new net ~{A17}: U27.11
- new net ~{A18}: U27.6
- new net ~{A19}: U27.5, U31.4
- new net ~{A20}: U27.4, U30.1
- new net ~{A21}: U27.3, U30.2
- new net ~{A22}: U27.2, U30.4
- new net ~{A23}: U27.1, U30.5
- new net ~{EXTRAM_CS}: U31.6
- new net ~{IO0}: U32.15 (O0)
- new net ~{IO1}: U32.14 (O1)
- new net ~{IO2}: U32.13 (O2)
- new net ~{IO3}: U32.12 (O3)
- new net ~{IO4}: U32.11 (O4)
- new net ~{IO5}: U32.10 (O5)
- new net ~{IO6}: U32.9 (O6)
- new net ~{IO7}: U32.7 (O7)
- no-connect marks 2 -> 0
Other:
- moved on the sheet: C40, C41

Commit message: Update for episode 20
Connections:
- net ~{BANK0}: now reaches U27.8, U31.12, U31.9, U32.5 (E2)
Other:
- moved on the sheet: U30C
Changed lines of the file:
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@@
   (title_block
     (title "Address Decoding Module")
-    (date "2022-03-01")
-    (rev "A.19")
+    (date "2022-03-25")
+    (rev "A.20")
     (comment 2 "https://github.com/adrienkohlbecker/65C816")
     (comment 3 "Licensed under CERN-OHL-W v2")
-    (comment 4 "Copyright © 2021 Adrien Kohlbecker")
+    (comment 4 "Copyright © 2022 Adrien Kohlbecker")
   )
   (junction (at 139.7 69.85) (diameter 0) (color 0 0 0 0)
@@
   (junction (at 134.62 172.72) (diameter 0) (color 0 0 0 0)
   )
+  (junction (at 158.75 90.17) (diameter 0) (color 0 0 0 0)
+  )
   (junction (at 100.33 172.72) (diameter 0) (color 0 0 0 0)
   )
@@
   (junction (at 146.05 177.8) (diameter 0) (color 0 0 0 0)
   )
-  (junction (at 161.29 90.17) (diameter 0) (color 0 0 0 0)
-  )
   (junction (at 144.78 64.77) (diameter 0) (color 0 0 0 0)
   )
@@
     (stroke (width 0) (type default) (color 0 0 0 0))
   )
-  (wire (pts (xy 161.29 92.71) (xy 162.56 92.71))
-    (stroke (width 0) (type default) (color 0 0 0 0))
-  )
   (wire (pts (xy 134.62 31.75) (xy 205.74 31.75))
     (stroke (width 0) (type default) (color 0 0 0 0))
@@
     (stroke (width 0) (type default) (color 0 0 0 0))
   )
-  (wire (pts (xy 161.29 90.17) (xy 161.29 87.63))
+  (wire (pts (xy 158.75 90.17) (xy 158.75 87.63))
     (stroke (width 0) (type default) (color 0 0 0 0))
   )
@@
     (stroke (width 0) (type default) (color 0 0 0 0))
   )
-  (wire (pts (xy 123.19 90.17) (xy 161.29 90.17))
+  (wire (pts (xy 123.19 90.17) (xy 158.75 90.17))
     (stroke (width 0) (type default) (color 0 0 0 0))
   )
@@
     (stroke (width 0) (type default) (color 0 0 0 0))
   )
-  (wire (pts (xy 177.8 90.17) (xy 187.96 90.17))
+  (wire (pts (xy 173.99 90.17) (xy 187.96 90.17))
     (stroke (width 0) (type default) (color 0 0 0 0))
   )
@@
     (stroke (width 0) (type default) (color 0 0 0 0))
   )
-  (wire (pts (xy 161.29 90.17) (xy 161.29 92.71))
+  (wire (pts (xy 158.75 90.17) (xy 158.75 92.71))
     (stroke (width 0) (type default) (color 0 0 0 0))
   )
@@
     (stroke (width 0) (type default) (color 0 0 0 0))
   )
-  (wire (pts (xy 161.29 87.63) (xy 162.56 87.63))
-    (stroke (width 0) (type default) (color 0 0 0 0))
-  )
   (label "A12" (at 123.19 102.87 0)
     (effects (font (size 1.27 1.27)) (justify left bottom))
@@
   )
   (label "{ADDRESS}" (at 93.98 59.69 0)
+    (effects (font (size 1.27 1.27)) (justify left bottom))
+  )
+  (label "~{BANK0}" (at 176.53 72.39 0)
     (effects (font (size 1.27 1.27)) (justify left bottom))
   )
@@
     (pin "3")
   )
-  (symbol (lib_id "74xx:74LS00") (at 170.18 90.17 0) (unit 3)
+  (symbol (lib_id "74xx:74LS00") (at 166.37 90.17 0) (unit 3)
     (in_bom yes) (on_board yes) (fields_autoplaced)
-    (property "Reference" "U30" (id 0) (at 170.18 81.28 0))
-    (property "Value" "74AHC00" (id 1) (at 170.18 83.82 0))
-    (property "Footprint" "" (id 2) (at 170.18 90.17 0)
-      (effects (font (size 1.27 1.27)) hide)
-    )
-    (property "Datasheet" "https://www.ti.com/lit/ds/symlink/sn74ahc00.pdf" (id 3) (at 170.18 90.17 0)
-      (effects (font (size 1.27 1.27)) hide)
-    )
+    (property "Reference" "U30" (id 0) (at 166.37 81.28 0))
+    (property "Value" "74AHC00" (id 1) (at 166.37 83.82 0))
+    (property "Footprint" "" (id 2) (at 166.37 90.17 0)
+      (effects (font (size 1.27 1.27)) hide)
+    )
+    (property "Datasheet" "https://www.ti.com/lit/ds/symlink/sn74ahc00.pdf" (id 3) (at 166.37 90.17 0)
+      (effects (font (size 1.27 1.27)) hide)
+    )
