File: hardware/address_decoding.kicad_sch (KiCad schematic)
At the start: 11 parts, among them U27 74HC30, U29 74HC30, U30 74AHC00, U31 74AHC32, U32 74AHC138

Commit message: Renumber
Parts:
- renumbered C40 to C35, C41 to C36, C44 to C37, C45 to C38, C46 to C39, C47 to C40, U27 to U22, U29 to U23, U30 to U24, U31 to U25, U32 to U26
Changed lines of the file:
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@@
   (symbol (lib_id "Device:C_Polarized_Small") (at 100.33 175.26 0) (unit 1)
     (in_bom yes) (on_board yes)
-    (property "Reference" "C40" (id 0) (at 102.87 173.99 0)
+    (property "Reference" "C35" (id 0) (at 102.87 173.99 0)
       (effects (font (size 1.27 1.27)) (justify left))
     )
@@
   (symbol (lib_id "74xx:74LS32") (at 74.93 175.26 0) (unit 5)
     (in_bom yes) (on_board yes)
-    (property "Reference" "U31" (id 0) (at 71.12 166.37 0))
+    (property "Reference" "U25" (id 0) (at 71.12 166.37 0))
     (property "Value" "74AHC32" (id 1) (at 80.01 166.37 0))
     (property "Footprint" "" (id 2) (at 74.93 175.26 0)
@@
   (symbol (lib_id "74xx:74LS32") (at 218.44 99.06 0) (unit 4)
     (in_bom yes) (on_board yes) (fields_autoplaced)
-    (property "Reference" "U31" (id 0) (at 218.44 90.17 0))
+    (property "Reference" "U25" (id 0) (at 218.44 90.17 0))
     (property "Value" "74AHC32" (id 1) (at 218.44 92.71 0))
     (property "Footprint" "" (id 2) (at 218.44 99.06 0)
@@
   (symbol (lib_id "74xx:74LS30") (at 25.4 175.26 0) (unit 2)
     (in_bom yes) (on_board yes)
-    (property "Reference" "U27" (id 0) (at 21.59 166.37 0))
+    (property "Reference" "U22" (id 0) (at 21.59 166.37 0))
     (property "Value" "74HC30" (id 1) (at 30.48 166.37 0))
     (property "Footprint" "" (id 2) (at 25.4 175.26 0)
@@
   (symbol (lib_id "74xx:74LS32") (at 218.44 78.74 0) (unit 3)
     (in_bom yes) (on_board yes) (fields_autoplaced)
-    (property "Reference" "U31" (id 0) (at 218.44 69.85 0))
+    (property "Reference" "U25" (id 0) (at 218.44 69.85 0))
     (property "Value" "74AHC32" (id 1) (at 218.44 72.39 0))
     (property "Footprint" "" (id 2) (at 218.44 78.74 0)
@@
   (symbol (lib_id "74xx:74LS00") (at 58.42 175.26 0) (unit 5)
     (in_bom yes) (on_board yes)
-    (property "Reference" "U30" (id 0) (at 54.61 166.37 0))
+    (property "Reference" "U24" (id 0) (at 54.61 166.37 0))
     (property "Value" "74AHC00" (id 1) (at 63.5 166.37 0))
     (property "Footprint" "" (id 2) (at 58.42 175.26 0)
@@
   (symbol (lib_id "power:GND") (at 210.82 149.86 0) (unit 1)
     (in_bom yes) (on_board yes) (fields_autoplaced)
-    (property "Reference" "#PWR0114" (id 0) (at 210.82 156.21 0)
+    (property "Reference" "#PWR086" (id 0) (at 210.82 156.21 0)
       (effects (font (size 1.27 1.27)) hide)
     )
@@
   (symbol (lib_id "power:VCC") (at 210.82 116.84 0) (unit 1)
     (in_bom yes) (on_board yes) (fields_autoplaced)
-    (property "Reference" "#PWR0113" (id 0) (at 210.82 120.65 0)
+    (property "Reference" "#PWR085" (id 0) (at 210.82 120.65 0)
       (effects (font (size 1.27 1.27)) hide)
     )
@@
   (symbol (lib_id "74xx:74LS00") (at 172.72 43.18 0) (unit 1)
     (in_bom yes) (on_board yes) (fields_autoplaced)
-    (property "Reference" "U30" (id 0) (at 172.72 34.29 0))
+    (property "Reference" "U24" (id 0) (at 172.72 34.29 0))
     (property "Value" "74AHC00" (id 1) (at 172.72 36.83 0))
     (property "Footprint" "" (id 2) (at 172.72 43.18 0)
@@
   (symbol (lib_id "74xx:74LS00") (at 166.37 90.17 0) (unit 3)
     (in_bom yes) (on_board yes) (fields_autoplaced)
-    (property "Reference" "U30" (id 0) (at 166.37 81.28 0))
+    (property "Reference" "U24" (id 0) (at 166.37 81.28 0))
     (property "Value" "74AHC00" (id 1) (at 166.37 83.82 0))
     (property "Footprint" "" (id 2) (at 166.37 90.17 0)
@@
   (symbol (lib_id "power:GND") (at 50.8 190.5 0) (unit 1)
     (in_bom yes) (on_board yes) (fields_autoplaced)
-    (property "Reference" "#PWR0101" (id 0) (at 50.8 196.85 0)
+    (property "Reference" "#PWR082" (id 0) (at 50.8 196.85 0)
       (effects (font (size 1.27 1.27)) hide)
     )
@@
   (symbol (lib_id "power:VCC") (at 50.8 161.29 0) (unit 1)
     (in_bom yes) (on_board yes) (fields_autoplaced)
-    (property "Reference" "#PWR099" (id 0) (at 50.8 165.1 0)
+    (property "Reference" "#PWR081" (id 0) (at 50.8 165.1 0)
       (effects (font (size 1.27 1.27)) hide)
     )
@@
   (symbol (lib_id "power:VCC") (at 100.33 171.45 0) (unit 1)
     (in_bom yes) (on_board yes) (fields_autoplaced)
-    (property "Reference" "#PWR0116" (id 0) (at 100.33 175.26 0)
+    (property "Reference" "#PWR083" (id 0) (at 100.33 175.26 0)
       (effects (font (size 1.27 1.27)) hide)
     )
@@
   (symbol (lib_id "74xx:74LS30") (at 41.91 175.26 0) (unit 2)
     (in_bom yes) (on_board yes)
-    (property "Reference" "U29" (id 0) (at 38.1 166.37 0))
+    (property "Reference" "U23" (id 0) (at 38.1 166.37 0))
     (property "Value" "74HC30" (id 1) (at 46.99 166.37 0))
     (property "Footprint" "" (id 2) (at 41.91 175.26 0)
@@
   (symbol (lib_id "74xx:74LS00") (at 172.72 58.42 0) (unit 2)
     (in_bom yes) (on_board yes) (fields_autoplaced)
-    (property "Reference" "U30" (id 0) (at 172.72 49.53 0))
+    (property "Reference" "U24" (id 0) (at 172.72 49.53 0))
     (property "Value" "74AHC00" (id 1) (at 172.72 52.07 0))
     (property "Footprint" "" (id 2) (at 172.72 58.42 0)
@@
   (symbol (lib_id "74xx:74LS00") (at 196.85 107.95 0) (unit 4)
     (in_bom yes) (on_board yes) (fields_autoplaced)
-    (property "Reference" "U30" (id 0) (at 196.85 99.06 0))
+    (property "Reference" "U24" (id 0) (at 196.85 99.06 0))
     (property "Value" "74AHC00" (id 1) (at 196.85 101.6 0))
     (property "Footprint" "" (id 2) (at 196.85 107.95 0)
@@
   (symbol (lib_id "74xx:74LS30") (at 152.4 72.39 0) (unit 1)
     (in_bom yes) (on_board yes)
-    (property "Reference" "U27" (id 0) (at 152.4 78.74 0))
+    (property "Reference" "U22" (id 0) (at 152.4 78.74 0))
     (property "Value" "74HC30" (id 1) (at 153.67 81.28 0))
     (property "Footprint" "" (id 2) (at 152.4 72.39 0)
@@
   (symbol (lib_id "74xx:74LS32") (at 195.58 50.8 0) (unit 1)
     (in_bom yes) (on_board yes) (fields_autoplaced)
-    (property "Reference" "U31" (id 0) (at 195.58 41.91 0))
+    (property "Reference" "U25" (id 0) (at 195.58 41.91 0))
     (property "Value" "74AHC32" (id 1) (at 195.58 44.45 0))
     (property "Footprint" "" (id 2) (at 195.58 50.8 0)
@@
   (symbol (lib_id "power:GND") (at 100.33 179.07 0) (unit 1)
     (in_bom yes) (on_board yes) (fields_autoplaced)
-    (property "Reference" "#PWR0117" (id 0) (at 100.33 185.42 0)
+    (property "Reference" "#PWR084" (id 0) (at 100.33 185.42 0)
       (effects (font (size 1.27 1.27)) hide)
     )
@@
   (symbol (lib_id "Device:C_Small") (at 157.48 175.26 0) (unit 1)
     (in_bom yes) (on_board yes) (fields_autoplaced)
-    (property "Reference" "C47" (id 0) (at 160.02 173.9962 0)
+    (property "Reference" "C40" (id 0) (at 160.02 173.9962 0)
       (effects (font (size 1.27 1.27)) (justify left))
     )
@@
   (symbol (lib_id "74xx:74LS138") (at 210.82 132.08 0) (unit 1)
     (in_bom yes) (on_board yes) (fields_autoplaced)
-    (property "Reference" "U32" (id 0) (at 212.8394 116.84 0)
+    (property "Reference" "U26" (id 0) (at 212.8394 116.84 0)
       (effects (font (size 1.27 1.27)) (justify left))
     )
@@
   (symbol (lib_id "Device:C_Small") (at 134.62 175.26 0) (unit 1)
     (in_bom yes) (on_board yes) (fields_autoplaced)
-    (property "Reference" "C45" (id 0) (at 137.16 173.9962 0)
+    (property "Reference" "C38" (id 0) (at 137.16 173.9962 0)
       (effects (font (size 1.27 1.27)) (justify left))
     )
@@
   (symbol (lib_id "74xx:74LS30") (at 152.4 105.41 0) (unit 1)
     (in_bom yes) (on_board yes)
-    (property "Reference" "U29" (id 0) (at 152.4 111.76 0))
+    (property "Reference" "U23" (id 0) (at 152.4 111.76 0))
     (property "Value" "74HC30" (id 1) (at 153.67 114.3 0))
     (property "Footprint" "" (id 2) (at 152.4 105.41 0)
@@
   (symbol (lib_id "Device:C_Small") (at 111.76 175.26 0) (unit 1)
     (in_bom yes) (on_board yes) (fields_autoplaced)
-    (property "Reference" "C41" (id 0) (at 114.3 173.9962 0)
+    (property "Reference" "C36" (id 0) (at 114.3 173.9962 0)
       (effects (font (size 1.27 1.27)) (justify left))
     )
@@
   (symbol (lib_id "74xx:74LS32") (at 218.44 43.18 0) (unit 2)
     (in_bom yes) (on_board yes) (fields_autoplaced)
-    (property "Reference" "U31" (id 0) (at 218.44 34.29 0))
+    (property "Reference" "U25" (id 0) (at 218.44 34.29 0))
     (property "Value" "74AHC32" (id 1) (at 218.44 36.83 0))
     (property "Footprint" "" (id 2) (at 218.44 43.18 0)
@@
   (symbol (lib_id "Device:C_Small") (at 146.05 175.26 0) (unit 1)
     (in_bom yes) (on_board yes) (fields_autoplaced)
-    (property "Reference" "C46" (id 0) (at 148.59 173.9962 0)
+    (property "Reference" "C39" (id 0) (at 148.59 173.9962 0)
       (effects (font (size 1.27 1.27)) (justify left))
     )
@@
   (symbol (lib_id "Device:C_Small") (at 123.19 175.26 0) (unit 1)
     (in_bom yes) (on_board yes) (fields_autoplaced)
-    (property "Reference" "C44" (id 0) (at 125.73 173.9962 0)
-      (effects (font (size 1.27 1.27)) (justify left))
-    )
+    (property "Reference" "C37" (id 0) (at 125.73 173.9962 0)
+      (effects (font (size 1.27 1.27)) (justify left))
+    )

Commit message: Snapshot ep 24 work
Parts:
- removed C40: 100n, symbol Device:C_Small
- removed U22: 74HC30, symbol 74xx:74LS30
Connections:
- net ~{A19} renamed A19
- net ~{A20} renamed A20
- net ~{A21} renamed A21
- net ~{A22} renamed A22
- net ~{A23} renamed A23
- no-connect marks 0 -> 3

Commit message: Update main project
Parts:
- renumbered C35 to C1, C36 to C2, C37 to C3, C38 to C4, C39 to C5, U23 to U2, U24 to U3, U25 to U4, U26 to U5
Changed lines of the file:
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@@
   (symbol (lib_id "Device:C_Polarized_Small") (at 100.33 175.26 0) (unit 1)
     (in_bom yes) (on_board yes)
-    (property "Reference" "C35" (id 0) (at 102.87 173.99 0)
+    (property "Reference" "C1" (id 0) (at 102.87 173.99 0)
       (effects (font (size 1.27 1.27)) (justify left))
     )
@@
   (symbol (lib_id "74xx:74LS32") (at 74.93 175.26 0) (unit 5)
     (in_bom yes) (on_board yes)
-    (property "Reference" "U25" (id 0) (at 71.12 166.37 0))
+    (property "Reference" "U4" (id 0) (at 71.12 166.37 0))
     (property "Value" "74AHC32" (id 1) (at 80.01 166.37 0))
     (property "Footprint" "" (id 2) (at 74.93 175.26 0)
@@
   (symbol (lib_id "74xx:74LS32") (at 218.44 99.06 0) (unit 4)
     (in_bom yes) (on_board yes) (fields_autoplaced)
-    (property "Reference" "U25" (id 0) (at 218.44 90.17 0))
+    (property "Reference" "U4" (id 0) (at 218.44 90.17 0))
     (property "Value" "74AHC32" (id 1) (at 218.44 92.71 0))
     (property "Footprint" "" (id 2) (at 218.44 99.06 0)
@@
   (symbol (lib_id "74xx:74LS32") (at 218.44 78.74 0) (unit 3)
     (in_bom yes) (on_board yes) (fields_autoplaced)
-    (property "Reference" "U25" (id 0) (at 218.44 69.85 0))
+    (property "Reference" "U4" (id 0) (at 218.44 69.85 0))
     (property "Value" "74AHC32" (id 1) (at 218.44 72.39 0))
     (property "Footprint" "" (id 2) (at 218.44 78.74 0)
@@
   (symbol (lib_id "74xx:74LS00") (at 58.42 175.26 0) (unit 5)
     (in_bom yes) (on_board yes)
-    (property "Reference" "U24" (id 0) (at 54.61 166.37 0))
+    (property "Reference" "U3" (id 0) (at 54.61 166.37 0))
     (property "Value" "74AHC00" (id 1) (at 63.5 166.37 0))
     (property "Footprint" "" (id 2) (at 58.42 175.26 0)
@@
   (symbol (lib_id "power:GND") (at 210.82 149.86 0) (unit 1)
     (in_bom yes) (on_board yes) (fields_autoplaced)
-    (property "Reference" "#PWR086" (id 0) (at 210.82 156.21 0)
+    (property "Reference" "#PWR011" (id 0) (at 210.82 156.21 0)
       (effects (font (size 1.27 1.27)) hide)
     )
@@
   (symbol (lib_id "power:VCC") (at 210.82 116.84 0) (unit 1)
     (in_bom yes) (on_board yes) (fields_autoplaced)
-    (property "Reference" "#PWR085" (id 0) (at 210.82 120.65 0)
+    (property "Reference" "#PWR010" (id 0) (at 210.82 120.65 0)
       (effects (font (size 1.27 1.27)) hide)
     )
@@
   (symbol (lib_id "74xx:74LS00") (at 172.72 43.18 0) (unit 1)
     (in_bom yes) (on_board yes) (fields_autoplaced)
-    (property "Reference" "U24" (id 0) (at 172.72 34.29 0))
+    (property "Reference" "U3" (id 0) (at 172.72 34.29 0))
     (property "Value" "74AHC00" (id 1) (at 172.72 36.83 0))
     (property "Footprint" "" (id 2) (at 172.72 43.18 0)
@@
   (symbol (lib_id "74xx:74LS00") (at 166.37 90.17 0) (unit 3)
     (in_bom yes) (on_board yes) (fields_autoplaced)
-    (property "Reference" "U24" (id 0) (at 166.37 81.28 0))
+    (property "Reference" "U3" (id 0) (at 166.37 81.28 0))
     (property "Value" "74AHC00" (id 1) (at 166.37 83.82 0))
     (property "Footprint" "" (id 2) (at 166.37 90.17 0)
@@
   (symbol (lib_id "power:GND") (at 50.8 190.5 0) (unit 1)
     (in_bom yes) (on_board yes) (fields_autoplaced)
-    (property "Reference" "#PWR082" (id 0) (at 50.8 196.85 0)
+    (property "Reference" "#PWR07" (id 0) (at 50.8 196.85 0)
       (effects (font (size 1.27 1.27)) hide)
     )
@@
   (symbol (lib_id "power:VCC") (at 50.8 161.29 0) (unit 1)
     (in_bom yes) (on_board yes) (fields_autoplaced)
-    (property "Reference" "#PWR081" (id 0) (at 50.8 165.1 0)
+    (property "Reference" "#PWR06" (id 0) (at 50.8 165.1 0)
       (effects (font (size 1.27 1.27)) hide)
     )
@@
   (symbol (lib_id "power:VCC") (at 100.33 171.45 0) (unit 1)
     (in_bom yes) (on_board yes) (fields_autoplaced)
-    (property "Reference" "#PWR083" (id 0) (at 100.33 175.26 0)
+    (property "Reference" "#PWR08" (id 0) (at 100.33 175.26 0)
       (effects (font (size 1.27 1.27)) hide)
     )
@@
   (symbol (lib_id "74xx:74LS30") (at 41.91 175.26 0) (unit 2)
     (in_bom yes) (on_board yes)
-    (property "Reference" "U23" (id 0) (at 38.1 166.37 0))
+    (property "Reference" "U2" (id 0) (at 38.1 166.37 0))
     (property "Value" "74HC30" (id 1) (at 46.99 166.37 0))
     (property "Footprint" "" (id 2) (at 41.91 175.26 0)
@@
   (symbol (lib_id "74xx:74LS00") (at 172.72 58.42 0) (unit 2)
     (in_bom yes) (on_board yes) (fields_autoplaced)
-    (property "Reference" "U24" (id 0) (at 172.72 49.53 0))
+    (property "Reference" "U3" (id 0) (at 172.72 49.53 0))
     (property "Value" "74AHC00" (id 1) (at 172.72 52.07 0))
     (property "Footprint" "" (id 2) (at 172.72 58.42 0)
@@
   (symbol (lib_id "74xx:74LS00") (at 196.85 107.95 0) (unit 4)
     (in_bom yes) (on_board yes) (fields_autoplaced)
-    (property "Reference" "U24" (id 0) (at 196.85 99.06 0))
+    (property "Reference" "U3" (id 0) (at 196.85 99.06 0))
     (property "Value" "74AHC00" (id 1) (at 196.85 101.6 0))
     (property "Footprint" "" (id 2) (at 196.85 107.95 0)
@@
   (symbol (lib_id "74xx:74LS32") (at 195.58 50.8 0) (unit 1)
     (in_bom yes) (on_board yes) (fields_autoplaced)
-    (property "Reference" "U25" (id 0) (at 195.58 41.91 0))
+    (property "Reference" "U4" (id 0) (at 195.58 41.91 0))
     (property "Value" "74AHC32" (id 1) (at 195.58 44.45 0))
     (property "Footprint" "" (id 2) (at 195.58 50.8 0)
@@
   (symbol (lib_id "power:GND") (at 100.33 179.07 0) (unit 1)
     (in_bom yes) (on_board yes) (fields_autoplaced)
-    (property "Reference" "#PWR084" (id 0) (at 100.33 185.42 0)
+    (property "Reference" "#PWR09" (id 0) (at 100.33 185.42 0)
       (effects (font (size 1.27 1.27)) hide)
     )
@@
   (symbol (lib_id "74xx:74LS138") (at 210.82 132.08 0) (unit 1)
     (in_bom yes) (on_board yes) (fields_autoplaced)
-    (property "Reference" "U26" (id 0) (at 212.8394 116.84 0)
+    (property "Reference" "U5" (id 0) (at 212.8394 116.84 0)
       (effects (font (size 1.27 1.27)) (justify left))
     )
@@
   (symbol (lib_id "Device:C_Small") (at 134.62 175.26 0) (unit 1)
     (in_bom yes) (on_board yes) (fields_autoplaced)
-    (property "Reference" "C38" (id 0) (at 137.16 173.9962 0)
+    (property "Reference" "C4" (id 0) (at 137.16 173.9962 0)
       (effects (font (size 1.27 1.27)) (justify left))
     )
@@
   (symbol (lib_id "74xx:74LS30") (at 152.4 105.41 0) (unit 1)
     (in_bom yes) (on_board yes)
-    (property "Reference" "U23" (id 0) (at 152.4 111.76 0))
+    (property "Reference" "U2" (id 0) (at 152.4 111.76 0))
     (property "Value" "74HC30" (id 1) (at 153.67 114.3 0))
     (property "Footprint" "" (id 2) (at 152.4 105.41 0)
@@
   (symbol (lib_id "Device:C_Small") (at 111.76 175.26 0) (unit 1)
     (in_bom yes) (on_board yes) (fields_autoplaced)
-    (property "Reference" "C36" (id 0) (at 114.3 173.9962 0)
+    (property "Reference" "C2" (id 0) (at 114.3 173.9962 0)
       (effects (font (size 1.27 1.27)) (justify left))
     )
@@
   (symbol (lib_id "74xx:74LS32") (at 218.44 43.18 0) (unit 2)
     (in_bom yes) (on_board yes) (fields_autoplaced)
-    (property "Reference" "U25" (id 0) (at 218.44 34.29 0))
+    (property "Reference" "U4" (id 0) (at 218.44 34.29 0))
     (property "Value" "74AHC32" (id 1) (at 218.44 36.83 0))
     (property "Footprint" "" (id 2) (at 218.44 43.18 0)
@@
   (symbol (lib_id "Device:C_Small") (at 146.05 175.26 0) (unit 1)
     (in_bom yes) (on_board yes) (fields_autoplaced)
-    (property "Reference" "C39" (id 0) (at 148.59 173.9962 0)
+    (property "Reference" "C5" (id 0) (at 148.59 173.9962 0)
       (effects (font (size 1.27 1.27)) (justify left))
     )
@@
   (symbol (lib_id "Device:C_Small") (at 123.19 175.26 0) (unit 1)
     (in_bom yes) (on_board yes) (fields_autoplaced)
-    (property "Reference" "C37" (id 0) (at 125.73 173.9962 0)
-      (effects (font (size 1.27 1.27)) (justify left))
-    )
+    (property "Reference" "C3" (id 0) (at 125.73 173.9962 0)
+      (effects (font (size 1.27 1.27)) (justify left))
+    )
