File: hardware/address_decoding.kicad_sch (KiCad schematic)
At the start: 9 parts, among them U2 74HC30, U3 74AHC00, U4 74AHC32, U5 74AHC138

Commit message: Add 65C51
Connections:
- net ~{IO0} renamed ~{IO_0}
- net ~{IO1} renamed ~{IO_1}
- net ~{IO2} renamed ~{IO_2}
- net ~{IO3} renamed ~{IO_3}
- net ~{IO4} renamed ~{IO_4}
- net ~{IO5} renamed ~{IO_5}
- net ~{IO6} renamed ~{IO_6}
- net ~{IO7} renamed ~{IO_7}
Changed lines of the file:
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@@
   (title_block
     (title "Address Decoding Module")
-    (date "2022-09-03")
-    (rev "A.28")
+    (date "2022-09-26")
+    (rev "A.30")
     (comment 2 "https://github.com/adrienkohlbecker/65C816")
     (comment 3 "Licensed under CERN-OHL-W v2")
@@
     (effects (font (size 1.27 1.27)) (justify left bottom))
   )
-  (label "~{IO0}" (at 46.99 34.29 0)
-    (effects (font (size 1.27 1.27)) (justify left bottom))
-  )
-  (label "~{IO0}" (at 234.95 124.46 180)
+  (label "~{IO_0}" (at 46.99 34.29 0)
+    (effects (font (size 1.27 1.27)) (justify left bottom))
+  )
+  (label "~{IO_0}" (at 234.95 124.46 180)
     (effects (font (size 1.27 1.27)) (justify right bottom))
   )
@@
     (effects (font (size 1.27 1.27)) (justify left bottom))
   )
-  (label "~{IO5}" (at 234.95 137.16 180)
+  (label "~{IO_5}" (at 234.95 137.16 180)
     (effects (font (size 1.27 1.27)) (justify right bottom))
   )
@@
     (effects (font (size 1.27 1.27)) (justify right bottom))
   )
-  (label "~{IO6}" (at 234.95 139.7 180)
-    (effects (font (size 1.27 1.27)) (justify right bottom))
-  )
-  (label "~{IO1}" (at 46.99 36.83 0)
+  (label "~{IO_6}" (at 234.95 139.7 180)
+    (effects (font (size 1.27 1.27)) (justify right bottom))
+  )
+  (label "~{IO_1}" (at 46.99 36.83 0)
     (effects (font (size 1.27 1.27)) (justify left bottom))
   )
@@
     (effects (font (size 1.27 1.27)) (justify left bottom))
   )
-  (label "~{IO6}" (at 46.99 49.53 0)
+  (label "~{IO_6}" (at 46.99 49.53 0)
     (effects (font (size 1.27 1.27)) (justify left bottom))
   )
@@
     (effects (font (size 1.27 1.27)) (justify left bottom))
   )
-  (label "~{IO3}" (at 46.99 41.91 0)
+  (label "~{IO_3}" (at 46.99 41.91 0)
     (effects (font (size 1.27 1.27)) (justify left bottom))
   )
@@
     (effects (font (size 1.27 1.27)) (justify left bottom))
   )
-  (label "~{IO3}" (at 234.95 132.08 180)
+  (label "~{IO_3}" (at 234.95 132.08 180)
     (effects (font (size 1.27 1.27)) (justify right bottom))
   )
@@
     (effects (font (size 1.27 1.27)) (justify left bottom))
   )
-  (label "~{IO7}" (at 234.95 142.24 180)
-    (effects (font (size 1.27 1.27)) (justify right bottom))
-  )
-  (label "~{IO4}" (at 46.99 44.45 0)
+  (label "~{IO_7}" (at 234.95 142.24 180)
+    (effects (font (size 1.27 1.27)) (justify right bottom))
+  )
+  (label "~{IO_4}" (at 46.99 44.45 0)
     (effects (font (size 1.27 1.27)) (justify left bottom))
   )
@@
     (effects (font (size 1.27 1.27)) (justify left bottom))
   )
-  (label "~{IO7}" (at 46.99 52.07 0)
+  (label "~{IO_7}" (at 46.99 52.07 0)
     (effects (font (size 1.27 1.27)) (justify left bottom))
   )
@@
     (effects (font (size 1.27 1.27)) (justify left bottom))
   )
-  (label "~{IO2}" (at 234.95 129.54 180)
+  (label "~{IO_2}" (at 234.95 129.54 180)
     (effects (font (size 1.27 1.27)) (justify right bottom))
   )
@@
     (effects (font (size 1.27 1.27)) (justify left bottom))
   )
-  (label "~{IO1}" (at 234.95 127 180)
-    (effects (font (size 1.27 1.27)) (justify right bottom))
-  )
-  (label "~{IO2}" (at 46.99 39.37 0)
-    (effects (font (size 1.27 1.27)) (justify left bottom))
-  )
-  (label "~{IO4}" (at 234.95 134.62 180)
+  (label "~{IO_1}" (at 234.95 127 180)
+    (effects (font (size 1.27 1.27)) (justify right bottom))
+  )
+  (label "~{IO_2}" (at 46.99 39.37 0)
+    (effects (font (size 1.27 1.27)) (justify left bottom))
+  )
+  (label "~{IO_4}" (at 234.95 134.62 180)
     (effects (font (size 1.27 1.27)) (justify right bottom))
   )
@@
     (effects (font (size 1.27 1.27)) (justify left bottom))
   )
-  (label "~{IO5}" (at 46.99 46.99 0)
+  (label "~{IO_5}" (at 46.99 46.99 0)
     (effects (font (size 1.27 1.27)) (justify left bottom))
   )
@@
     (effects (font (size 1.27 1.27)) (justify left bottom))
   )
-  (hierarchical_label "~{IO6}" (shape output) (at 59.69 49.53 0)
+  (hierarchical_label "~{IO_6}" (shape output) (at 59.69 49.53 0)
     (effects (font (size 1.27 1.27)) (justify left))
   )
@@
     (effects (font (size 1.27 1.27)) (justify right))
   )
-  (hierarchical_label "~{IO0}" (shape output) (at 59.69 34.29 0)
-    (effects (font (size 1.27 1.27)) (justify left))
-  )
-  (hierarchical_label "~{IO3}" (shape output) (at 59.69 41.91 0)
-    (effects (font (size 1.27 1.27)) (justify left))
-  )
-  (hierarchical_label "~{IO5}" (shape output) (at 59.69 46.99 0)
+  (hierarchical_label "~{IO_0}" (shape output) (at 59.69 34.29 0)
+    (effects (font (size 1.27 1.27)) (justify left))
+  )
+  (hierarchical_label "~{IO_3}" (shape output) (at 59.69 41.91 0)
+    (effects (font (size 1.27 1.27)) (justify left))
+  )
+  (hierarchical_label "~{IO_5}" (shape output) (at 59.69 46.99 0)
     (effects (font (size 1.27 1.27)) (justify left))
   )
@@
     (effects (font (size 1.27 1.27)) (justify left))
   )
-  (hierarchical_label "~{IO2}" (shape output) (at 59.69 39.37 0)
+  (hierarchical_label "~{IO_2}" (shape output) (at 59.69 39.37 0)
     (effects (font (size 1.27 1.27)) (justify left))
   )
@@
     (effects (font (size 1.27 1.27)) (justify left))
   )
-  (hierarchical_label "~{IO7}" (shape output) (at 59.69 52.07 0)
-    (effects (font (size 1.27 1.27)) (justify left))
-  )
-  (hierarchical_label "~{IO4}" (shape output) (at 59.69 44.45 0)
-    (effects (font (size 1.27 1.27)) (justify left))
-  )
-  (hierarchical_label "~{IO1}" (shape output) (at 59.69 36.83 0)
-    (effects (font (size 1.27 1.27)) (justify left))
-  )
+  (hierarchical_label "~{IO_7}" (shape output) (at 59.69 52.07 0)
+    (effects (font (size 1.27 1.27)) (justify left))
+  )
+  (hierarchical_label "~{IO_4}" (shape output) (at 59.69 44.45 0)
+    (effects (font (size 1.27 1.27)) (justify left))
+  )
+  (hierarchical_label "~{IO_1}" (shape output) (at 59.69 36.83 0)
+    (effects (font (size 1.27 1.27)) (justify left))
+  )
