File: hardware/address_decoding.kicad_sch (KiCad schematic)
At the start: 9 parts, among them U2 74HC30, U3 74AHC00, U4 74AHC32, U5 74AHC138

Commit message: Update schematic
Connections:
- no-connect marks 3 -> 0
Changed lines of the file:
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@@
   (title_block
     (title "Address Decoding Module")
-    (date "2022-09-26")
-    (rev "A.30")
+    (date "2023-02-24")
+    (rev "A.31")
     (comment 2 "https://github.com/adrienkohlbecker/65C816")
     (comment 3 "Licensed under CERN-OHL-W v2")
@@
   (junction (at 111.76 172.72) (diameter 0) (color 0 0 0 0)
   )
-  (no_connect (at 134.62 77.47))
-  (no_connect (at 134.62 82.55))
-  (no_connect (at 134.62 80.01))
   (bus_entry (at 120.65 105.41) (size 2.54 2.54)
     (stroke (width 0) (type default) (color 0 0 0 0))
@@
     (stroke (width 0) (type default) (color 0 0 0 0))
   )
-  (bus_entry (at 120.65 74.93) (size 2.54 2.54)
-    (stroke (width 0) (type default) (color 0 0 0 0))
-  )
   (bus_entry (at 120.65 102.87) (size 2.54 2.54)
     (stroke (width 0) (type default) (color 0 0 0 0))
   )
-  (bus_entry (at 120.65 80.01) (size 2.54 2.54)
-    (stroke (width 0) (type default) (color 0 0 0 0))
-  )
-  (bus_entry (at 120.65 77.47) (size 2.54 2.54)
-    (stroke (width 0) (type default) (color 0 0 0 0))
-  )
   (bus_entry (at 120.65 87.63) (size 2.54 2.54)
     (stroke (width 0) (type default) (color 0 0 0 0))
@@
     (stroke (width 0) (type default) (color 0 0 0 0))
   )
-  (wire (pts (xy 123.19 82.55) (xy 134.62 82.55))
-    (stroke (width 0) (type default) (color 0 0 0 0))
-  )
   (bus (pts (xy 120.65 102.87) (xy 120.65 105.41))
     (stroke (width 0) (type default) (color 0 0 0 0))
@@
     (stroke (width 0) (type default) (color 0 0 0 0))
   )
-  (wire (pts (xy 123.19 77.47) (xy 134.62 77.47))
-    (stroke (width 0) (type default) (color 0 0 0 0))
-  )
   (wire (pts (xy 59.69 52.07) (xy 46.99 52.07))
     (stroke (width 0) (type default) (color 0 0 0 0))
   )
   (bus (pts (xy 93.98 59.69) (xy 120.65 59.69))
-    (stroke (width 0) (type default) (color 0 0 0 0))
-  )
-  (wire (pts (xy 123.19 80.01) (xy 134.62 80.01))
     (stroke (width 0) (type default) (color 0 0 0 0))
   )
@@
     (effects (font (size 1.27 1.27)) (justify left bottom))
   )
-  (label "A16" (at 123.19 82.55 0)
-    (effects (font (size 1.27 1.27)) (justify left bottom))
-  )
   (label "~{IO_5}" (at 234.95 137.16 180)
     (effects (font (size 1.27 1.27)) (justify right bottom))
   )
-  (label "A18" (at 123.19 77.47 0)
-    (effects (font (size 1.27 1.27)) (justify left bottom))
-  )
-  (label "A17" (at 123.19 80.01 0)
-    (effects (font (size 1.27 1.27)) (justify left bottom))
-  )
   (label "A[0..23]" (at 39.37 25.4 180)

Commit message: CLeanup
Changed lines of the file:
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@@
-    (stroke (width 0) (type default) (color 0 0 0 0))
-  )
-  (bus (pts (xy 120.65 80.01) (xy 120.65 87.63))
     (stroke (width 0) (type default) (color 0 0 0 0))
   )
@@
     (stroke (width 0) (type default) (color 0 0 0 0))
   )
-  (bus (pts (xy 120.65 74.93) (xy 120.65 77.47))
+  (bus (pts (xy 120.65 72.39) (xy 120.65 87.63))
     (stroke (width 0) (type default) (color 0 0 0 0))
   )
@@
     (stroke (width 0) (type default) (color 0 0 0 0))
   )
-  (bus (pts (xy 120.65 72.39) (xy 120.65 74.93))
-    (stroke (width 0) (type default) (color 0 0 0 0))
-  )
   (wire (pts (xy 205.74 50.8) (xy 205.74 45.72))
     (stroke (width 0) (type default) (color 0 0 0 0))
@@
     (stroke (width 0) (type default) (color 0 0 0 0))
   )
-  (bus (pts (xy 120.65 77.47) (xy 120.65 80.01))
-    (stroke (width 0) (type default) (color 0 0 0 0))
-  )
