File: hardware/monitor.kicad_sch (KiCad schematic)
At the start: 1 part, among them U33 Teensy++2.0

Commit message: Update for episode 18
Connections:
- net GND: now also U33.32 (AREF), U33.33 (GND)
- net SYNC: now reaches U33.2 (27_PWM)
- net VA: now reaches U33.42 (26_PWM)
- no-connect marks 5 -> 1
Changed lines of the file:
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@@
 (kicad_sch (version 20211123) (generator eeschema)
   (paper "A4")
+  (title_block
+    (date "2022-02-21")
+    (rev "A.18")
+    (comment 2 "https://github.com/adrienkohlbecker/65C816")
+    (comment 3 "Licensed under CERN-OHL-W v2")
+    (comment 4 "Copyright © 2021 Adrien Kohlbecker")
+  )
+  (junction (at 165.1 88.9) (diameter 0) (color 0 0 0 0)
+  )
   (junction (at 119.38 46.99) (diameter 0) (color 0 0 0 0)
   )
-  (no_connect (at 163.83 66.04))
-  (no_connect (at 163.83 88.9))
-  (no_connect (at 163.83 91.44))
-  (no_connect (at 128.27 66.04))
   (no_connect (at 163.83 63.5))
   (bus_entry (at 173.99 96.52) (size -2.54 2.54)
@@
     (stroke (width 0) (type default) (color 0 0 0 0))
   )
-  (bus (pts (xy 33.02 30.48) (xy 48.26 30.48))
+  (wire (pts (xy 33.02 29.21) (xy 48.26 29.21))
+    (stroke (width 0) (type default) (color 0 0 0 0))
+  )
+  (bus (pts (xy 33.02 39.37) (xy 48.26 39.37))
+    (stroke (width 0) (type default) (color 0 0 0 0))
+  )
+  (wire (pts (xy 121.92 66.04) (xy 128.27 66.04))
     (stroke (width 0) (type default) (color 0 0 0 0))
   )
@@
     (stroke (width 0) (type default) (color 0 0 0 0))
   )
+  (wire (pts (xy 165.1 88.9) (xy 179.07 88.9))
+    (stroke (width 0) (type default) (color 0 0 0 0))
+  )
   (bus (pts (xy 119.38 114.3) (xy 119.38 133.35))
     (stroke (width 0) (type default) (color 0 0 0 0))
@@
     (stroke (width 0) (type default) (color 0 0 0 0))
   )
+  (wire (pts (xy 163.83 66.04) (xy 171.45 66.04))
+    (stroke (width 0) (type default) (color 0 0 0 0))
+  )
   (bus (pts (xy 119.38 99.06) (xy 119.38 101.6))
     (stroke (width 0) (type default) (color 0 0 0 0))
@@
     (stroke (width 0) (type default) (color 0 0 0 0))
   )
+  (wire (pts (xy 165.1 91.44) (xy 165.1 88.9))
+    (stroke (width 0) (type default) (color 0 0 0 0))
+  )
   (wire (pts (xy 121.92 109.22) (xy 128.27 109.22))
     (stroke (width 0) (type default) (color 0 0 0 0))
@@
     (stroke (width 0) (type default) (color 0 0 0 0))
   )
+  (wire (pts (xy 115.57 63.5) (xy 128.27 63.5))
+    (stroke (width 0) (type default) (color 0 0 0 0))
+  )
   (bus (pts (xy 173.99 46.99) (xy 173.99 66.04))
     (stroke (width 0) (type default) (color 0 0 0 0))
@@
     (stroke (width 0) (type default) (color 0 0 0 0))
   )
+  (wire (pts (xy 163.83 91.44) (xy 165.1 91.44))
+    (stroke (width 0) (type default) (color 0 0 0 0))
+  )
   (wire (pts (xy 121.92 91.44) (xy 128.27 91.44))
     (stroke (width 0) (type default) (color 0 0 0 0))
@@
     (stroke (width 0) (type default) (color 0 0 0 0))
   )
+  (wire (pts (xy 163.83 88.9) (xy 165.1 88.9))
+    (stroke (width 0) (type default) (color 0 0 0 0))
+  )
   (wire (pts (xy 121.92 81.28) (xy 128.27 81.28))
     (stroke (width 0) (type default) (color 0 0 0 0))
@@
     (stroke (width 0) (type default) (color 0 0 0 0))
   )
-  (bus (pts (xy 33.02 33.02) (xy 48.26 33.02))
+  (bus (pts (xy 33.02 41.91) (xy 48.26 41.91))
     (stroke (width 0) (type default) (color 0 0 0 0))
   )
@@
     (stroke (width 0) (type default) (color 0 0 0 0))
   )
+  (wire (pts (xy 33.02 33.02) (xy 48.26 33.02))
+    (stroke (width 0) (type default) (color 0 0 0 0))
+  )
   (bus (pts (xy 173.99 104.14) (xy 173.99 106.68))
     (stroke (width 0) (type default) (color 0 0 0 0))
@@
   (label "A5" (at 121.92 78.74 0)
     (effects (font (size 1.27 1.27)) (justify left bottom))
+  )
+  (label "VA" (at 171.45 66.04 180)
+    (effects (font (size 1.27 1.27)) (justify right bottom))
   )
   (label "D6" (at 121.92 96.52 0)
@@
     (effects (font (size 1.27 1.27)) (justify left bottom))
   )
+  (label "VA" (at 48.26 33.02 180)
+    (effects (font (size 1.27 1.27)) (justify right bottom))
+  )
   (label "~{A23}" (at 167.64 68.58 0)
     (effects (font (size 1.27 1.27)) (justify left bottom))
@@
     (effects (font (size 1.27 1.27)) (justify left bottom))
   )
-  (label "{ADDRESS}" (at 48.26 30.48 180)
+  (label "{ADDRESS}" (at 48.26 39.37 180)
     (effects (font (size 1.27 1.27)) (justify right bottom))
   )
@@
     (effects (font (size 1.27 1.27)) (justify left bottom))
   )
+  (label "SYNC" (at 121.92 66.04 0)
+    (effects (font (size 1.27 1.27)) (justify left bottom))
+  )
   (label "~{A22}" (at 167.64 71.12 0)
     (effects (font (size 1.27 1.27)) (justify left bottom))
@@
     (effects (font (size 1.27 1.27)) (justify left bottom))
   )
+  (label "SYNC" (at 48.26 29.21 180)
+    (effects (font (size 1.27 1.27)) (justify right bottom))
+  )
   (label "D5" (at 121.92 99.06 0)
     (effects (font (size 1.27 1.27)) (justify left bottom))
   )
-  (label "D[0..7]" (at 48.26 33.02 180)
+  (label "D[0..7]" (at 48.26 41.91 180)
     (effects (font (size 1.27 1.27)) (justify right bottom))
   )
@@
     (effects (font (size 1.27 1.27)) (justify right))
   )
-  (hierarchical_label "{ADDRESS}" (shape input) (at 33.02 30.48 180)
+  (hierarchical_label "VA" (shape input) (at 33.02 33.02 180)
     (effects (font (size 1.27 1.27)) (justify right))
   )
-  (hierarchical_label "D[0..7]" (shape input) (at 33.02 33.02 180)
+  (hierarchical_label "{ADDRESS}" (shape input) (at 33.02 39.37 180)
     (effects (font (size 1.27 1.27)) (justify right))
+  )
+  (hierarchical_label "D[0..7]" (shape input) (at 33.02 41.91 180)
+    (effects (font (size 1.27 1.27)) (justify right))
+  )
+  (hierarchical_label "SYNC" (shape input) (at 33.02 29.21 180)
+    (effects (font (size 1.27 1.27)) (justify right))
+  )
+  (symbol (lib_id "power:GND") (at 179.07 88.9 0) (unit 1)
+    (in_bom yes) (on_board yes) (fields_autoplaced)
+    (property "Reference" "#PWR0102" (id 0) (at 179.07 95.25 0)
+      (effects (font (size 1.27 1.27)) hide)
+    )
+    (property "Value" "GND" (id 1) (at 179.07 93.98 0))
+    (property "Footprint" "" (id 2) (at 179.07 88.9 0)
+      (effects (font (size 1.27 1.27)) hide)
+    )
+    (property "Datasheet" "" (id 3) (at 179.07 88.9 0)
+      (effects (font (size 1.27 1.27)) hide)
+    )
+    (pin "1")
   )
   (symbol (lib_id "65C816:Teensy++2.0") (at 146.05 97.79 0) (unit 1)
@@
     (pin "9")
   )
-  (symbol (lib_id "power:GND") (at 128.27 63.5 270) (unit 1)
+  (symbol (lib_id "power:GND") (at 115.57 63.5 0) (unit 1)
     (in_bom yes) (on_board yes) (fields_autoplaced)
-    (property "Reference" "#PWR025" (id 0) (at 121.92 63.5 0)
+    (property "Reference" "#PWR025" (id 0) (at 115.57 69.85 0)
       (effects (font (size 1.27 1.27)) hide)
     )
-    (property "Value" "GND" (id 1) (at 124.46 63.4999 90)
-      (effects (font (size 1.27 1.27)) (justify right))
-    )
-    (property "Footprint" "" (id 2) (at 128.27 63.5 0)
+    (property "Value" "GND" (id 1) (at 115.57 68.58 0))
+    (property "Footprint" "" (id 2) (at 115.57 63.5 0)
       (effects (font (size 1.27 1.27)) hide)
     )
-    (property "Datasheet" "" (id 3) (at 128.27 63.5 0)
+    (property "Datasheet" "" (id 3) (at 115.57 63.5 0)
       (effects (font (size 1.27 1.27)) hide)
     )

Commit message: Update for episode 19
Connections:
- net CLK is gone; now on net MONCLK: U33.3 (0_INT0_PWM)
Changed lines of the file:
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@@
   (paper "A4")
   (title_block
-    (date "2022-02-21")
-    (rev "A.18")
+    (date "2022-03-01")
+    (rev "A.19")
     (comment 2 "https://github.com/adrienkohlbecker/65C816")
     (comment 3 "Licensed under CERN-OHL-W v2")
@@
     (effects (font (size 1.27 1.27)) (justify right bottom))
   )
-  (label "CLK" (at 121.92 68.58 0)
-    (effects (font (size 1.27 1.27)) (justify left bottom))
-  )
+  (label "MONCLK" (at 121.92 68.58 0)
+    (effects (font (size 1.27 1.27)) (justify left bottom))
+  )

Commit message: More episode 19 updates
Other:
- note added: "Note: Do not connect the +5V pin comming from USB power, as the project is already powered by your power supply. It could break either your USB port or bench power supply."
Changed lines of the file:
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@@
     (stroke (width 0) (type default) (color 0 0 0 0))
   )
-  (bus (pts (xy 80.01 133.35) (xy 119.38 133.35))
+  (bus (pts (xy 86.36 133.35) (xy 119.38 133.35))
     (stroke (width 0) (type default) (color 0 0 0 0))
   )
@@
   (wire (pts (xy 121.92 106.68) (xy 128.27 106.68))
     (stroke (width 0) (type default) (color 0 0 0 0))
+  )
+  (text "Note: Do not connect the +5V pin comming from USB power,\nas the project is already powered by your power supply.\nIt could break either your USB port or bench power supply."
+    (at 191.77 62.23 0)
+    (effects (font (size 1.27 1.27)) (justify left bottom))
   )
   (label "R~{W}" (at 121.92 71.12 0)
@@
     (effects (font (size 1.27 1.27)) (justify left bottom))
   )
-  (label "D[0..7]" (at 80.01 133.35 0)
+  (label "D[0..7]" (at 86.36 133.35 0)
     (effects (font (size 1.27 1.27)) (justify left bottom))
   )

Commit message: Update for episode 20
Connections:
- net A0: now also U33.3 (D0_0_INT0_PWM); no longer U33.12 (9)
- net A1: now also U33.4 (D1_1_INT1_PWM); no longer U33.11 (8)
- net A10: now also U33.29 (F2_40_A2); no longer U33.26 (43_A5)
- net A11: now also U33.28 (F3_41_A3); no longer U33.27 (42_A4)
- net A12: now also U33.27 (F4_42_A4); no longer U33.28 (41_A3)
- net A13: now also U33.26 (F5_43_A5); no longer U33.29 (40_A2)
- net A14: now also U33.25 (F6_44_A6); no longer U33.30 (39_A1)
- net A15: now also U33.24 (F7_45_A7); no longer U33.31 (38_A0)
- net A2: now also U33.5 (D2_2_INT2_RX); no longer U33.10 (7)
- net A3: now also U33.6 (D3_3_INT3_TX); no longer U33.9 (6_LED)
- net A4: now also U33.7 (D4_4); no longer U33.8 (5)
- net A5: now also U33.8 (D5_5); no longer U33.7 (4)
- net A6: now also U33.9 (D6_6_LED); no longer U33.6 (3_INT3_TX)
- net A7: now also U33.10 (D7_7); no longer U33.5 (2_INT2_RX)
- net A8: now also U33.31 (F0_38_A0); no longer U33.24 (45_A7)
- net A9: now also U33.30 (F1_39_A1); no longer U33.25 (44_A6)
- net D0: now also U33.13 (C0_10); no longer U33.20 (17)
- net D1: now also U33.14 (C1_11); no longer U33.19 (16_PWM)
- net D2: now also U33.15 (C2_12); no longer U33.18 (15_PWM)
- net D3: now also U33.16 (C3_13); no longer U33.17 (14_PWM)
- net D4: now also U33.17 (C4_14_PWM); no longer U33.16 (13)
- net D5: now also U33.18 (C5_15_PWM); no longer U33.15 (12)
- net D6: now also U33.19 (C6_16_PWM); no longer U33.14 (11)
- net D7: now also U33.20 (C7_17); no longer U33.13 (10)
- net GND: no longer U33.32 (AREF)
- net MONCLK: now also U33.34 (E6_18_INT6); no longer U33.3 (0_INT0_PWM)
- net R~{W}: now also U33.11 (E0_8); no longer U33.4 (1_INT1_PWM)
- net SYNC: now also U33.12 (E1_9); no longer U33.2 (27_PWM)
- net VA: now also U33.35 (E7_19_INT7); no longer U33.42 (26_PWM)
- net ~{A16}: now also U33.36 (B0_20); no longer U33.34 (18_INT6)
- net ~{A17}: now also U33.37 (B1_21); no longer U33.35 (19_INT7)
- net ~{A18}: now also U33.38 (B2_22); no longer U33.36 (20)
- net ~{A19}: now also U33.39 (B3_23); no longer U33.37 (21)
- net ~{A20}: now also U33.40 (B4_24_PWM); no longer U33.38 (22)
- net ~{A21}: now also U33.41 (B5_25_PWM); no longer U33.39 (23)
- net ~{A22}: now also U33.42 (B6_26_PWM); no longer U33.40 (24_PWM)
- net ~{A23}: now also U33.2 (B7_27_PWM); no longer U33.41 (25_PWM)
- no-connect marks 1 -> 2
Other:
- note added: "Note: Do not connect the +5V pin coming from USB power, as the project is already powered by your power supply. It could break either your USB port or bench power supply."
- note removed: "Note: Do not connect the +5V pin comming from USB power, as the project is already powered by your power supply. It could break either your USB port or bench power supply."
- moved on the sheet: U33

Commit message: Updates for episode 20
Other:
- note added: "Note: Do not connect the +5V pin coming from USB power, as the project is already powered by your bench power supply. It could break either your USB port or bench power supply."
- note removed: "Note: Do not connect the +5V pin coming from USB power, as the project is already powered by your power supply. It could break either your USB port or bench power supply."
Changed lines of the file:
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@@
     )
   )
-  (text "Note: Do not connect the +5V pin coming from USB power,\nas the project is already powered by your power supply.\nIt could break either your USB port or bench power supply."
+  (text "Note: Do not connect the +5V pin coming from USB power,\nas the project is already powered by your bench power supply.\nIt could break either your USB port or bench power supply."
     (at 187.96 50.8 0)
     (effects (font (size 1.27 1.27)) (justify left bottom))

Commit message: Update for episode 21
Other:
- title: (none) -> Monitor Module
Changed lines of the file:
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@@
   (paper "A4")
   (title_block
-    (date "2022-03-25")
-    (rev "A.20")
+    (title "Monitor Module")
+    (date "2022-04-15")
+    (rev "A.21")
     (comment 2 "https://github.com/adrienkohlbecker/65C816")
     (comment 3 "Licensed under CERN-OHL-W v2")

Commit message: Renumber
Parts:
- renumbered U33 to U36
Changed lines of the file:
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@@
   (symbol (lib_id "power:GND") (at 181.61 88.9 0) (unit 1)
     (in_bom yes) (on_board yes) (fields_autoplaced)
-    (property "Reference" "#PWR0102" (id 0) (at 181.61 95.25 0)
+    (property "Reference" "#PWR0125" (id 0) (at 181.61 95.25 0)
       (effects (font (size 1.27 1.27)) hide)
     )
@@
   (symbol (lib_id "65C816:Teensy++2.0") (at 146.05 97.79 0) (unit 1)
     (in_bom yes) (on_board yes)
-    (property "Reference" "U33" (id 0) (at 133.35 58.42 0)
+    (property "Reference" "U36" (id 0) (at 133.35 58.42 0)
       (effects (font (size 1.524 1.524)) (justify left))
     )
@@
   (symbol (lib_id "power:GND") (at 115.57 63.5 0) (unit 1)
     (in_bom yes) (on_board yes) (fields_autoplaced)
-    (property "Reference" "#PWR025" (id 0) (at 115.57 69.85 0)
+    (property "Reference" "#PWR0124" (id 0) (at 115.57 69.85 0)
       (effects (font (size 1.27 1.27)) hide)
     )
