File: hardware/monitor.kicad_sch (KiCad schematic)
At the start: 2 parts, among them U25 Teensy++2.0

Commit message: Rename
Parts:
- U25: footprint 65C816:Teensy2.0++ -> BB816:Teensy2.0++; symbol 65C816:Teensy++2.0 -> BB816:Teensy++2.0
Changed lines of the file:
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@@
   (title_block
     (title "Monitor Module")
-    (date "2023-05-14")
+    (date "2023-05-23")
     (rev "A.32")
-    (comment 2 "https://github.com/adrienkohlbecker/65C816")
+    (comment 2 "https://github.com/adrienkohlbecker/BB816")
     (comment 3 "Licensed under CERN-OHL-W v2")
-    (comment 4 "Copyright © 2022 Adrien Kohlbecker")
+    (comment 4 "Copyright © 2022-2023 Adrien Kohlbecker")
   )
   (junction (at 119.38 46.99) (diameter 0) (color 0 0 0 0)
@@
     (pin "1")
   )
-  (symbol (lib_id "65C816:Teensy++2.0") (at 146.05 97.79 0) (unit 1)
+  (symbol (lib_id "BB816:Teensy++2.0") (at 146.05 97.79 0) (unit 1)
     (in_bom yes) (on_board yes)
     (property "Reference" "U25" (id 0) (at 133.35 58.42 0)
@@
       (effects (font (size 1.524 1.524)) (justify left))
     )
-    (property "Footprint" "65C816:Teensy2.0++" (id 2) (at 148.0694 59.69 0)
+    (property "Footprint" "BB816:Teensy2.0++" (id 2) (at 148.0694 59.69 0)
       (effects (font (size 1.524 1.524)) (justify left) hide)
     )

Commit message: Kicad 7
Parts:
- U25: footprint BB816:Teensy2.0++ -> 65C816:Teensy2.0++
