File: hardware/breakout.kicad_sch (KiCad schematic)
At the start: 16 parts, among them J1 Jack-DC, J5 Conn_01x13, J6 Conn_01x40, J7 Conn_01x10, U1 W65C816SxP

Commit message: Snapshot ep 24 work
Connections:
- net E: now also J5.8 (Pin_8)
Changed lines of the file:
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@@
+    (effects (font (size 1.27 1.27)) (justify left bottom))
+  )
+  (label "E" (at 209.55 43.18 0)
     (effects (font (size 1.27 1.27)) (justify left bottom))
   )

Commit message: More updates
Parts:
- removed F1: Fuse, symbol Device:Fuse
- removed J5: Conn_01x13, symbol Connector_Generic:Conn_01x13
- added J5: Conn_01x12, symbol Connector_Generic:Conn_01x12
Connections:
- net +5V is gone; now on net VCC: C1.1, J1.1, J6.1 (Pin_1)
- net E: now also J5.7 (Pin_7)
- net GND: now also J5.12 (Pin_12)
- net MX: now also J5.8 (Pin_8), J5.9 (Pin_9)
- net RDY⎒: now also J5.3 (Pin_3)
- net RST: now also J5.2 (Pin_2)
- net VDA: now also J5.4 (Pin_4)
- net VPA: now also J5.5 (Pin_5)
- net ~{ABORT}: now also J5.6 (Pin_6)
- net ~{CLK}: now also J5.1 (Pin_1)
- net ~{ML}: now also J5.11 (Pin_11)
- net ~{VP}: now also J5.10 (Pin_10)
- net CLK_IN renamed CLK_SRC
Other:
- sheet Clock & Reset ports: added CLK_SRC; removed 8MHz, CLK
- sheet Glue Logic ports: added CLK_SRC; removed CLK_IN

Commit message: Updates for episode 25
Parts:
- removed J5: Conn_01x12, symbol Connector_Generic:Conn_01x12
- added J5: Conn_01x13, symbol Connector_Generic:Conn_01x13
Connections:
- net E: now also J5.8 (Pin_8)
- net GND: now also J5.13 (Pin_13)
- net MX: now also J5.6 (Pin_6)
- net RDY⎒: now also J5.3 (Pin_3)
- net RST: now also J5.2 (Pin_2)
- net SYNC: now also J6.13 (Pin_13); no longer J6.14 (Pin_14)
- net VA: now also J6.14 (Pin_14); no longer J6.13 (Pin_13)
- net VDA: now also J5.4 (Pin_4)
- net VPA: now also J5.5 (Pin_5)
- net ~{ABORT}: now also J5.7 (Pin_7)
- net ~{CLK}: now also J5.1 (Pin_1)
- net ~{ML}: now also J5.12 (Pin_12)
- net ~{VP}: now also J5.11 (Pin_11)
- net CLK_SRC renamed CLK_IN
- net ~{CLK_EN_IN} renamed ~{CLK_EN}
- new net M: J5.9 (Pin_9)
- new net X: J5.10 (Pin_10)
Other:
- sheet Clock & Reset ports: added CLK_IN, ~{CLK_EN}; removed CLK_SRC, ~{CLK_EN_IN}
- sheet Glue Logic ports: added M, MX, X; removed none
- note removed: "TODO: Decode MX into M and X"
