File: hardware/clock_reset.kicad_sch (KiCad schematic)
At the start: 12 parts, among them SW7 Reset, U11 DS1813-5, U14 74AHC125, U41 74HC74, U42 74HC74, X2 8MHz

Commit message: More updates
Parts:
- added J3: Conn_01x02, symbol Connector_Generic:Conn_01x02
Connections:
- net CLK_IN is gone; now on net CLK_SRC: U41.3 (C), U42.11 (C), U42.3 (C)
- net 8MHz: now also J3.1 (Pin_1)
- net GND: now also J3.2 (Pin_2)
- net ~{MR}⎒: now also U42.12 (D); no longer U42.2 (D)
- net at U41.2 (D): now also U42.5 (Q); no longer U42.9 (Q)
- net CLK renamed CLK_SRC
- new net: U42.2 (D), U42.9 (Q)
Other:
- note added: "Generates a ~{RST} pulse of 150ms + 3 clock rising edges Ensures the CPU registers the reset even with slow or stopped clock"
- note removed: "Generates a ~{RST} pulse of 150ms + 3 clock rising edges Ensures CPU registers the reset even with slow or stopped clock"
- moved on the sheet: U41A, U42A, U42B

Commit message: Updates for episode 25
Parts:
- removed R46: 3.3k, symbol Device:R_Small
Connections:
- net CLK_SRC renamed CLK_IN
- net ~{CLK_EN_IN} renamed ~{CLK_EN}
Other:
- moved on the sheet: C24, SW7, U11
