File: hardware/gpio.kicad_sch (KiCad schematic)
At the start: 10 parts, among them U37 W65C22SxP, U38 74HC541, U39 74HC541

Commit message: Renumber
Parts:
- renumbered RN1 to RN12, RN9 to RN13
Changed lines of the file:
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@@
   (symbol (lib_id "Device:R_Network08") (at 224.79 90.17 270) (mirror x) (unit 1)
     (in_bom yes) (on_board yes)
-    (property "Reference" "RN9" (id 0) (at 224.79 76.835 90))
+    (property "Reference" "RN13" (id 0) (at 224.79 76.835 90))
     (property "Value" "1.5k" (id 1) (at 224.79 79.1464 90))
     (property "Footprint" "Resistor_THT:R_Array_SIP9" (id 2) (at 224.79 78.105 90)
@@
   (symbol (lib_id "power:GND") (at 91.44 134.62 0) (unit 1)
     (in_bom yes) (on_board yes) (fields_autoplaced)
-    (property "Reference" "#PWR0112" (id 0) (at 91.44 140.97 0)
+    (property "Reference" "#PWR0127" (id 0) (at 91.44 140.97 0)
       (effects (font (size 1.27 1.27)) hide)
     )
@@
   (symbol (lib_id "power:VCC") (at 91.44 60.96 0) (unit 1)
     (in_bom yes) (on_board yes) (fields_autoplaced)
-    (property "Reference" "#PWR069" (id 0) (at 91.44 64.77 0)
+    (property "Reference" "#PWR0126" (id 0) (at 91.44 64.77 0)
       (effects (font (size 1.27 1.27)) hide)
     )
@@
   (symbol (lib_id "Device:R_Network08") (at 224.79 36.83 270) (mirror x) (unit 1)
     (in_bom yes) (on_board yes)
-    (property "Reference" "RN1" (id 0) (at 224.79 23.495 90))
+    (property "Reference" "RN12" (id 0) (at 224.79 23.495 90))
     (property "Value" "1.5k" (id 1) (at 224.79 25.8064 90))
     (property "Footprint" "Resistor_THT:R_Array_SIP9" (id 2) (at 224.79 24.765 90)

Commit message: Updates for episode 22
Other:
- note added: "W65C22 pin features: -------------------- CB1: Interrupt, SR clock, Write Handshake Data Taken CB2: Interrupt, SR data, Write Handshake Data Ready, Output Bit PB6: T2 pulse input PB7: T1 output CA1: Interrupt, Read/Write Handshake Data Taken CA2: Interrupt, Read/Write Handshake Data Ready, Output Bit"
Changed lines of the file:
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@@
   (title_block
     (title "GPIO module")
-    (date "2022-04-15")
-    (rev "A.21")
+    (date "2022-05-06")
+    (rev "A.22")
     (comment 2 "https://github.com/adrienkohlbecker/65C816")
     (comment 3 "Licensed under CERN-OHL-W v2")
@@
     (stroke (width 0) (type default) (color 0 0 0 0))
   )
+  (bus (pts (xy 44.45 25.4) (xy 55.88 25.4))
+    (stroke (width 0) (type default) (color 0 0 0 0))
+  )
   (wire (pts (xy 68.58 85.09) (xy 76.2 85.09))
     (stroke (width 0) (type default) (color 0 0 0 0))
@@
     (stroke (width 0) (type default) (color 0 0 0 0))
   )
+  (bus (pts (xy 44.45 22.86) (xy 55.88 22.86))
+    (stroke (width 0) (type default) (color 0 0 0 0))
+  )
   (wire (pts (xy 204.47 92.71) (xy 201.93 92.71))
     (stroke (width 0) (type default) (color 0 0 0 0))
@@
     (stroke (width 0) (type default) (color 0 0 0 0))
   )
+  (text "W65C22 pin features:\n--------------------\nCB1: Interrupt, SR clock, Write Handshake Data Taken\nCB2: Interrupt, SR data, Write Handshake Data Ready, Output Bit\nPB6: T2 pulse input\nPB7: T1 output\nCA1: Interrupt, Read/Write Handshake Data Taken\nCA2: Interrupt, Read/Write Handshake Data Ready, Output Bit"
+    (at 68.58 162.56 0)
+    (effects (font (size 1.27 1.27)) (justify left bottom))
+  )
   (label "PB3" (at 114.3 107.95 180)
     (effects (font (size 1.27 1.27)) (justify right bottom))
@@
     (effects (font (size 1.27 1.27)) (justify left bottom))
   )
+  (label "{PORTB}" (at 44.45 25.4 0)
+    (effects (font (size 1.27 1.27)) (justify left bottom))
+  )
   (label "CA2" (at 114.3 95.25 180)
     (effects (font (size 1.27 1.27)) (justify right bottom))
@@
     (effects (font (size 1.27 1.27)) (justify left bottom))
   )
+  (label "{PORTA}" (at 44.45 22.86 0)
+    (effects (font (size 1.27 1.27)) (justify left bottom))
+  )
   (label "D1" (at 68.58 110.49 0)
     (effects (font (size 1.27 1.27)) (justify left bottom))
@@
   (label "A0" (at 68.58 90.17 0)
     (effects (font (size 1.27 1.27)) (justify left bottom))
+  )
+  (hierarchical_label "{PORTA}" (shape output) (at 55.88 22.86 0)
+    (effects (font (size 1.27 1.27)) (justify left))
   )
   (hierarchical_label "VA" (shape input) (at 27.94 30.48 180)
@@
     (effects (font (size 1.27 1.27)) (justify right))
   )
+  (hierarchical_label "{PORTB}" (shape output) (at 55.88 25.4 0)
+    (effects (font (size 1.27 1.27)) (justify left))
+  )
   (hierarchical_label "CLK" (shape input) (at 27.94 25.4 180)

Commit message: Snapshot ep 24 work
Changed lines of the file:
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@@
   (title_block
     (title "GPIO module")
-    (date "2022-05-23")
-    (rev "A.23")
+    (date "2022-07-04")
+    (rev "A.24")
     (comment 2 "https://github.com/adrienkohlbecker/65C816")
     (comment 3 "Licensed under CERN-OHL-W v2")
@@
     (effects (font (size 1.27 1.27)) (justify right bottom))
   )
-  (label "{ADDRESS}" (at 53.34 85.09 0)
+  (label "A[0..23]" (at 53.34 85.09 0)
     (effects (font (size 1.27 1.27)) (justify left bottom))
   )
@@
     (effects (font (size 1.27 1.27)) (justify left bottom))
   )
-  (label "{ADDRESS}" (at 39.37 39.37 180)
+  (label "A[0..23]" (at 39.37 39.37 180)
     (effects (font (size 1.27 1.27)) (justify right bottom))
   )
@@
     (effects (font (size 1.27 1.27)) (justify right))
   )
-  (hierarchical_label "{ADDRESS}" (shape input) (at 27.94 39.37 180)
+  (hierarchical_label "A[0..23]" (shape input) (at 27.94 39.37 180)
     (effects (font (size 1.27 1.27)) (justify right))
   )

Commit message: Update main project
Parts:
- renumbered BAR7 to BAR6, BAR8 to BAR7, C52 to C34, C53 to C35, C54 to C36, RN12 to RN5, RN13 to RN6, U37 to U26, U38 to U27, U39 to U28
Changed lines of the file:
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@@
   (symbol (lib_id "Device:R_Network08") (at 224.79 90.17 270) (mirror x) (unit 1)
     (in_bom yes) (on_board yes)
-    (property "Reference" "RN13" (id 0) (at 224.79 76.835 90))
+    (property "Reference" "RN6" (id 0) (at 224.79 76.835 90))
     (property "Value" "1.5k" (id 1) (at 224.79 79.1464 90))
     (property "Footprint" "Resistor_THT:R_Array_SIP9" (id 2) (at 224.79 78.105 90)
@@
   (symbol (lib_id "Device:C_Small") (at 250.19 21.59 0) (unit 1)
     (in_bom yes) (on_board yes) (fields_autoplaced)
-    (property "Reference" "C52" (id 0) (at 252.73 20.3262 0)
+    (property "Reference" "C34" (id 0) (at 252.73 20.3262 0)
       (effects (font (size 1.27 1.27)) (justify left))
     )
@@
   (symbol (lib_id "power:GND") (at 175.26 57.15 0) (unit 1)
     (in_bom yes) (on_board yes)
-    (property "Reference" "#PWR0128" (id 0) (at 175.26 63.5 0)
+    (property "Reference" "#PWR096" (id 0) (at 175.26 63.5 0)
       (effects (font (size 1.27 1.27)) hide)
     )
@@
   (symbol (lib_id "74xx:74LS541") (at 189.23 41.91 0) (unit 1)
     (in_bom yes) (on_board yes) (fields_autoplaced)
-    (property "Reference" "U38" (id 0) (at 191.2494 21.59 0)
+    (property "Reference" "U27" (id 0) (at 191.2494 21.59 0)
       (effects (font (size 1.27 1.27)) (justify left))
     )
@@
   (symbol (lib_id "power:GND") (at 175.26 110.49 0) (unit 1)
     (in_bom yes) (on_board yes)
-    (property "Reference" "#PWR0129" (id 0) (at 175.26 116.84 0)
+    (property "Reference" "#PWR097" (id 0) (at 175.26 116.84 0)
       (effects (font (size 1.27 1.27)) hide)
     )
@@
   (symbol (lib_id "65C816:W65C22SxP") (at 91.44 97.79 0) (unit 1)
     (in_bom yes) (on_board yes)
-    (property "Reference" "U37" (id 0) (at 81.28 64.77 0)
+    (property "Reference" "U26" (id 0) (at 81.28 64.77 0)
       (effects (font (size 1.27 1.27)) (justify left))
     )
@@
   (symbol (lib_id "74xx:74LS541") (at 189.23 95.25 0) (unit 1)
     (in_bom yes) (on_board yes) (fields_autoplaced)
-    (property "Reference" "U39" (id 0) (at 191.2494 74.93 0)
+    (property "Reference" "U28" (id 0) (at 191.2494 74.93 0)
       (effects (font (size 1.27 1.27)) (justify left))
     )
@@
   (symbol (lib_id "power:GND") (at 231.14 101.6 0) (unit 1)
     (in_bom yes) (on_board yes)
-    (property "Reference" "#PWR0135" (id 0) (at 231.14 107.95 0)
+    (property "Reference" "#PWR0103" (id 0) (at 231.14 107.95 0)
       (effects (font (size 1.27 1.27)) hide)
     )
@@
   (symbol (lib_id "power:VCC") (at 250.19 19.05 0) (unit 1)
     (in_bom yes) (on_board yes)
-    (property "Reference" "#PWR0136" (id 0) (at 250.19 22.86 0)
+    (property "Reference" "#PWR0104" (id 0) (at 250.19 22.86 0)
       (effects (font (size 1.27 1.27)) hide)
     )
@@
   (symbol (lib_id "power:VCC") (at 189.23 21.59 0) (unit 1)
     (in_bom yes) (on_board yes)
-    (property "Reference" "#PWR0130" (id 0) (at 189.23 25.4 0)
+    (property "Reference" "#PWR098" (id 0) (at 189.23 25.4 0)
       (effects (font (size 1.27 1.27)) hide)
     )
@@
   (symbol (lib_id "Device:C_Small") (at 273.05 21.59 0) (unit 1)
     (in_bom yes) (on_board yes) (fields_autoplaced)
-    (property "Reference" "C54" (id 0) (at 275.59 20.3262 0)
+    (property "Reference" "C36" (id 0) (at 275.59 20.3262 0)
       (effects (font (size 1.27 1.27)) (justify left))
     )
@@
   (symbol (lib_id "power:GND") (at 250.19 24.13 0) (unit 1)
     (in_bom yes) (on_board yes)
-    (property "Reference" "#PWR0137" (id 0) (at 250.19 30.48 0)
+    (property "Reference" "#PWR0105" (id 0) (at 250.19 30.48 0)
       (effects (font (size 1.27 1.27)) hide)
     )
@@
   (symbol (lib_id "power:VCC") (at 189.23 74.93 0) (unit 1)
     (in_bom yes) (on_board yes)
-    (property "Reference" "#PWR0132" (id 0) (at 189.23 78.74 0)
+    (property "Reference" "#PWR0100" (id 0) (at 189.23 78.74 0)
       (effects (font (size 1.27 1.27)) hide)
     )
@@
   (symbol (lib_id "power:GND") (at 231.14 48.26 0) (unit 1)
     (in_bom yes) (on_board yes)
-    (property "Reference" "#PWR0134" (id 0) (at 231.14 54.61 0)
+    (property "Reference" "#PWR0102" (id 0) (at 231.14 54.61 0)
       (effects (font (size 1.27 1.27)) hide)
     )
@@
   (symbol (lib_id "power:GND") (at 91.44 134.62 0) (unit 1)
     (in_bom yes) (on_board yes) (fields_autoplaced)
-    (property "Reference" "#PWR0127" (id 0) (at 91.44 140.97 0)
+    (property "Reference" "#PWR095" (id 0) (at 91.44 140.97 0)
       (effects (font (size 1.27 1.27)) hide)
     )
@@
   (symbol (lib_id "65C816:LED-Array-8") (at 209.55 38.1 0) (unit 1)
     (in_bom yes) (on_board yes)
-    (property "Reference" "BAR7" (id 0) (at 209.55 23.241 0))
+    (property "Reference" "BAR6" (id 0) (at 209.55 23.241 0))
     (property "Value" "Red" (id 1) (at 209.55 25.5524 0))
     (property "Footprint" "" (id 2) (at 210.312 52.705 0)
@@
   (symbol (lib_id "power:GND") (at 189.23 62.23 0) (unit 1)
     (in_bom yes) (on_board yes)
-    (property "Reference" "#PWR0131" (id 0) (at 189.23 68.58 0)
+    (property "Reference" "#PWR099" (id 0) (at 189.23 68.58 0)
       (effects (font (size 1.27 1.27)) hide)
     )
@@
   (symbol (lib_id "power:GND") (at 189.23 115.57 0) (unit 1)
     (in_bom yes) (on_board yes)
-    (property "Reference" "#PWR0133" (id 0) (at 189.23 121.92 0)
+    (property "Reference" "#PWR0101" (id 0) (at 189.23 121.92 0)
       (effects (font (size 1.27 1.27)) hide)
     )
@@
   (symbol (lib_id "Device:C_Small") (at 261.62 21.59 0) (unit 1)
     (in_bom yes) (on_board yes) (fields_autoplaced)
-    (property "Reference" "C53" (id 0) (at 264.16 20.3262 0)
+    (property "Reference" "C35" (id 0) (at 264.16 20.3262 0)
       (effects (font (size 1.27 1.27)) (justify left))
     )
@@
   (symbol (lib_id "power:VCC") (at 91.44 60.96 0) (unit 1)
     (in_bom yes) (on_board yes) (fields_autoplaced)
-    (property "Reference" "#PWR0126" (id 0) (at 91.44 64.77 0)
+    (property "Reference" "#PWR094" (id 0) (at 91.44 64.77 0)
       (effects (font (size 1.27 1.27)) hide)
     )
@@
   (symbol (lib_id "65C816:LED-Array-8") (at 209.55 91.44 0) (unit 1)
     (in_bom yes) (on_board yes)
-    (property "Reference" "BAR8" (id 0) (at 209.55 76.581 0))
+    (property "Reference" "BAR7" (id 0) (at 209.55 76.581 0))
     (property "Value" "Red" (id 1) (at 209.55 78.8924 0))
     (property "Footprint" "" (id 2) (at 210.312 106.045 0)
@@
   (symbol (lib_id "Device:R_Network08") (at 224.79 36.83 270) (mirror x) (unit 1)
     (in_bom yes) (on_board yes)
-    (property "Reference" "RN12" (id 0) (at 224.79 23.495 90))
+    (property "Reference" "RN5" (id 0) (at 224.79 23.495 90))
     (property "Value" "1.5k" (id 1) (at 224.79 25.8064 90))
     (property "Footprint" "Resistor_THT:R_Array_SIP9" (id 2) (at 224.79 24.765 90)
