File: hardware/serial.kicad_sch (KiCad schematic)
At the start: 20 parts, among them J2 USB_B, J3 Conn_01x04, U29 W65C51NxP, U30 MCP2221AxP, X2 1.8432MHz

Commit message: Episode 30
Parts:
- added J4: USB Reset, symbol Connector_Generic:Conn_01x02
- C40: value .47u -> 470n
Connections:
- net GND: now also J4.2 (Pin_2)
- net at R34.2, U30.4 (~{RST}): now also J4.1 (Pin_1)
Other:
- moved on the sheet: J2, J3, R35, R36

Commit message: Update for ep 30
Parts:
- J3: value Conn_01x04 -> USB_I2C
Changed lines of the file:
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@@
       (effects (font (size 1.27 1.27)) (justify left))
     )
-    (property "Value" "Conn_01x04" (id 1) (at 248.92 92.7099 0)
+    (property "Value" "USB_I2C" (id 1) (at 248.92 92.7099 0)
       (effects (font (size 1.27 1.27)) (justify left))
     )
