File: hardware/serial.kicad_sch (KiCad schematic)
At the start: 21 parts, among them J2 USB_B, J3 USB_I2C, J4 USB Reset, U29 W65C51NxP, U30 MCP2221AxP, X2 1.8432MHz

Commit message: Update schematic
Parts:
- removed U29: W65C51NxP, symbol 65xx:W65C51NxP
- added U29: W65C51NxP, symbol 65C816:W65C51NxP
Connections:
- net A0: now also U29.13 (RS0)
- net A1: now also U29.14 (RS1)
- net CLK: now also U29.27 (ϕ2)
- net D0: now also U29.18 (D0)
- net D1: now also U29.19 (D1)
- net D2: now also U29.20 (D2)
- net D3: now also U29.21 (D3)
- net D4: now also U29.22 (D4)
- net D5: now also U29.23 (D5)
- net D6: now also U29.24 (D6)
- net D7: now also U29.25 (D7)
- net GND: now also U29.1 (VSS), U29.16 (~{DCD}), U29.17 (~{DSR}), U29.9 (~{CTS})
- net R~{W}: now also U29.28 (R/~{W})
- net UART->USB: now also U29.10 (TxD)
- net USB->UART: now also U29.12 (RxD)
- net VA: now also U29.2 (CS1)
- net VCC: now also U29.15 (VCC)
- net ~{ACIA_CS}: now also U29.3 (~{CS2})
- net ~{IRQ}: now also U29.26 (~{IRQ})
- net ~{RST}: now also U29.4 (~{RES})
- net at X2.5 (OUT): now also U29.6 (XTAL1)
Changed lines of the file:
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@@
   (title_block
     (title "Serial Module")
-    (date "2022-09-26")
-    (rev "A.30")
+    (date "2023-02-24")
+    (rev "A.31")
     (comment 2 "https://github.com/adrienkohlbecker/65C816")
     (comment 3 "Licensed under CERN-OHL-W v2")
@@
     (pin "1")
   )
+  (symbol (lib_id "power:VCC") (at 76.2 67.31 0) (unit 1)
+    (in_bom yes) (on_board yes) (fields_autoplaced)
+    (property "Reference" "#PWR0115" (id 0) (at 76.2 71.12 0)
+      (effects (font (size 1.27 1.27)) hide)
+    )
+    (property "Value" "VCC" (id 1) (at 76.2 62.23 0))
+    (property "Footprint" "" (id 2) (at 76.2 67.31 0)
+      (effects (font (size 1.27 1.27)) hide)
+    )
+    (property "Datasheet" "" (id 3) (at 76.2 67.31 0)
+      (effects (font (size 1.27 1.27)) hide)
+    )
+    (pin "1")
+  )
   (symbol (lib_id "power:GND") (at 93.98 58.42 0) (unit 1)
     (in_bom yes) (on_board yes) (fields_autoplaced)
@@
     (pin "1")
   )
-  (symbol (lib_id "65xx:W65C51NxP") (at 76.2 104.14 0) (unit 1)
+  (symbol (lib_id "65C816:W65C51NxP") (at 76.2 104.14 0) (unit 1)
     (in_bom yes) (on_board yes) (fields_autoplaced)
     (property "Reference" "U29" (id 0) (at 78.2194 67.31 0)
@@
       (effects (font (size 1.27 1.27)) hide)
     )
-    (pin "1")
-  )
-  (symbol (lib_id "power:VCC") (at 76.2 67.31 0) (unit 1)
-    (in_bom yes) (on_board yes) (fields_autoplaced)
-    (property "Reference" "#PWR0115" (id 0) (at 76.2 71.12 0)
-      (effects (font (size 1.27 1.27)) hide)
-    )
-    (property "Value" "VCC" (id 1) (at 76.2 62.23 0))
-    (property "Footprint" "" (id 2) (at 76.2 67.31 0)
-      (effects (font (size 1.27 1.27)) hide)
-    )
-    (property "Datasheet" "" (id 3) (at 76.2 67.31 0)
-      (effects (font (size 1.27 1.27)) hide)
-    )

Commit message: Update for Episode 32
Parts:
- removed D3: Rx, symbol Device:LED_Small
- removed D4: Tx, symbol Device:LED_Small
- removed D5: USBCFG, symbol Device:LED_Small
- removed D6: I2C, symbol Device:LED_Small
- removed R30, R31, R32, R33: 1k, symbol Device:R_Small
- added U19: 74HC04, symbol 74xx:74HC04
Connections:
- net ~{LED_RX}: now reaches U30.3 (GP1)
- net ~{LED_RX}: now also U19.3
- net ~{LED_TX}: now reaches U30.2 (GP0)
- net ~{LED_TX}: now also U19.1
- net ~{LED_I2C}: now reaches U30.8 (GP3)
- net ~{LED_I2C}: now also U19.5
- net ~{USBCFG}: now reaches U30.7 (GP2)
- new net LED_I2C: U19.6
- new net LED_RX: U19.4
- new net LED_TX: U19.2
