File: hardware/serial.kicad_sch (KiCad schematic)
At the start: 14 parts, among them J2 USB_B, J3 USB_I2C, J4 USB Reset, U19 74HC04, U29 W65C51NxP, U30 MCP2221AxP, X2 1.8432MHz

Commit message: Rename
Parts:
- U29: symbol 65C816:W65C51NxP -> BB816:W65C51NxP
Changed lines of the file:
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@@
   (title_block
     (title "Serial Module")
-    (date "2023-05-14")
+    (date "2023-05-23")
     (rev "A.32")
-    (comment 2 "https://github.com/adrienkohlbecker/65C816")
+    (comment 2 "https://github.com/adrienkohlbecker/BB816")
     (comment 3 "Licensed under CERN-OHL-W v2")
-    (comment 4 "Copyright © 2022 Adrien Kohlbecker")
+    (comment 4 "Copyright © 2022-2023 Adrien Kohlbecker")
   )
   (junction (at 231.14 95.25) (diameter 0) (color 0 0 0 0)
@@
     (pin "1")
   )
-  (symbol (lib_id "65C816:W65C51NxP") (at 76.2 104.14 0) (unit 1)
+  (symbol (lib_id "BB816:W65C51NxP") (at 76.2 104.14 0) (unit 1)
     (in_bom yes) (on_board yes) (fields_autoplaced)
     (property "Reference" "U29" (id 0) (at 78.2194 67.31 0)
