File: hardware/debug_clock.kicad_sch (KiCad schematic)
At the start: 53 parts, among them SW1 Pulse, SW2 Mode, SW3 Speed, SW4 SW_DIP_SPDT_x02, SW5 SW_DIP_x03, U10 74AC151, U2 74HC14, U3 74HC74, U4 74HC193, U40 74HC251, U5 74AC112, U6 74HC74, U7 74AC112, U8 LMC555xN, U9 74HC283, X1 20MHz

Commit message: Snapshot ep 24 work
Parts:
- added NT1: NetTie_2, symbol Device:NetTie_2
- R13, R14, R15, R16, R17, R18, R19, R20: value 10k -> 3.3k
Connections:
- net VCC: now also NT1.1
- net ~{CLK_EN} renamed ~{CLK_EN_IN}
- new net ~{CLK_EN_OUT}: NT1.2
Other:
- note added: "CLOCK ENABLE"
- moved on the sheet: R17, U2G, U3C, U5C, U6C, U7B, U7C

Commit message: More updates
Parts:
- NT1: now left out of the parts list
Changed lines of the file:
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@@
   )
   (symbol (lib_id "Device:NetTie_2") (at 177.8 185.42 0) (unit 1)
-    (in_bom yes) (on_board yes) (fields_autoplaced)
+    (in_bom no) (on_board yes) (fields_autoplaced)
     (property "Reference" "NT1" (id 0) (at 177.8 180.34 0))
     (property "Value" "NetTie_2" (id 1) (at 177.8 182.88 0))

Commit message: Updates for episode 25
Parts:
- removed NT1: NetTie_2, symbol Device:NetTie_2
Connections:
- net ~{CLK_EN_IN} renamed ~{CLK_EN}
Other:
- note removed: "CLOCK ENABLE"
- moved on the sheet: U2G, U3C, U5C, U6C, U7B, U7C

Commit message: Update main project
Parts:
- renumbered C4 to C10, C5 to C11, C6 to C12, C7 to C13, C8 to C14, C9 to C15, C10 to C16, C11 to C17, C12 to C18, C13 to C19, C14 to C20, C15 to C21, C16 to C22, C17 to C23, C18 to C24, C19 to C25, C20 to C26, D2 to D1, R14 to R10, R15 to R11, R16 to R12, R18 to R13, R19 to R14, R20 to R15, R21 to R16, R22 to R17, R23 to R18, R17 to R19, R6 to R2, R7 to R3, R8 to R4, R9 to R5, R10 to R6, R11 to R7, R12 to R8, R13 to R9, U3 to U10, U9 to U11, U5 to U12, U4 to U13, U6 to U14, U7 to U15, U8 to U16, U40 to U17, U10 to U18, U2 to U9

Commit message: Update schematic
Parts:
- removed U11: 74HC283, symbol 74xx:74LS283
- removed U12, U15: 74AC112, symbol 74xx:74LS112
- removed U18: 74AC151, symbol 74xx:74LS151
- added C41, C42: 100n, symbol Device:C_Small
- added D10: Pulse, symbol Device:LED_Small
- added D8: Slow, symbol Device:LED_Small
- added D9: Fast, symbol Device:LED_Small
- added R37, R38, R39: 1k, symbol Device:R_Small
- added U11: 74HC32, symbol 74xx:74LS32
- added U12: 74HC74, symbol 74xx:74LS74
- added U15, U31: 74AHC74, symbol 74xx:74LS74
- added U18: 74HC153, symbol 74xx:74LS153
- U13: value 74HC193 -> 74HCT193
- X1: value 20MHz -> 8MHz
Connections:
- net FAST: now also U15.3 (C), U18.11 (I1b), U18.13 (I3b), U18.5 (I1a), U31.3 (C); no longer U17.1 (I3), U17.2 (I2)
- net FAST_ON_RST: now also U10.4 (~{S}), U12.4 (~{S}), U15.4 (~{S}), U31.4 (~{S}); no longer U10.10 (~{S})
- net FAST_~{SLOW}: now also U11.2, U18.14 (S0), U31.5 (Q); no longer U17.10 (S1), U17.11 (S0)
- net GND: now also U13.9 (D), U17.1 (I3), U17.10 (S1), U17.11 (S0), U17.12 (I7), U17.13 (I6), U17.14 (I5), U17.15 (I4), U17.2 (I2), U17.3 (I1), U17.9 (S2), C41.2, C42.2, U11.7 (GND), U12.7 (GND), U15.7 (GND), U18.1 (Ea), U18.15 (Eb), U18.8 (GND), U31.7 (GND); no longer R16.1
- net MODE: now also U10.11 (C); no longer U10.3 (C)
- net PULSE: now also U9.4, U18.3 (I3a), U18.4 (I2a); no longer U17.12 (I7), U17.13 (I6), U17.14 (I5), U17.15 (I4), U9.2
- net PULSE_ON_RST: now also U10.10 (~{S}), U15.10 (~{S}), U31.10 (~{S}); no longer U10.4 (~{S})
- net PULSE_~{RUN}: now also U11.1, U11.4, U18.2 (S1), U31.9 (Q); no longer U17.9 (S2)
- net RUN: now also U15.11 (C), U18.9 (Zb), U31.11 (C)
- net RUN_ON_RST: now also U10.13 (~{R}), U15.13 (~{R}), U31.13 (~{R}); no longer U10.1 (~{R})
- net SLOW: now also U12.3 (C), U18.10 (I0b), U18.12 (I2b), U18.6 (I0a); no longer U17.3 (I1), U17.4 (I0)
- net SLOW_ON_RST: now also U10.1 (~{R}), U12.1 (~{R}), U15.1 (~{R}), U31.1 (~{R}); no longer U10.13 (~{R})
- net SPEED: now also U10.3 (C), U9.8; no longer U10.11 (C), U9.4
- net VCC: now also R16.1, C41.1, C42.1, R37.1, R38.1, R39.1, U11.10, U11.14 (VCC), U11.9, U12.10 (~{S}), U12.11 (C), U12.12 (D), U12.13 (~{R}), U12.14 (VCC), U15.14 (VCC), U18.16 (VCC), U31.14 (VCC)
- net ~{CLK}: now also U11.12, U11.13; no longer U9.11
- net at C15.1, R8.2: now also U9.9; no longer U9.3
- net at U10.5 (Q): now also U12.2 (D)
- net at U10.9 (Q): now also U15.12 (D)
- net at U13.1 (B): now also R14.2, SW5.5
- net at U13.10 (C): now also R13.2, SW5.6
- net at U13.15 (A): now also R15.2, SW5.4
- net at U9.13: now also C11.1, R2.1; no longer U9.8
- net at U9.10: now also SW4.1, SW4.2, SW4.3, SW4.4; no longer D1.2 (A)
- net at D1.1 (K): now also U11.11; no longer R16.2
- new net: U9.2, U9.3
- new net: U9.11, U9.12
- new net: D1.2 (A), R16.2
- new net: D8.2 (A), R37.2
- new net: D10.2 (A), R39.2
- new net: D9.2 (A), R38.2
- new net: D8.1 (K), U11.3
- new net: U12.5 (Q), U15.2 (D)
- new net: U15.5 (Q), U31.2 (D)
- new net: U15.9 (Q), U31.12 (D)
- new net: D9.1 (K), U11.6
- new net OUT_CLK: U17.4 (I0), U18.7 (Za)
- new net ~{FAST}_SLOW: U11.5, U31.6 (~{Q})
- new net ~{PULSE}_RUN: D10.1 (K), U31.8 (~{Q})
Other:
- note added: "000 /2 4MHz 001 /4 2MHz 010 /6 1.33MHz 011 /8 1MHz 100 /10 0.80MHz 101 /12 0.66MHz 110 /14 0.57MHz 111 /16 0.50MHz"
- note added: "=> overall, maximum frequency of the fast clock is 5.31MHz"
- note added: "CLOCK SELECT"
- note added: "Fast clock falling edge => 2 * 10.5 ns (74AHC74) => FAST_SLOW selection bit => 38 ns (74HC153) => CLK We want the whole chain to happen before the fast clock has a rising edge => minimum half period of the fast clock 2*10.5+38ns = 59ns => maximum frequency of the fast clock 1000/59/2 = 8.47MHz"
- note added: "Fast clock falling edge => 35 ns (74HC153) => RUN => 2 * 10.5 ns (74AHC74) => PULSE_RUN selection bit => 38 ns (74HC153) => OUT_CLK We want the whole chain to happen before the fast clock has a rising edge => minimum half period of the fast clock 35+2*10.5+38ns = 94ns => maximum frequency of the fast clock 1000/94/2 = 5.31MHz"
- note added: "Max oscillator frequency: 74HC193 20MHz 74HCT193 18MHz"
- note removed: "000 5Mhz 001 3.33Mhz 010 2.5Mhz 011 2Mhz 100 1.67Mhz 101 1.43Mhz 110 1.25Mhz 111 1.11Mhz"
- note removed: "=> overall, maximum frequency of the fast clock is 6.87MHz"
- note removed: "Fast clock falling edge => 12.3 ns (74AC151) => RUN => 9.4 ns (74AC112) => PULSE_RUN selection bit => 51 ns (74HC251) => CLK We want the whole chain to happen before the fast clock has a rising edge => minimum half period of the fast clock 12.3+9.4+51ns = 72.7ns => maximum frequency of the fast clock 1000/72.7/2 = 6.87MHz"
- note removed: "Fast clock falling edge => 9.4 ns (74AC112) => FAST_SLOW selection bit => 51 ns (74HC251) => CLK We want the whole chain to happen before the fast clock has a rising edge => minimum half period of the fast clock 9.4+51ns = 60.4ns => maximum frequency of the fast clock 1000/60.4/2 = 8.27MHz"
- note removed: "RUN CLOCK"
- moved on the sheet: C13, D1, R13, R14, R15, R16, R19, R3, R4, SW1, SW5, U10A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

Commit message: CLeanup
Connections:
- net FAST: now also U15.11 (C); no longer U31.3 (C)
- net FAST_ON_RST: now also U15.10 (~{S}); no longer U31.4 (~{S})
- net FAST_~{SLOW}: now also U15.9 (Q); no longer U31.5 (Q)
- net PULSE_ON_RST: now also U31.4 (~{S}); no longer U15.10 (~{S})
- net RUN: now also U31.3 (C); no longer U15.11 (C)
- net RUN_ON_RST: now also U31.1 (~{R}); no longer U15.13 (~{R})
- net SLOW_ON_RST: now also U15.13 (~{R}); no longer U31.1 (~{R})
- net ~{FAST}_SLOW: now also U15.8 (~{Q}); no longer U31.6 (~{Q})
- net at U10.9 (Q): now also U31.2 (D); no longer U15.12 (D)
- net at U15.5 (Q): now also U15.12 (D); no longer U31.2 (D)
- net at U31.12 (D): now also U31.5 (Q); no longer U15.9 (Q)
Other:
- moved on the sheet: U15B, U31A
Changed lines of the file:
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@@
     (pin "2")
   )
-  (symbol (lib_id "74xx:74LS74") (at 163.83 114.3 0) (unit 1)
-    (in_bom yes) (on_board yes)
-    (property "Reference" "U31" (id 0) (at 158.75 107.95 0))
-    (property "Value" "74AHC74" (id 1) (at 168.91 107.95 0))
-    (property "Footprint" "" (id 2) (at 163.83 114.3 0)
-      (effects (font (size 1.27 1.27)) hide)
-    )
-    (property "Datasheet" "https://www.ti.com/lit/ds/symlink/sn74ahc74.pdf" (id 3) (at 163.83 114.3 0)
+  (symbol (lib_id "74xx:74LS74") (at 240.03 114.3 0) (unit 1)
+    (in_bom yes) (on_board yes)
+    (property "Reference" "U31" (id 0) (at 234.95 107.95 0))
+    (property "Value" "74AHC74" (id 1) (at 245.11 107.95 0))
+    (property "Footprint" "" (id 2) (at 240.03 114.3 0)
+      (effects (font (size 1.27 1.27)) hide)
+    )
+    (property "Datasheet" "https://www.ti.com/lit/ds/symlink/sn74ahc74.pdf" (id 3) (at 240.03 114.3 0)
       (effects (font (size 1.27 1.27)) hide)
     )
@@
     (pin "7")
   )
-  (symbol (lib_id "74xx:74LS74") (at 240.03 114.3 0) (unit 2)
-    (in_bom yes) (on_board yes)
-    (property "Reference" "U15" (id 0) (at 234.95 107.95 0))
-    (property "Value" "74AHC74" (id 1) (at 245.11 107.95 0))
-    (property "Footprint" "" (id 2) (at 240.03 114.3 0)
-      (effects (font (size 1.27 1.27)) hide)
-    )
-    (property "Datasheet" "https://www.ti.com/lit/ds/symlink/sn74ahc74.pdf" (id 3) (at 240.03 114.3 0)
-      (effects (font (size 1.27 1.27)) hide)
-    )
+  (symbol (lib_id "74xx:74LS74") (at 163.83 114.3 0) (unit 2)
+    (in_bom yes) (on_board yes)
+    (property "Reference" "U15" (id 0) (at 158.75 107.95 0))
+    (property "Value" "74AHC74" (id 1) (at 168.91 107.95 0))
+    (property "Footprint" "" (id 2) (at 163.83 114.3 0)
+      (effects (font (size 1.27 1.27)) hide)
+    )
+    (property "Datasheet" "https://www.ti.com/lit/ds/symlink/sn74ahc74.pdf" (id 3) (at 163.83 114.3 0)
+      (effects (font (size 1.27 1.27)) hide)
+    )
