File: hardware/debug_clock.kicad_sch (KiCad schematic)
At the start: 62 parts, among them SW1 Pulse, SW2 Mode, SW3 Speed, SW4 SW_DIP_SPDT_x02, SW5 SW_DIP_x03, U10 74HC74, U11 74HC32, U12 74HC74, U13 74HCT193, U14 74HC74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

Commit message: Rename
Parts:
- SW4: symbol 65C816:SW_DIP_SPDT_x02 -> BB816:SW_DIP_SPDT_x02
- U16: symbol 65C816:LMC555xN -> BB816:LMC555xN
Changed lines of the file:
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@@
   (title_block
     (title "Clock Module")
-    (date "2023-05-14")
+    (date "2023-05-23")
     (rev "A.32")
-    (comment 2 "https://github.com/adrienkohlbecker/65C816")
+    (comment 2 "https://github.com/adrienkohlbecker/BB816")
     (comment 3 "Licensed under CERN-OHL-W v2")
-    (comment 4 "Copyright © 2022 Adrien Kohlbecker")
+    (comment 4 "Copyright © 2022-2023 Adrien Kohlbecker")
   )
   (junction (at 92.71 123.19) (diameter 0) (color 0 0 0 0)
@@
     (pin "1")
   )
-  (symbol (lib_id "65C816:LMC555xN") (at 224.79 52.07 0) (unit 1)
+  (symbol (lib_id "BB816:LMC555xN") (at 224.79 52.07 0) (unit 1)
     (in_bom yes) (on_board yes)
     (property "Reference" "U16" (id 0) (at 218.44 43.18 0))
@@
     (pin "1")
   )
-  (symbol (lib_id "65C816:SW_DIP_SPDT_x02") (at 67.31 193.04 0) (unit 1)
+  (symbol (lib_id "BB816:SW_DIP_SPDT_x02") (at 67.31 193.04 0) (unit 1)
     (in_bom yes) (on_board yes)
     (property "Reference" "SW4" (id 0) (at 67.31 181.1782 0))
