File: hardware/BB816.kicad_sch (KiCad schematic)
At the start: 1 part, among them U1 65C816-Breakout

Commit message: Rename
Other:
- title: 65C816 Homebrew Computer -> BB816 Homebrew Computer
Changed lines of the file:
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@@
   (paper "A4")
   (title_block
-    (title "65C816 Homebrew Computer")
-    (date "2023-05-14")
+    (title "BB816 Homebrew Computer")
+    (date "2023-05-23")
     (rev "A.32")
-    (comment 2 "https://github.com/adrienkohlbecker/65C816")
+    (comment 2 "https://github.com/adrienkohlbecker/BB816")
     (comment 3 "Licensed under CERN-OHL-W v2")
-    (comment 4 "Copyright © 2022 Adrien Kohlbecker")
+    (comment 4 "Copyright © 2022-2023 Adrien Kohlbecker")
   )
   (no_connect (at 38.1 53.34))
@@
       (effects (font (size 1.27 1.27)) hide)
     )
-    (property "Datasheet" "https://github.com/adrienkohlbecker/65C816/tree/main/hardware/breakout" (id 3) (at 41.91 33.02 0)
+    (property "Datasheet" "https://github.com/adrienkohlbecker/BB816/tree/main/hardware/breakout" (id 3) (at 41.91 33.02 0)
       (effects (font (size 1.27 1.27)) hide)
     )
