File: hardware/breakout/clock_reset.kicad_sch (KiCad schematic)
At the start: 12 parts, among them J3 Conn_01x02, SW7 Reset, U11 DS1813-5, U14 74AHC125, U41 74HC74, U42 74HC74, X2 8MHz

Commit message: Update main project
Parts:
- renumbered C24 to C16, C22 to C17, C23 to C18, C55 to C19, J3 to J6, R42 to R17, SW7 to SW1, U41 to U14, U42 to U15, U11 to U16, U14 to U7, X2 to X1
Changed lines of the file:
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@@
   (symbol (lib_id "Switch:SW_Push") (at 72.39 93.98 90) (unit 1)
     (in_bom yes) (on_board yes)
-    (property "Reference" "SW7" (id 0) (at 73.6092 92.8116 90)
+    (property "Reference" "SW1" (id 0) (at 73.6092 92.8116 90)
       (effects (font (size 1.27 1.27)) (justify right))
     )
@@
   (symbol (lib_id "power:GND") (at 72.39 102.87 0) (unit 1)
     (in_bom yes) (on_board yes)
-    (property "Reference" "#PWR058" (id 0) (at 72.39 109.22 0)
+    (property "Reference" "#PWR048" (id 0) (at 72.39 109.22 0)
       (effects (font (size 1.27 1.27)) hide)
     )
@@
   (symbol (lib_id "Device:C_Small") (at 72.39 161.29 0) (unit 1)
     (in_bom yes) (on_board yes)
-    (property "Reference" "C22" (id 0) (at 74.7268 160.1216 0)
+    (property "Reference" "C17" (id 0) (at 74.7268 160.1216 0)
       (effects (font (size 1.27 1.27)) (justify left))
     )
@@
   (symbol (lib_id "Device:C_Small") (at 85.09 161.29 0) (unit 1)
     (in_bom yes) (on_board yes)
-    (property "Reference" "C23" (id 0) (at 87.4268 160.1216 0)
+    (property "Reference" "C18" (id 0) (at 87.4268 160.1216 0)
       (effects (font (size 1.27 1.27)) (justify left))
     )
@@
   (symbol (lib_id "power:VCC") (at 72.39 158.75 0) (unit 1)
     (in_bom yes) (on_board yes)
-    (property "Reference" "#PWR056" (id 0) (at 72.39 162.56 0)
+    (property "Reference" "#PWR049" (id 0) (at 72.39 162.56 0)
       (effects (font (size 1.27 1.27)) hide)
     )
@@
   (symbol (lib_id "power:GND") (at 72.39 163.83 0) (unit 1)
     (in_bom yes) (on_board yes)
-    (property "Reference" "#PWR057" (id 0) (at 72.39 170.18 0)
+    (property "Reference" "#PWR050" (id 0) (at 72.39 170.18 0)
       (effects (font (size 1.27 1.27)) hide)
     )
@@
   (symbol (lib_id "Device:C_Small") (at 62.23 93.98 0) (unit 1)
     (in_bom yes) (on_board yes)
-    (property "Reference" "C24" (id 0) (at 64.5668 92.8116 0)
+    (property "Reference" "C16" (id 0) (at 64.5668 92.8116 0)
       (effects (font (size 1.27 1.27)) (justify left))
     )
@@
   (symbol (lib_id "power:GND") (at 201.93 100.33 0) (unit 1)
     (in_bom yes) (on_board yes)
-    (property "Reference" "#PWR0165" (id 0) (at 201.93 106.68 0)
+    (property "Reference" "#PWR056" (id 0) (at 201.93 106.68 0)
       (effects (font (size 1.27 1.27)) hide)
     )
@@
   (symbol (lib_id "power:VCC") (at 48.26 69.85 0) (unit 1)
     (in_bom yes) (on_board yes)
-    (property "Reference" "#PWR0146" (id 0) (at 48.26 73.66 0)
+    (property "Reference" "#PWR046" (id 0) (at 48.26 73.66 0)
       (effects (font (size 1.27 1.27)) hide)
     )
@@
   (symbol (lib_id "Device:C_Small") (at 96.52 161.29 0) (unit 1)
     (in_bom yes) (on_board yes)
-    (property "Reference" "C55" (id 0) (at 98.8568 160.1216 0)
+    (property "Reference" "C19" (id 0) (at 98.8568 160.1216 0)
       (effects (font (size 1.27 1.27)) (justify left))
     )
@@
   (symbol (lib_id "power:GND") (at 238.76 92.71 0) (unit 1)
     (in_bom yes) (on_board yes)
-    (property "Reference" "#PWR0161" (id 0) (at 238.76 99.06 0)
+    (property "Reference" "#PWR059" (id 0) (at 238.76 99.06 0)
       (effects (font (size 1.27 1.27)) hide)
     )
@@
   (symbol (lib_id "74xx:74LS125") (at 238.76 76.2 0) (unit 3)
     (in_bom yes) (on_board yes) (fields_autoplaced)
-    (property "Reference" "U14" (id 0) (at 238.76 67.31 0))
+    (property "Reference" "U7" (id 0) (at 238.76 67.31 0))
     (property "Value" "74AHC125" (id 1) (at 238.76 69.85 0))
     (property "Footprint" "" (id 2) (at 238.76 76.2 0)
@@
   (symbol (lib_id "power:GND") (at 48.26 85.09 0) (unit 1)
     (in_bom yes) (on_board yes)
-    (property "Reference" "#PWR0147" (id 0) (at 48.26 91.44 0)
+    (property "Reference" "#PWR047" (id 0) (at 48.26 91.44 0)
       (effects (font (size 1.27 1.27)) hide)
     )
@@
   (symbol (lib_id "power:VCC") (at 121.92 72.39 0) (unit 1)
     (in_bom yes) (on_board yes)
-    (property "Reference" "#PWR0144" (id 0) (at 121.92 76.2 0)
+    (property "Reference" "#PWR052" (id 0) (at 121.92 76.2 0)
       (effects (font (size 1.27 1.27)) hide)
     )
@@
   (symbol (lib_id "Connector_Generic:Conn_01x02") (at 208.28 96.52 0) (unit 1)
     (in_bom yes) (on_board yes) (fields_autoplaced)
-    (property "Reference" "J3" (id 0) (at 210.82 96.5199 0)
+    (property "Reference" "J6" (id 0) (at 210.82 96.5199 0)
       (effects (font (size 1.27 1.27)) (justify left))
     )
@@
   (symbol (lib_id "power:GND") (at 38.1 172.72 0) (unit 1)
     (in_bom yes) (on_board yes)
-    (property "Reference" "#PWR0152" (id 0) (at 38.1 179.07 0)
+    (property "Reference" "#PWR045" (id 0) (at 38.1 179.07 0)
       (effects (font (size 1.27 1.27)) hide)
     )
@@
   (symbol (lib_id "power:VCC") (at 146.05 72.39 0) (unit 1)
     (in_bom yes) (on_board yes)
-    (property "Reference" "#PWR0145" (id 0) (at 146.05 76.2 0)
+    (property "Reference" "#PWR053" (id 0) (at 146.05 76.2 0)
       (effects (font (size 1.27 1.27)) hide)
     )
@@
   (symbol (lib_id "65C816:DS1813") (at 49.53 77.47 0) (unit 1)
     (in_bom yes) (on_board yes) (fields_autoplaced)
-    (property "Reference" "U11" (id 0) (at 43.18 76.1999 0)
+    (property "Reference" "U16" (id 0) (at 43.18 76.1999 0)
       (effects (font (size 1.27 1.27)) (justify right))
     )
@@
   (symbol (lib_id "74xx:74LS74") (at 146.05 80.01 0) (unit 1)
     (in_bom yes) (on_board yes)
-    (property "Reference" "U41" (id 0) (at 140.97 73.66 0))
+    (property "Reference" "U14" (id 0) (at 140.97 73.66 0))
     (property "Value" "74HC74" (id 1) (at 151.13 73.66 0))
     (property "Footprint" "" (id 2) (at 146.05 80.01 0)
@@
   (symbol (lib_id "power:VCC") (at 38.1 148.59 0) (unit 1)
     (in_bom yes) (on_board yes)
-    (property "Reference" "#PWR0151" (id 0) (at 38.1 152.4 0)
+    (property "Reference" "#PWR044" (id 0) (at 38.1 152.4 0)
       (effects (font (size 1.27 1.27)) hide)
     )
@@
   (symbol (lib_id "74xx:74LS74") (at 96.52 80.01 0) (unit 2)
     (in_bom yes) (on_board yes)
-    (property "Reference" "U42" (id 0) (at 91.44 73.66 0))
+    (property "Reference" "U15" (id 0) (at 91.44 73.66 0))
     (property "Value" "74HC74" (id 1) (at 101.6 73.66 0))
     (property "Footprint" "" (id 2) (at 96.52 80.01 0)
@@
   (symbol (lib_id "power:VCC") (at 187.96 71.12 0) (unit 1)
     (in_bom yes) (on_board yes)
-    (property "Reference" "#PWR0148" (id 0) (at 187.96 74.93 0)
+    (property "Reference" "#PWR054" (id 0) (at 187.96 74.93 0)
       (effects (font (size 1.27 1.27)) hide)
     )
@@
   (symbol (lib_id "74xx:74LS74") (at 215.9 78.74 0) (unit 2)
     (in_bom yes) (on_board yes)
-    (property "Reference" "U41" (id 0) (at 210.82 72.39 0))
+    (property "Reference" "U14" (id 0) (at 210.82 72.39 0))
     (property "Value" "74HC74" (id 1) (at 220.98 72.39 0))
     (property "Footprint" "" (id 2) (at 215.9 78.74 0)
@@
   (symbol (lib_id "power:VCC") (at 215.9 71.12 0) (unit 1)
     (in_bom yes) (on_board yes)
-    (property "Reference" "#PWR0154" (id 0) (at 215.9 74.93 0)
+    (property "Reference" "#PWR058" (id 0) (at 215.9 74.93 0)
       (effects (font (size 1.27 1.27)) hide)
     )
@@
   (symbol (lib_id "Oscillator:CXO_DIP14") (at 187.96 78.74 0) (unit 1)
     (in_bom yes) (on_board yes)
-    (property "Reference" "X2" (id 0) (at 181.61 72.39 0)
+    (property "Reference" "X1" (id 0) (at 181.61 72.39 0)
       (effects (font (size 1.27 1.27)) (justify left))
     )
@@
   (symbol (lib_id "power:VCC") (at 96.52 72.39 0) (unit 1)
     (in_bom yes) (on_board yes)
-    (property "Reference" "#PWR059" (id 0) (at 96.52 76.2 0)
+    (property "Reference" "#PWR051" (id 0) (at 96.52 76.2 0)
       (effects (font (size 1.27 1.27)) hide)
     )
@@
   (symbol (lib_id "74xx:74LS74") (at 29.21 161.29 0) (unit 3)
     (in_bom yes) (on_board yes)
-    (property "Reference" "U41" (id 0) (at 24.13 152.4 0))
+    (property "Reference" "U14" (id 0) (at 24.13 152.4 0))
     (property "Value" "74HC74" (id 1) (at 34.29 152.4 0))
     (property "Footprint" "" (id 2) (at 29.21 161.29 0)
@@
   (symbol (lib_id "74xx:74LS74") (at 121.92 80.01 0) (unit 1)
     (in_bom yes) (on_board yes)
-    (property "Reference" "U42" (id 0) (at 116.84 73.66 0))
+    (property "Reference" "U15" (id 0) (at 116.84 73.66 0))
     (property "Value" "74HC74" (id 1) (at 127 73.66 0))
     (property "Footprint" "" (id 2) (at 121.92 80.01 0)
@@
   (symbol (lib_id "Device:R_Small") (at 238.76 88.9 0) (unit 1)
     (in_bom yes) (on_board yes) (fields_autoplaced)
-    (property "Reference" "R42" (id 0) (at 241.3 87.6299 0)
+    (property "Reference" "R17" (id 0) (at 241.3 87.6299 0)
       (effects (font (size 1.27 1.27)) (justify left))
     )
@@
   (symbol (lib_id "74xx:74LS74") (at 46.99 161.29 0) (unit 3)
     (in_bom yes) (on_board yes)
-    (property "Reference" "U42" (id 0) (at 41.91 152.4 0))
+    (property "Reference" "U15" (id 0) (at 41.91 152.4 0))
     (property "Value" "74HC74" (id 1) (at 52.07 152.4 0))
     (property "Footprint" "" (id 2) (at 46.99 161.29 0)
@@
   (symbol (lib_id "power:VCC") (at 210.82 87.63 0) (unit 1)
     (in_bom yes) (on_board yes)
-    (property "Reference" "#PWR0153" (id 0) (at 210.82 91.44 0)
+    (property "Reference" "#PWR057" (id 0) (at 210.82 91.44 0)
       (effects (font (size 1.27 1.27)) hide)
     )
@@
   (symbol (lib_id "power:GND") (at 187.96 86.36 0) (unit 1)
     (in_bom yes) (on_board yes)
-    (property "Reference" "#PWR0149" (id 0) (at 187.96 92.71 0)
-      (effects (font (size 1.27 1.27)) hide)
-    )
+    (property "Reference" "#PWR055" (id 0) (at 187.96 92.71 0)
+      (effects (font (size 1.27 1.27)) hide)
+    )

Commit message: Episode 25
Parts:
- renumbered C16 to C4, C17 to C5, C18 to C6, C19 to C7, J6 to J5, R17 to R7, U14 to U2, U15 to U3, U16 to U4, U7 to U5
Connections:
- net CLK_IN renamed CLK_SRC
