File: hardware/breakout/glue_logic.kicad_sch (KiCad schematic)
At the start: 41 parts, among them J4 Conn_01x10, U12 74AHC32, U13 74AHC74, U14 74AHC125, U15 DS1035-10, U16 74AHC00, U17 74AHC02, U18 74AHC32, U19 74AC10, U20 74AHCT245, U21 74AHC573, U22 74AHC32, U43 74AC112

Commit message: Update main project
Parts:
- renumbered C31 to C10, C32 to C11, C33 to C12, C34 to C13, C25 to C14, C40 to C15, C21 to C4, C26 to C5, C27 to C6, C28 to C7, C29 to C8, C30 to C9, D3 to D2, J4 to J5, R29 to R10, R30 to R11, R46 to R12, R24 to R13, R43 to R14, R44 to R15, R45 to R16, R26 to R7, R27 to R8, R28 to R9, U12 to U10, U15 to U11, U20 to U12, U21 to U13, U17 to U2, U18 to U3, U13 to U4, U22 to U5, U19 to U6, U14 to U7, U16 to U8, U43 to U9

Commit message: Episode 25
Parts:
- removed J5: Conn_01x10, symbol Connector_Generic:Conn_01x10
- added J6: Conn_01x11, symbol Connector_Generic:Conn_01x11
- renumbered C6 to C10, C7 to C11, C8 to C12, C9 to C13, C10 to C14, C11 to C15, C12 to C16, C13 to C17, C14 to C18, C15 to C19, C4 to C8, C5 to C9, R9 to R10, R10 to R11, R11 to R12, R12 to R13, R13 to R14, R14 to R15, R15 to R16, R16 to R17, R7 to R8, R8 to R9, U6 to U10, U8 to U11, U9 to U12, U10 to U13, U11 to U14, U12 to U15, U13 to U16, U7 to U5, U2 to U6, U3 to U7, U4 to U8, U5 to U9
Connections:
- net BUFFER_CLK: now also J6.3 (Pin_3)
- net B_~{OE}: now also J6.9 (Pin_9)
- net CLK+: now also J6.2 (Pin_2)
- net CLK-: now also J6.1 (Pin_1)
- net GND: now also J6.11 (Pin_11)
- net RDY_REG: now also J6.7 (Pin_7)
- net READ_CLK: now also J6.5 (Pin_5)
- net WRITE_CLK: now also J6.6 (Pin_6)
- net ~{BE}: now also J6.10 (Pin_10)
- net ~{RDY_REG}: now also J6.8 (Pin_8)
- net ~{READ_CLK}: now also J6.4 (Pin_4)
