File: hardware/breakout/breakout.kicad_sch (KiCad schematic)
At the start: 15 parts, among them J1 Jack-DC, J5 Conn_01x13, J6 Conn_01x40, J7 Conn_01x10, U1 W65C816SxP

Commit message: Update main project
Parts:
- renumbered C3 to C1, C1 to C2, C2 to C3, J5 to J2, J6 to J3, J7 to J4, R2 to R1, R25 to R2, R1 to R6

Commit message: Episode 25
Connections:
- net CLK_IN renamed CLK_SRC
Other:
- sheet Clock & Reset ports: added CLK_SRC; removed CLK_IN

Commit message: Move breakout to single sheet
Parts:
- removed C1: 100n, symbol Device:C_Small
- removed C2: 220u, symbol Device:C_Polarized_Small
- removed J2: Conn_01x13, symbol Connector_Generic:Conn_01x13
- removed J4: Conn_01x10, symbol Connector_Generic:Conn_01x10
- removed U1: W65C816SxP, Package_DIP:DIP-40_W15.24mm, symbol 65C816:W65C816SxP
- added C1: 220u, symbol Device:C_Polarized_Small
- added C10, C11, C12, C13, C14, C15, C16, C17, C18, C19, C2, C4, C5, C6, C7, C8, C9: 100n, symbol Device:C_Small
- added D2: 1N5817, Diode_THT:D_DO-41_SOD81_P10.16mm_Horizontal, symbol Diode:1N5817
- added J2: Conn_01x16, symbol Connector_Generic:Conn_01x16
- added J4: Conn_01x18, symbol Connector_Generic:Conn_01x18
- added R10, R16: 3.3k, symbol Device:R_Small
- added R11, R7, R8, R9: 0R, symbol Device:R_Small
- added R12, R13, R14, R15: 100k, symbol Device:R_Small
- added R17: 1k, symbol Device:R_Small
- added RN1, RN2, RN3, RN4, RN5: 100k, Resistor_THT:R_Array_SIP9, symbol Device:R_Network08
- added SW1: Reset, symbol Switch:SW_Push
- added U1: 74AHC02, symbol 74xx:74LS02
- added U10: DS1813-5, Package_TO_SOT_THT:TO-92_Inline, symbol 65C816:DS1813
- added U11, U15: 74HC74, symbol 74xx:74LS74
- added U12: 74AHCT245, symbol 65C816:74AC245
- added U13: 74AHC573, symbol 74xx:74LS573
- added U14, U7, U8: 74AHC32, symbol 74xx:74LS32
- added U16: DS1035-10, symbol 65C816:DS1035-10
- added U2: 74AC10, symbol 74xx:74LS10
- added U3: 74AHC00, symbol 74xx:74HC00
- added U4: 74AC112, symbol 74xx:74LS112
- added U5: W65C816SxP, Package_DIP:DIP-40_W15.24mm, symbol 65C816:W65C816SxP
- added U6: 74AHC74, symbol 74xx:74LS74
- added U9: 74AHC125, symbol 74xx:74LS125
- added X1: 8MHz, Oscillator:Oscillator_DIP-14, symbol Oscillator:CXO_DIP14
Connections:
- net A0: now also J4.10 (Pin_10), RN2.2 (R1), U5.9 (A0)
- net A1: now also J4.9 (Pin_9), RN2.3 (R2), U5.10 (A1)
- net A10: now also J3.40 (Pin_40), RN3.4 (R3), U5.19 (A10); no longer J3.32 (Pin_32)
- net A11: now also J3.39 (Pin_39), RN3.5 (R4), U5.20 (A11); no longer J3.31 (Pin_31)
- net A12: now also J3.38 (Pin_38), RN3.6 (R5), U5.22 (A12); no longer J3.30 (Pin_30)
- net A13: now also J3.37 (Pin_37), RN3.7 (R6), U5.23 (A13); no longer J3.29 (Pin_29)
- net A14: now also J3.36 (Pin_36), RN3.8 (R7), U5.24 (A14); no longer J3.28 (Pin_28)
- net A15: now also J3.35 (Pin_35), RN3.9 (R8), U5.25 (A15); no longer J3.27 (Pin_27)
- net A16: now also J3.34 (Pin_34), RN5.2 (R1), U13.19 (Q0), U7.1; no longer J3.26 (Pin_26)
- net A17: now also J3.33 (Pin_33), RN5.3 (R2), U13.18 (Q1), U7.2; no longer J3.25 (Pin_25)
- net A18: now also J3.32 (Pin_32), RN5.4 (R3), U13.17 (Q2), U7.4; no longer J3.24 (Pin_24)
- net A19: now also J3.31 (Pin_31), RN5.5 (R4), U13.16 (Q3), U7.5; no longer J3.23 (Pin_23)
- net A2: now also J4.8 (Pin_8), RN2.4 (R3), U5.11 (A2); no longer J3.40 (Pin_40)
- net A20: now also J3.30 (Pin_30), RN5.6 (R5), U13.15 (Q4), U7.9; no longer J3.22 (Pin_22)
- net A21: now also J3.29 (Pin_29), RN5.7 (R6), U13.14 (Q5), U7.10; no longer J3.21 (Pin_21)
- net A22: now also J3.28 (Pin_28), RN5.8 (R7), U13.13 (Q6), U7.12; no longer J3.20 (Pin_20)
- net A23: now also J3.27 (Pin_27), RN5.9 (R8), U13.12 (Q7), U7.13; no longer J3.19 (Pin_19)
- net A3: now also J4.7 (Pin_7), RN2.5 (R4), U5.12 (A3); no longer J3.39 (Pin_39)
- net A4: now also J4.6 (Pin_6), RN2.6 (R5), U5.13 (A4); no longer J3.38 (Pin_38)
- net A5: now also J4.5 (Pin_5), RN2.7 (R6), U5.14 (A5); no longer J3.37 (Pin_37)
- net A6: now also J4.4 (Pin_4), RN2.8 (R7), U5.15 (A6); no longer J3.36 (Pin_36)
- net A7: now also J4.3 (Pin_3), RN2.9 (R8), U5.16 (A7); no longer J3.35 (Pin_35)
- net A8: now also J4.2 (Pin_2), RN3.2 (R1), U5.17 (A8); no longer J3.34 (Pin_34)
- net A9: now also J4.1 (Pin_1), RN3.3 (R2), U5.18 (A9); no longer J3.33 (Pin_33)
- net BE: now also J3.13 (Pin_13), U1.5, U1.6, U2.10, U2.11, U5.36 (BE); no longer J3.10 (Pin_10)
- net CLK: now also J3.8 (Pin_8), R9.2, U1.12, U1.2, U1.3, U11.11 (C), U11.3 (C), U14.10, U15.3 (C), U4.13 (C), U5.37 (ϕ0), U6.11 (C), U6.3 (C); no longer J3.7 (Pin_7)
- net CLK_SRC: now also J3.6 (Pin_6), R12.1, U14.5, U16.1, U9.8; no longer J3.5 (Pin_5)
- net D0: now also J4.18 (Pin_18), RN4.2 (R1), U12.2 (A0)
- net D1: now also J4.17 (Pin_17), RN4.3 (R2), U12.3 (A1)
- net D2: now also J4.16 (Pin_16), RN4.4 (R3), U12.4 (A2)
- net D3: now also J4.15 (Pin_15), RN4.5 (R4), U12.5 (A3)
- net D4: now also J4.14 (Pin_14), RN4.6 (R5), U12.6 (A4)
- net D5: now also J4.13 (Pin_13), RN4.7 (R6), U12.7 (A5)
- net D6: now also J4.12 (Pin_12), RN4.8 (R7), U12.8 (A6)
- net D7: now also J4.11 (Pin_11), RN4.9 (R8), U12.9 (A7)
- net DBA0: now also RN1.2 (R1), U12.18 (B0), U13.2 (D0), U5.33 (D0)
- net DBA1: now also RN1.3 (R2), U12.17 (B1), U13.3 (D1), U5.32 (D1)
- net DBA2: now also RN1.4 (R3), U12.16 (B2), U13.4 (D2), U5.31 (D2)
- net DBA3: now also RN1.5 (R4), U12.15 (B3), U13.5 (D3), U5.30 (D3)
- net DBA4: now also RN1.6 (R5), U12.14 (B4), U13.6 (D4), U5.29 (D4)
- net DBA5: now also RN1.7 (R6), U12.13 (B5), U13.7 (D5), U5.28 (D5)
- net DBA6: now also RN1.8 (R7), U12.12 (B6), U13.8 (D6), U5.27 (D6)
- net DBA7: now also RN1.9 (R8), U12.11 (B7), U13.9 (D7), U5.26 (D7)
- net E: now also J3.21 (Pin_21), U5.35 (E)
- net GND: now also C1.2, C10.2, C11.2, C12.2, C13.2, C14.2, C15.2, C16.2, C17.2, C18.2, C19.2, C2.2, C4.2, C5.2, C6.2, C7.2, C8.2, C9.2, J2.16 (Pin_16), R10.2, R12.2, R15.2, RN1.1 (common), RN4.1 (common), SW1.1, U1.7 (GND), U10.3 (GND), U11.7 (GND), U12.10 (GND), U13.10 (GND), U14.7 (GND), U15.7 (GND), U16.4 (GND), U2.7 (GND), U3.7 (GND), U4.8 (GND), U5.21 (VSS), U6.7 (GND), U7.7 (GND), U8.7 (GND), U9.7 (GND), X1.7 (GND)
- net M: now also J3.22 (Pin_22), R7.2
- net MX: now also J2.5 (Pin_5), U3.12, U3.13, U4.11 (J), U5.38 (MX), U6.2 (D)
- net RDY_IN: now also J3.14 (Pin_14), R16.2, U6.12 (D); no longer J3.11 (Pin_11)
- net RDY⎒: now also D2.2 (A), J2.2 (Pin_2), R17.1, U14.12, U5.2 (RDY⎒)
- net RST: now also J3.3 (Pin_3), U15.6 (~{Q})
- net R~{W}: now also J3.18 (Pin_18), U1.8, U1.9, U12.1 (A->B), U2.13, U5.34 (R/~{W}); no longer J3.15 (Pin_15)
- net SYNC: now also J3.16 (Pin_16), U3.6; no longer J3.13 (Pin_13)
- net VA: now also J3.17 (Pin_17), R15.1, U9.11; no longer J3.14 (Pin_14)
- net VCC: now also C1.1, C10.1, C11.1, C12.1, C13.1, C14.1, C15.1, C16.1, C17.1, C18.1, C19.1, C2.1, C4.1, C5.1, C6.1, C7.1, C9.1, R13.1, R14.1, R16.1, R17.2, RN2.1 (common), RN3.1 (common), RN5.1 (common), U1.14 (VCC), U10.2 (VDD), U11.10 (~{S}), U11.14 (VCC), U11.4 (~{S}), U12.20 (VCC), U13.20 (VCC), U14.14 (VCC), U15.10 (~{S}), U15.13 (~{R}), U15.14 (VCC), U15.4 (~{S}), U16.8 (VCC), U2.14 (VCC), U3.10, U3.14 (VCC), U3.9, U4.1 (C), U4.10 (~{S}), U4.14 (~{R}), U4.15 (~{R}), U4.16 (VCC), U4.2 (K), U4.3 (J), U4.4 (~{S}), U5.8 (VDD), U6.1 (~{R}), U6.10 (~{S}), U6.13 (~{R}), U6.14 (VCC), U6.4 (~{S}), U7.14 (VCC), U8.14 (VCC), U9.14 (VCC), X1.14 (Vcc)
- net VDA: now also J2.3 (Pin_3), U14.1, U3.1, U5.39 (VDA)
- net VPA: now also J2.4 (Pin_4), U14.2, U3.2, U5.7 (VPA)
- net X: now also J3.23 (Pin_23), U6.5 (Q)
- net ~{ABORT}: now also J3.12 (Pin_12), U5.3 (~{ABORT})
- net ~{BANK0}: now also J3.26 (Pin_26), U8.8; no longer J3.18 (Pin_18)
- net ~{CLK_EN}: now also J3.7 (Pin_7), R10.1, U9.10; no longer J3.6 (Pin_6)
- net ~{CLK}: now also J3.9 (Pin_9), U1.1
- net ~{IRQ}: now also J3.10 (Pin_10), U5.4 (~{IRQ}); no longer J3.8 (Pin_8)
- net ~{ML}: now also J3.25 (Pin_25), U5.5 (~{ML})
- net ~{MR}⎒: now also J3.5 (Pin_5), C8.1, SW1.2, U10.1 (~{RST}⎒), U11.1 (~{R}), U11.12 (D), U11.13 (~{R}), U15.1 (~{R}); no longer J3.4 (Pin_4)
- net ~{NMI}: now also J3.11 (Pin_11), U5.6 (~{NMI}); no longer J3.9 (Pin_9)
- net ~{RD}: now also J3.19 (Pin_19), R13.2, U9.3; no longer J3.16 (Pin_16)
- net ~{RST}: now also J3.4 (Pin_4), U15.5 (Q), U5.40 (~{RES}); no longer J3.3 (Pin_3)
- net ~{VP}: now also J3.24 (Pin_24), U5.1 (~{VP})
- net ~{WAI}: now also J3.15 (Pin_15), U14.11; no longer J3.12 (Pin_12)
- net ~{WR}: now also J3.20 (Pin_20), R14.2, U9.6; no longer J3.17 (Pin_17)
- new net: U1.10, U2.3
- new net: R9.1, U16.3, U16.6
- new net: R11.1, U16.5
- new net: U14.3, U2.2, U2.4, U9.12
- new net: U11.2 (D), U11.9 (Q)
- new net: U2.12, U9.2
- new net: U7.8, U8.4
- new net: U7.3, U8.1
- new net: U7.6, U8.2
- new net: U8.3, U8.9
- new net: U7.11, U8.5
- new net: U8.10, U8.6
- new net: U2.6, U9.5
- new net: U11.5 (Q), U15.2 (D)
- new net: U15.12 (D), U15.8 (~{Q})
- new net: U15.9 (Q), U9.9
- new net: R8.1, U16.2, U16.7
- new net: U3.3, U3.4, U3.5
- new net: U3.11, U4.12 (K)
- new net: R7.1, U4.9 (Q)
- new net 8MHz: J2.1 (Pin_1), U15.11 (C), X1.8 (OUT)
- new net BUFFER_CLK: J2.8 (Pin_8), U1.11, U14.9, U2.9, U8.11
- new net B_~{OE}: J2.14 (Pin_14), U12.19 (CE), U2.8
- new net CLK+: J2.7 (Pin_7), R11.2, U8.13
- new net CLK-: J2.6 (Pin_6), R8.2
- new net RDY_REG: D2.1 (K), J2.12 (Pin_12), U6.9 (Q)
- new net READ_CLK: J2.10 (Pin_10), U14.8, U2.1
- new net WRITE_CLK: J2.11 (Pin_11), U14.6, U2.5
- new net ~{BE}: J2.15 (Pin_15), U1.4, U13.1 (OE), U9.1, U9.13, U9.4
- new net ~{RDY_REG}: J2.13 (Pin_13), U14.13, U14.4, U6.8 (~{Q}), U8.12
- new net ~{READ_CLK}: J2.9 (Pin_9), U1.13, U13.11 (Load)
- no-connect marks 0 -> 8
Other:
- removed sheet Clock & Reset
- removed sheet Glue Logic
- note added: "BANK ZERO"
- note added: "BUFFER_CLK +10ns"
- note added: "BUS ENABLE"
- note added: "CLK"
- note added: "CLOCK"
- note added: "CLOCK PHASES"
- note added: "CPU & BUS MANAGEMENT"
- note added: "Generates a ~{RST} pulse of 150ms + 3 clock rising edges Ensures the CPU registers the reset even with slow or stopped clock"
- note added: "I/O CONTROL"
- note added: "M/X DEMUX"
- note added: "OUTPUT"
- note added: "POWER"
- note added: "READY PIN"
- note added: "READ_CLK +10ns (falling-edge only)"
- note added: "RESET"
- note added: "SYNC"
- note added: "TEST POINTS"
- note added: "Two delay lines options: DS1035-10 is DIP but obsolete DS1135-10 is a drop-in SMD replacement that is still active"
- note added: "WRITE_CLK -20ns"
- note added: "pull-down on buffer data bus is useful if you stop the clock, since the data bus is only driven for half the cycle pull-up/down on address bus and cpu data bus are useful only if you plan to tie BE low with nothing else driving the bus"
- note added: "~{MR} is open-collector Do not connect to logic gate output directly"

Commit message: Footprints
Parts:
- removed J1: Jack-DC, symbol Connector:Jack-DC
- added J1: Barrel_Jack_Switch, 65C816:163179PHEX, symbol Connector:Barrel_Jack_Switch
- C1: footprint (none) -> Capacitor_THT:CP_Radial_D6.3mm_P2.50mm
- C10, C11, C12, C13, C14, C15, C16, C17, C18, C19, C2, C4, C5, C6, C7, C8, C9: footprint (none) -> Capacitor_THT:C_Disc_D3.4mm_W2.1mm_P2.50mm
- C3: footprint (none) -> Capacitor_THT:CP_Radial_D4.0mm_P1.50mm
- D1: footprint (none) -> LED_THT:LED_D3.0mm
- D2: footprint Diode_THT:D_DO-41_SOD81_P10.16mm_Horizontal -> Diode_THT:D_DO-41_SOD81_P7.62mm_Horizontal
- J2: footprint (none) -> Connector_PinHeader_2.54mm:PinHeader_1x16_P2.54mm_Vertical
- J3: footprint (none) -> Connector_PinHeader_2.54mm:PinHeader_1x40_P2.54mm_Vertical
- J4: footprint (none) -> Connector_PinHeader_2.54mm:PinHeader_1x18_P2.54mm_Vertical
- R1, R10, R12, R13, R14, R15, R16, R17, R2, R3, R4, R5, R6: footprint (none) -> Resistor_THT:R_Axial_DIN0207_L6.3mm_D2.5mm_P7.62mm_Horizontal
- R11, R7, R8, R9: footprint (none) -> 65C816:0R_Jumper_R_Axial_DIN0207_L6.3mm_D2.5mm_P7.62mm_Horizontal
- SW1: footprint (none) -> Button_Switch_THT:SW_PUSH_6mm
- U1, U11, U14, U15, U2, U3, U6, U7, U8, U9: footprint (none) -> Package_DIP:DIP-14_W7.62mm
- U12, U13: footprint (none) -> Package_DIP:DIP-20_W7.62mm
- U16: footprint (none) -> Package_DIP:DIP-8_W7.62mm
- U4: footprint (none) -> Package_DIP:DIP-16_W7.62mm
- X1: footprint Oscillator:Oscillator_DIP-14 -> Oscillator:Oscillator_DIP-8
Connections:
- net GND: now also J1.2
- net VCC: now also J1.1
- no-connect marks 8 -> 9

Commit message: Update breakout
Parts:
- removed J2: Conn_01x16, Connector_PinHeader_2.54mm:PinHeader_1x16_P2.54mm_Vertical, symbol Connector_Generic:Conn_01x16
- removed J3: Conn_01x40, Connector_PinHeader_2.54mm:PinHeader_1x40_P2.54mm_Vertical, symbol Connector_Generic:Conn_01x40
- removed J4: Conn_01x18, Connector_PinHeader_2.54mm:PinHeader_1x18_P2.54mm_Vertical, symbol Connector_Generic:Conn_01x18
- added H1, H2: MountingHole_Pad, MountingHole:MountingHole_3.2mm_M3_Pad, symbol Mechanical:MountingHole_Pad
- added J2: Conn_02x40_Odd_Even, Connector_PinHeader_2.54mm:PinHeader_2x40_P2.54mm_Vertical, symbol Connector_Generic:Conn_02x40_Odd_Even
- added J3: Conn_02x18_Odd_Even, Connector_PinHeader_2.54mm:PinHeader_2x18_P2.54mm_Vertical, symbol Connector_Generic:Conn_02x18_Odd_Even
- added TP1: 8MHz, TestPoint:TestPoint_THTPad_D1.5mm_Drill0.7mm, symbol Connector:TestPoint
- added TP10: READ_CLK, TestPoint:TestPoint_THTPad_D1.5mm_Drill0.7mm, symbol Connector:TestPoint
- added TP11: WRITE_CLK, TestPoint:TestPoint_THTPad_D1.5mm_Drill0.7mm, symbol Connector:TestPoint
- added TP12: RDY_REG, TestPoint:TestPoint_THTPad_D1.5mm_Drill0.7mm, symbol Connector:TestPoint
- added TP13: ~{RDY_REG}, TestPoint:TestPoint_THTPad_D1.5mm_Drill0.7mm, symbol Connector:TestPoint
- added TP14: B_~{OE}, TestPoint:TestPoint_THTPad_D1.5mm_Drill0.7mm, symbol Connector:TestPoint
- added TP15: ~{BE}, TestPoint:TestPoint_THTPad_D1.5mm_Drill0.7mm, symbol Connector:TestPoint
- added TP2: RDY⎒, TestPoint:TestPoint_THTPad_D1.5mm_Drill0.7mm, symbol Connector:TestPoint
- added TP3: VDA, TestPoint:TestPoint_THTPad_D1.5mm_Drill0.7mm, symbol Connector:TestPoint
- added TP4: VPA, TestPoint:TestPoint_THTPad_D1.5mm_Drill0.7mm, symbol Connector:TestPoint
- added TP5: MX, TestPoint:TestPoint_THTPad_D1.5mm_Drill0.7mm, symbol Connector:TestPoint
- added TP6: CLK-, TestPoint:TestPoint_THTPad_D1.5mm_Drill0.7mm, symbol Connector:TestPoint
- added TP7: CLK+, TestPoint:TestPoint_THTPad_D1.5mm_Drill0.7mm, symbol Connector:TestPoint
- added TP8: BUFFER_CLK, TestPoint:TestPoint_THTPad_D1.5mm_Drill0.7mm, symbol Connector:TestPoint
- added TP9: ~{READ_CLK}, TestPoint:TestPoint_THTPad_D1.5mm_Drill0.7mm, symbol Connector:TestPoint
- J1: footprint 65C816:163179PHEX -> Connector_BarrelJack:BarrelJack_Horizontal
- SW1: value Reset -> RESET
- X1: symbol Oscillator:CXO_DIP14 -> Oscillator:CXO_DIP8
- renumbered R11 to R10, R10 to R11, R17 to R16, R16 to R17, U6 to U1, U12 to U10, U13 to U11, U14 to U12, U1 to U13, U15 to U14, U2 to U15, U3 to U2, U4 to U3, U5 to U4, U7 to U5, U8 to U6, U9 to U7, U10 to U8, U11 to U9
Connections:
- net 8MHz: now also U9.11 (C), X1.5 (OUT), TP1.1; no longer U14.11 (C), X1.8 (OUT)
- net A0: now also J3.19 (Pin_19)
- net A1: now also J3.17 (Pin_17)
- net A10: now also J2.79 (Pin_79)
- net A11: now also J2.77 (Pin_77)
- net A12: now also J2.75 (Pin_75)
- net A13: now also J2.73 (Pin_73)
- net A14: now also J2.71 (Pin_71)
- net A15: now also J2.69 (Pin_69)
- net A16: now also RN5.9 (R8), U11.12 (Q7), U5.9, J2.67 (Pin_67); no longer RN5.2 (R1), U11.19 (Q0), U5.1
- net A17: now also RN5.8 (R7), U11.13 (Q6), U5.10, J2.65 (Pin_65); no longer RN5.3 (R2), U11.18 (Q1), U5.2
- net A18: now also RN5.7 (R6), U11.14 (Q5), U5.5, J2.63 (Pin_63); no longer RN5.4 (R3), U11.17 (Q2), U5.4
- net A19: now also RN5.6 (R5), U11.15 (Q4), U5.4, J2.61 (Pin_61); no longer RN5.5 (R4), U11.16 (Q3), U5.5
- net A2: now also J3.15 (Pin_15)
- net A20: now also RN5.5 (R4), U11.16 (Q3), U5.12, J2.59 (Pin_59); no longer RN5.6 (R5), U11.15 (Q4), U5.9
- net A21: now also RN5.4 (R3), U11.17 (Q2), U5.13, J2.57 (Pin_57); no longer RN5.7 (R6), U11.14 (Q5), U5.10
- net A22: now also RN5.3 (R2), U11.18 (Q1), U5.2, J2.55 (Pin_55); no longer RN5.8 (R7), U11.13 (Q6), U5.12
- net A23: now also RN5.2 (R1), U11.19 (Q0), U5.1, J2.53 (Pin_53); no longer RN5.9 (R8), U11.12 (Q7), U5.13
- net A3: now also J3.13 (Pin_13)
- net A4: now also J3.11 (Pin_11)
- net A5: now also J3.9 (Pin_9)
- net A6: now also J3.7 (Pin_7)
- net A7: now also J3.5 (Pin_5)
- net A8: now also J3.3 (Pin_3)
- net A9: now also J3.1 (Pin_1)
- net BE: now also J2.25 (Pin_25)
- net BUFFER_CLK: now also U12.11, TP8.1; no longer U6.11
- net B_~{OE}: now also TP14.1
- net CLK: now also U14.11 (C), J2.15 (Pin_15); no longer U9.11 (C)
- net CLK+: now also U12.13, TP7.1; no longer U6.13
- net CLK-: now also TP6.1
- net CLK_SRC: now also J2.13 (Pin_13)
- net D0: now also U10.9 (A7), J3.35 (Pin_35); no longer U10.2 (A0)
- net D1: now also U10.8 (A6), J3.33 (Pin_33); no longer U10.3 (A1)
- net D2: now also U10.7 (A5), J3.31 (Pin_31); no longer U10.4 (A2)
- net D3: now also U10.6 (A4), J3.29 (Pin_29); no longer U10.5 (A3)
- net D4: now also U10.5 (A3), J3.27 (Pin_27); no longer U10.6 (A4)
- net D5: now also U10.4 (A2), J3.25 (Pin_25); no longer U10.7 (A5)
- net D6: now also U10.3 (A1), J3.23 (Pin_23); no longer U10.8 (A6)
- net D7: now also U10.2 (A0), J3.21 (Pin_21); no longer U10.9 (A7)
- net DBA0: now also U10.11 (B7), U11.9 (D7); no longer U10.18 (B0), U11.2 (D0)
- net DBA1: now also U10.12 (B6), U11.8 (D6); no longer U10.17 (B1), U11.3 (D1)
- net DBA2: now also U10.13 (B5), U11.7 (D5); no longer U10.16 (B2), U11.4 (D2)
- net DBA3: now also U10.14 (B4), U11.6 (D4); no longer U10.15 (B3), U11.5 (D3)
- net DBA4: now also U10.15 (B3), U11.5 (D3); no longer U10.14 (B4), U11.6 (D4)
- net DBA5: now also U10.16 (B2), U11.4 (D2); no longer U10.13 (B5), U11.7 (D5)
- net DBA6: now also U10.17 (B1), U11.3 (D1); no longer U10.12 (B6), U11.8 (D6)
- net DBA7: now also U10.18 (B0), U11.2 (D0); no longer U10.11 (B7), U11.9 (D7)
- net E: now also J2.43 (Pin_43)
- net GND: now also X1.4 (GND), H1.1, H2.1, J2.10 (Pin_10), J2.12 (Pin_12), J2.14 (Pin_14), J2.16 (Pin_16), J2.18 (Pin_18), J2.2 (Pin_2), J2.20 (Pin_20), J2.22 (Pin_22), J2.24 (Pin_24), J2.26 (Pin_26), J2.28 (Pin_28), J2.3 (Pin_3), J2.30 (Pin_30), J2.32 (Pin_32), J2.34 (Pin_34), J2.36 (Pin_36), J2.38 (Pin_38), J2.4 (Pin_4), J2.40 (Pin_40), J2.42 (Pin_42), J2.44 (Pin_44), J2.46 (Pin_46), J2.48 (Pin_48), J2.50 (Pin_50), J2.52 (Pin_52), J2.54 (Pin_54), J2.56 (Pin_56), J2.58 (Pin_58), J2.6 (Pin_6), J2.60 (Pin_60), J2.62 (Pin_62), J2.64 (Pin_64), J2.66 (Pin_66), J2.68 (Pin_68), J2.70 (Pin_70), J2.72 (Pin_72), J2.74 (Pin_74), J2.76 (Pin_76), J2.78 (Pin_78), J2.8 (Pin_8), J2.80 (Pin_80), J3.10 (Pin_10), J3.12 (Pin_12), J3.14 (Pin_14), J3.16 (Pin_16), J3.18 (Pin_18), J3.2 (Pin_2), J3.20 (Pin_20), J3.22 (Pin_22), J3.24 (Pin_24), J3.26 (Pin_26), J3.28 (Pin_28), J3.30 (Pin_30), J3.32 (Pin_32), J3.34 (Pin_34), J3.36 (Pin_36), J3.4 (Pin_4), J3.6 (Pin_6), J3.8 (Pin_8); no longer X1.7 (GND)
- net M: now also J2.45 (Pin_45)
- net MX: now also TP5.1
- net RDY_IN: now also J2.27 (Pin_27)
- net RDY_REG: now also TP12.1
- net RDY⎒: now also U6.12, TP2.1; no longer U12.12
- net READ_CLK: now also TP10.1
- net RST: now also J2.9 (Pin_9)
- net R~{W}: now also J2.35 (Pin_35)
- net SYNC: now also J2.31 (Pin_31)
- net VA: now also J2.33 (Pin_33)
- net VCC: now also U9.13 (~{R}), X1.8 (Vcc), J2.1 (Pin_1); no longer U14.13 (~{R}), X1.14 (Vcc)
- net VDA: now also TP3.1
- net VPA: now also TP4.1
- net WRITE_CLK: now also TP11.1
- net X: now also J2.47 (Pin_47)
- net ~{ABORT}: now also J2.23 (Pin_23)
- net ~{BANK0}: now also J2.41 (Pin_41)
- net ~{BE}: now also TP15.1
- net ~{CLK_EN}: now also J2.11 (Pin_11)
- net ~{CLK}: now also J2.17 (Pin_17)
- net ~{IRQ}: now also J2.19 (Pin_19)
- net ~{ML}: now also J2.51 (Pin_51)
- net ~{MR}⎒: now also U14.13 (~{R}), U9.2 (D), J2.5 (Pin_5); no longer U9.12 (D), U9.13 (~{R})
- net ~{NMI}: now also J2.21 (Pin_21)
- net ~{RDY_REG}: now also U12.12, U6.13, TP13.1; no longer U12.13, U6.12
- net ~{RD}: now also J2.37 (Pin_37)
- net ~{READ_CLK}: now also TP9.1
- net ~{RST}: now also J2.7 (Pin_7)
- net ~{VP}: now also J2.49 (Pin_49)
- net ~{WAI}: now also U6.11, J2.29 (Pin_29); no longer U12.11
- net ~{WR}: now also J2.39 (Pin_39)
- net at U9.8 (~{Q}): now also U9.12 (D)
- net at U9.9 (Q): now also U7.9; no longer U9.2 (D)
- net at U5.8: now also U6.1; no longer U6.4
- net at U5.3: now also U6.5; no longer U6.1
- net at U6.3: now also U6.10; no longer U6.9
- net at U5.11: now also U6.4; no longer U6.5
- net at U6.6: now also U6.9; no longer U6.10
- net at U14.2 (D): now also U14.9 (Q); no longer U9.5 (Q)
- net at U14.12 (D): now also U9.5 (Q); no longer U14.8 (~{Q})
Other:
- note added: "Two delay lines options: DS1035M-10 is DIP but obsolete DS1135Z-10 is a drop-in SMD replacement that is still active"
- note removed: "Two delay lines options: DS1035-10 is DIP but obsolete DS1135-10 is a drop-in SMD replacement that is still active"
- moved on the sheet: U12D, U14B, U5A, U5C, U5D, U6D, U9A, U9B

Commit message: Update breakout
Other:
- note added: "Note: 74'112 triggers on the falling edge of the clock, whereas 74'74 triggers on the rising edge"
- moved on the sheet: J2, J3

Commit message: Update
Parts:
- H1, H2, TP1, TP10, TP11, TP12, TP13, TP14, TP15, TP2, TP3, TP4, TP5, TP6, TP7, TP8, TP9: now left out of the parts list
Changed lines of the file:
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@@
   )
   (symbol (lib_id "Connector:TestPoint") (at 383.54 208.28 270) (unit 1)
-    (in_bom yes) (on_board yes)
+    (in_bom no) (on_board yes)
     (property "Reference" "TP2" (id 0) (at 388.62 208.28 90)
       (effects (font (size 1.27 1.27)) (justify left))
@@
   )
   (symbol (lib_id "Connector:TestPoint") (at 383.54 215.9 270) (unit 1)
-    (in_bom yes) (on_board yes)
+    (in_bom no) (on_board yes)
     (property "Reference" "TP5" (id 0) (at 388.62 215.9 90)
       (effects (font (size 1.27 1.27)) (justify left))
@@
   )
   (symbol (lib_id "Connector:TestPoint") (at 383.54 236.22 270) (unit 1)
-    (in_bom yes) (on_board yes)
+    (in_bom no) (on_board yes)
     (property "Reference" "TP13" (id 0) (at 388.62 236.22 90)
       (effects (font (size 1.27 1.27)) (justify left))
@@
   )
   (symbol (lib_id "Connector:TestPoint") (at 383.54 213.36 270) (unit 1)
-    (in_bom yes) (on_board yes)
+    (in_bom no) (on_board yes)
     (property "Reference" "TP4" (id 0) (at 388.62 213.36 90)
       (effects (font (size 1.27 1.27)) (justify left))
@@
   )
   (symbol (lib_id "Connector:TestPoint") (at 383.54 231.14 270) (unit 1)
-    (in_bom yes) (on_board yes)
+    (in_bom no) (on_board yes)
     (property "Reference" "TP11" (id 0) (at 388.62 231.14 90)
       (effects (font (size 1.27 1.27)) (justify left))
@@
   )
   (symbol (lib_id "Connector:TestPoint") (at 383.54 228.6 270) (unit 1)
-    (in_bom yes) (on_board yes)
+    (in_bom no) (on_board yes)
     (property "Reference" "TP10" (id 0) (at 388.62 228.6 90)
       (effects (font (size 1.27 1.27)) (justify left))
@@
   )
   (symbol (lib_id "Connector:TestPoint") (at 383.54 223.52 270) (unit 1)
-    (in_bom yes) (on_board yes)
+    (in_bom no) (on_board yes)
     (property "Reference" "TP8" (id 0) (at 388.62 223.52 90)
       (effects (font (size 1.27 1.27)) (justify left))
@@
   )
   (symbol (lib_id "Connector:TestPoint") (at 383.54 238.76 270) (unit 1)
-    (in_bom yes) (on_board yes)
+    (in_bom no) (on_board yes)
     (property "Reference" "TP14" (id 0) (at 388.62 238.76 90)
       (effects (font (size 1.27 1.27)) (justify left))
@@
   )
   (symbol (lib_id "Connector:TestPoint") (at 383.54 233.68 270) (unit 1)
-    (in_bom yes) (on_board yes)
+    (in_bom no) (on_board yes)
     (property "Reference" "TP12" (id 0) (at 388.62 233.68 90)
       (effects (font (size 1.27 1.27)) (justify left))
@@
   )
   (symbol (lib_id "Connector:TestPoint") (at 383.54 218.44 270) (unit 1)
-    (in_bom yes) (on_board yes)
+    (in_bom no) (on_board yes)
     (property "Reference" "TP6" (id 0) (at 388.62 218.44 90)
       (effects (font (size 1.27 1.27)) (justify left))
@@
   )
   (symbol (lib_id "Connector:TestPoint") (at 383.54 205.74 270) (unit 1)
-    (in_bom yes) (on_board yes)
+    (in_bom no) (on_board yes)
     (property "Reference" "TP1" (id 0) (at 388.62 205.74 90)
       (effects (font (size 1.27 1.27)) (justify left))
@@
   )
   (symbol (lib_id "Mechanical:MountingHole_Pad") (at 285.75 245.11 270) (unit 1)
-    (in_bom yes) (on_board yes)
+    (in_bom no) (on_board yes)
     (property "Reference" "H2" (id 0) (at 290.83 246.38 90))
     (property "Value" "MountingHole_Pad" (id 1) (at 298.45 243.84 90))
@@
   )
   (symbol (lib_id "Connector:TestPoint") (at 383.54 220.98 270) (unit 1)
-    (in_bom yes) (on_board yes)
+    (in_bom no) (on_board yes)
     (property "Reference" "TP7" (id 0) (at 388.62 220.98 90)
       (effects (font (size 1.27 1.27)) (justify left))
@@
   )
   (symbol (lib_id "Mechanical:MountingHole_Pad") (at 285.75 238.76 270) (unit 1)
-    (in_bom yes) (on_board yes)
+    (in_bom no) (on_board yes)
     (property "Reference" "H1" (id 0) (at 290.83 240.03 90))
     (property "Value" "MountingHole_Pad" (id 1) (at 298.45 237.49 90))
@@
   )
   (symbol (lib_id "Connector:TestPoint") (at 383.54 210.82 270) (unit 1)
-    (in_bom yes) (on_board yes)
+    (in_bom no) (on_board yes)
     (property "Reference" "TP3" (id 0) (at 388.62 210.82 90)
       (effects (font (size 1.27 1.27)) (justify left))
@@
   )
   (symbol (lib_id "Connector:TestPoint") (at 383.54 226.06 270) (unit 1)
-    (in_bom yes) (on_board yes)
+    (in_bom no) (on_board yes)
     (property "Reference" "TP9" (id 0) (at 388.62 226.06 90)
       (effects (font (size 1.27 1.27)) (justify left))
@@
   )
   (symbol (lib_id "Connector:TestPoint") (at 383.54 241.3 270) (unit 1)
-    (in_bom yes) (on_board yes)
+    (in_bom no) (on_board yes)
     (property "Reference" "TP15" (id 0) (at 388.62 241.3 90)
       (effects (font (size 1.27 1.27)) (justify left))

Commit message: Prep ep 28
Other:
- note added: "Do not solder the ground side when using the PCB on a breadboard"
Changed lines of the file:
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@@
     (effects (font (size 2.54 2.54)) (justify left bottom))
+  )
+  (text "Do not solder the ground side \nwhen using the PCB on a breadboard"
+    (at 361.95 190.5 0)
+    (effects (font (size 1.27 1.27)) (justify left bottom))
   )
   (text "POWER" (at 19.05 146.05 0)
