File: hardware/breakout/breakout.kicad_sch (KiCad schematic)
At the start: 81 parts, among them J1 Barrel_Jack_Switch, J2 Conn_02x40_Odd_Even, J3 Conn_02x18_Odd_Even, SW1 RESET, U1 74AHC74, U10 74AHCT245, U11 74AHC573, U12 74AHC32, U13 74AHC02, U14 74HC74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

Commit message: Rename
Parts:
- R10, R7, R8, R9: footprint 65C816:0R_Jumper_R_Axial_DIN0207_L6.3mm_D2.5mm_P7.62mm_Horizontal -> BB816:0R_Jumper_R_Axial_DIN0207_L6.3mm_D2.5mm_P7.62mm_Horizontal
- U10: symbol 65C816:74AC245 -> BB816:74AC245
- U16: symbol 65C816:DS1035-10 -> BB816:DS1035-10
- U4: symbol 65C816:W65C816SxP -> BB816:W65C816SxP
- U8: symbol 65C816:DS1813 -> BB816:DS1813
Changed lines of the file:
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@@
     (date "2022-08-31")
     (rev "A.27")
-    (comment 2 "https://github.com/adrienkohlbecker/65C816/tree/main/hardware/breakout")
+    (comment 2 "https://github.com/adrienkohlbecker/BB816/tree/main/hardware/breakout")
     (comment 3 "Licensed under CERN-OHL-W v2")
     (comment 4 "Copyright © 2022 Adrien Kohlbecker")
@@
       (effects (font (size 1.27 1.27)) (justify left))
     )
-    (property "Footprint" "65C816:0R_Jumper_R_Axial_DIN0207_L6.3mm_D2.5mm_P7.62mm_Horizontal" (id 2) (at 229.87 78.74 0)
+    (property "Footprint" "BB816:0R_Jumper_R_Axial_DIN0207_L6.3mm_D2.5mm_P7.62mm_Horizontal" (id 2) (at 229.87 78.74 0)
       (effects (font (size 1.27 1.27)) hide)
     )
@@
       (effects (font (size 1.27 1.27)) (justify left))
     )
-    (property "Footprint" "65C816:0R_Jumper_R_Axial_DIN0207_L6.3mm_D2.5mm_P7.62mm_Horizontal" (id 2) (at 245.11 78.74 0)
+    (property "Footprint" "BB816:0R_Jumper_R_Axial_DIN0207_L6.3mm_D2.5mm_P7.62mm_Horizontal" (id 2) (at 245.11 78.74 0)
       (effects (font (size 1.27 1.27)) hide)
     )
@@
     (pin "7")
   )
-  (symbol (lib_id "65C816:W65C816SxP") (at 59.69 68.58 0) (unit 1)
+  (symbol (lib_id "BB816:W65C816SxP") (at 59.69 68.58 0) (unit 1)
     (in_bom yes) (on_board yes)
     (property "Reference" "U4" (id 0) (at 50.8 33.02 0))
@@
     (pin "9")
   )
-  (symbol (lib_id "65C816:DS1035-10") (at 222.25 72.39 0) (unit 2)
+  (symbol (lib_id "BB816:DS1035-10") (at 222.25 72.39 0) (unit 2)
     (in_bom yes) (on_board yes) (fields_autoplaced)
     (property "Reference" "U16" (id 0) (at 222.25 63.5 0))
@@
     (pin "1")
   )
-  (symbol (lib_id "65C816:DS1035-10") (at 237.49 72.39 0) (unit 3)
+  (symbol (lib_id "BB816:DS1035-10") (at 237.49 72.39 0) (unit 3)
     (in_bom yes) (on_board yes) (fields_autoplaced)
     (property "Reference" "U16" (id 0) (at 237.49 63.5 0))
@@
       (effects (font (size 1.27 1.27)) (justify left))
     )
-    (property "Footprint" "65C816:0R_Jumper_R_Axial_DIN0207_L6.3mm_D2.5mm_P7.62mm_Horizontal" (id 2) (at 214.63 78.74 0)
+    (property "Footprint" "BB816:0R_Jumper_R_Axial_DIN0207_L6.3mm_D2.5mm_P7.62mm_Horizontal" (id 2) (at 214.63 78.74 0)
       (effects (font (size 1.27 1.27)) hide)
     )
@@
     (pin "7")
   )
-  (symbol (lib_id "65C816:74AC245") (at 132.08 44.45 0) (unit 1)
+  (symbol (lib_id "BB816:74AC245") (at 132.08 44.45 0) (unit 1)
     (in_bom yes) (on_board yes)
     (property "Reference" "U10" (id 0) (at 125.73 27.94 0))
@@
     (pin "7")
   )
-  (symbol (lib_id "65C816:DS1813") (at 115.57 157.48 0) (unit 1)
+  (symbol (lib_id "BB816:DS1813") (at 115.57 157.48 0) (unit 1)
     (in_bom yes) (on_board yes) (fields_autoplaced)
     (property "Reference" "U8" (id 0) (at 109.22 156.2099 0)
@@
     (property "Reference" "R7" (id 0) (at 109.22 203.2 90))
     (property "Value" "0R" (id 1) (at 109.22 205.74 90))
-    (property "Footprint" "65C816:0R_Jumper_R_Axial_DIN0207_L6.3mm_D2.5mm_P7.62mm_Horizontal" (id 2) (at 109.22 208.28 0)
+    (property "Footprint" "BB816:0R_Jumper_R_Axial_DIN0207_L6.3mm_D2.5mm_P7.62mm_Horizontal" (id 2) (at 109.22 208.28 0)
       (effects (font (size 1.27 1.27)) hide)
     )
@@
     (pin "7")
   )
-  (symbol (lib_id "65C816:DS1035-10") (at 207.01 72.39 0) (unit 1)
+  (symbol (lib_id "BB816:DS1035-10") (at 207.01 72.39 0) (unit 1)
     (in_bom yes) (on_board yes) (fields_autoplaced)
     (property "Reference" "U16" (id 0) (at 207.01 63.5 0))
@@
     (pin "1")
   )
-  (symbol (lib_id "65C816:DS1035-10") (at 265.43 264.16 0) (unit 4)
+  (symbol (lib_id "BB816:DS1035-10") (at 265.43 264.16 0) (unit 4)
     (in_bom yes) (on_board yes)
     (property "Reference" "U16" (id 0) (at 259.08 255.27 0)
@@
     )
     (path "/d6d346d6-40ef-4c34-9f22-cac2f4c66c6f"
-      (reference "R7") (unit 1) (value "0R") (footprint "65C816:0R_Jumper_R_Axial_DIN0207_L6.3mm_D2.5mm_P7.62mm_Horizontal")
+      (reference "R7") (unit 1) (value "0R") (footprint "BB816:0R_Jumper_R_Axial_DIN0207_L6.3mm_D2.5mm_P7.62mm_Horizontal")
     )
     (path "/b5964721-e3de-4566-85dd-0c256270f346"
-      (reference "R8") (unit 1) (value "0R") (footprint "65C816:0R_Jumper_R_Axial_DIN0207_L6.3mm_D2.5mm_P7.62mm_Horizontal")
+      (reference "R8") (unit 1) (value "0R") (footprint "BB816:0R_Jumper_R_Axial_DIN0207_L6.3mm_D2.5mm_P7.62mm_Horizontal")
     )
     (path "/085a7467-8de8-4115-8e8c-8c9437d7a02d"
-      (reference "R9") (unit 1) (value "0R") (footprint "65C816:0R_Jumper_R_Axial_DIN0207_L6.3mm_D2.5mm_P7.62mm_Horizontal")
+      (reference "R9") (unit 1) (value "0R") (footprint "BB816:0R_Jumper_R_Axial_DIN0207_L6.3mm_D2.5mm_P7.62mm_Horizontal")
     )
     (path "/1d602cdc-4f53-4f7d-92e7-1303cadcd74f"
-      (reference "R10") (unit 1) (value "0R") (footprint "65C816:0R_Jumper_R_Axial_DIN0207_L6.3mm_D2.5mm_P7.62mm_Horizontal")
+      (reference "R10") (unit 1) (value "0R") (footprint "BB816:0R_Jumper_R_Axial_DIN0207_L6.3mm_D2.5mm_P7.62mm_Horizontal")
     )
     (path "/a544b3d7-ac91-4278-a0d6-3fe0a4a7bdbe"
